File: FAN_PWM_DRIVER.sch (KiCad schematic (older format))
At the start: 3 parts, among them Q3 SS9013_J3

Commit message: update,
Parts:
- R7, R8: footprint (none) -> Resistor_SMD:R_0805_2012Metric_Pad1.15x1.40mm_HandSolder
Changed lines of the file:
@@
 $EndDescr
 $Comp
-L stm32_bottom_board_respin-rescue:SS9013_J3-taobao-transistor Q3
+L stm32_bottom_board_respin-rescue:SS9013_J3-taobao-transistor Q?
 U 1 1 5BCBA2C4
 P 2750 2200
-AR Path="/5BCBA2C4" Ref="Q3"  Part="1"
+AR Path="/5BCBA2C4" Ref="Q?"  Part="1"
 AR Path="/5BCBA20B/5BCBA2C4" Ref="Q3"  Part="1"
 F 0 "Q3" H 2941 2246 50  0000 L CNN
@@
 F 0 "R7" V 1954 2200 50  0000 C CNN
 F 1 "R471" V 2045 2200 50  0000 C CNN
-F 2 "" H 2150 2200 50  0001 C CNN
+F 2 "Resistor_SMD:R_0805_2012Metric_Pad1.15x1.40mm_HandSolder" H 2150 2200 50  0001 C CNN
 F 3 "~" H 2150 2200 50  0001 C CNN
 	1    2150 2200
@@
 F 0 "R8" H 2909 1646 50  0000 L CNN
 F 1 "R331" H 2909 1555 50  0000 L CNN
-F 2 "" H 2850 1600 50  0001 C CNN
+F 2 "Resistor_SMD:R_0805_2012Metric_Pad1.15x1.40mm_HandSolder" H 2850 1600 50  0001 C CNN
 F 3 "~" H 2850 1600 50  0001 C CNN
 	1    2850 1600
@@
 	2850 1700 2850 1850
 $Comp
-L power:GND #PWR0112
+L power:GND #PWR016
 U 1 1 5BCBA643
 P 2850 2700
-F 0 "#PWR0112" H 2850 2450 50  0001 C CNN
+F 0 "#PWR016" H 2850 2450 50  0001 C CNN
 F 1 "GND" H 2855 2527 50  0000 C CNN
 F 2 "" H 2850 2700 50  0001 C CNN
@@
 FAN_PWM_GND
 $Comp
-L power:VDD #PWR0111
+L power:VDD #PWR015
 U 1 1 5BCBA5C6
 P 2850 1300
-F 0 "#PWR0111" H 2850 1150 50  0001 C CNN
+F 0 "#PWR015" H 2850 1150 50  0001 C CNN
 F 1 "VDD" H 2867 1473 50  0000 C CNN
 F 2 "" H 2850 1300 50  0001 C CNN

Commit message: update,
Parts:
- removed Q3: SS9013_J3, Package_TO_SOT_THT:TO-92_Inline, symbol stm32_bottom_board_respin-rescue:SS9013_J3-taobao-transistor
- added Q?: SS9013_J3, Package_TO_SOT_THT:TO-92_Inline, symbol taobao-transistor:SS9013_J3
Connections:
- net FAN_PWM_OUTPUT: now also Q?.3 (C)
- net GND: now also Q?.2 (E)
- net at R7.1: now also Q?.1 (B)
Changed lines of the file:
@@
 $EndDescr
-$Comp
-L stm32_bottom_board_respin-rescue:SS9013_J3-taobao-transistor Q?
-U 1 1 5BCBA2C4
-P 2750 2200
-AR Path="/5BCBA2C4" Ref="Q?"  Part="1"
-AR Path="/5BCBA20B/5BCBA2C4" Ref="Q3"  Part="1"
-F 0 "Q3" H 2941 2246 50  0000 L CNN
-F 1 "SS9013_J3" H 2941 2155 50  0000 L CNN
-F 2 "Package_TO_SOT_THT:TO-92_Inline" H 2950 2125 50  0001 L CIN
-F 3 "https://www.fairchildsemi.com/datasheets/2N/2N3904.pdf" H 2750 2200 50  0001 L CNN
-	1    2750 2200
-	1    0    0    -1
-$EndComp
 $Comp
 L taobao-r:R471 R7
@@
 	1    0    0    -1
 $EndComp
+$Comp
+L taobao-transistor:SS9013_J3 Q?
+U 1 1 5BCBC4D0
+P 2750 2200
+F 0 "Q?" H 2950 2250 50  0000 L CNN
+F 1 "SS9013_J3" H 2950 2200 50  0000 L CNN
+F 2 "Package_TO_SOT_THT:TO-92_Inline" H 2950 2125 50  0001 L CIN
+F 3 "https://www.fairchildsemi.com/datasheets/2N/2N3904.pdf" H 2750 2200 50  0001 L CNN
+	1    2750 2200
+	1    0    0    -1
+$EndComp

Commit message: update,
Parts:
- Q2: renamed from Q?; footprint Package_TO_SOT_THT:TO-92_Inline -> Package_TO_SOT_SMD:SOT-23_Handsoldering
Changed lines of the file:
@@
 $Descr A4 11693 8268
 encoding utf-8
-Sheet 5 6
+Sheet 4 6
 Title ""
 Date ""
@@
 $EndComp
 $Comp
-L taobao-transistor:SS9013_J3 Q?
+L taobao-transistor:SS9013_J3 Q2
 U 1 1 5BCBC4D0
 P 2750 2200
-F 0 "Q?" H 2950 2250 50  0000 L CNN
+F 0 "Q2" H 2950 2250 50  0000 L CNN
 F 1 "SS9013_J3" H 2950 2200 50  0000 L CNN
-F 2 "Package_TO_SOT_THT:TO-92_Inline" H 2950 2125 50  0001 L CIN
+F 2 "Package_TO_SOT_SMD:SOT-23_Handsoldering" H 2950 2125 50  0001 L CIN
 F 3 "https://www.fairchildsemi.com/datasheets/2N/2N3904.pdf" H 2750 2200 50  0001 L CNN
 	1    2750 2200
