File: SSR-25-DA_DRIVER.sch (KiCad schematic (older format))
At the start: 3 parts, among them Q2 SS9013_J3

Commit message: update,
Parts:
- R5, R6: footprint (none) -> Resistor_SMD:R_0805_2012Metric_Pad1.15x1.40mm_HandSolder
Changed lines of the file:
@@
 $EndDescr
 $Comp
-L power:VDD #PWR0109
+L power:VDD #PWR013
 U 1 1 5BCB697F
 P 6250 1900
-F 0 "#PWR0109" H 6250 1750 50  0001 C CNN
+F 0 "#PWR013" H 6250 1750 50  0001 C CNN
 F 1 "VDD" H 6267 2073 50  0000 C CNN
 F 2 "" H 6250 1900 50  0001 C CNN
@@
 F 0 "R6" H 6309 2146 50  0000 L CNN
 F 1 "R101" H 6309 2055 50  0000 L CNN
-F 2 "" H 6250 2100 50  0001 C CNN
+F 2 "Resistor_SMD:R_0805_2012Metric_Pad1.15x1.40mm_HandSolder" H 6250 2100 50  0001 C CNN
 F 3 "~" H 6250 2100 50  0001 C CNN
 	1    6250 2100
@@
 F 0 "R5" V 5304 3100 50  0000 C CNN
 F 1 "R471" V 5395 3100 50  0000 C CNN
-F 2 "" H 5500 3100 50  0001 C CNN
+F 2 "Resistor_SMD:R_0805_2012Metric_Pad1.15x1.40mm_HandSolder" H 5500 3100 50  0001 C CNN
 F 3 "~" H 5500 3100 50  0001 C CNN
 	1    5500 3100
@@
 	5050 3100 5400 3100
 $Comp
-L power:GND #PWR0110
+L power:GND #PWR014
 U 1 1 5BCB6BDC
 P 6250 3600
-F 0 "#PWR0110" H 6250 3350 50  0001 C CNN
+F 0 "#PWR014" H 6250 3350 50  0001 C CNN
 F 1 "GND" H 6255 3427 50  0000 C CNN
 F 2 "" H 6250 3600 50  0001 C CNN
@@
 	6250 2600 6250 2900
 $Comp
-L stm32_bottom_board_respin-rescue:SS9013_J3-taobao-transistor Q2
+L stm32_bottom_board_respin-rescue:SS9013_J3-taobao-transistor Q?
 U 1 1 5BCB856E
 P 6150 3100
-AR Path="/5BCB856E" Ref="Q2"  Part="1"
+AR Path="/5BCB856E" Ref="Q?"  Part="1"
 AR Path="/5BCB679F/5BCB856E" Ref="Q2"  Part="1"
 F 0 "Q2" H 6341 3146 50  0000 L CNN

Commit message: update,
Parts:
- removed Q2: SS9013_J3, Package_TO_SOT_SMD:TSOT-23_HandSoldering, symbol stm32_bottom_board_respin-rescue:SS9013_J3-taobao-transistor
- added Q3: SS9013_J3, Package_TO_SOT_SMD:SOT-23_Handsoldering, symbol taobao-transistor:SS9013_J3
Connections:
- net GND: now also Q3.2 (E)
- net SSR-25-DA2: now also Q3.3 (C)
- net at R5.1: now also Q3.1 (B)
Changed lines of the file:
@@
 Wire Wire Line
 	6250 2600 6250 2900
-$Comp
-L stm32_bottom_board_respin-rescue:SS9013_J3-taobao-transistor Q?
-U 1 1 5BCB856E
-P 6150 3100
-AR Path="/5BCB856E" Ref="Q?"  Part="1"
-AR Path="/5BCB679F/5BCB856E" Ref="Q2"  Part="1"
-F 0 "Q2" H 6341 3146 50  0000 L CNN
-F 1 "SS9013_J3" H 6341 3055 50  0000 L CNN
-F 2 "Package_TO_SOT_SMD:TSOT-23_HandSoldering" H 6350 3025 50  0001 L CIN
-F 3 "https://www.fairchildsemi.com/datasheets/2N/2N3904.pdf" H 6150 3100 50  0001 L CNN
-	1    6150 3100
-	1    0    0    -1
-$EndComp
 Text HLabel 7350 2400 2    50   Input ~ 0
 SSR-25-DA1
@@
 Wire Wire Line
 	6250 2600 7350 2600
+$Comp
+L taobao-transistor:SS9013_J3 Q3
+U 1 1 5BCBD15E
+P 6150 3100
+F 0 "Q3" H 6350 3150 50  0000 L CNN
+F 1 "SS9013_J3" H 6350 3100 50  0000 L CNN
+F 2 "Package_TO_SOT_SMD:SOT-23_Handsoldering" H 6350 3025 50  0001 L CIN
+F 3 "https://www.fairchildsemi.com/datasheets/2N/2N3904.pdf" H 6150 3100 50  0001 L CNN
+	1    6150 3100
+	1    0    0    -1
+$EndComp
 $EndSCHEMATC
