File: STM32_CORE.sch (KiCad schematic (older format))
At the start: 31 parts, among them J1 Conn_01x14, J3 Conn_01x12, J4 Conn_01x12, SW1 SW_Push, U1 STM32F103C8T6, U2 AMS1117-3.3, Y1 O8M, Y2 O32.768K

Commit message: update,
Parts:
- C7, C8: renamed from C?; footprint (none) -> Capacitor_Tantalum_SMD:CP_EIA-3216-12_Kemet-S_Pad1.58x1.35mm_HandSolder
- R10: renamed from R2; footprint Resistor_SMD:R_0603_1608Metric_Pad1.05x0.95mm_HandSolder -> Resistor_SMD:R_0805_2012Metric_Pad1.15x1.40mm_HandSolder
- R11: renamed from R3; footprint Resistor_SMD:R_0603_1608Metric_Pad1.05x0.95mm_HandSolder -> Resistor_SMD:R_0805_2012Metric_Pad1.15x1.40mm_HandSolder
- R12: renamed from R4; footprint Resistor_SMD:R_0603_1608Metric_Pad1.05x0.95mm_HandSolder -> Resistor_SMD:R_0805_2012Metric_Pad1.15x1.40mm_HandSolder
- R13: renamed from R5; footprint Resistor_SMD:R_0603_1608Metric_Pad1.05x0.95mm_HandSolder -> Resistor_SMD:R_0805_2012Metric_Pad1.15x1.40mm_HandSolder
- R9: renamed from R1; footprint Resistor_SMD:R_0603_1608Metric_Pad1.05x0.95mm_HandSolder -> Resistor_SMD:R_0805_2012Metric_Pad1.15x1.40mm_HandSolder
- renumbered BOOT0 to BOOT1, BOOT1 to BOOT2, C9 to C10, C10 to C11, C11 to C12, C12 to C13, C13 to C14, C8 to C2, C1 to C3, C2 to C4, C3 to C5, C4 to C6, C7 to C9, D1 to D2, D2 to D3, J1 to J6, J3 to J7, J4 to J8, JP3 to JP1, U1 to U3, U2 to U4

Commit message: update,
Parts:
- Y1: footprint Crystal:Crystal_SMD_HC49-SD -> w_crystal:hc-49_smd
Changed lines of the file:
@@
 $Descr A3 16535 11693
 encoding utf-8
-Sheet 6 6
+Sheet 5 6
 Title ""
 Date ""
@@
 F 0 "Y1" V 14654 6788 50  0000 L CNN
 F 1 "O8M" V 14745 6788 50  0000 L CNN
-F 2 "Crystal:Crystal_SMD_HC49-SD" H 14700 6700 50  0001 C CNN
+F 2 "w_crystal:hc-49_smd" H 14700 6700 50  0001 C CNN
 F 3 "~" H 14700 6700 50  0001 C CNN
 	1    14700 6700

Commit message: update,
Parts:
- BOOT0: renamed from BOOT1; value SolderJumper_3_Open -> JUMPER
- BOOT1: renamed from BOOT2; value SolderJumper_3_Open -> JUMPER
Changed lines of the file:
@@
 	14500 3100 14500 3350
 $Comp
-L Jumper:SolderJumper_3_Open BOOT1
+L Jumper:SolderJumper_3_Open BOOT0
 U 1 1 5BCF8FA5
 P 11800 2850
-F 0 "BOOT1" V 11754 2918 50  0000 L CNN
-F 1 "SolderJumper_3_Open" V 11845 2918 50  0000 L CNN
+F 0 "BOOT0" V 11754 2918 50  0000 L CNN
+F 1 "JUMPER" V 11845 2918 50  0000 L CNN
 F 2 "Jumper:SolderJumper-3_P2.0mm_Open_TrianglePad1.0x1.5mm" H 11800 2850 50  0001 C CNN
 F 3 "~" H 11800 2850 50  0001 C CNN
@@
 $EndComp
 $Comp
-L Jumper:SolderJumper_3_Open BOOT2
+L Jumper:SolderJumper_3_Open BOOT1
 U 1 1 5BCF9021
 P 12650 2850
-F 0 "BOOT2" V 12604 2918 50  0000 L CNN
-F 1 "SolderJumper_3_Open" V 12695 2918 50  0000 L CNN
+F 0 "BOOT1" V 12604 2918 50  0000 L CNN
+F 1 "JUMPER" V 12695 2918 50  0000 L CNN
 F 2 "Jumper:SolderJumper-3_P2.0mm_Open_TrianglePad1.0x1.5mm" H 12650 2850 50  0001 C CNN
 F 3 "~" H 12650 2850 50  0001 C CNN

Commit message: update,
Connections:
- net PC13: now also J6.13 (Pin_13); no longer J6.14 (Pin_14)
- net at JP1.1: now also J6.14 (Pin_14); no longer J8.1 (Pin_1)
Other:
- moved on the sheet: JP1
Changed lines of the file:
@@
 $EndComp
 Wire Wire Line
-	4200 4800 4200 4950
+	2250 3800 2250 3950
 Wire Wire Line
 	2150 2400 2150 2500
@@
 L Device:Jumper_NO_Small JP1
 U 1 1 5BE05EFF
-P 4450 4800
-F 0 "JP1" H 4450 4985 50  0000 C CNN
-F 1 "Jumper_NO_Small" H 4450 4894 50  0000 C CNN
-F 2 "Jumper:SolderJumper-2_P1.3mm_Open_TrianglePad1.0x1.5mm" H 4450 4800 50  0001 C CNN
-F 3 "~" H 4450 4800 50  0001 C CNN
-	1    4450 4800
-	-1   0    0    1
-$EndComp
-Wire Wire Line
-	4750 4800 4550 4800
-Wire Wire Line
-	4350 4800 4200 4800
+P 2000 3800
+F 0 "JP1" H 2000 3985 50  0000 C CNN
+F 1 "Jumper_NO_Small" H 2000 3894 50  0000 C CNN
+F 2 "Jumper:SolderJumper-2_P1.3mm_Open_TrianglePad1.0x1.5mm" H 2000 3800 50  0001 C CNN
+F 3 "~" H 2000 3800 50  0001 C CNN
+	1    2000 3800
+	1    0    0    1
+$EndComp
+Wire Wire Line
+	1700 3800 1900 3800
+Wire Wire Line
+	2100 3800 2250 3800
 Text Label 2000 3600 2    50   ~ 0
 PB9
@@
 Wire Wire Line
 	3950 4600 4750 4600
-Text Label 2000 3800 2    50   ~ 0
+Text Label 2000 3700 2    50   ~ 0
 PC13
 Wire Wire Line
-	2000 3800 1700 3800
-Wire Wire Line
-	1700 3700 2150 3700
-Wire Wire Line
-	2150 3700 2150 3650
+	2000 3700 1700 3700
 $Comp
 L power:+3V3 #PWR017
@@
 L power:+5V #PWR021
 U 1 1 5BCACB86
-P 4200 4950
-F 0 "#PWR021" H 4200 4800 50  0001 C CNN
-F 1 "+5V" H 4200 5150 50  0000 C CNN
-F 2 "" H 4200 4950 50  0001 C CNN
-F 3 "" H 4200 4950 50  0001 C CNN
-	1    4200 4950
-	-1   0    0    1
-$EndComp
-$Comp
+P 2250 3950
+F 0 "#PWR021" H 2250 3800 50  0001 C CNN
+F 1 "+5V" H 2250 4150 50  0000 C CNN
+F 2 "" H 2250 3950 50  0001 C CNN
+F 3 "" H 2250 3950 50  0001 C CNN
+	1    2250 3950
+	1    0    0    1
+$EndComp
+$Comp

Commit message: update,
Parts:
- removed D2: LED_GREEN, LED_SMD:LED_0805_2012Metric_Pad1.15x1.40mm_HandSolder, symbol taobao-components:LED_GREEN
- removed D3: LED_ORANGE, LED_SMD:LED_0805_2012Metric_Pad1.15x1.40mm_HandSolder, symbol taobao-components:LED_GREEN
- added D?: LED_GREEN, symbol taobao-components:LED_GREEN
- added D?: LED_ORANGE, symbol taobao-components:LED_ORANGE
Connections:
- net +3V3: now also D?.2 (A), D?.2 (A)
- net at R11.1: now also D?.1 (K)
- net at R13.1: now also D?.1 (K)
Changed lines of the file:
@@
 Connection ~ 14700 6850
-$Comp
-L taobao-components:LED_GREEN D2
-U 1 1 5BCD1BF1
-P 14200 5000
-F 0 "D2" V 14246 4932 50  0000 R CNN
-F 1 "LED_GREEN" V 14155 4932 50  0000 R CNN
-F 2 "LED_SMD:LED_0805_2012Metric_Pad1.15x1.40mm_HandSolder" V 14200 5000 50  0001 C CNN
-F 3 "~" V 14200 5000 50  0001 C CNN
-	1    14200 5000
-	0    -1   -1   0
-$EndComp
 $Comp
 L taobao-r:R511 R11
@@
 Wire Wire Line
 	14200 5400 14200 5500
-$Comp
-L taobao-components:LED_GREEN D3
-U 1 1 5BCD7CA2
-P 14850 5000
-F 0 "D3" V 14896 4932 50  0000 R CNN
-F 1 "LED_ORANGE" V 14805 4932 50  0000 R CNN
-F 2 "LED_SMD:LED_0805_2012Metric_Pad1.15x1.40mm_HandSolder" V 14850 5000 50  0001 C CNN
-F 3 "~" V 14850 5000 50  0001 C CNN
-	1    14850 5000
-	0    -1   -1   0
-$EndComp
 $Comp
 L taobao-r:R511 R13
@@
 	1    0    0    -1
 $EndComp
+$Comp
+L taobao-components:LED_GREEN D?
+U 1 1 5BCEC9BE
+P 14200 5000
+F 0 "D?" V 14246 4932 50  0000 R CNN
+F 1 "LED_GREEN" V 14155 4932 50  0000 R CNN
+F 2 "" V 14200 5000 50  0001 C CNN
+F 3 "" V 14200 5000 50  0001 C CNN
+	1    14200 5000
+	0    -1   -1   0
+$EndComp
+$Comp
+L taobao-components:LED_ORANGE D?
+U 1 1 5BD0511E
+P 14850 5000
+F 0 "D?" V 14896 4932 50  0000 R CNN
+F 1 "LED_ORANGE" V 14805 4932 50  0000 R CNN
+F 2 "" V 14850 5000 50  0001 C CNN
+F 3 "" V 14850 5000 50  0001 C CNN
+	1    14850 5000
+	0    -1   -1   0
+$EndComp
 $EndSCHEMATC

Commit message: update,
Parts:
- D2, D3: renamed from D?; footprint (none) -> LED_SMD:LED_0805_2012Metric_Pad1.15x1.40mm_HandSolder
Changed lines of the file:
@@
 $EndComp
 $Comp
-L taobao-components:LED_GREEN D?
+L taobao-components:LED_GREEN D2
 U 1 1 5BCEC9BE
 P 14200 5000
-F 0 "D?" V 14246 4932 50  0000 R CNN
+F 0 "D2" V 14246 4932 50  0000 R CNN
 F 1 "LED_GREEN" V 14155 4932 50  0000 R CNN
-F 2 "" V 14200 5000 50  0001 C CNN
+F 2 "LED_SMD:LED_0805_2012Metric_Pad1.15x1.40mm_HandSolder" V 14200 5000 50  0001 C CNN
 F 3 "" V 14200 5000 50  0001 C CNN
 	1    14200 5000
@@
 $EndComp
 $Comp
-L taobao-components:LED_ORANGE D?
+L taobao-components:LED_ORANGE D3
 U 1 1 5BD0511E
 P 14850 5000
-F 0 "D?" V 14896 4932 50  0000 R CNN
+F 0 "D3" V 14896 4932 50  0000 R CNN
 F 1 "LED_ORANGE" V 14805 4932 50  0000 R CNN
-F 2 "" V 14850 5000 50  0001 C CNN
+F 2 "LED_SMD:LED_0805_2012Metric_Pad1.15x1.40mm_HandSolder" V 14850 5000 50  0001 C CNN
 F 3 "" V 14850 5000 50  0001 C CNN
 	1    14850 5000
