File: stm32_bottom_board_respin.sch (KiCad schematic (older format))
At the start: 2 parts

Commit message: update,
Parts:
- added C?: CP1000uf,10V, symbol taobao-cp:CP1000uf,10V
- added J3: Conn_01x03, symbol Connector_Generic:Conn_01x02
- added J4: Conn_01x04, symbol Connector_Generic:Conn_01x04
- added J?: Conn_01x02, symbol Connector_Generic:Conn_01x02
- gave numbers to parts that had none: 2
Connections:
- net GND: now also J1.2 (Pin_2), C?.2, J?.2 (Pin_2); no longer J1.3 (Pin_3)
- net VWS2812: now also C?.1
- net WS2812_PWM_TERMINAL: now also J1.3 (Pin_3); no longer J1.2 (Pin_2)
- new net FAN_48V: J4.1 (Pin_1), J?.1 (Pin_1)
- new net FAN_PWM_GND: J4.3 (Pin_3)
- new net FAN_PWM_OUTPUT: J4.2 (Pin_2)
- new net FAN_RPM: J4.4 (Pin_4)
- new net SSR-25-DA1: J3.1 (Pin_1)
- new net SSR-25-DA2: J3.2 (Pin_2)
Other:
- note added: "connect the main power supply to VWS2812"
- note added: "the power of driver circuit is by VDD instead of +5V\nto provision the power control of the driver circuit"
- moved on the sheet: J1, J2

Commit message: update,
Parts:
- C1: renamed from C?; footprint (none) -> Capacitor_SMD:CP_Elec_10x10.5
- J1: renamed from J?; footprint (none) -> Connector_PinHeader_2.00mm:PinHeader_1x02_P2.00mm_Vertical
- J2: renamed from J1; footprint (none) -> Connector_PinHeader_1.27mm:PinHeader_1x03_P1.27mm_Vertical
- J3: renamed from J4; footprint (none) -> Connector_PinHeader_1.27mm:PinHeader_1x04_P1.27mm_Horizontal
- J4: renamed from J3; value Conn_01x03 -> Conn_01x02; footprint (none) -> Connector_PinHeader_1.27mm:PinHeader_1x02_P1.27mm_Vertical
- J5: renamed from J2; value Conn_01x03 -> Conn_01x02; footprint (none) -> Connector_PinHeader_1.27mm:PinHeader_1x02_P1.27mm_Vertical
Changed lines of the file:
@@
 $EndSheet
 $Comp
-L Connector_Generic:Conn_01x03 J1
+L Connector_Generic:Conn_01x03 J2
 U 1 1 5BCB416C
 P 8700 8400
-F 0 "J1" H 8780 8442 50  0000 L CNN
+F 0 "J2" H 8780 8442 50  0000 L CNN
 F 1 "Conn_01x03" H 8780 8351 50  0000 L CNN
-F 2 "" H 8700 8400 50  0001 C CNN
+F 2 "Connector_PinHeader_1.27mm:PinHeader_1x03_P1.27mm_Vertical" H 8700 8400 50  0001 C CNN
 F 3 "~" H 8700 8400 50  0001 C CNN
 	1    8700 8400
@@
 $EndComp
 $Comp
-L taobao-components:VWS2812 #PWR0101
+L taobao-components:VWS2812 #PWR05
 U 1 1 5BCB42EE
 P 8300 8150
-F 0 "#PWR0101" H 8300 8000 50  0001 C CNN
+F 0 "#PWR05" H 8300 8000 50  0001 C CNN
 F 1 "VWS2812" H 8317 8323 50  0000 C CNN
 F 2 "" H 8300 8150 50  0001 C CNN
@@
 	8300 8300 8500 8300
 $Comp
-L power:GND #PWR0102
+L power:GND #PWR04
 U 1 1 5BCB4355
 P 7850 8450
-F 0 "#PWR0102" H 7850 8200 50  0001 C CNN
+F 0 "#PWR04" H 7850 8200 50  0001 C CNN
 F 1 "GND" H 7855 8277 50  0000 C CNN
 F 2 "" H 7850 8450 50  0001 C CNN
@@
 	13150 6450 14500 6450
 $Comp
-L Connector_Generic:Conn_01x02 J2
+L Connector_Generic:Conn_01x02 J5
 U 1 1 5BCB6490
 P 9650 6450
-F 0 "J2" H 9730 6442 50  0000 L CNN
-F 1 "Conn_01x03" H 9730 6351 50  0000 L CNN
-F 2 "" H 9650 6450 50  0001 C CNN
+F 0 "J5" H 9730 6442 50  0000 L CNN
+F 1 "Conn_01x02" H 9730 6351 50  0000 L CNN
+F 2 "Connector_PinHeader_1.27mm:PinHeader_1x02_P1.27mm_Vertical" H 9650 6450 50  0001 C CNN
 F 3 "~" H 9650 6450 50  0001 C CNN
 	1    9650 6450
@@
 	9400 4950 8600 4950
 $Comp
-L Connector_Generic:Conn_01x02 J3
+L Connector_Generic:Conn_01x02 J4
 U 1 1 5BCB931B
 P 9600 4950
-F 0 "J3" H 9680 4942 50  0000 L CNN
-F 1 "Conn_01x03" H 9680 4851 50  0000 L CNN
-F 2 "" H 9600 4950 50  0001 C CNN
+F 0 "J4" H 9680 4942 50  0000 L CNN
+F 1 "Conn_01x02" H 9680 4851 50  0000 L CNN
+F 2 "Connector_PinHeader_1.27mm:PinHeader_1x02_P1.27mm_Vertical" H 9600 4950 50  0001 C CNN
 F 3 "~" H 9600 4950 50  0001 C CNN
 	1    9600 4950
@@
 	9350 3800 8550 3800
 $Comp
-L Connector_Generic:Conn_01x04 J4
+L Connector_Generic:Conn_01x04 J3
 U 1 1 5BCBC3BF
 P 9550 3800
-F 0 "J4" H 9630 3792 50  0000 L CNN
+F 0 "J3" H 9630 3792 50  0000 L CNN
 F 1 "Conn_01x04" H 9630 3701 50  0000 L CNN
-F 2 "" H 9550 3800 50  0001 C CNN
+F 2 "Connector_PinHeader_1.27mm:PinHeader_1x04_P1.27mm_Horizontal" H 9550 3800 50  0001 C CNN
 F 3 "~" H 9550 3800 50  0001 C CNN
 	1    9550 3800
@@
 connect the main power supply to VWS2812
 $Comp
-L taobao-components:VWS2812 #PWR0113
+L taobao-components:VWS2812 #PWR06
 U 1 1 5BCB629E
 P 9650 8150
-F 0 "#PWR0113" H 9650 8000 50  0001 C CNN
+F 0 "#PWR06" H 9650 8000 50  0001 C CNN
 F 1 "VWS2812" H 9667 8323 50  0000 C CNN
 F 2 "" H 9650 8150 50  0001 C CNN
@@
 $EndComp
 $Comp
-L power:GND #PWR0114
+L power:GND #PWR07
 U 1 1 5BCB62B1
 P 9650 8600
-F 0 "#PWR0114" H 9650 8350 50  0001 C CNN
+F 0 "#PWR07" H 9650 8350 50  0001 C CNN
 F 1 "GND" H 9655 8427 50  0000 C CNN
 F 2 "" H 9650 8600 50  0001 C CNN
@@
 	9650 8450 9650 8600
 $Comp
-L taobao-cp:CP1000uf,10V C?
+L taobao-cp:CP1000uf,10V C1
 U 1 1 5BCB6CCE
 P 9650 8350
-F 0 "C?" H 9738 8396 50  0000 L CNN
+F 0 "C1" H 9738 8396 50  0000 L CNN
 F 1 "CP1000uf,10V" H 9738 8305 50  0000 L CNN
-F 2 "" H 9650 8350 50  0001 C CNN
+F 2 "Capacitor_SMD:CP_Elec_10x10.5" H 9650 8350 50  0001 C CNN
 F 3 "~" H 9650 8350 50  0001 C CNN
 	1    9650 8350
@@
 $EndSheet
 $Comp
-L tinkerforge:+5V #PWR?
+L tinkerforge:+5V #PWR01
 U 1 1 5BCBF96D
 P 6700 1050
-F 0 "#PWR?" H 6700 900 50  0001 C CNN
+F 0 "#PWR01" H 6700 900 50  0001 C CNN
 F 1 "+5V" H 6715 1223 50  0000 C CNN
 F 2 "" H 6700 1050 50  0000 C CNN
@@
 $EndComp
 $Comp
-L power:VDD #PWR?
+L power:VDD #PWR02
 U 1 1 5BCBFA5F
 P 7150 1050
-F 0 "#PWR?" H 7150 900 50  0001 C CNN
+F 0 "#PWR02" H 7150 900 50  0001 C CNN
 F 1 "VDD" H 7167 1223 50  0000 C CNN
 F 2 "" H 7150 1050 50  0001 C CNN
@@
 	8550 3700 9350 3700
 $Comp
-L Connector_Generic:Conn_01x02 J?
+L Connector_Generic:Conn_01x02 J1
 U 1 1 5BCC1C7F
 P 7800 3700
-F 0 "J?" H 7880 3692 50  0000 L CNN
+F 0 "J1" H 7880 3692 50  0000 L CNN
 F 1 "Conn_01x02" H 7880 3601 50  0000 L CNN
-F 2 "" H 7800 3700 50  0001 C CNN
+F 2 "Connector_PinHeader_2.00mm:PinHeader_1x02_P2.00mm_Vertical" H 7800 3700 50  0001 C CNN
 F 3 "~" H 7800 3700 50  0001 C CNN
 	1    7800 3700
@@
 	6800 3700 7600 3700
 $Comp
-L power:GND #PWR?
+L power:GND #PWR03
 U 1 1 5BCC7684
 P 7550 3900
-F 0 "#PWR?" H 7550 3650 50  0001 C CNN
+F 0 "#PWR03" H 7550 3650 50  0001 C CNN
 F 1 "GND" H 7555 3727 50  0000 C CNN
 F 2 "" H 7550 3900 50  0001 C CNN

Commit message: update,
Changed lines of the file:
@@
 Comment4 ""
 $EndDescr
-$Sheet
-S 11450 7850 1950 1050
-U 5BCB4060
-F0 "WS2812_PWM_DRIVER" 50
-F1 "WS2812_PWM_DRIVER.sch" 50
-F2 "STM32_WS2812_PWM" I L 11450 8200 50
-F3 "WS2812_PWM_OUTPUT" I R 13400 8500 50
-$EndSheet
 $Comp
 L Connector_Generic:Conn_01x03 J2
@@
 Text Label 7000 8700 0    50   ~ 0
 WS2812_PWM_TERMINAL
-Text Label 14500 8500 2    50   ~ 0
+Text Label 14250 8550 2    50   ~ 0
 WS2812_PWM_TERMINAL
 Wire Wire Line
-	14500 8500 13400 8500
-Text Label 10400 8200 0    50   ~ 0
+	14250 8550 13150 8550
+Text Label 10550 8250 0    50   ~ 0
 STM32_WS2812_OUTPUT
 Wire Wire Line
-	10400 8200 11450 8200
-$Sheet
-S 11600 5950 1550 950
+	10550 8250 11650 8250
+$Sheet
+S 11650 5950 1500 900
 U 5BCB4A39
 F0 "SSR_DRIVER" 50
 F1 "SSR_DRIVER.sch" 50
-F2 "STM32_SSR_OUTPUT" I L 11600 6200 50
+F2 "STM32_SSR_OUTPUT" I L 11650 6200 50
 F3 "SSR_CH1_OUTPUT1" I R 13150 6450 50
 F4 "SSR_CH1_OUTPUT2" I R 13150 6600 50
@@
 STM32_SSR_OUTPUT
 Wire Wire Line
-	10400 6200 11600 6200
+	10400 6200 11650 6200
 Text Label 14500 6450 2    50   ~ 0
 SSR_CH1_OUTPUT1
@@
 $EndSheet
 $Comp
-L tinkerforge:+5V #PWR01
+L stm32_bottom_board_respin-rescue:+5V-tinkerforge #PWR01
 U 1 1 5BCBF96D
 P 6700 1050
@@
 Wire Wire Line
 	7550 3800 6800 3800
+$Sheet
+S 11650 7900 1500 850
+U 5BCB4060
+F0 "WS2812_PWM_DRIVER" 50
+F1 "WS2812_PWM_DRIVER.sch" 50
+F2 "STM32_WS2812_PWM" I L 11650 8250 50
+F3 "WS2812_PWM_OUTPUT" I R 13150 8550 50
+$EndSheet
 $EndSCHEMATC

Commit message: update,
Parts:
- J2: value Conn_01x03 -> WS2812; footprint Connector_PinHeader_1.27mm:PinHeader_1x03_P1.27mm_Vertical -> w_conn_mkds:mkds_1,5-3
- J3: value Conn_01x04 -> FAN_PWM; footprint Connector_PinHeader_1.27mm:PinHeader_1x04_P1.27mm_Horizontal -> w_conn_mkds:mkds_1,5-4
- J4: value Conn_01x02 -> SSR; footprint Connector_PinHeader_1.27mm:PinHeader_1x02_P1.27mm_Vertical -> w_conn_mkds:mkds_1,5-2
- J5: value Conn_01x02 -> PURFUME; footprint Connector_PinHeader_1.27mm:PinHeader_1x02_P1.27mm_Vertical -> w_conn_mkds:mkds_1,5-2
Changed lines of the file:
@@
 P 8700 8400
 F 0 "J2" H 8780 8442 50  0000 L CNN
-F 1 "Conn_01x03" H 8780 8351 50  0000 L CNN
-F 2 "Connector_PinHeader_1.27mm:PinHeader_1x03_P1.27mm_Vertical" H 8700 8400 50  0001 C CNN
+F 1 "WS2812" H 8780 8351 50  0000 L CNN
+F 2 "w_conn_mkds:mkds_1,5-3" H 8700 8400 50  0001 C CNN
 F 3 "~" H 8700 8400 50  0001 C CNN
 	1    8700 8400
@@
 P 9650 6450
 F 0 "J5" H 9730 6442 50  0000 L CNN
-F 1 "Conn_01x02" H 9730 6351 50  0000 L CNN
-F 2 "Connector_PinHeader_1.27mm:PinHeader_1x02_P1.27mm_Vertical" H 9650 6450 50  0001 C CNN
+F 1 "PURFUME" H 9730 6351 50  0000 L CNN
+F 2 "w_conn_mkds:mkds_1,5-2" H 9650 6450 50  0001 C CNN
 F 3 "~" H 9650 6450 50  0001 C CNN
 	1    9650 6450
@@
 P 9600 4950
 F 0 "J4" H 9680 4942 50  0000 L CNN
-F 1 "Conn_01x02" H 9680 4851 50  0000 L CNN
-F 2 "Connector_PinHeader_1.27mm:PinHeader_1x02_P1.27mm_Vertical" H 9600 4950 50  0001 C CNN
+F 1 "SSR" H 9680 4851 50  0000 L CNN
+F 2 "w_conn_mkds:mkds_1,5-2" H 9600 4950 50  0001 C CNN
 F 3 "~" H 9600 4950 50  0001 C CNN
 	1    9600 4950
@@
 P 9550 3800
 F 0 "J3" H 9630 3792 50  0000 L CNN
-F 1 "Conn_01x04" H 9630 3701 50  0000 L CNN
-F 2 "Connector_PinHeader_1.27mm:PinHeader_1x04_P1.27mm_Horizontal" H 9550 3800 50  0001 C CNN
+F 1 "FAN_PWM" H 9630 3701 50  0000 L CNN
+F 2 "w_conn_mkds:mkds_1,5-4" H 9550 3800 50  0001 C CNN
 F 3 "~" H 9550 3800 50  0001 C CNN
 	1    9550 3800

Commit message: update,
Parts:
- J1: footprint Connector_PinHeader_2.00mm:PinHeader_1x02_P2.00mm_Vertical -> w_conn_mkds:mkds_1,5-2
Changed lines of the file:
@@
 F 0 "J1" H 7880 3692 50  0000 L CNN
 F 1 "Conn_01x02" H 7880 3601 50  0000 L CNN
-F 2 "Connector_PinHeader_2.00mm:PinHeader_1x02_P2.00mm_Vertical" H 7800 3700 50  0001 C CNN
+F 2 "w_conn_mkds:mkds_1,5-2" H 7800 3700 50  0001 C CNN
 F 3 "~" H 7800 3700 50  0001 C CNN
 	1    7800 3700

Commit message: update,
Changed lines of the file:
@@
 $EndSheet
-$Comp
-L stm32_bottom_board_respin-rescue:+5V-tinkerforge #PWR01
-U 1 1 5BCBF96D
-P 6700 1050
-F 0 "#PWR01" H 6700 900 50  0001 C CNN
-F 1 "+5V" H 6715 1223 50  0000 C CNN
-F 2 "" H 6700 1050 50  0000 C CNN
-F 3 "" H 6700 1050 50  0000 C CNN
-	1    6700 1050
-	1    0    0    -1
-$EndComp
 $Comp
 L power:VDD #PWR02
@@
 F3 "WS2812_PWM_OUTPUT" I R 13150 8550 50
 $EndSheet
+$Comp
+L tinkerforge:+5V #PWR?
+U 1 1 5BCEC385
+P 6700 1050
+F 0 "#PWR?" H 6700 900 50  0001 C CNN
+F 1 "+5V" H 6715 1223 50  0000 C CNN
+F 2 "" H 6700 1050 50  0000 C CNN
+F 3 "" H 6700 1050 50  0000 C CNN
+	1    6700 1050
+	1    0    0    -1
+$EndComp
 $EndSCHEMATC

Commit message: update,
Parts:
- added J?: SSR, w_conn_mkds:mkds_1,5-2, symbol Connector_Generic:Conn_01x02
Connections:
- new net IONAIR_RX: J?.2 (Pin_2)
- new net IONAIR_TX: J?.1 (Pin_1)
Changed lines of the file:
@@
 $Descr A3 16535 11693
 encoding utf-8
-Sheet 1 6
+Sheet 1 7
 Title ""
 Date ""
@@
 	1    0    0    -1
 $EndComp
+$Sheet
+S 11650 2250 1500 850
+U 5BCE47B4
+F0 "rs232_level_switch" 50
+F1 "rs232_level_switch.sch" 50
+F2 "TTL-TX1" I L 11650 2550 50
+F3 "TTL-TX2" I L 11650 2650 50
+F4 "TTL-RX1" I L 11650 2750 50
+F5 "TTL-RX2" I L 11650 2850 50
+F6 "RS232-TX1" I R 13150 2550 50
+F7 "RS232-TX2" I R 13150 2650 50
+F8 "RS232-RX1" I R 13150 2750 50
+F9 "RS232-RX2" I R 13150 2850 50
+$EndSheet
+Text Label 13900 2550 2    50   ~ 0
+IONAIR_TX
+Wire Wire Line
+	13900 2550 13150 2550
+Wire Wire Line
+	13900 2750 13150 2750
+Text Label 13900 2750 2    50   ~ 0
+IONAIR_RX
+Text Label 11000 2550 0    50   ~ 0
+IONAIR-TTL-TX
+Text Label 11000 2750 0    50   ~ 0
+IONAIR-TTL-RX
+Wire Wire Line
+	11000 2550 11650 2550
+Wire Wire Line
+	11000 2750 11650 2750
+$Comp
+L Connector_Generic:Conn_01x02 J?
+U 1 1 5BCF033A
+P 9600 2550
+F 0 "J?" H 9680 2542 50  0000 L CNN
+F 1 "SSR" H 9680 2451 50  0000 L CNN
+F 2 "w_conn_mkds:mkds_1,5-2" H 9600 2550 50  0001 C CNN
+F 3 "~" H 9600 2550 50  0001 C CNN
+	1    9600 2550
+	1    0    0    -1
+$EndComp
+Text Label 8650 2550 0    50   ~ 0
+IONAIR_TX
+Wire Wire Line
+	8650 2550 9400 2550
+Wire Wire Line
+	8650 2650 9400 2650
+Text Label 8650 2650 0    50   ~ 0
+IONAIR_RX
 $EndSCHEMATC
