File: stm32_bottom_board_respin.kicad_pcb (KiCad board)
At the start: 2 copper layers, 90 x 60 mm, 49 parts, among them J1 Conn_01x02, J2 WS2812, J3 FAN_PWM, J4 SSR, J5 PURFUME, J6 Conn_01x14, J7 Conn_01x12, J8 Conn_01x12, Q1 2N3904(1AM), Q2 SS9013_J3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

Commit message: update,
Parts:
- removed BOOT2: SolderJumper_3_Open, Jumper:SolderJumper-3_P2.0mm_Open_TrianglePad1.0x1.5mm
- added BOOT0: JUMPER, Jumper:SolderJumper-3_P2.0mm_Open_TrianglePad1.0x1.5mm, F.Cu at (43.3, 16.1)
- added Q3: SS9013_J3, Package_TO_SOT_SMD:SOT-23_Handsoldering, F.Cu at (68.3, 43.2)
- BOOT1: value SolderJumper_3_Open -> JUMPER
- J1: footprint Connector_PinHeader_2.00mm:PinHeader_1x02_P2.00mm_Vertical -> w_conn_mkds:mkds_1,5-2
- moved J1 63.4 mm to (11.4, 58.7), turned to 270 degrees
- moved R4 47.9 mm to (65.3, 52.1), turned to 180 degrees
- moved J7 44.8 mm to (56.0, 34.6), turned to 180 degrees
- moved D1 43.4 mm to (60.7, 52.1)
- moved J8 42.5 mm to (26.2, 51.1), turned to 90 degrees
- moved Q2 40.0 mm to (64.5, 29.0)
- moved Q1 36.8 mm to (47.2, 58.9)
- moved J6 35.1 mm to (49.7, 7.89), turned to 270 degrees
- moved R5 35.1 mm to (61.0, 36.8), turned to 180 degrees
- moved R8 33.5 mm to (70.6, 28.2)
- moved C14 32.9 mm to (13.6, 47.8)
- moved R6 32.5 mm to (69.3, 47.5)
- moved R3 31.7 mm to (56.4, 52.1), turned to 180 degrees
- moved BOOT1 30.1 mm to (44.5, 40.9), turned to 90 degrees
- moved R7 29.3 mm to (62.0, 24.6), turned to 180 degrees
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Connections:
- R10 pad 2: Net-(BOOT2-Pad2) -> Net-(BOOT1-Pad2)
- R9 pad 1: Net-(BOOT1-Pad2) -> Net-(BOOT0-Pad2)

Commit message: update,
Parts:
- moved J1 83.0 mm to (83.1, 16.7), turned to 90 degrees
- moved JP1 42.9 mm to (27.1, 7.56), turned to 180 degrees
- moved C12 32.8 mm to (11.6, 40.1), turned to 0 degrees
- moved C10 26.3 mm to (15.1, 48.3)
- moved R12 26.3 mm to (18.9, 48.3), turned to 180 degrees
- moved C14 25.1 mm to (26.3, 26.0), turned to 270 degrees
- moved Y1 25.0 mm to (15.8, 35.6), turned to 180 degrees
- moved C11 22.7 mm to (19.8, 40.1), turned to 180 degrees
- moved Y2 21.8 mm to (28.3, 27.2), turned to 90 degrees
- moved SW1 21.8 mm to (15.8, 45.2)
- moved C13 20.0 mm to (24.6, 28.0), turned to 90 degrees
- moved J2 15.3 mm to (68.3, 10.6), turned to 180 degrees
- moved R8 8.07 mm to (70.9, 36.3)
- moved R5 8.04 mm to (57.9, 44.3)
- moved R7 7.59 mm to (64.1, 31.9)
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Connections:
- J6 pad 13: Net-(J6-Pad13) -> /STM32_CORE/PC13
- J6 pad 14: /STM32_CORE/PC13 -> Net-(J6-Pad14)
- JP1 pad 1: Net-(J8-Pad1) -> Net-(J6-Pad14)
Routing:
- net GND: track 0.00 -> 218.4 mm
- net +3V3: track 0.00 -> 111.4 mm
- net /STM32_CORE/OSCIN: track 0.00 -> 34.0 mm
- net /STM32_CORE/RESET: track 0.00 -> 32.0 mm
- net +5V: track 0.00 -> 27.5 mm
- net /STM32_CORE/OSCOUT: track 0.00 -> 23.9 mm
- net /STM32_CORE/SWIO: track 0.00 -> 23.7 mm
- net /STM32_CORE/PA0: track 0.00 -> 23.5 mm
- net /STM32_CORE/PB1: track 0.00 -> 23.0 mm
- net /STM32_CORE/PA1: track 0.00 -> 22.7 mm
- net /STM32_CORE/PB0: track 0.00 -> 22.6 mm
- net /STM32_CORE/PA7: track 0.00 -> 22.2 mm
- net /STM32_CORE/PC13: track 0.00 -> 21.8 mm
- net /STM32_CORE/PB11: track 0.00 -> 21.8 mm
- net /STM32_CORE/PA2: track 0.00 -> 21.4 mm
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
Commit message: update,
Parts:
- U2: footprint Package_SIP:SIP4_Sharp-SSR_P7.62mm_Straight -> footprint-lib:OMRON-G3MB-202P
- moved U2 5.10 mm to (64.0, 60.0)
Changed lines of the file:
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@@
     (add_net VWS2812)
+  )
+  (module footprint-lib:OMRON-G3MB-202P (layer F.Cu)
+    (at 64 60 180)
+    (descr "relay, 34.51series")
+    (fp_text reference U2 (at 0 -3.8 180) (layer F.SilkS)
+      (effects (font (size 1.524 1.524) (thickness 0.3048)))
+    )
+    (fp_text value S102S01 (at 0 4.3 180) (layer F.SilkS)
+      (effects (font (size 1.524 1.524) (thickness 0.3048)))
+    )
+    (fp_arc (start 11.74962 -2.24962) (end 11.74962 -2.75) (angle 90) (layer F.SilkS) (width 0.3048))
+    (fp_arc (start -11.74962 -2.24962) (end -12.25 -2.24962) (angle 90) (layer F.SilkS) (width 0.3048))
+    (fp_line (start -11.74962 -2.75) (end 11.74962 -2.75) (layer F.SilkS) (width 0.3048))
+    (fp_line (start -11.74962 2.75) (end 11.74962 2.75) (layer F.SilkS) (width 0.3048))
+    (fp_line (start -12.25 -2.24962) (end -12.25 2.24962) (layer F.SilkS) (width 0.3048))
+    (fp_line (start 12.25 -2.24962) (end 12.25 2.24962) (layer F.SilkS) (width 0.3048))
+    (fp_line (start 11.437241 -0.281265) (end 11.437241 -1.681265) (layer F.SilkS) (width 0.3048))
+    (fp_line (start 6.437241 -0.581265) (end 7.437241 -1.881265) (layer F.SilkS) (width 0.3048))
+    (fp_line (start 11.437241 -1.681265) (end 7.137241 -1.681265) (layer F.SilkS) (width 0.3048))
+    (fp_line (start 5.737241 -1.681265) (end 1.437241 -1.681265) (layer F.SilkS) (width 0.3048))
+    (fp_line (start 1.437241 -0.281265) (end 1.437241 -1.681265) (layer F.SilkS) (width 0.3048))
+    (fp_line (start -9.293278 -2.316312) (end -9.293278 -0.116312) (layer F.SilkS) (width 0.3048))
+    (fp_line (start -7.693278 -2.316312) (end -9.293278 -2.316312) (layer F.SilkS) (width 0.3048))
+    (fp_line (start -7.693278 -0.116312) (end -7.693278 -2.316312) (layer F.SilkS) (width 0.3048))
+    (fp_line (start -9.293278 -0.116312) (end -7.693278 -0.116312) (layer F.SilkS) (width 0.3048))
+    (fp_line (start -7.693278 -2.316312) (end -9.293278 -0.116312) (layer F.SilkS) (width 0.3048))
+    (fp_line (start -7.693278 -1.216312) (end -6.593278 -1.216312) (layer F.SilkS) (width 0.3048))
+    (fp_line (start -9.293278 -1.216312) (end -10.293278 -1.216312) (layer F.SilkS) (width 0.3048))
+    (fp_line (start -6.593278 -0.216312) (end -6.593278 -1.216312) (layer F.SilkS) (width 0.3048))
+    (fp_line (start -10.293278 -0.216312) (end -10.293278 -1.216312) (layer F.SilkS) (width 0.3048))
+    (fp_arc (start 11.74962 2.24962) (end 12.25 2.24962) (angle 90) (layer F.SilkS) (width 0.3048))
+    (fp_arc (start -11.74962 2.24962) (end -11.74962 2.75) (angle 90) (layer F.SilkS) (width 0.3048))
+    (pad 2 thru_hole circle (at 2.54 1.48 180) (size 2.5 2.5) (drill 1.1) (layers *.Cu *.Mask)
+      (net 23 /SSR_CH1_OUTPUT1))
+    (pad 4 thru_hole circle (at -10.16 1.48 180) (size 2 2) (drill 0.8) (layers *.Cu *.Mask)
+      (net 16 "Net-(Q1-Pad3)"))
+    (pad 1 thru_hole circle (at 10.16 1.48 180) (size 2.5 2.5) (drill 1.1) (layers *.Cu *.Mask)
+      (net 22 /SSR_CH1_OUTPUT2))
+    (pad 3 thru_hole circle (at -6.61 1.48 180) (size 2 2) (drill 0.8) (layers *.Cu *.Mask)
+      (net 15 "Net-(R4-Pad2)"))
   )
   (module w_conn_mkds:mkds_1,5-2 (layer F.Cu)
@@
       (net 18 +3V3))
     (model ${KISYS3DMOD}/Package_QFP.3dshapes/LQFP-48_7x7mm_P0.5mm.wrl
-      (at (xyz 0 0 0))
-      (scale (xyz 1 1 1))
-      (rotate (xyz 0 0 0))
-    )
-  )
-  (module Package_SIP:SIP4_Sharp-SSR_P7.62mm_Straight (layer F.Cu)
-    (at 69 59 180)
-    (descr "SIP4 Footprint for SSR made by Sharp")
-    (tags "Solid State relais SSR Sharp")
-    (fp_text reference U2 (at 0.508 -2.54 180) (layer F.SilkS)
-      (effects (font (size 1 1) (thickness 0.15)))
-    )
-    (fp_text value S102S01 (at 7.62 5 180) (layer F.Fab)
-      (effects (font (size 1 1) (thickness 0.15)))
-    )
-    (fp_text user %R (at 7.62 0 180) (layer F.Fab)
-      (effects (font (size 1 1) (thickness 0.15)))
-    )
-    (fp_line (start 1.27 -0.3) (end 3.81 -0.3) (layer F.SilkS) (width 0.15))
-    (fp_line (start 6.35 -0.3) (end 11.43 -0.3) (layer F.SilkS) (width 0.15))
-    (fp_line (start 17.25 -1.95) (end 17.25 4.25) (layer F.CrtYd) (width 0.05))
-    (fp_line (start 17.25 4.25) (end -2 4.25) (layer F.CrtYd) (width 0.05))
-    (fp_line (start -2 4.25) (end -2 -1.95) (layer F.CrtYd) (width 0.05))
-    (fp_line (start -2 -1.95) (end 17.25 -1.95) (layer F.CrtYd) (width 0.05))
-    (fp_line (start 2.62 4) (end 1.28 1.5) (layer F.SilkS) (width 0.15))
-    (fp_line (start 12.62 4) (end 13.96 1.5) (layer F.SilkS) (width 0.15))
-    (fp_line (start -1.73 -1.7) (end 16.97 -1.7) (layer F.SilkS) (width 0.15))
-    (fp_line (start 16.97 -1.7) (end 16.97 4) (layer F.SilkS) (width 0.15))
-    (fp_line (start 16.97 4) (end -1.73 4) (layer F.SilkS) (width 0.15))
-    (fp_line (start -1.73 4) (end -1.73 -1.7) (layer F.SilkS) (width 0.15))
-    (fp_line (start -1.6 3.9) (end 16.8 3.9) (layer F.Fab) (width 0.1))
-    (fp_line (start 16.8 3.9) (end 16.8 -1.6) (layer F.Fab) (width 0.1))
-    (fp_line (start 16.8 -1.6) (end -0.6 -1.6) (layer F.Fab) (width 0.1))
-    (fp_line (start -0.6 -1.6) (end -1.6 -0.6) (layer F.Fab) (width 0.1))
-    (fp_line (start -1.6 -0.6) (end -1.6 3.9) (layer F.Fab) (width 0.1))
-    (pad 1 thru_hole rect (at 0 0 180) (size 2 3) (drill 1.2) (layers *.Cu *.Mask)
-      (net 22 /SSR_CH1_OUTPUT2))
-    (pad 2 thru_hole oval (at 5.08 0 180) (size 2 3) (drill 1.2) (layers *.Cu *.Mask)
-      (net 23 /SSR_CH1_OUTPUT1))
-    (pad 3 thru_hole oval (at 12.7 0 180) (size 2 3) (drill 1.2) (layers *.Cu *.Mask)
-      (net 15 "Net-(R4-Pad2)"))
-    (pad 4 thru_hole oval (at 15.24 0 180) (size 2 3) (drill 1.2) (layers *.Cu *.Mask)
-      (net 16 "Net-(Q1-Pad3)"))
-    (model ${KISYS3DMOD}/Package_SIP.3dshapes/SIP4_Sharp-SSR_P7.62mm_Straight.wrl
       (at (xyz 0 0 0))
       (scale (xyz 1 1 1))
@@
   (segment (start 20.261497 24.379003) (end 23.622 21.0185) (width 0.25) (layer F.Cu) (net 6))
   (segment (start 18.344088 24.379003) (end 20.261497 24.379003) (width 0.25) (layer F.Cu) (net 6))
-  (segment (start 28.177003 7.894003) (end 27.8395 7.5565) (width 0.25) (layer F.Cu) (net 76))
   (segment (start 44.460088 40.914003) (end 44.492088 40.946003) (width 0.25) (layer F.Cu) (net 7) (status 30))
   (segment (start 41.952088 40.914003) (end 44.460088 40.914003) (width 0.25) (layer F.Cu) (net 7) (status 30))
@@
   (segment (start 37.843503 15.609503) (end 37.719 15.485) (width 0.25) (layer F.Cu) (net 75) (status 30))
   (segment (start 39.729588 15.609503) (end 37.843503 15.609503) (width 0.25) (layer F.Cu) (net 75) (status 30))
+  (segment (start 28.177003 7.894003) (end 27.8395 7.5565) (width 0.25) (layer F.Cu) (net 76))
   (segment (start 32.851585 7.5565) (end 33.189088 7.894003) (width 0.25) (layer F.Cu) (net 76))
   (segment (start 27.8395 7.5565) (end 32.851585 7.5565) (width 0.25) (layer F.Cu) (net 76))

Commit message: update,
Parts:
- added U1: 74AHCT1G125, Package_TO_SOT_SMD:SOT-23-5_HandSoldering, F.Cu at (56.0, 15.0)
- U2: value S102S01 -> OMRON-G3MB-202P
Connections:
- D1 pad 2: VDD -> +5V
- R4 pad 1: VDD -> +5V
- R6 pad 1: VDD -> +5V
- R8 pad 1: VDD -> +5V
Changed lines of the file:
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@@
     (tracks 338)
     (zones 0)
-    (modules 50)
+    (modules 51)
     (nets 77)
   )
@@
   (net 72 VWS2812)
   (net 73 "Net-(Q1-Pad1)")
-  (net 74 VDD)
-  (net 75 "Net-(BOOT0-Pad2)")
-  (net 76 "Net-(J6-Pad14)")
+  (net 74 "Net-(BOOT0-Pad2)")
+  (net 75 "Net-(J6-Pad14)")
+  (net 76 /STM32_WS2812_OUTPUT)
   (net_class Default "This is the default net class."
     (clearance 0.2)
@@
     (add_net /STM32_SSR-25-DA_OUTPUT)
     (add_net /STM32_SSR_OUTPUT)
+    (add_net /STM32_WS2812_OUTPUT)
     (add_net /WS2812_PWM_TERMINAL)
     (add_net GND)
@@
     (add_net "Net-(Q3-Pad1)")
     (add_net "Net-(R4-Pad2)")
-    (add_net VDD)
     (add_net VWS2812)
+  )
+  (module Package_TO_SOT_SMD:SOT-23-5_HandSoldering (layer F.Cu)
+    (at 56 15)
+    (descr "5-pin SOT23 package")
+    (tags "SOT-23-5 hand-soldering")
+    (attr smd)
+    (fp_text reference U1 (at 0 -2.9) (layer F.SilkS)
+      (effects (font (size 1 1) (thickness 0.15)))
+    )
+    (fp_text value 74AHCT1G125 (at 0 2.9) (layer F.Fab)
+      (effects (font (size 1 1) (thickness 0.15)))
+    )
+    (fp_text user %R (at 0 0 90) (layer F.Fab)
+      (effects (font (size 0.5 0.5) (thickness 0.075)))
+    )
+    (fp_line (start -0.9 1.61) (end 0.9 1.61) (layer F.SilkS) (width 0.12))
+    (fp_line (start 0.9 -1.61) (end -1.55 -1.61) (layer F.SilkS) (width 0.12))
+    (fp_line (start -0.9 -0.9) (end -0.25 -1.55) (layer F.Fab) (width 0.1))
+    (fp_line (start 0.9 -1.55) (end -0.25 -1.55) (layer F.Fab) (width 0.1))
+    (fp_line (start -0.9 -0.9) (end -0.9 1.55) (layer F.Fab) (width 0.1))
+    (fp_line (start 0.9 1.55) (end -0.9 1.55) (layer F.Fab) (width 0.1))
+    (fp_line (start 0.9 -1.55) (end 0.9 1.55) (layer F.Fab) (width 0.1))
+    (fp_line (start -2.38 -1.8) (end 2.38 -1.8) (layer F.CrtYd) (width 0.05))
+    (fp_line (start -2.38 -1.8) (end -2.38 1.8) (layer F.CrtYd) (width 0.05))
+    (fp_line (start 2.38 1.8) (end 2.38 -1.8) (layer F.CrtYd) (width 0.05))
+    (fp_line (start 2.38 1.8) (end -2.38 1.8) (layer F.CrtYd) (width 0.05))
+    (pad 1 smd rect (at -1.35 -0.95) (size 1.56 0.65) (layers F.Cu F.Paste F.Mask)
+      (net 1 GND))
+    (pad 2 smd rect (at -1.35 0) (size 1.56 0.65) (layers F.Cu F.Paste F.Mask)
+      (net 76 /STM32_WS2812_OUTPUT))
+    (pad 3 smd rect (at -1.35 0.95) (size 1.56 0.65) (layers F.Cu F.Paste F.Mask)
+      (net 1 GND))
+    (pad 4 smd rect (at 1.35 0.95) (size 1.56 0.65) (layers F.Cu F.Paste F.Mask)
+      (net 21 /WS2812_PWM_TERMINAL))
+    (pad 5 smd rect (at 1.35 -0.95) (size 1.56 0.65) (layers F.Cu F.Paste F.Mask)
+      (net 6 +5V))
+    (model ${KISYS3DMOD}/Package_TO_SOT_SMD.3dshapes/SOT-23-5.wrl
+      (at (xyz 0 0 0))
+      (scale (xyz 1 1 1))
+      (rotate (xyz 0 0 0))
+    )
   )
   (module footprint-lib:OMRON-G3MB-202P (layer F.Cu)
@@
       (effects (font (size 1.524 1.524) (thickness 0.3048)))
     )
-    (fp_text value S102S01 (at 0 4.3 180) (layer F.SilkS)
+    (fp_text value OMRON-G3MB-202P (at 0 4.3 180) (layer F.SilkS)
       (effects (font (size 1.524 1.524) (thickness 0.3048)))
     )
@@
       ))
     (pad 2 smd custom (at 0 0 90) (size 0.3 0.3) (layers F.Cu)
-      (net 75 "Net-(BOOT0-Pad2)") (zone_connect 0)
+      (net 74 "Net-(BOOT0-Pad2)") (zone_connect 0)
       (options (clearance outline) (anchor rect))
       (primitives
@@
       (net 25 /STM32_CORE/PC13))
     (pad 14 thru_hole oval (at 0 16.51 270) (size 1 1) (drill 0.65) (layers *.Cu *.Mask)
-      (net 76 "Net-(J6-Pad14)"))
+      (net 75 "Net-(J6-Pad14)"))
     (model ${KISYS3DMOD}/Connector_PinHeader_1.27mm.3dshapes/PinHeader_1x14_P1.27mm_Vertical.wrl
       (at (xyz 0 0 0))
@@
       ))
     (pad 1 smd custom (at -0.725 0 180) (size 0.3 0.3) (layers F.Cu F.Mask)
-      (net 76 "Net-(J6-Pad14)") (zone_connect 0)
+      (net 75 "Net-(J6-Pad14)") (zone_connect 0)
       (options (clearance outline) (anchor rect))
       (primitives
@@
       (net 17 "Net-(D1-Pad1)"))
     (pad 2 smd roundrect (at 1.025 0) (size 1.15 1.4) (layers F.Cu F.Paste F.Mask) (roundrect_rratio 0.217391)
-      (net 74 VDD))
+      (net 6 +5V))
     (model ${KISYS3DMOD}/LED_SMD.3dshapes/LED_0805_2012Metric.wrl
       (at (xyz 0 0 0))
@@
     )
     (pad 1 smd roundrect (at -1.025 0 180) (size 1.15 1.4) (layers F.Cu F.Paste F.Mask) (roundrect_rratio 0.217391)
-      (net 74 VDD))
+      (net 6 +5V))
     (pad 2 smd roundrect (at 1.025 0 180) (size 1.15 1.4) (layers F.Cu F.Paste F.Mask) (roundrect_rratio 0.217391)
       (net 15 "Net-(R4-Pad2)"))
@@
     )
     (pad 1 smd roundrect (at -1.025 0) (size 1.15 1.4) (layers F.Cu F.Paste F.Mask) (roundrect_rratio 0.217391)
-      (net 74 VDD))
+      (net 6 +5V))
     (pad 2 smd roundrect (at 1.025 0) (size 1.15 1.4) (layers F.Cu F.Paste F.Mask) (roundrect_rratio 0.217391)
       (net 12 /SSR-25-DA1))
@@
     )
     (pad 1 smd roundrect (at -1.025 0 270) (size 1.15 1.4) (layers F.Cu F.Paste F.Mask) (roundrect_rratio 0.217391)
-      (net 75 "Net-(BOOT0-Pad2)"))
+      (net 74 "Net-(BOOT0-Pad2)"))
     (pad 2 smd roundrect (at 1.025 0 270) (size 1.15 1.4) (layers F.Cu F.Paste F.Mask) (roundrect_rratio 0.217391)
       (net 8 /STM32_CORE/BOOT0))
@@
       (net 5 /FAN_PWM_OUTPUT))
     (pad 1 smd roundrect (at -1.025 0) (size 1.15 1.4) (layers F.Cu F.Paste F.Mask) (roundrect_rratio 0.217391)
-      (net 74 VDD))
+      (net 6 +5V))
     (model ${KISYS3DMOD}/Resistor_SMD.3dshapes/R_0805_2012Metric.wrl
       (at (xyz 0 0 0))
@@
   (segment (start 73.326 23.0125) (end 72.907 23.4315) (width 0.25) (layer F.Cu) (net 72) (status 30))
   (segment (start 73.326 10.6045) (end 73.326 23.0125) (width 0.25) (layer F.Cu) (net 72) (status 30))
-  (segment (start 37.843503 15.609503) (end 37.719 15.485) (width 0.25) (layer F.Cu) (net 75) (status 30))
-  (segment (start 39.729588 15.609503) (end 37.843503 15.609503) (width 0.25) (layer F.Cu) (net 75) (status 30))
-  (segment (start 28.177003 7.894003) (end 27.8395 7.5565) (width 0.25) (layer F.Cu) (net 76))
-  (segment (start 32.851585 7.5565) (end 33.189088 7.894003) (width 0.25) (layer F.Cu) (net 76))
-  (segment (start 27.8395 7.5565) (end 32.851585 7.5565) (width 0.25) (layer F.Cu) (net 76))
+  (segment (start 37.843503 15.609503) (end 37.719 15.485) (width 0.25) (layer F.Cu) (net 74) (status 30))
+  (segment (start 39.729588 15.609503) (end 37.843503 15.609503) (width 0.25) (layer F.Cu) (net 74) (status 30))
+  (segment (start 28.177003 7.894003) (end 27.8395 7.5565) (width 0.25) (layer F.Cu) (net 75))
+  (segment (start 32.851585 7.5565) (end 33.189088 7.894003) (width 0.25) (layer F.Cu) (net 75))
+  (segment (start 27.8395 7.5565) (end 32.851585 7.5565) (width 0.25) (layer F.Cu) (net 75))
 )

Commit message: update,
Parts:
- added C15: C104, Capacitor_SMD:C_0805_2012Metric_Pad1.15x1.40mm_HandSolder, F.Cu at (9.00, 53.0)
- added C16: C104, Capacitor_SMD:C_0805_2012Metric_Pad1.15x1.40mm_HandSolder, F.Cu at (8.97, 60.0)
- added C17: C104, Capacitor_SMD:C_0805_2012Metric_Pad1.15x1.40mm_HandSolder, F.Cu at (25.0, 55.0)
- added C18: C104, Capacitor_SMD:C_0805_2012Metric_Pad1.15x1.40mm_HandSolder, F.Cu at (18.0, 52.0)
- added C19: C104, Capacitor_SMD:C_0805_2012Metric_Pad1.15x1.40mm_HandSolder, F.Cu at (8.97, 57.0)
- added J9: SSR, w_conn_mkds:mkds_1,5-2, F.Cu at (32.0, 59.0)
- added U5: SP3232EEN, footprint-lib:SOP-16_4.4x10.4mm_Pitch1.27mm, F.Cu at (18.0, 59.0)

Commit message: update,
Routing:
- net +3V3: track 111.4 -> 128.6 mm, vias 0 -> 1
Changed lines of the file:
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@@
     (thickness 1.6)
     (drawings 16)
-    (tracks 338)
+    (tracks 345)
     (zones 0)
     (modules 58)
@@
   (segment (start 28.744088 49.191088) (end 28.744088 51.074003) (width 0.25) (layer F.Cu) (net 18))
   (segment (start 27.8765 48.3235) (end 28.744088 49.191088) (width 0.25) (layer F.Cu) (net 18))
+  (segment (start 46.496 21.504) (end 46.496 23.749) (width 0.25) (layer F.Cu) (net 18))
+  (segment (start 49.699088 18.300912) (end 49.699088 7.894003) (width 0.25) (layer B.Cu) (net 18))
+  (segment (start 47.244 20.447) (end 46.496 21.504) (width 0.25) (layer F.Cu) (net 18))
+  (via (at 47.244 20.447) (size 1.2) (drill 0.4) (layers F.Cu B.Cu) (net 18))
+  (segment (start 47.244 20.447) (end 49.699088 18.300912) (width 0.25) (layer B.Cu) (net 18))
   (segment (start 27.813 38.1) (end 20.680997 45.232003) (width 0.25) (layer F.Cu) (net 19))
   (segment (start 27.813 35.6235) (end 27.813 38.1) (width 0.25) (layer F.Cu) (net 19))
@@
   (segment (start 48.429088 20.616088) (end 48.429088 7.894003) (width 0.25) (layer F.Cu) (net 51) (status 20))
   (segment (start 50.038 22.225) (end 48.429088 20.616088) (width 0.25) (layer F.Cu) (net 51))
-  (segment (start 47.159088 19.642912) (end 47.159088 7.894003) (width 0.25) (layer F.Cu) (net 52) (status 20))
-  (segment (start 44.194088 22.607912) (end 47.159088 19.642912) (width 0.25) (layer F.Cu) (net 52))
-  (segment (start 44.194088 24.880003) (end 44.194088 22.607912) (width 0.25) (layer F.Cu) (net 52) (status 10))
+  (segment (start 46 20.802) (end 44.194088 22.607912) (width 0.25) (layer F.Cu) (net 52))
+  (segment (start 46 19) (end 46 20.802) (width 0.25) (layer F.Cu) (net 52))
+  (segment (start 47.159088 17.840912) (end 46 19) (width 0.25) (layer F.Cu) (net 52))
+  (segment (start 44.194088 22.607912) (end 44.194088 24.880003) (width 0.25) (layer F.Cu) (net 52))
+  (segment (start 47.159088 7.894003) (end 47.159088 17.840912) (width 0.25) (layer F.Cu) (net 52))
   (segment (start 44.619088 7.894003) (end 44.619088 8.551088) (width 0.25) (layer F.Cu) (net 53) (status 10))
   (segment (start 44.619088 8.551088) (end 44.957295 8.889295) (width 0.25) (layer F.Cu) (net 53))
