File: pcb/stm32_bottom_board_respin.kicad_pcb (KiCad board)
At the start: 2 copper layers, 90 x 60 mm, 58 parts, among them J1 Conn_01x02, J2 WS2812, J3 FAN_PWM, J4 SSR, J5 PURFUME, J6 Conn_01x14, J7 Conn_01x12, J8 Conn_01x12, J9 SSR, Q1 2N3904(1AM)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

Commit message: update,
Parts:
- added J10: Conn_01x08, Connector_FFC-FPC:TE_84952-8_1x08-1MP_P1.0mm_Horizontal, F.Cu at (9.65, 38.0)
- J9: footprint w_conn_mkds:mkds_1,5-2 -> w_conn_mkds:mkds_1,5-3
- moved C12 8.45 mm to (20.1, 40.0)
- moved Y1 4.56 mm to (20.3, 35.8)
- moved C11 4.45 mm to (24.3, 40.1)
- moved C17 3.05 mm to (23.7, 52.2)
- moved J9 1.45 mm to (32.0, 60.5)
- turned Q3 to 270 degrees
- turned R8 to 180 degrees
- turned U2 to 0 degrees
Connections:
- net /IONAIR-TTL-RX renamed IONAIR-TTL-RX
- net /IONAIR-TTL-TX renamed IONAIR-TTL-TX
- net /STM32_CORE/PA3 renamed SPI1_SCK
- net /STM32_CORE/PA4 renamed SPI1_MISO
- net /STM32_CORE/PA5 renamed SPI1_MOSI
- net /STM32_CORE/PB8 renamed I2C_SCL
- net /STM32_CORE/PB9 renamed I2C_SDA
- net /STM32_FAN_PWM_OUTPUT renamed STM32_FAN_PWM_OUTPUT
- net /STM32_SSR-25-DA_OUTPUT renamed STM32_SSR-25-DA_OUTPUT
- net /STM32_SSR_OUTPUT renamed STM32_SSR_OUTPUT
- net /STM32_WS2812_OUTPUT renamed STM32_WS2812_OUTPUT
- J9 pad 1: /IONAIR_TX -> /IONAIR_RX
- J9 pad 2: /IONAIR_RX -> /IONAIR_TX
Routing:
- net /FAN_48V: track 0.00 -> 31.9 mm
- net GND: track 218.4 -> 247.5 mm
- net /FAN_PWM_OUTPUT: track 0.00 -> 20.5 mm
- net /SSR_CH1_OUTPUT1: track 0.00 -> 17.8 mm
- net Net-(Q1-Pad3): track 0.00 -> 15.8 mm
- net /SSR-25-DA2: track 0.00 -> 15.0 mm
- net /SSR-25-DA1: track 0.00 -> 13.9 mm
- net Net-(R4-Pad2): track 0.00 -> 12.3 mm
- net /IONAIR_TX: track 0.00 -> 12.2 mm
- net +5V: track 27.5 -> 39.4 mm
- net Net-(Q3-Pad1): track 0.00 -> 11.8 mm
- net /SSR_CH1_OUTPUT2: track 0.00 -> 10.9 mm
- net /WS2812_PWM_TERMINAL: track 0.00 -> 9.22 mm
- net Net-(Q1-Pad1): track 0.00 -> 8.52 mm
- net /IONAIR_RX: track 0.00 -> 6.72 mm
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
Commit message: update,
Parts:
- added D4: LED_GREEN, LED_SMD:LED_0805_2012Metric_Pad1.15x1.40mm_HandSolder, F.Cu at (34.4, 51.8)
- added D5: LED_GREEN, LED_SMD:LED_0805_2012Metric_Pad1.15x1.40mm_HandSolder, F.Cu at (34.3, 53.8)
- added R14: R102, Resistor_SMD:R_0805_2012Metric_Pad1.15x1.40mm_HandSolder, F.Cu at (28.3, 51.8)
- added R15: R102, Resistor_SMD:R_0805_2012Metric_Pad1.15x1.40mm_HandSolder, F.Cu at (29.7, 53.8)
- J8: value Conn_01x12 -> Conn_01x15; footprint Connector_PinHeader_1.27mm:PinHeader_1x20_P1.27mm_Vertical -> Connector_PinHeader_1.27mm:PinHeader_1x15_P1.27mm_Vertical
- moved J10 46.0 mm to (41.4, 4.70), turned to 180 degrees
- moved C17 25.5 mm to (19.1, 27.2), turned to 0 degrees
- moved BOOT0 8.76 mm to (31.2, 17.8)
- moved R10 8.11 mm to (49.2, 43.6)
- moved BOOT1 7.86 mm to (51.8, 43.7)
- moved J8 6.75 mm to (32.6, 49.0)
- moved Q1 6.34 mm to (50.7, 53.6)
- moved R2 6.03 mm to (46.1, 57.1)
- moved Y1 5.22 mm to (25.3, 37.5), turned to 90 degrees
- moved R1 5.03 mm to (46.1, 52.6), turned to 90 degrees
- moved J9 4.70 mm to (36.7, 60.3)
- moved J6 4.00 mm to (49.7, 11.9)
- moved C9 3.98 mm to (13.7, 27.1)
- moved C11 3.54 mm to (21.0, 41.4), turned to 90 degrees
- moved C7 3.30 mm to (19.7, 24.9)
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Connections:
- J10 pad 1: GND -> +5V
- J10 pad 2: +5V -> GND
- J10 pad 3: I2C_SDA -> SPI1_SCK
- J10 pad 4: I2C_SCL -> SPI1_MISO
- J10 pad 6: SPI1_MISO -> I2C_SCL
- J10 pad 7: SPI1_SCK -> I2C_SDA
- J6 pad 6: /STM32_CORE/PB3 -> SPI1_SCK
- J6 pad 7: /STM32_CORE/PB4 -> SPI1_MISO
- J6 pad 8: /STM32_CORE/PB5 -> SPI1_MOSI
- J7 pad 2: /STM32_CORE/PB13 -> STM32_FAN_PWM_OUTPUT
- J8 pad 1: Net-(J8-Pad1) -> GND
- J8 pad 10: /STM32_CORE/PA1 -> STM32_WS2812_OUTPUT
- J8 pad 11: /STM32_CORE/PA2 -> /STM32_CORE/PA7
- J8 pad 12: SPI1_SCK -> STM32_SSR_OUTPUT
- J8 pad 13: SPI1_MISO -> STM32_SSR-25-DA_OUTPUT
- J8 pad 14: SPI1_MOSI -> /STM32_CORE/PB10
- J8 pad 15: /STM32_CORE/PA6 -> /STM32_CORE/PB11
- J8 pad 2: GND -> +3V3
- J8 pad 3: +3V3 -> Net-(J8-Pad3)
- J8 pad 4: Net-(J8-Pad4) -> /STM32_CORE/PA0
- J8 pad 5: Net-(J8-Pad5) -> /STM32_CORE/PA1
- J8 pad 6: Net-(J8-Pad6) -> IONAIR-TTL-TX
- J8 pad 7: Net-(J8-Pad7) -> IONAIR-TTL-RX
- J8 pad 8: Net-(J8-Pad8) -> /STM32_CORE/PA4
- J8 pad 9: /STM32_CORE/PA0 -> /STM32_CORE/PA5
- U3 pad 12: /STM32_CORE/PA2 -> IONAIR-TTL-TX
- U3 pad 13: SPI1_SCK -> IONAIR-TTL-RX
- U3 pad 14: SPI1_MISO -> /STM32_CORE/PA4
- U3 pad 15: SPI1_MOSI -> /STM32_CORE/PA5
- U3 pad 16: /STM32_CORE/PA6 -> STM32_WS2812_OUTPUT
- U3 pad 18: /STM32_CORE/PB0 -> STM32_SSR_OUTPUT
- U3 pad 19: /STM32_CORE/PB1 -> STM32_SSR-25-DA_OUTPUT
- U3 pad 26: /STM32_CORE/PB13 -> STM32_FAN_PWM_OUTPUT
- U3 pad 39: /STM32_CORE/PB3 -> SPI1_SCK
- U3 pad 40: /STM32_CORE/PB4 -> SPI1_MISO
- U3 pad 41: /STM32_CORE/PB5 -> SPI1_MOSI
- U5 pad 3: Net-(C19-Pad2) -> Net-(C15-Pad2)
- U5 pad 6: (no net) -> Net-(C19-Pad2)
Routing:
- net GND: track 247.5 -> 475.4 mm, vias 0 -> 8
- net +5V: track 39.4 -> 219.6 mm, vias 0 -> 4
- net +3V3: track 128.6 -> 226.3 mm, vias 1 -> 6
- net IONAIR-TTL-TX: track 0.00 -> 58.6 mm, vias 0 -> 1
- net STM32_WS2812_OUTPUT: track 0.00 -> 48.1 mm, vias 0 -> 2
- net IONAIR-TTL-RX: track 0.00 -> 45.5 mm
- net STM32_SSR-25-DA_OUTPUT: track 0.00 -> 33.3 mm
- net /STM32_CORE/PB1: track 23.0 -> 0.00 mm
- net /STM32_CORE/PB0: track 22.6 -> 0.00 mm
- net /STM32_CORE/PA2: track 21.4 -> 0.00 mm
- net /STM32_CORE/PA6: track 21.3 -> 0.00 mm
- net /STM32_CORE/PB3: track 20.6 -> 0.00 mm
- net STM32_SSR_OUTPUT: track 0.00 -> 20.5 mm
- net /STM32_CORE/PB5: track 18.0 -> 0.00 mm
- net /STM32_CORE/PB4: track 17.9 -> 0.00 mm
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Other:
- net class Default: trace_width 0.25 -> 0.3; via_dia 0.8 -> 1.5; via_drill 0.4 -> 1
- net class PWR added: clearance 0.2, trace_width 0.5, via_dia 2, via_drill 1

Commit message: update,
Parts:
- moved Q3 3.21 mm to (67.3, 40.1)
Routing:
- net GND: track 475.4 -> 511.5 mm, vias 8 -> 7
- net IONAIR-TTL-TX: track 58.6 -> 64.8 mm
- net +5V: track 219.6 -> 213.5 mm
- net +3V3: track 226.3 -> 221.7 mm
- net /SSR-25-DA2: track 19.1 -> 22.9 mm
- net Net-(C19-Pad2): track 11.4 -> 14.1 mm
- net Net-(Q3-Pad1): track 17.0 -> 18.6 mm
- net Net-(C15-Pad2): track 7.11 -> 8.39 mm
- net I2C_SDA: track 23.0 -> 24.1 mm
- net I2C_SCL: track 22.9 -> 23.9 mm
- net /FAN_PWM_OUTPUT: track 20.8 -> 21.6 mm
- net Net-(C15-Pad1): track 6.91 -> 7.54 mm
- added copper zone on F.Cu, net GND
Other:
- rule trace_min: 0.2 -> 0.3

Commit message: update,
Connections:
- J5 pad 1: /SSR_CH1_OUTPUT1 -> /SSR_CH1_OUTPUT2
- J5 pad 2: /SSR_CH1_OUTPUT2 -> /SSR_CH1_OUTPUT1
Routing:
- net /SSR_CH1_OUTPUT2: track 12.6 -> 8.85 mm
Other:
- net class HIGH_PWR added: clearance 0.2, trace_width 1, via_dia 2, via_drill 1
Changed lines of the file:
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@@
     (thickness 1.6)
     (drawings 16)
-    (tracks 735)
+    (tracks 732)
     (zones 0)
     (modules 63)
@@
     (uvia_dia 0.3)
     (uvia_drill 0.1)
+    (diff_pair_gap 0.25)
+    (diff_pair_width 0.3)
     (add_net /FAN_PWM_OUTPUT)
     (add_net /FAN_RPM)
@@
     (add_net /SSR-25-DA1)
     (add_net /SSR-25-DA2)
-    (add_net /SSR_CH1_OUTPUT1)
-    (add_net /SSR_CH1_OUTPUT2)
     (add_net /STM32_CORE/BOOT0)
     (add_net /STM32_CORE/BOOT1)
@@
     (add_net VWS2812)
   )
+  (net_class HIGH_PWR ""
+    (clearance 0.2)
+    (trace_width 1)
+    (via_dia 2)
+    (via_drill 1)
+    (uvia_dia 0.3)
+    (uvia_drill 0.1)
+    (diff_pair_gap 0.25)
+    (diff_pair_width 0.3)
+    (add_net /SSR_CH1_OUTPUT1)
+    (add_net /SSR_CH1_OUTPUT2)
+  )
   (net_class PWR ""
     (clearance 0.2)
@@
     (uvia_dia 0.3)
     (uvia_drill 0.1)
+    (diff_pair_gap 0.25)
+    (diff_pair_width 0.3)
     (add_net +3V3)
     (add_net +5V)
@@
     (fp_line (start -5 -5.2) (end -5 4.6) (layer F.SilkS) (width 0.381))
     (pad 1 thru_hole circle (at -2.5 0 90) (size 2.5 2.5) (drill 1.3) (layers *.Cu *.Mask F.SilkS)
-      (net 20 /SSR_CH1_OUTPUT1))
-    (pad 2 thru_hole circle (at 2.5 0 90) (size 2.5 2.5) (drill 1.3) (layers *.Cu *.Mask F.SilkS)
       (net 19 /SSR_CH1_OUTPUT2))
+    (pad 2 thru_hole circle (at 2.5 0 90) (size 2.5 2.5) (drill 1.3) (layers *.Cu *.Mask F.SilkS)
+      (net 20 /SSR_CH1_OUTPUT1))
     (model ${HOME}/_workspace/kicad/kicad_library/smisioto-footprints/modules/packages3d/walter/conn_mkds/mkds_1,5-2.wrl
       (at (xyz 0 0 0))
@@
   (segment (start 61.1759 10.6045) (end 61.558234 10.6045) (width 0.3) (layer B.Cu) (net 18))
   (segment (start 60.2234 11.557) (end 61.1759 10.6045) (width 0.3) (layer B.Cu) (net 18))
-  (segment (start 74.16 61.48) (end 74.16 58.666) (width 0.3) (layer B.Cu) (net 19) (status 10))
-  (segment (start 76.326 56.5) (end 83 56.5) (width 0.3) (layer B.Cu) (net 19) (status 20))
-  (segment (start 74.16 58.666) (end 76.326 56.5) (width 0.3) (layer B.Cu) (net 19))
-  (segment (start 67.046234 63.754) (end 66.54 63.247766) (width 0.3) (layer B.Cu) (net 20))
-  (segment (start 66.54 63.247766) (end 66.54 61.48) (width 0.3) (layer B.Cu) (net 20))
-  (segment (start 83 63.267766) (end 82.513766 63.754) (width 0.3) (layer B.Cu) (net 20))
-  (segment (start 82.513766 63.754) (end 67.046234 63.754) (width 0.3) (layer B.Cu) (net 20))
-  (segment (start 83 61.5) (end 83 63.267766) (width 0.3) (layer B.Cu) (net 20))
+  (segment (start 74.18 61.5) (end 74.16 61.48) (width 1) (layer B.Cu) (net 19))
+  (segment (start 83 61.5) (end 74.18 61.5) (width 1) (layer B.Cu) (net 19))
+  (segment (start 66.54 61.48) (end 66.54 57.92) (width 1) (layer B.Cu) (net 20))
+  (segment (start 67.96 56.5) (end 66.54 57.92) (width 1) (layer B.Cu) (net 20))
+  (segment (start 83 56.5) (end 67.96 56.5) (width 1) (layer B.Cu) (net 20))
   (segment (start 34.459088 12.657912) (end 34.459088 11.894003) (width 0.3) (layer F.Cu) (net 22))
   (segment (start 33.02 14.097) (end 34.459088 12.657912) (width 0.3) (layer F.Cu) (net 22))

Commit message: update,
Parts:
- J6: footprint Connector_PinHeader_1.27mm:PinHeader_1x14_P1.27mm_Vertical -> footprint-lib:PinHeader_1x14_P1.27mm_Vertical
- J7: footprint Connector_PinHeader_1.27mm:PinHeader_1x12_P1.27mm_Vertical -> footprint-lib:PinHeader_1x12_P1.27mm_Vertical
- J8: footprint Connector_PinHeader_1.27mm:PinHeader_1x15_P1.27mm_Vertical -> footprint-lib:PinHeader_1x15_P1.27mm_Vertical
- U2: value OMRON-G3MB-202P -> OMRON G3MB-202P
Routing:
- net /IONAIR_TX: track 17.9 -> 20.5 mm
- net GND: track 511.5 -> 513.5 mm, vias 7 -> 8
Other:
- net class Default: via_dia 1.5 -> 2
- net class GND added: clearance 0.2, trace_width 1, via_dia 2, via_drill 1

Commit message: update,
Routing:
- net Net-(Q1-Pad3): track 11.7 -> 15.1 mm, vias 0 -> 1
- net Net-(R4-Pad2): track 14.3 -> 17.5 mm
- net +3V3: track 221.7 -> 219.0 mm
- net STM32_WS2812_OUTPUT: track 48.1 -> 50.5 mm
- net /STM32_CORE/BOOT1: track 13.8 -> 12.3 mm
- net /STM32_CORE/PB10: track 20.8 -> 19.6 mm
- net IONAIR-TTL-RX: track 45.5 -> 46.6 mm
- net /STM32_CORE/PA4: track 17.1 -> 18.2 mm
- net /STM32_CORE/PB11: track 23.0 -> 22.0 mm
- net IONAIR-TTL-TX: track 64.8 -> 65.8 mm
- net /STM32_CORE/PA5: track 17.4 -> 18.2 mm
- net GND: track 513.5 -> 512.7 mm
Other:
- net class Default: via_dia 2 -> 2.5
- net class GND: via_dia 2 -> 2.5
- net class HIGH_PWR: via_dia 2 -> 2.5
- net class PWR: via_dia 2 -> 2.5

Commit message: update,
Parts:
- added J11: Conn_01x04, footprint-lib:Pin_Header_Straight_1x04_Pitch2.54mm, F.Cu at (53.3, 7.92)
- added J12: Conn_01x04, footprint-lib:Pin_Header_Straight_1x03_Pitch2.54mm, F.Cu at (18.7, 9.40)
- added REF**: MountingHole_3.2mm_M3_DIN965, MountingHole:MountingHole_3.2mm_M3_DIN965, F.Cu at (95.0, 5.00)
- added REF**: MountingHole_3.2mm_M3_DIN965, MountingHole:MountingHole_3.2mm_M3_DIN965, F.Cu at (5.00, 5.00)
- added REF**: MountingHole_3.2mm_M3_DIN965, MountingHole:MountingHole_3.2mm_M3_DIN965, F.Cu at (5.00, 65.0)
- added REF**: MountingHole_3.2mm_M3_DIN965, MountingHole:MountingHole_3.2mm_M3_DIN965, F.Cu at (95.0, 65.0)
- J6: footprint footprint-lib:PinHeader_1x14_P1.27mm_Vertical -> footprint-lib:Pin_Header_Straight_1x14_Pitch1.27mm
- J7: footprint footprint-lib:PinHeader_1x12_P1.27mm_Vertical -> footprint-lib:Pin_Header_Straight_1x12_Pitch1.27mm
- J8: footprint footprint-lib:PinHeader_1x15_P1.27mm_Vertical -> footprint-lib:Pin_Header_Straight_1x15_Pitch1.27mm
- U2: value OMRON G3MB-202P -> OMRON-G3MB-202P
- moved C9 10.3 mm to (8.51, 35.9)
- moved C7 10.3 mm to (14.5, 33.8)
- moved C8 10.3 mm to (9.40, 33.8)
- moved C17 10.3 mm to (13.8, 36.1)
- moved U4 8.78 mm to (10.4, 25.4)
- moved J2 7.87 mm to (76.2, 10.6)
- moved J4 5.90 mm to (88.9, 48.2)
- moved J3 5.90 mm to (88.9, 33.0)
- moved J1 5.84 mm to (88.9, 16.7)
- moved D3 5.62 mm to (9.63, 13.2)
- moved D2 4.43 mm to (10.5, 16.7)
- moved R13 3.56 mm to (13.9, 11.1)
- moved R11 2.93 mm to (15.7, 15.2)
- moved J5 2.24 mm to (85.0, 60.0), turned to 0 degrees
Connections:
- D2 pad 2: +3V3 -> +5V
- J6 pad 1: +3V3 -> Net-(J6-Pad1)
Routing:
- net GND: track 512.7 -> 586.3 mm
- net +5V: track 213.3 -> 283.0 mm
- net +3V3: track 219.0 -> 235.2 mm
- net /SSR_CH1_OUTPUT1: track 20.6 -> 36.8 mm
- net /STM32_CORE/SWIO: track 21.8 -> 35.2 mm
- net /STM32_CORE/SWCLK: track 14.2 -> 26.6 mm
- net /FAN_PWM_OUTPUT: track 21.6 -> 33.7 mm
- net /SSR-25-DA2: track 22.9 -> 30.0 mm
- net IONAIR-TTL-TX: track 65.8 -> 58.9 mm
- net /FAN_48V: track 27.3 -> 34.0 mm
- net /SSR-25-DA1: track 13.9 -> 19.9 mm
- net /WS2812_PWM_TERMINAL: track 11.4 -> 16.7 mm
- net VWS2812: track 13.0 -> 17.2 mm
- net Net-(D3-Pad1): track 4.05 -> 3.05 mm
- added copper zone on B.Cu, net GND

Commit message: update,
Parts:
- moved Q2 1.58 mm to (63.7, 34.4)
- moved J7 1.50 mm to (57.1, 35.6)
Routing:
- net +3V3: track 235.2 -> 249.4 mm, vias 6 -> 5
- net +5V: track 283.0 -> 292.0 mm
- net /FAN_PWM_OUTPUT: track 33.7 -> 39.2 mm
- net GND: track 586.3 -> 582.8 mm
- net STM32_FAN_PWM_OUTPUT: track 16.8 -> 19.5 mm
- net /STM32_CORE/PB14: track 10.7 -> 13.0 mm
- net /SSR_CH1_OUTPUT1: track 36.8 -> 34.8 mm
- net /STM32_CORE/PB12: track 11.3 -> 13.2 mm
- net Net-(Q2-Pad1): track 4.46 -> 2.82 mm
- net /STM32_CORE/PB15: track 10.4 -> 11.9 mm
- net VWS2812: track 17.2 -> 18.5 mm
- net /STM32_CORE/PA8: track 10.5 -> 11.7 mm
- net /STM32_CORE/PA9: track 10.8 -> 11.4 mm
- net /STM32_CORE/PA12: track 11.7 -> 12.3 mm
- net /STM32_CORE/PA11: track 11.4 -> 12.0 mm
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