File: pcb/stm32_bottom_board_respin.kicad_pcb (KiCad board)
At the start: 2 copper layers, 100 x 70 mm, 93 parts, among them J1 48V_SRC, J10 FCC_B2B, J11 SSR2_CTRL, J12 POWER, J13 PMS7003S_CONN, J14 MAINBOARD_CONN, J2 WS2812_CTRL, J3 FAN_CTRL, J4 SSR_OUTPUT, J5 PURFUME_CTRL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

Commit message: basic rout complete,
Parts:
- moved J4 49.5 mm to (86.6, 93.6), turned to 0 degrees
- moved Q4 46.6 mm to (76.7, 88.2), turned to 270 degrees
- moved R23 44.1 mm to (85.0, 89.6), turned to 180 degrees
- moved R22 39.1 mm to (85.5, 86.1), turned to 180 degrees
- moved D7 38.9 mm to (90.1, 86.1), turned to 0 degrees
- moved R21 36.4 mm to (80.5, 83.1), turned to 180 degrees
- moved R20 33.7 mm to (83.6, 82.0), turned to 90 degrees
- moved U2 13.0 mm to (101.1, 79.1)
- moved U6 13.0 mm to (101.1, 72.1)
- moved R17 12.2 mm to (94.1, 65.0)
- moved R25 12.2 mm to (114.7, 64.9)
- moved Q3 12.2 mm to (102.6, 63.6)
- moved R19 12.2 mm to (92.3, 64.4)
- moved Q2 12.0 mm to (98.9, 53.5)
- moved R8 11.3 mm to (105.1, 55.8), turned to 0 degrees
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Connections:
- J6 pad 1: Net-(J6-Pad1) -> +5V
- J6 pad 14: +5V -> Net-(J6-Pad14)
Routing:
- net +3V3: track 207.8 -> 312.8 mm, vias 5 -> 6
- net GND: track 407.4 -> 446.3 mm, vias 5 -> 12
- net /SSR-25-DA_N: track 15.4 -> 52.5 mm
- net STM32_SSR-25-DA_OUTPUT: track 75.0 -> 38.3 mm, vias 2 -> 1
- net /SSR-25-DA_P: track 7.32 -> 29.6 mm, vias 1 -> 0
- net Net-(Q1-Pad3): track 54.2 -> 40.6 mm, vias 0 -> 1
- net /SSR_CH1_OUTPUT1: track 19.3 -> 30.4 mm
- net STM32_PMS7003S_SET: track 66.6 -> 56.9 mm
- net +5V: track 333.7 -> 325.3 mm, vias 10 -> 11
- net STM32_SSR2_OUTPUT: track 39.4 -> 47.8 mm
- net /SSR_CH1_OUTPUT2: track 5.68 -> 13.9 mm
- net STM32_PMS7003S_RXD: track 69.8 -> 77.6 mm, vias 0 -> 2
- net STM32_FAN_RPM: track 66.6 -> 74.2 mm
- net /FAN_PWM_OUTPUT: track 41.5 -> 34.1 mm, vias 0 -> 1
- net Net-(R4-Pad2): track 10.6 -> 17.7 mm
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- added copper zone on B.Cu, net GND
- added copper zone on F.Cu, net GND

Commit message: basic rout complete,
Parts:
- moved D7 5.34 mm to (86.7, 90.2)
- moved R23 2.15 mm to (86.7, 88.3)
Connections:
- J4 pad 1: /SSR-25-DA_P -> /SSR-25-DA_N
- J4 pad 2: /SSR-25-DA_N -> /SSR-25-DA_P
Routing:
- net /SSR-25-DA_N: track 52.5 -> 39.7 mm
- net /SSR-25-DA_P: track 29.6 -> 39.7 mm
- net +5V: track 325.3 -> 333.2 mm, vias 11 -> 12
- net STM32_SSR2_OUTPUT: track 47.8 -> 41.2 mm
- net Net-(D7-Pad1): track 2.70 -> 6.34 mm
- net Net-(Q1-Pad3): track 40.6 -> 44.2 mm
- net Net-(Q3-Pad3): track 54.8 -> 52.1 mm
- net GND: vias 12 -> 27

Commit message: remove jumper,
Parts:
- moved JP5 2.73 mm to (50.0, 35.0), turned to 0 degrees
- turned JP3 to 0 degrees
Routing:
- net Net-(J10-Pad7): track 34.9 -> 32.4 mm
- net Net-(J10-Pad6): track 28.3 -> 30.2 mm
- net B2B_UART_RX: track 52.6 -> 51.7 mm

Commit message: remove jumper,
Parts:
- removed JP2: SCL_EN, Jumper:SolderJumper-2_P1.3mm_Open_TrianglePad1.0x1.5mm
- removed JP3: SDA_EN, Jumper:SolderJumper-2_P1.3mm_Open_TrianglePad1.0x1.5mm
- removed JP4: TX_EN, Jumper:SolderJumper-2_P1.3mm_Open_TrianglePad1.0x1.5mm
- removed JP5: RX_EN, Jumper:SolderJumper-2_P1.3mm_Open_TrianglePad1.0x1.5mm
- R5, R6: value R472,0603 -> R472,0603,NC
Connections:
- J10 pad 6: Net-(J10-Pad6) -> B2B_UART_TX
- J10 pad 7: Net-(J10-Pad7) -> B2B_UART_RX
Routing:
- net Net-(J10-Pad7): track 32.4 -> 0.00 mm
- net B2B_UART_RX: track 51.7 -> 82.8 mm
- net Net-(J10-Pad6): track 30.2 -> 0.00 mm
- net B2B_UART_TX: track 45.6 -> 69.6 mm

Commit message: update,
Routing:
- net B2B_UART_RX: track 82.8 -> 62.3 mm
- net B2B_UART_TX: track 69.6 -> 52.1 mm
- net +5V: track 333.2 -> 323.5 mm
- net +3V3: track 312.8 -> 311.3 mm
Other:
- net class GND: trace_width 1 -> 1.2; via_dia 1 -> 1.4
- net class HIGH_PWR: via_dia 1 -> 1.2
- net class PWR: trace_width 0.5 -> 0.75

Commit message: update,
Parts:
- added D9: LED_GREEN, LED_SMD:LED_0603_1608Metric_Pad1.05x0.95mm_HandSolder, F.Cu at (56.1, 49.3)
- added R27: R102,0603, Resistor_SMD:R_0603_1608Metric_Pad1.05x0.95mm_HandSolder, F.Cu at (57.6, 49.3)
- U2: footprint footprint-lib:OMRON-G3MB-202P -> footprint-lib.pretty:OMRON-G3MB-202P
- moved R13 20.4 mm to (58.3, 33.8), turned to 270 degrees
- moved D3 20.0 mm to (55.5, 33.8), turned to 270 degrees
- moved R6 17.5 mm to (67.4, 47.3)
- moved R5 16.2 mm to (70.2, 47.3)
- moved R11 10.5 mm to (51.9, 33.8), turned to 270 degrees
- moved D2 10.3 mm to (49.1, 33.8), turned to 270 degrees
- moved U7 6.91 mm to (83.0, 35.7), turned to 90 degrees
- moved R26 6.65 mm to (110.5, 64.6), turned to 90 degrees
- moved C10 6.27 mm to (39.0, 77.0)
- moved R12 6.01 mm to (43.0, 77.0)
- moved R2 5.10 mm to (66.8, 82.6)
- moved R9 3.22 mm to (65.0, 47.3), turned to 90 degrees
- moved R25 0.34 mm to (114.7, 64.6)
Connections:
- J7 pad 8: STM32_PMS7003S_SET -> STM32_PMS7003S_RESET
- J7 pad 9: STM32_PMS7003S_RESET -> STM32_PMS7003S_SET
- R25 pad 2: STM32_PMS7003S_RESET -> +3V3
- U3 pad 32: STM32_PMS7003S_SET -> STM32_PMS7003S_RESET
- U3 pad 33: STM32_PMS7003S_RESET -> STM32_PMS7003S_SET
Routing:
- net +5V: track 323.5 -> 442.3 mm, vias 12 -> 11
- net GND: track 446.3 -> 503.5 mm, vias 27 -> 26
- net +3V3: track 311.3 -> 365.4 mm, vias 6 -> 9
- net STM32_FAN_RPM: track 74.4 -> 22.5 mm, vias 1 -> 0
- net B2B_UART_RX: track 62.3 -> 23.7 mm, vias 1 -> 0
- net /STM32_CORE/RESET: track 49.0 -> 16.8 mm, vias 2 -> 0
- net B2B_UART_TX: track 52.1 -> 20.1 mm, vias 1 -> 0
- net STM32_PMS7003S_TXD: track 80.4 -> 95.7 mm, vias 1 -> 0
- net STM32_PMS7003S_RXD: track 77.6 -> 63.9 mm, vias 2 -> 1
- net /STM32_CORE/PC13: track 20.1 -> 30.2 mm
- net STM32_FAN_PWM_OUTPUT: track 21.5 -> 11.6 mm
- net STM32_PMS7003S_RESET: track 65.6 -> 57.4 mm, vias 1 -> 0
- net IONAIR-TTL-RX: track 42.5 -> 48.5 mm
- net Net-(Q3-Pad3): track 52.1 -> 57.5 mm
- net /STM32_CORE/BOOT0: track 7.74 -> 13.0 mm
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Other:
- rule trace_min: 0.3 -> 0.25

Commit message: update,
Parts:
- moved C10 23.8 mm to (60.9, 67.7), turned to 270 degrees
- moved R12 22.3 mm to (60.9, 63.7), turned to 270 degrees
- moved C12 17.6 mm to (52.7, 49.7), turned to 90 degrees
- moved SW1 15.8 mm to (56.7, 66.1), turned to 90 degrees
- moved Y1 11.0 mm to (50.5, 57.6)
- moved C11 4.00 mm to (51.1, 67.4), turned to 270 degrees
- moved C3 2.45 mm to (63.3, 61.4)
Routing:
- net +5V: track 442.3 -> 375.3 mm
- net STM32_PMS7003S_RXD: track 63.9 -> 97.3 mm, vias 1 -> 0
- net STM32_FAN_RPM: track 22.5 -> 50.6 mm, vias 0 -> 2
- net GND: track 503.5 -> 521.9 mm, vias 26 -> 32
- net +3V3: track 365.4 -> 353.1 mm
- net STM32_FAN_PWM_OUTPUT: track 11.6 -> 22.2 mm, vias 0 -> 1
- net /SSR_CH2_OUTPUT1: track 35.9 -> 41.4 mm
- net /STM32_CORE/OSCIN: track 21.4 -> 26.8 mm
- net STM32_SSR2_OUTPUT: track 41.9 -> 46.7 mm
- net /WS2812_PWM_TERMINAL: track 31.1 -> 35.7 mm
- net /FAN_PWM_OUTPUT: track 34.1 -> 30.1 mm, vias 1 -> 0
- net /STM32_CORE/RESET: track 16.8 -> 20.9 mm
- net STM32_PMS7003S_TXD: track 95.7 -> 99.2 mm
- net /STM32_CORE/OSCOUT: track 25.7 -> 22.4 mm
- net STM32_PMS7003S_SET: track 57.8 -> 55.8 mm
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
Commit message: update,
Connections:
- J14 pad 1: /SSR-25-DA_P -> GND
- J14 pad 2: /SSR-25-DA_N -> /SSR-25-DA_P
- J14 pad 3: /IONAIR_RX -> /SSR-25-DA_N
- J14 pad 4: /IONAIR_TX -> /IONAIR_RX
- J14 pad 5: GND -> /IONAIR_TX
- J14 pad 6: Net-(J14-Pad6) -> PCB1_ALARM_COM
- J14 pad 8: Net-(J14-Pad8) -> +5V
- J8 pad 9: /STM32_CORE/PA5 -> PCB1_ALARM_COM
- U3 pad 15: /STM32_CORE/PA5 -> PCB1_ALARM_COM
Routing:
- net PCB1_ALARM_COM: track 0.00 -> 16.0 mm
- net /STM32_CORE/PA5: track 16.0 -> 0.00 mm
