File: pcb/stm32_bottom_board_respin.sch (KiCad schematic (older format))
At the start: 8 parts, among them J1 Conn_01x02, J10 Conn_01x08, J2 WS2812, J3 FAN_PWM, J4 SSR, J5 PURFUME, J9 SSR

Commit message: update,
Connections:
- net SSR_CH1_OUTPUT1: now also J5.2 (Pin_2); no longer J5.1 (Pin_1)
- net SSR_CH1_OUTPUT2: now also J5.1 (Pin_1); no longer J5.2 (Pin_2)
Changed lines of the file:
@@
 	1    0    0    -1
 $EndComp
+Text Label 8650 6550 0    50   ~ 0
+SSR_CH1_OUTPUT1
+Wire Wire Line
+	8650 6550 9450 6550
 Text Label 8650 6450 0    50   ~ 0
-SSR_CH1_OUTPUT1
+SSR_CH1_OUTPUT2
 Wire Wire Line
 	8650 6450 9450 6450
-Text Label 8650 6550 0    50   ~ 0
-SSR_CH1_OUTPUT2
-Wire Wire Line
-	8650 6550 9450 6550
 $Sheet
 S 11650 4450 1500 950
@@
 IONAIR_RX
 $Comp
-L power:+5V #PWR?
+L power:+5V #PWR0101
 U 1 1 5BCE34B6
 P 5150 2650
-F 0 "#PWR?" H 5150 2500 50  0001 C CNN
+F 0 "#PWR0101" H 5150 2500 50  0001 C CNN
 F 1 "+5V" H 5200 2850 50  0000 C CNN
 F 2 "" H 5150 2650 50  0001 C CNN
@@
 $EndComp
 $Comp
-L power:+5V #PWR?
+L power:+5V #PWR0106
 U 1 1 5BCE34D8
 P 6400 1450
-F 0 "#PWR?" H 6400 1300 50  0001 C CNN
+F 0 "#PWR0106" H 6400 1300 50  0001 C CNN
 F 1 "+5V" H 6450 1650 50  0000 C CNN
 F 2 "" H 6400 1450 50  0001 C CNN

Commit message: update,
Other:
- moved on the sheet: C1, J2
Changed lines of the file:
@@
 $Descr A3 16535 11693
 encoding utf-8
-Sheet 1 7
+Sheet 1 8
 Title ""
 Date ""
@@
 L Connector_Generic:Conn_01x03 J2
 U 1 1 5BCB416C
-P 8700 8400
-F 0 "J2" H 8780 8442 50  0000 L CNN
-F 1 "WS2812" H 8780 8351 50  0000 L CNN
-F 2 "w_conn_mkds:mkds_1,5-3" H 8700 8400 50  0001 C CNN
-F 3 "~" H 8700 8400 50  0001 C CNN
-	1    8700 8400
+P 8700 7700
+F 0 "J2" H 8780 7742 50  0000 L CNN
+F 1 "WS2812" H 8780 7651 50  0000 L CNN
+F 2 "w_conn_mkds:mkds_1,5-3" H 8700 7700 50  0001 C CNN
+F 3 "~" H 8700 7700 50  0001 C CNN
+	1    8700 7700
 	1    0    0    -1
 $EndComp
@@
 L taobao-components:VWS2812 #PWR05
 U 1 1 5BCB42EE
-P 8300 8150
-F 0 "#PWR05" H 8300 8000 50  0001 C CNN
-F 1 "VWS2812" H 8317 8323 50  0000 C CNN
-F 2 "" H 8300 8150 50  0001 C CNN
-F 3 "" H 8300 8150 50  0001 C CNN
-	1    8300 8150
-	1    0    0    -1
-$EndComp
-Wire Wire Line
-	8300 8150 8300 8300
-Wire Wire Line
-	8300 8300 8500 8300
+P 8300 7450
+F 0 "#PWR05" H 8300 7300 50  0001 C CNN
+F 1 "VWS2812" H 8317 7623 50  0000 C CNN
+F 2 "" H 8300 7450 50  0001 C CNN
+F 3 "" H 8300 7450 50  0001 C CNN
+	1    8300 7450
+	1    0    0    -1
+$EndComp
+Wire Wire Line
+	8300 7450 8300 7600
+Wire Wire Line
+	8300 7600 8500 7600
 $Comp
 L power:GND #PWR04
 U 1 1 5BCB4355
-P 7850 8450
-F 0 "#PWR04" H 7850 8200 50  0001 C CNN
-F 1 "GND" H 7855 8277 50  0000 C CNN
-F 2 "" H 7850 8450 50  0001 C CNN
-F 3 "" H 7850 8450 50  0001 C CNN
-	1    7850 8450
-	1    0    0    -1
-$EndComp
-Wire Wire Line
-	8300 8700 8300 8500
-Wire Wire Line
-	8300 8500 8500 8500
-Text Label 7000 8700 0    50   ~ 0
+P 7850 7750
+F 0 "#PWR04" H 7850 7500 50  0001 C CNN
+F 1 "GND" H 7855 7577 50  0000 C CNN
+F 2 "" H 7850 7750 50  0001 C CNN
+F 3 "" H 7850 7750 50  0001 C CNN
+	1    7850 7750
+	1    0    0    -1
+$EndComp
+Wire Wire Line
+	8300 8000 8300 7800
+Wire Wire Line
+	8300 7800 8500 7800
+Text Label 7000 8000 0    50   ~ 0
 WS2812_PWM_TERMINAL
-Text Label 14250 8550 2    50   ~ 0
+Text Label 14250 7850 2    50   ~ 0
 WS2812_PWM_TERMINAL
 Wire Wire Line
-	14250 8550 13150 8550
+	14250 7850 13150 7850
 $Sheet
 S 11650 5950 1500 900
@@
 $EndComp
 Wire Wire Line
-	8500 8400 7850 8400
-Wire Wire Line
-	7850 8400 7850 8450
-Wire Wire Line
-	7000 8700 8300 8700
-Text Notes 6150 8050 0    50   ~ 0
+	8500 7700 7850 7700
+Wire Wire Line
+	7850 7700 7850 7750
+Wire Wire Line
+	7000 8000 8300 8000
+Text Notes 6150 7350 0    50   ~ 0
 connect the main power supply to VWS2812
 $Comp
 L taobao-components:VWS2812 #PWR06
 U 1 1 5BCB629E
-P 9650 8150
-F 0 "#PWR06" H 9650 8000 50  0001 C CNN
-F 1 "VWS2812" H 9667 8323 50  0000 C CNN
-F 2 "" H 9650 8150 50  0001 C CNN
-F 3 "" H 9650 8150 50  0001 C CNN
-	1    9650 8150
+P 9650 7450
+F 0 "#PWR06" H 9650 7300 50  0001 C CNN
+F 1 "VWS2812" H 9667 7623 50  0000 C CNN
+F 2 "" H 9650 7450 50  0001 C CNN
+F 3 "" H 9650 7450 50  0001 C CNN
+	1    9650 7450
 	1    0    0    -1
 $EndComp
@@
 L power:GND #PWR07
 U 1 1 5BCB62B1
-P 9650 8600
-F 0 "#PWR07" H 9650 8350 50  0001 C CNN
-F 1 "GND" H 9655 8427 50  0000 C CNN
-F 2 "" H 9650 8600 50  0001 C CNN
-F 3 "" H 9650 8600 50  0001 C CNN
-	1    9650 8600
-	1    0    0    -1
-$EndComp
-Wire Wire Line
-	9650 8150 9650 8250
-Wire Wire Line
-	9650 8450 9650 8600
+P 9650 7900
+F 0 "#PWR07" H 9650 7650 50  0001 C CNN
+F 1 "GND" H 9655 7727 50  0000 C CNN
+F 2 "" H 9650 7900 50  0001 C CNN
+F 3 "" H 9650 7900 50  0001 C CNN
+	1    9650 7900
+	1    0    0    -1
+$EndComp
+Wire Wire Line
+	9650 7450 9650 7550
+Wire Wire Line
+	9650 7750 9650 7900
 $Comp
 L taobao-cp:CP1000uf,10V C1
 U 1 1 5BCB6CCE
-P 9650 8350
-F 0 "C1" H 9738 8396 50  0000 L CNN
-F 1 "CP1000uf,10V" H 9738 8305 50  0000 L CNN
-F 2 "Capacitor_SMD:CP_Elec_10x10.5" H 9650 8350 50  0001 C CNN
-F 3 "~" H 9650 8350 50  0001 C CNN
-	1    9650 8350
+P 9650 7650
+F 0 "C1" H 9738 7696 50  0000 L CNN
+F 1 "CP1000uf,10V" H 9738 7605 50  0000 L CNN
+F 2 "Capacitor_SMD:CP_Elec_10x10.5" H 9650 7650 50  0001 C CNN
+F 3 "~" H 9650 7650 50  0001 C CNN
+	1    9650 7650
 	1    0    0    -1
 $EndComp
@@
 	7550 3800 6800 3800
 $Sheet
-S 11650 7900 1500 850
+S 11650 7200 1500 850
 U 5BCB4060
 F0 "WS2812_PWM_DRIVER" 50
 F1 "WS2812_PWM_DRIVER.sch" 50
-F2 "STM32_WS2812_PWM" I L 11650 8250 50
-F3 "WS2812_PWM_OUTPUT" I R 13150 8550 50
+F2 "STM32_WS2812_PWM" I L 11650 7550 50
+F3 "WS2812_PWM_OUTPUT" I R 13150 7850 50
 $EndSheet
 $Sheet
@@
 Text GLabel 11450 6200 0    50   Input ~ 0
 STM32_SSR_OUTPUT
-Text GLabel 11450 8250 0    50   Input ~ 0
+Text GLabel 11450 7550 0    50   Input ~ 0
 STM32_WS2812_OUTPUT
 Wire Wire Line
@@
 	11450 6200 11650 6200
 Wire Wire Line
-	11450 8250 11650 8250
+	11450 7550 11650 7550
 $Comp
 L power:GND #PWR0107
@@
 	1    0    0    -1
 $EndComp
+$Sheet
+S 11650 8450 1500 950
+U 5BDCE0AC
+F0 "PMS5003S_interface" 50
+F1 "PMS5003S_interface.sch" 50
+F2 "PMS5003S_RX" I L 11650 8750 50
+F3 "PMS5003S_TX" I L 11650 8950 50
+$EndSheet
+Text GLabel 11450 8750 0    50   Input ~ 0
+STM32_PMS5003S_RX
+Wire Wire Line
+	11450 8750 11650 8750
+Text GLabel 11450 8950 0    50   Input ~ 0
+STM32_PMS5003S_TX
+Wire Wire Line
+	11450 8950 11650 8950
 $EndSCHEMATC

Commit message: update,
Parts:
- J10: value Conn_01x08 -> FCC_01_10; symbol Connector_Generic:Conn_01x08 -> Connector_Generic:Conn_01x10
Connections:
- net labels added: B2B_UART_RX, B2B_UART_TX, STM32_PMS7003S_RESET, STM32_PMS7003S_RXD, STM32_PMS7003S_SET, STM32_PMS7003S_TXD
- net labels removed: STM32_PMS5003S_RX, STM32_PMS5003S_TX
- wire segments 54 -> 58
Changed lines of the file:
@@
 Wire Wire Line
 	8650 2550 9400 2550
-$Comp
-L Connector_Generic:Conn_01x08 J10
-U 1 1 5BD05062
-P 5750 3000
-F 0 "J10" H 5830 2992 50  0000 L CNN
-F 1 "Conn_01x08" H 5830 2901 50  0000 L CNN
-F 2 "Connector_FFC-FPC:TE_84952-8_1x08-1MP_P1.0mm_Horizontal" H 5750 3000 50  0001 C CNN
-F 3 "~" H 5750 3000 50  0001 C CNN
-	1    5750 3000
-	1    0    0    -1
-$EndComp
 Wire Wire Line
 	4800 3300 5550 3300
@@
 F0 "PMS5003S_interface" 50
 F1 "PMS5003S_interface.sch" 50
-F2 "PMS5003S_RX" I L 11650 8750 50
-F3 "PMS5003S_TX" I L 11650 8950 50
+F2 "PMS7003S_RESET_5" I L 11650 9100 50
+F3 "PMS7003S_RXD_7" I L 11650 8750 50
+F4 "PMS7003S_TXD_9" I L 11650 8950 50
+F5 "PMS7003S_SET_10" I L 11650 9250 50
 $EndSheet
-Text GLabel 11450 8750 0    50   Input ~ 0
-STM32_PMS5003S_RX
+Text GLabel 11450 8950 0    50   Input ~ 0
+STM32_PMS7003S_RXD
 Wire Wire Line
 	11450 8750 11650 8750
-Text GLabel 11450 8950 0    50   Input ~ 0
-STM32_PMS5003S_TX
+Text GLabel 11450 8750 0    50   Input ~ 0
+STM32_PMS7003S_TXD
 Wire Wire Line
 	11450 8950 11650 8950
+Text GLabel 11450 9100 0    50   Input ~ 0
+STM32_PMS7003S_RESET
+Wire Wire Line
+	11450 9100 11650 9100
+Text GLabel 11450 9250 0    50   Input ~ 0
+STM32_PMS7003S_SET
+Wire Wire Line
+	11450 9250 11650 9250
+$Comp
+L Connector_Generic:Conn_01x10 J10
+U 1 1 5BD05062
+P 5750 3100
+F 0 "J10" H 5830 3092 50  0000 L CNN
+F 1 "FCC_01_10" H 5830 3001 50  0000 L CNN
+F 2 "Connector_FFC-FPC:TE_84952-8_1x08-1MP_P1.0mm_Horizontal" H 5750 3100 50  0001 C CNN
+F 3 "~" H 5750 3100 50  0001 C CNN
+	1    5750 3100
+	1    0    0    -1
+$EndComp
+Text GLabel 4800 3400 0    50   Input ~ 0
+B2B_UART_TX
+Text GLabel 4800 3500 0    50   Input ~ 0
+B2B_UART_RX
+Wire Wire Line
+	4800 3400 5550 3400
+Wire Wire Line
+	4800 3500 5550 3500
 $EndSCHEMATC

Commit message: update,
Parts:
- J10: value FCC_01_10 -> FCC_B2B
Changed lines of the file:
@@
 P 5750 3100
 F 0 "J10" H 5830 3092 50  0000 L CNN
-F 1 "FCC_01_10" H 5830 3001 50  0000 L CNN
+F 1 "FCC_B2B" H 5830 3001 50  0000 L CNN
 F 2 "Connector_FFC-FPC:TE_84952-8_1x08-1MP_P1.0mm_Horizontal" H 5750 3100 50  0001 C CNN
 F 3 "~" H 5750 3100 50  0001 C CNN

Commit message: update,
Parts:
- added R? (x2): R472,0603, symbol taobao-r:R472,0603
Connections:
- net labels added: 3V3
- wire segments 58 -> 66
Changed lines of the file:
@@
 	8650 2550 9400 2550
 Wire Wire Line
-	4800 3300 5550 3300
-Wire Wire Line
-	4800 3200 5550 3200
+	3500 3300 3950 3300
+Wire Wire Line
+	3500 3200 3750 3200
 Wire Wire Line
 	4800 3100 5550 3100
@@
 Wire Wire Line
 	5150 2700 5550 2700
-Text GLabel 4800 3300 0    50   Input ~ 0
+Text GLabel 3500 3300 0    50   Input ~ 0
 I2C_SDA
-Text GLabel 4800 3200 0    50   Input ~ 0
+Text GLabel 3500 3200 0    50   Input ~ 0
 I2C_SCL
 Text GLabel 4800 3100 0    50   Input ~ 0
@@
 Wire Wire Line
 	4800 3500 5550 3500
+$Comp
+L tinkerforge:3V3 #PWR?
+U 1 1 5BDD6C93
+P 3750 2650
+F 0 "#PWR?" H 3750 2500 50  0001 C CNN
+F 1 "3V3" H 3765 2823 50  0000 C CNN
+F 2 "" H 3750 2650 50  0000 C CNN
+F 3 "" H 3750 2650 50  0000 C CNN
+	1    3750 2650
+	1    0    0    -1
+$EndComp
+$Comp
+L taobao-r:R472,0603 R?
+U 1 1 5BDDACA3
+P 3750 2850
+F 0 "R?" H 3809 2896 50  0000 L CNN
+F 1 "R472,0603" H 3809 2805 50  0000 L CNN
+F 2 "" H 3750 2850 50  0001 C CNN
+F 3 "~" H 3750 2850 50  0001 C CNN
+	1    3750 2850
+	1    0    0    -1
+$EndComp
+$Comp
+L taobao-r:R472,0603 R?
+U 1 1 5BDDACCF
+P 3950 2850
+F 0 "R?" H 4009 2896 50  0000 L CNN
+F 1 "R472,0603" H 4009 2805 50  0000 L CNN
+F 2 "" H 3950 2850 50  0001 C CNN
+F 3 "~" H 3950 2850 50  0001 C CNN
+	1    3950 2850
+	1    0    0    -1
+$EndComp
+Wire Wire Line
+	3750 2650 3750 2700
+Wire Wire Line
+	3750 2700 3950 2700
+Wire Wire Line
+	3950 2700 3950 2750
+Connection ~ 3750 2700
+Wire Wire Line
+	3750 2700 3750 2750
+Wire Wire Line
+	3750 2950 3750 3200
+Connection ~ 3750 3200
+Wire Wire Line
+	3750 3200 5550 3200
+Wire Wire Line
+	3950 2950 3950 3300
+Connection ~ 3950 3300
+Wire Wire Line
+	3950 3300 5550 3300
 $EndSCHEMATC

Commit message: update adding SSR2 on pcb and ioc,
Parts:
- added JP? (x4): Jumper_NO_Small, symbol Device:Jumper_NO_Small
- J10: symbol Connector_Generic:Conn_01x10 -> Connector_Generic:Conn_01x08
Connections:
- net labels added: SSR_CH2_OUTPUT1, SSR_CH2_OUTPUT2, STM32_SSR1_OUTPUT, STM32_SSR2_OUTPUT
- net labels removed: STM32_SSR_OUTPUT
- wire segments 66 -> 77
Changed lines of the file:
@@
 F0 "SSR_DRIVER" 50
 F1 "SSR_DRIVER.sch" 50
-F2 "STM32_SSR_OUTPUT" I L 11650 6200 50
-F3 "SSR_CH1_OUTPUT1" I R 13150 6450 50
-F4 "SSR_CH1_OUTPUT2" I R 13150 6600 50
-$EndSheet
+F2 "STM32_SSR1_OUTPUT" I L 11650 6200 50
+F3 "SSR_CH1_OUTPUT1" I R 13150 6350 50
+F4 "SSR_CH1_OUTPUT2" I R 13150 6450 50
+F5 "STM32_SSR2_OUTPUT" I L 11650 6550 50
+F6 "SSR_CH2_OUTPUT1" I R 13150 6650 50
+F7 "SSR_CH2_OUTPUT2" I R 13150 6750 50
+$EndSheet
+Text Label 14500 6350 2    50   ~ 0
+SSR_CH1_OUTPUT1
 Text Label 14500 6450 2    50   ~ 0
-SSR_CH1_OUTPUT1
-Text Label 14500 6600 2    50   ~ 0
 SSR_CH1_OUTPUT2
 Wire Wire Line
-	13150 6600 14500 6600
-Wire Wire Line
 	13150 6450 14500 6450
+Wire Wire Line
+	13150 6350 14500 6350
 $Comp
 L Connector_Generic:Conn_01x02 J5
@@
 STM32_SSR-25-DA_OUTPUT
 Text GLabel 11450 6200 0    50   Input ~ 0
-STM32_SSR_OUTPUT
+STM32_SSR1_OUTPUT
 Text GLabel 11450 7550 0    50   Input ~ 0
 STM32_WS2812_OUTPUT
@@
 Wire Wire Line
 	11450 9250 11650 9250
-$Comp
-L Connector_Generic:Conn_01x10 J10
-U 1 1 5BD05062
-P 5750 3100
-F 0 "J10" H 5830 3092 50  0000 L CNN
-F 1 "FCC_B2B" H 5830 3001 50  0000 L CNN
-F 2 "Connector_FFC-FPC:TE_84952-8_1x08-1MP_P1.0mm_Horizontal" H 5750 3100 50  0001 C CNN
-F 3 "~" H 5750 3100 50  0001 C CNN
-	1    5750 3100
-	1    0    0    -1
-$EndComp
-Text GLabel 4800 3400 0    50   Input ~ 0
+Text GLabel 3700 3600 0    50   Input ~ 0
 B2B_UART_TX
-Text GLabel 4800 3500 0    50   Input ~ 0
+Text GLabel 3700 3700 0    50   Input ~ 0
 B2B_UART_RX
-Wire Wire Line
-	4800 3400 5550 3400
-Wire Wire Line
-	4800 3500 5550 3500
 $Comp
 L tinkerforge:3V3 #PWR?
@@
 Wire Wire Line
 	3750 2950 3750 3200
+Wire Wire Line
+	3950 2950 3950 3300
+$Comp
+L Connector_Generic:Conn_01x08 J10
+U 1 1 5BD05062
+P 5750 3000
+F 0 "J10" H 5830 2992 50  0000 L CNN
+F 1 "FCC_B2B" H 5830 2901 50  0000 L CNN
+F 2 "Connector_FFC-FPC:TE_84952-8_1x08-1MP_P1.0mm_Horizontal" H 5750 3000 50  0001 C CNN
+F 3 "~" H 5750 3000 50  0001 C CNN
+	1    5750 3000
+	1    0    0    -1
+$EndComp
+Wire Wire Line
+	3700 3600 4250 3600
+Wire Wire Line
+	3700 3700 4250 3700
+Wire Wire Line
+	4450 3700 5050 3700
+Wire Wire Line
+	5050 3700 5050 3300
+Wire Wire Line
+	5050 3300 5550 3300
+Wire Wire Line
+	5550 3200 4950 3200
+Wire Wire Line
+	4950 3200 4950 3600
+Wire Wire Line
+	4950 3600 4450 3600
+$Comp
+L Device:Jumper_NO_Small JP?
+U 1 1 5BDDECBA
+P 4350 3200
+F 0 "JP?" H 4350 3385 50  0000 C CNN
+F 1 "Jumper_NO_Small" H 4350 3294 50  0000 C CNN
+F 2 "" H 4350 3200 50  0001 C CNN
+F 3 "~" H 4350 3200 50  0001 C CNN
+	1    4350 3200
+	1    0    0    -1
+$EndComp
+$Comp
+L Device:Jumper_NO_Small JP?
+U 1 1 5BDDED1D
+P 4350 3300
+F 0 "JP?" H 4350 3485 50  0000 C CNN
+F 1 "Jumper_NO_Small" H 4350 3394 50  0000 C CNN
+F 2 "" H 4350 3300 50  0001 C CNN
+F 3 "~" H 4350 3300 50  0001 C CNN
+	1    4350 3300
+	1    0    0    -1
+$EndComp
+Wire Wire Line
+	4450 3300 5050 3300
+Connection ~ 5050 3300
+Wire Wire Line
+	4450 3200 4950 3200
+Connection ~ 4950 3200
+Wire Wire Line
+	3750 3200 4250 3200
 Connection ~ 3750 3200
 Wire Wire Line
-	3750 3200 5550 3200
-Wire Wire Line
-	3950 2950 3950 3300
+	3950 3300 4250 3300
 Connection ~ 3950 3300
-Wire Wire Line
-	3950 3300 5550 3300
+$Comp
+L Device:Jumper_NO_Small JP?
+U 1 1 5BE40594
+P 4350 3700
+F 0 "JP?" H 4350 3885 50  0000 C CNN
+F 1 "Jumper_NO_Small" H 4350 3794 50  0000 C CNN
+F 2 "" H 4350 3700 50  0001 C CNN
+F 3 "~" H 4350 3700 50  0001 C CNN
+	1    4350 3700
+	1    0    0    -1
+$EndComp
+$Comp
+L Device:Jumper_NO_Small JP?
+U 1 1 5BE405D0
+P 4350 3600
+F 0 "JP?" H 4350 3785 50  0000 C CNN
+F 1 "Jumper_NO_Small" H 4350 3694 50  0000 C CNN
+F 2 "" H 4350 3600 50  0001 C CNN
+F 3 "~" H 4350 3600 50  0001 C CNN
+	1    4350 3600
+	1    0    0    -1
+$EndComp
+Text Label 14500 6650 2    50   ~ 0
+SSR_CH2_OUTPUT1
+Text Label 14500 6750 2    50   ~ 0
+SSR_CH2_OUTPUT2
+Wire Wire Line
+	13150 6750 14500 6750
+Wire Wire Line
+	13150 6650 14500 6650
+Text GLabel 11450 6550 0    50   Input ~ 0
+STM32_SSR2_OUTPUT
+Wire Wire Line
+	11450 6550 11650 6550
 $EndSCHEMATC

Commit message: updat,
Parts:
- added J?: SSR_CH2_OUTPUT, w_conn_mkds:mkds_1,5-2, symbol Connector_Generic:Conn_01x02
Connections:
- wire segments 77 -> 79
Other:
- moved on the sheet: J5
Changed lines of the file:
@@
 L Connector_Generic:Conn_01x02 J5
 U 1 1 5BCB6490
-P 9650 6450
-F 0 "J5" H 9730 6442 50  0000 L CNN
-F 1 "PURFUME" H 9730 6351 50  0000 L CNN
-F 2 "w_conn_mkds:mkds_1,5-2" H 9650 6450 50  0001 C CNN
-F 3 "~" H 9650 6450 50  0001 C CNN
-	1    9650 6450
-	1    0    0    -1
-$EndComp
-Text Label 8650 6550 0    50   ~ 0
+P 9650 6100
+F 0 "J5" H 9730 6092 50  0000 L CNN
+F 1 "PURFUME" H 9730 6001 50  0000 L CNN
+F 2 "w_conn_mkds:mkds_1,5-2" H 9650 6100 50  0001 C CNN
+F 3 "~" H 9650 6100 50  0001 C CNN
+	1    9650 6100
+	1    0    0    -1
+$EndComp
+Text Label 8650 6200 0    50   ~ 0
 SSR_CH1_OUTPUT1
 Wire Wire Line
-	8650 6550 9450 6550
-Text Label 8650 6450 0    50   ~ 0
+	8650 6200 9450 6200
+Text Label 8650 6100 0    50   ~ 0
 SSR_CH1_OUTPUT2
 Wire Wire Line
-	8650 6450 9450 6450
+	8650 6100 9450 6100
 $Sheet
 S 11650 4450 1500 950
@@
 Wire Wire Line
 	11450 6550 11650 6550
+$Comp
+L Connector_Generic:Conn_01x02 J?
+U 1 1 5BE5623C
+P 9650 6450
+F 0 "J?" H 9730 6442 50  0000 L CNN
+F 1 "SSR_CH2_OUTPUT" H 9730 6351 50  0000 L CNN
+F 2 "w_conn_mkds:mkds_1,5-2" H 9650 6450 50  0001 C CNN
+F 3 "~" H 9650 6450 50  0001 C CNN
+	1    9650 6450
+	1    0    0    -1
+$EndComp
+Text Label 8650 6550 0    50   ~ 0
+SSR_CH2_OUTPUT1
+Wire Wire Line
+	8650 6550 9450 6550
+Text Label 8650 6450 0    50   ~ 0
+SSR_CH2_OUTPUT2
+Wire Wire Line
+	8650 6450 9450 6450
 $EndSCHEMATC

Commit message: update,
Connections:
- net labels added: STM32_FAN_RPM
- wire segments 79 -> 81
Changed lines of the file:
@@
 F3 "FAN_PWM_OUTPUT" I R 13150 3750 50
 F4 "FAN_PWM_GND" I R 13150 3850 50
+F5 "STM32_FAN_RPM" I L 11650 3700 50
+F6 "FAN_RPM" I R 13150 3950 50
 $EndSheet
 Text Label 14200 3750 2    50   ~ 0
@@
 Wire Wire Line
 	8650 6450 9450 6450
+Text Label 14200 3950 2    50   ~ 0
+FAN_RPM
+Wire Wire Line
+	13150 3950 14200 3950
+Text GLabel 11450 3700 0    50   Input ~ 0
+STM32_FAN_RPM
+Wire Wire Line
+	11450 3700 11650 3700
 $EndSCHEMATC
