File: pcb/stm32_bottom_board_respin.sch (KiCad schematic (older format))
At the start: 15 parts, among them J1 Conn_01x02, J10 FCC_B2B, J2 WS2812, J3 FAN_PWM, J4 SSR, J5 PURFUME, J9 SSR

Commit message: update,
Parts:
- J1: value Conn_01x02 -> 48V source
Connections:
- net labels removed: FAN_PWM_GND
- wire segments 81 -> 80
Changed lines of the file:
@@
 F2 "STM32_FAN_PWM" I L 11650 3600 50
 F3 "FAN_PWM_OUTPUT" I R 13150 3750 50
-F4 "FAN_PWM_GND" I R 13150 3850 50
-F5 "STM32_FAN_RPM" I L 11650 3700 50
-F6 "FAN_RPM" I R 13150 3950 50
+F4 "STM32_FAN_RPM" I L 11650 3700 50
+F5 "FAN_RPM" I R 13150 3950 50
 $EndSheet
 Text Label 14200 3750 2    50   ~ 0
 FAN_PWM_OUTPUT
-Text Label 14200 3850 2    50   ~ 0
-FAN_PWM_GND
-Wire Wire Line
-	13150 3850 14200 3850
 Wire Wire Line
 	13150 3750 14200 3750
-Text Label 8550 3800 0    50   ~ 0
-FAN_PWM_OUTPUT
-Text Label 8550 3900 0    50   ~ 0
-FAN_PWM_GND
-Wire Wire Line
-	9350 3900 8550 3900
-Wire Wire Line
-	9350 3800 8550 3800
 $Comp
 L Connector_Generic:Conn_01x04 J3
@@
 Text Notes 6000 1850 0    50   ~ 0
 the power of driver circuit is by VDD instead of +5V\nto provision the power control of the driver circuit
-Text Label 8550 3700 0    50   ~ 0
+Text Label 8550 3800 0    50   ~ 0
 FAN_48V
-Text Label 8550 4000 0    50   ~ 0
+Text Label 8550 3900 0    50   ~ 0
 FAN_RPM
 Wire Wire Line
-	8550 4000 9350 4000
-Wire Wire Line
-	8550 3700 9350 3700
+	8550 3900 9350 3900
+Wire Wire Line
+	8550 3800 9350 3800
 $Comp
 L Connector_Generic:Conn_01x02 J1
@@
 P 7800 3700
 F 0 "J1" H 7880 3692 50  0000 L CNN
-F 1 "Conn_01x02" H 7880 3601 50  0000 L CNN
+F 1 "48V source" H 7880 3601 50  0000 L CNN
 F 2 "w_conn_mkds:mkds_1,5-2" H 7800 3700 50  0001 C CNN
 F 3 "~" H 7800 3700 50  0001 C CNN
@@
 Wire Wire Line
 	11450 3700 11650 3700
+Text Label 8550 3700 0    50   ~ 0
+FAN_48V_GND
+Wire Wire Line
+	8550 3700 9350 3700
+Wire Wire Line
+	9350 4000 8550 4000
+Text Label 8550 4000 0    50   ~ 0
+FAN_PWM_OUTPUT
 $EndSCHEMATC

Commit message: update,
Parts:
- J1: value 48V source -> 48V_SRC
- J2: value WS2812 -> WS2812_CTRL
- J3: value FAN_PWM -> FAN_CTRL
- J4: value SSR -> SSR_OUTPUT
- J5: value PURFUME -> PURFUME_CTRL
- J9: value SSR -> MAIN_CTRL
- J?: value SSR_CH2_OUTPUT -> SSR2_CTRL
Other:
- note added: "follows PC fan ordering"
Changed lines of the file:
@@
 P 8700 7700
 F 0 "J2" H 8780 7742 50  0000 L CNN
-F 1 "WS2812" H 8780 7651 50  0000 L CNN
+F 1 "WS2812_CTRL" H 8780 7651 50  0000 L CNN
 F 2 "w_conn_mkds:mkds_1,5-3" H 8700 7700 50  0001 C CNN
 F 3 "~" H 8700 7700 50  0001 C CNN
@@
 P 9650 6100
 F 0 "J5" H 9730 6092 50  0000 L CNN
-F 1 "PURFUME" H 9730 6001 50  0000 L CNN
+F 1 "PURFUME_CTRL" H 9730 6001 50  0000 L CNN
 F 2 "w_conn_mkds:mkds_1,5-2" H 9650 6100 50  0001 C CNN
 F 3 "~" H 9650 6100 50  0001 C CNN
@@
 P 9600 4950
 F 0 "J4" H 9680 4942 50  0000 L CNN
-F 1 "SSR" H 9680 4851 50  0000 L CNN
+F 1 "SSR_OUTPUT" H 9680 4851 50  0000 L CNN
 F 2 "w_conn_mkds:mkds_1,5-2" H 9600 4950 50  0001 C CNN
 F 3 "~" H 9600 4950 50  0001 C CNN
@@
 P 9550 3800
 F 0 "J3" H 9630 3792 50  0000 L CNN
-F 1 "FAN_PWM" H 9630 3701 50  0000 L CNN
+F 1 "FAN_CTRL" H 9630 3701 50  0000 L CNN
 F 2 "w_conn_mkds:mkds_1,5-4" H 9550 3800 50  0001 C CNN
 F 3 "~" H 9550 3800 50  0001 C CNN
@@
 P 7800 3700
 F 0 "J1" H 7880 3692 50  0000 L CNN
-F 1 "48V source" H 7880 3601 50  0000 L CNN
+F 1 "48V_SRC" H 7880 3601 50  0000 L CNN
 F 2 "w_conn_mkds:mkds_1,5-2" H 7800 3700 50  0001 C CNN
 F 3 "~" H 7800 3700 50  0001 C CNN
@@
 	1    0    0    -1
 $EndComp
-Text Label 6800 3800 0    50   ~ 0
+Text Label 6850 3700 0    50   ~ 0
 FAN_48V_GND
 Wire Wire Line
 	7600 3800 7550 3800
-Text Label 6800 3700 0    50   ~ 0
+Text Label 6750 3800 0    50   ~ 0
 FAN_48V
 Wire Wire Line
-	6800 3700 7600 3700
+	6750 3800 7550 3800
 $Comp
 L power:GND #PWR03
@@
 Wire Wire Line
 	7550 3800 7550 3900
-Connection ~ 7550 3800
-Wire Wire Line
-	7550 3800 6800 3800
+Wire Wire Line
+	7600 3700 6850 3700
 $Sheet
 S 11650 7200 1500 850
@@
 P 9600 2650
 F 0 "J9" H 9680 2642 50  0000 L CNN
-F 1 "SSR" H 9680 2551 50  0000 L CNN
+F 1 "MAIN_CTRL" H 9680 2551 50  0000 L CNN
 F 2 "w_conn_mkds:mkds_1,5-3" H 9600 2650 50  0001 C CNN
 F 3 "~" H 9600 2650 50  0001 C CNN
@@
 P 9650 6450
 F 0 "J?" H 9730 6442 50  0000 L CNN
-F 1 "SSR_CH2_OUTPUT" H 9730 6351 50  0000 L CNN
+F 1 "SSR2_CTRL" H 9730 6351 50  0000 L CNN
 F 2 "w_conn_mkds:mkds_1,5-2" H 9650 6450 50  0001 C CNN
 F 3 "~" H 9650 6450 50  0001 C CNN
@@
 Text Label 8550 4000 0    50   ~ 0
 FAN_PWM_OUTPUT
+Connection ~ 7550 3800
+Text Notes 8650 4250 0    50   ~ 0
+follows PC fan ordering
 $EndSCHEMATC

Commit message: update,
Parts:
- J9: value MAIN_CTRL -> PCB_UART
Connections:
- wire segments 80 -> 82
Changed lines of the file:
@@
 P 9600 2650
 F 0 "J9" H 9680 2642 50  0000 L CNN
-F 1 "MAIN_CTRL" H 9680 2551 50  0000 L CNN
+F 1 "PCB_UART" H 9680 2551 50  0000 L CNN
 F 2 "w_conn_mkds:mkds_1,5-3" H 9600 2650 50  0001 C CNN
 F 3 "~" H 9600 2650 50  0001 C CNN
@@
 Text Notes 8650 4250 0    50   ~ 0
 follows PC fan ordering
+$Comp
+L power:GND #PWR?
+U 1 1 5BE0459B
+P 5400 3600
+F 0 "#PWR?" H 5400 3350 50  0001 C CNN
+F 1 "GND" H 5405 3427 50  0000 C CNN
+F 2 "" H 5400 3600 50  0001 C CNN
+F 3 "" H 5400 3600 50  0001 C CNN
+	1    5400 3600
+	1    0    0    -1
+$EndComp
+Wire Wire Line
+	5400 3600 5400 3400
+Wire Wire Line
+	5400 3400 5550 3400
 $EndSCHEMATC

Commit message: update,
Connections:
- net labels added: +3V3, SSR-25-DA_N, SSR-25-DA_P
- net labels removed: 3V3, SSR-25-DA1, SSR-25-DA2
Changed lines of the file:
@@
 F1 "SSR-25-DA_DRIVER.sch" 50
 F2 "STM32_SSR-25-DA_OUTPUT" I L 11650 4750 50
-F3 "SSR-25-DA1" I R 13150 5000 50
-F4 "SSR-25-DA2" I R 13150 5100 50
+F3 "SSR-25-DA_P" I R 13150 5000 50
+F4 "SSR-25-DA_N" I R 13150 5100 50
 $EndSheet
 Text Label 14500 5000 2    50   ~ 0
-SSR-25-DA1
+SSR-25-DA_P
 Text Label 14500 5100 2    50   ~ 0
-SSR-25-DA2
+SSR-25-DA_N
 Wire Wire Line
 	13150 5100 14500 5100
@@
 	13150 5000 14500 5000
 Text Label 8600 4950 0    50   ~ 0
-SSR-25-DA1
+SSR-25-DA_P
 Text Label 8600 5050 0    50   ~ 0
-SSR-25-DA2
+SSR-25-DA_N
 Wire Wire Line
 	9400 5050 8600 5050
@@
 B2B_UART_RX
 $Comp
-L tinkerforge:3V3 #PWR?
-U 1 1 5BDD6C93
-P 3750 2650
-F 0 "#PWR?" H 3750 2500 50  0001 C CNN
-F 1 "3V3" H 3765 2823 50  0000 C CNN
-F 2 "" H 3750 2650 50  0000 C CNN
-F 3 "" H 3750 2650 50  0000 C CNN
-	1    3750 2650
-	1    0    0    -1
-$EndComp
-$Comp
 L taobao-r:R472,0603 R?
 U 1 1 5BDDACA3
@@
 Wire Wire Line
 	5400 3400 5550 3400
+$Comp
+L power:+3V3 #PWR?
+U 1 1 5BE0CC9B
+P 3750 2650
+F 0 "#PWR?" H 3750 2500 50  0001 C CNN
+F 1 "+3V3" H 3765 2823 50  0000 C CNN
+F 2 "" H 3750 2650 50  0001 C CNN
+F 3 "" H 3750 2650 50  0001 C CNN
+	1    3750 2650
+	1    0    0    -1
+$EndComp
 $EndSCHEMATC

Commit message: categorize pinout,
Parts:
- added J?: PCB_UART, w_conn_mkds:mkds_1,5-3, symbol Connector_Generic:Conn_01x10
Connections:
- wire segments 82 -> 88
Other:
- note added: "TO MAIN LANDING BOARD"
- moved on the sheet: C1, J1, J2, J3, J4, J5, J9, J?

Commit message: update,
Parts:
- gave numbers to parts that had none: 8
Changed lines of the file:
@@
 B2B_UART_RX
 $Comp
-L taobao-r:R472,0603 R?
+L taobao-r:R472,0603 R5
 U 1 1 5BDDACA3
 P 3750 2850
-F 0 "R?" H 3809 2896 50  0000 L CNN
+F 0 "R5" H 3809 2896 50  0000 L CNN
 F 1 "R472,0603" H 3809 2805 50  0000 L CNN
 F 2 "" H 3750 2850 50  0001 C CNN
@@
 $EndComp
 $Comp
-L taobao-r:R472,0603 R?
+L taobao-r:R472,0603 R6
 U 1 1 5BDDACCF
 P 3950 2850
-F 0 "R?" H 4009 2896 50  0000 L CNN
+F 0 "R6" H 4009 2896 50  0000 L CNN
 F 1 "R472,0603" H 4009 2805 50  0000 L CNN
 F 2 "" H 3950 2850 50  0001 C CNN
@@
 	4950 3600 4450 3600
 $Comp
-L Device:Jumper_NO_Small JP?
+L Device:Jumper_NO_Small JP2
 U 1 1 5BDDECBA
 P 4350 3200
-F 0 "JP?" H 4350 3385 50  0000 C CNN
+F 0 "JP2" H 4350 3385 50  0000 C CNN
 F 1 "Jumper_NO_Small" H 4350 3294 50  0000 C CNN
 F 2 "" H 4350 3200 50  0001 C CNN
@@
 $EndComp
 $Comp
-L Device:Jumper_NO_Small JP?
+L Device:Jumper_NO_Small JP3
 U 1 1 5BDDED1D
 P 4350 3300
-F 0 "JP?" H 4350 3485 50  0000 C CNN
+F 0 "JP3" H 4350 3485 50  0000 C CNN
 F 1 "Jumper_NO_Small" H 4350 3394 50  0000 C CNN
 F 2 "" H 4350 3300 50  0001 C CNN
@@
 Connection ~ 3950 3300
 $Comp
-L Device:Jumper_NO_Small JP?
+L Device:Jumper_NO_Small JP5
 U 1 1 5BE40594
 P 4350 3700
-F 0 "JP?" H 4350 3885 50  0000 C CNN
+F 0 "JP5" H 4350 3885 50  0000 C CNN
 F 1 "Jumper_NO_Small" H 4350 3794 50  0000 C CNN
 F 2 "" H 4350 3700 50  0001 C CNN
@@
 $EndComp
 $Comp
-L Device:Jumper_NO_Small JP?
+L Device:Jumper_NO_Small JP4
 U 1 1 5BE405D0
 P 4350 3600
-F 0 "JP?" H 4350 3785 50  0000 C CNN
+F 0 "JP4" H 4350 3785 50  0000 C CNN
 F 1 "Jumper_NO_Small" H 4350 3694 50  0000 C CNN
 F 2 "" H 4350 3600 50  0001 C CNN
@@
 	6000 7750 6200 7750
 $Comp
-L Connector_Generic:Conn_01x02 J?
+L Connector_Generic:Conn_01x02 J11
 U 1 1 5BE5623C
 P 4200 7650
-F 0 "J?" H 4280 7642 50  0000 L CNN
+F 0 "J11" H 4280 7642 50  0000 L CNN
 F 1 "SSR2_CTRL" H 4280 7551 50  0000 L CNN
 F 2 "w_conn_mkds:mkds_1,5-2" H 4200 7650 50  0001 C CNN
@@
 follows PC fan ordering
 $Comp
-L power:GND #PWR?
+L power:GND #PWR0117
 U 1 1 5BE0459B
 P 5400 3600
-F 0 "#PWR?" H 5400 3350 50  0001 C CNN
+F 0 "#PWR0117" H 5400 3350 50  0001 C CNN
 F 1 "GND" H 5405 3427 50  0000 C CNN
 F 2 "" H 5400 3600 50  0001 C CNN
@@
 	5400 3400 5550 3400
 $Comp
-L power:+3V3 #PWR?
+L power:+3V3 #PWR0118
 U 1 1 5BE0CC9B
 P 3750 2650
-F 0 "#PWR?" H 3750 2500 50  0001 C CNN
+F 0 "#PWR0118" H 3750 2500 50  0001 C CNN
 F 1 "+3V3" H 3765 2823 50  0000 C CNN
 F 2 "" H 3750 2650 50  0001 C CNN
@@
 $EndComp
 $Comp
-L Connector_Generic:Conn_01x10 J?
+L Connector_Generic:Conn_01x10 J14
 U 1 1 5BDC7136
 P 11350 9350
-F 0 "J?" H 11430 9342 50  0000 L CNN
+F 0 "J14" H 11430 9342 50  0000 L CNN
 F 1 "PCB_UART" H 11430 9251 50  0000 L CNN
 F 2 "w_conn_mkds:mkds_1,5-3" H 11350 9350 50  0001 C CNN
@@
 	10400 9150 11150 9150
 $Comp
-L power:GND #PWR?
+L power:GND #PWR0119
 U 1 1 5BDC7281
 P 11000 9450
-F 0 "#PWR?" H 11000 9200 50  0001 C CNN
+F 0 "#PWR0119" H 11000 9200 50  0001 C CNN
 F 1 "GND" H 11005 9277 50  0000 C CNN
 F 2 "" H 11000 9450 50  0001 C CNN

Commit message: assign footprint,
Parts:
- JP2, JP3, JP4, JP5: footprint (none) -> Jumper:SolderJumper-2_P1.3mm_Open_TrianglePad1.0x1.5mm
- R5, R6: footprint (none) -> Resistor_SMD:R_0603_1608Metric_Pad1.05x0.95mm_HandSolder
Changed lines of the file:
@@
 	10050 6650 10800 6650
-Wire Wire Line
-	3500 3300 3950 3300
 Wire Wire Line
 	3500 3200 3750 3200
@@
 F 0 "R5" H 3809 2896 50  0000 L CNN
 F 1 "R472,0603" H 3809 2805 50  0000 L CNN
-F 2 "" H 3750 2850 50  0001 C CNN
+F 2 "Resistor_SMD:R_0603_1608Metric_Pad1.05x0.95mm_HandSolder" H 3750 2850 50  0001 C CNN
 F 3 "~" H 3750 2850 50  0001 C CNN
 	1    3750 2850
@@
 F 0 "R6" H 4009 2896 50  0000 L CNN
 F 1 "R472,0603" H 4009 2805 50  0000 L CNN
-F 2 "" H 3950 2850 50  0001 C CNN
+F 2 "Resistor_SMD:R_0603_1608Metric_Pad1.05x0.95mm_HandSolder" H 3950 2850 50  0001 C CNN
 F 3 "~" H 3950 2850 50  0001 C CNN
 	1    3950 2850
@@
 Wire Wire Line
 	3750 2700 3950 2700
-Wire Wire Line
-	3950 2700 3950 2750
 Connection ~ 3750 2700
 Wire Wire Line
@@
 Wire Wire Line
 	3750 2950 3750 3200
-Wire Wire Line
-	3950 2950 3950 3300
 $Comp
 L Connector_Generic:Conn_01x08 J10
@@
 $EndComp
 Wire Wire Line
-	3700 3600 4250 3600
-Wire Wire Line
-	3700 3700 4250 3700
-Wire Wire Line
-	4450 3700 5050 3700
-Wire Wire Line
-	5050 3700 5050 3300
-Wire Wire Line
 	5050 3300 5550 3300
-Wire Wire Line
-	5550 3200 4950 3200
-Wire Wire Line
-	4950 3200 4950 3600
-Wire Wire Line
-	4950 3600 4450 3600
-$Comp
-L Device:Jumper_NO_Small JP2
-U 1 1 5BDDECBA
-P 4350 3200
-F 0 "JP2" H 4350 3385 50  0000 C CNN
-F 1 "Jumper_NO_Small" H 4350 3294 50  0000 C CNN
-F 2 "" H 4350 3200 50  0001 C CNN
-F 3 "~" H 4350 3200 50  0001 C CNN
-	1    4350 3200
-	1    0    0    -1
-$EndComp
-$Comp
-L Device:Jumper_NO_Small JP3
-U 1 1 5BDDED1D
-P 4350 3300
-F 0 "JP3" H 4350 3485 50  0000 C CNN
-F 1 "Jumper_NO_Small" H 4350 3394 50  0000 C CNN
-F 2 "" H 4350 3300 50  0001 C CNN
-F 3 "~" H 4350 3300 50  0001 C CNN
-	1    4350 3300
-	1    0    0    -1
-$EndComp
-Wire Wire Line
-	4450 3300 5050 3300
-Connection ~ 5050 3300
-Wire Wire Line
-	4450 3200 4950 3200
-Connection ~ 4950 3200
-Wire Wire Line
-	3750 3200 4250 3200
 Connection ~ 3750 3200
-Wire Wire Line
-	3950 3300 4250 3300
-Connection ~ 3950 3300
-$Comp
-L Device:Jumper_NO_Small JP5
-U 1 1 5BE40594
-P 4350 3700
-F 0 "JP5" H 4350 3885 50  0000 C CNN
-F 1 "Jumper_NO_Small" H 4350 3794 50  0000 C CNN
-F 2 "" H 4350 3700 50  0001 C CNN
-F 3 "~" H 4350 3700 50  0001 C CNN
-	1    4350 3700
-	1    0    0    -1
-$EndComp
-$Comp
-L Device:Jumper_NO_Small JP4
-U 1 1 5BE405D0
-P 4350 3600
-F 0 "JP4" H 4350 3785 50  0000 C CNN
-F 1 "Jumper_NO_Small" H 4350 3694 50  0000 C CNN
-F 2 "" H 4350 3600 50  0001 C CNN
-F 3 "~" H 4350 3600 50  0001 C CNN
-	1    4350 3600
-	1    0    0    -1
-$EndComp
 Text Label 9050 7850 2    50   ~ 0
 SSR_CH2_OUTPUT1
@@
 Text Notes 10150 5800 0    300  ~ 0
 TO MAIN LANDING BOARD
+Wire Wire Line
+	3950 3300 4250 3300
+Wire Wire Line
+	3500 3300 3950 3300
+Connection ~ 3950 3300
+Wire Wire Line
+	3950 2700 3950 2750
+Wire Wire Line
+	3950 2950 3950 3300
+Wire Wire Line
+	3700 3700 4250 3700
+Wire Wire Line
+	3750 3200 4250 3200
+Wire Wire Line
+	3700 3600 4250 3600
+Wire Wire Line
+	5050 3700 5050 3300
+Wire Wire Line
+	4450 3700 5050 3700
+Wire Wire Line
+	4950 3600 4450 3600
+Wire Wire Line
+	4450 3200 4950 3200
+Wire Wire Line
+	5550 3200 4950 3200
+Connection ~ 4950 3200
+Wire Wire Line
+	4950 3200 4950 3600
+Connection ~ 5050 3300
+Wire Wire Line
+	4450 3300 5050 3300
+$Comp
+L Device:Jumper_NO_Small JP4
+U 1 1 5BE405D0
+P 4350 3600
+F 0 "JP4" H 4350 3785 50  0000 C CNN
+F 1 "Jumper_NO_Small" H 4350 3694 50  0000 C CNN
+F 2 "Jumper:SolderJumper-2_P1.3mm_Open_TrianglePad1.0x1.5mm" H 4350 3600 50  0001 C CNN
+F 3 "~" H 4350 3600 50  0001 C CNN
+	1    4350 3600
+	1    0    0    -1
+$EndComp
+$Comp
+L Device:Jumper_NO_Small JP5
+U 1 1 5BE40594
+P 4350 3700
+F 0 "JP5" H 4350 3885 50  0000 C CNN
+F 1 "Jumper_NO_Small" H 4350 3794 50  0000 C CNN
+F 2 "Jumper:SolderJumper-2_P1.3mm_Open_TrianglePad1.0x1.5mm" H 4350 3700 50  0001 C CNN
+F 3 "~" H 4350 3700 50  0001 C CNN
+	1    4350 3700
+	1    0    0    -1
+$EndComp
+$Comp
+L Device:Jumper_NO_Small JP3
+U 1 1 5BDDED1D
+P 4350 3300
+F 0 "JP3" H 4350 3485 50  0000 C CNN
+F 1 "Jumper_NO_Small" H 4350 3394 50  0000 C CNN
+F 2 "Jumper:SolderJumper-2_P1.3mm_Open_TrianglePad1.0x1.5mm" H 4350 3300 50  0001 C CNN
+F 3 "~" H 4350 3300 50  0001 C CNN
+	1    4350 3300
+	1    0    0    -1
+$EndComp
+$Comp
+L Device:Jumper_NO_Small JP2
+U 1 1 5BDDECBA
+P 4350 3200
+F 0 "JP2" H 4350 3385 50  0000 C CNN
+F 1 "Jumper_NO_Small" H 4350 3294 50  0000 C CNN
+F 2 "Jumper:SolderJumper-2_P1.3mm_Open_TrianglePad1.0x1.5mm" H 4350 3200 50  0001 C CNN
+F 3 "~" H 4350 3200 50  0001 C CNN
+	1    4350 3200
+	1    0    0    -1
+$EndComp
 $EndSCHEMATC

Commit message: init commit,
Parts:
- J14: footprint w_conn_mkds:mkds_1,5-3 -> footprint-lib:s8b-ph-kl; symbol Connector_Generic:Conn_01x10 -> Connector_Generic:Conn_01x08
Changed lines of the file:
@@
 $EndComp
 $Comp
-L Connector_Generic:Conn_01x10 J14
+L Connector_Generic:Conn_01x08 J14
 U 1 1 5BDC7136
-P 11350 9350
-F 0 "J14" H 11430 9342 50  0000 L CNN
-F 1 "PCB_UART" H 11430 9251 50  0000 L CNN
-F 2 "w_conn_mkds:mkds_1,5-3" H 11350 9350 50  0001 C CNN
-F 3 "~" H 11350 9350 50  0001 C CNN
-	1    11350 9350
+P 11350 9250
+F 0 "J14" H 11430 9242 50  0000 L CNN
+F 1 "PCB_UART" H 11430 9151 50  0000 L CNN
+F 2 "footprint-lib:s8b-ph-kl" H 11350 9250 50  0001 C CNN
+F 3 "~" H 11350 9250 50  0001 C CNN
+	1    11350 9250
 	1    0    0    -1
 $EndComp
