File: pcb/stm32_bottom_board_respin.sch (KiCad schematic (older format))
At the start: 16 parts, among them J1 48V_SRC, J10 FCC_B2B, J11 SSR2_CTRL, J14 PCB_UART, J2 WS2812_CTRL, J3 FAN_CTRL, J4 SSR_OUTPUT, J5 PURFUME_CTRL, J9 PCB_UART

Commit message: update existing footprint to smaller one,
Parts:
- J1, J11: footprint w_conn_mkds:mkds_1,5-2 -> footprint-lib:s2b-ph-kl
- J2: footprint w_conn_mkds:mkds_1,5-3 -> footprint-lib:s3b-ph-kl
- J3: footprint w_conn_mkds:mkds_1,5-4 -> footprint-lib:s4b-ph-kl
- JP2: value Jumper_NO_Small -> SCL_EN
- JP3: value Jumper_NO_Small -> SDA_EN
- JP4: value Jumper_NO_Small -> TX_EN
- JP5: value Jumper_NO_Small -> RX_EN
Changed lines of the file:
@@
 F 0 "J2" H 3330 8942 50  0000 L CNN
 F 1 "WS2812_CTRL" H 3330 8851 50  0000 L CNN
-F 2 "w_conn_mkds:mkds_1,5-3" H 3250 8900 50  0001 C CNN
+F 2 "footprint-lib:s3b-ph-kl" H 3250 8900 50  0001 C CNN
 F 3 "~" H 3250 8900 50  0001 C CNN
 	1    3250 8900
@@
 F 0 "J3" H 4430 6342 50  0000 L CNN
 F 1 "FAN_CTRL" H 4430 6251 50  0000 L CNN
-F 2 "w_conn_mkds:mkds_1,5-4" H 4350 6350 50  0001 C CNN
+F 2 "footprint-lib:s4b-ph-kl" H 4350 6350 50  0001 C CNN
 F 3 "~" H 4350 6350 50  0001 C CNN
 	1    4350 6350
@@
 F 0 "J1" H 2680 6242 50  0000 L CNN
 F 1 "48V_SRC" H 2680 6151 50  0000 L CNN
-F 2 "w_conn_mkds:mkds_1,5-2" H 2600 6250 50  0001 C CNN
+F 2 "footprint-lib:s2b-ph-kl" H 2600 6250 50  0001 C CNN
 F 3 "~" H 2600 6250 50  0001 C CNN
 	1    2600 6250
@@
 F 0 "J11" H 4280 7642 50  0000 L CNN
 F 1 "SSR2_CTRL" H 4280 7551 50  0000 L CNN
-F 2 "w_conn_mkds:mkds_1,5-2" H 4200 7650 50  0001 C CNN
+F 2 "footprint-lib:s2b-ph-kl" H 4200 7650 50  0001 C CNN
 F 3 "~" H 4200 7650 50  0001 C CNN
 	1    4200 7650
@@
 P 4350 3600
 F 0 "JP4" H 4350 3785 50  0000 C CNN
-F 1 "Jumper_NO_Small" H 4350 3694 50  0000 C CNN
+F 1 "TX_EN" H 4350 3694 50  0000 C CNN
 F 2 "Jumper:SolderJumper-2_P1.3mm_Open_TrianglePad1.0x1.5mm" H 4350 3600 50  0001 C CNN
 F 3 "~" H 4350 3600 50  0001 C CNN
@@
 P 4350 3700
 F 0 "JP5" H 4350 3885 50  0000 C CNN
-F 1 "Jumper_NO_Small" H 4350 3794 50  0000 C CNN
+F 1 "RX_EN" H 4350 3794 50  0000 C CNN
 F 2 "Jumper:SolderJumper-2_P1.3mm_Open_TrianglePad1.0x1.5mm" H 4350 3700 50  0001 C CNN
 F 3 "~" H 4350 3700 50  0001 C CNN
@@
 P 4350 3300
 F 0 "JP3" H 4350 3485 50  0000 C CNN
-F 1 "Jumper_NO_Small" H 4350 3394 50  0000 C CNN
+F 1 "SDA_EN" H 4350 3394 50  0000 C CNN
 F 2 "Jumper:SolderJumper-2_P1.3mm_Open_TrianglePad1.0x1.5mm" H 4350 3300 50  0001 C CNN
 F 3 "~" H 4350 3300 50  0001 C CNN
@@
 P 4350 3200
 F 0 "JP2" H 4350 3385 50  0000 C CNN
-F 1 "Jumper_NO_Small" H 4350 3294 50  0000 C CNN
+F 1 "SCL_EN" H 4350 3294 50  0000 C CNN
 F 2 "Jumper:SolderJumper-2_P1.3mm_Open_TrianglePad1.0x1.5mm" H 4350 3200 50  0001 C CNN
 F 3 "~" H 4350 3200 50  0001 C CNN

Commit message: update existing footprint to smaller one,
Parts:
- J4, J5: footprint w_conn_mkds:mkds_1,5-2 -> footprint-lib:s2b-ph-kl
- J9: footprint w_conn_mkds:mkds_1,5-3 -> footprint-lib:s3b-ph-kl
Changed lines of the file:
@@
 F 0 "J5" H 4280 7292 50  0000 L CNN
 F 1 "PURFUME_CTRL" H 4280 7201 50  0000 L CNN
-F 2 "w_conn_mkds:mkds_1,5-2" H 4200 7300 50  0001 C CNN
+F 2 "footprint-lib:s2b-ph-kl" H 4200 7300 50  0001 C CNN
 F 3 "~" H 4200 7300 50  0001 C CNN
 	1    4200 7300
@@
 F 0 "J4" H 11080 7992 50  0000 L CNN
 F 1 "SSR_OUTPUT" H 11080 7901 50  0000 L CNN
-F 2 "w_conn_mkds:mkds_1,5-2" H 11000 8000 50  0001 C CNN
+F 2 "footprint-lib:s2b-ph-kl" H 11000 8000 50  0001 C CNN
 F 3 "~" H 11000 8000 50  0001 C CNN
 	1    11000 8000
@@
 F 0 "J9" H 11080 6742 50  0000 L CNN
 F 1 "PCB_UART" H 11080 6651 50  0000 L CNN
-F 2 "w_conn_mkds:mkds_1,5-3" H 11000 6750 50  0001 C CNN
+F 2 "footprint-lib:s3b-ph-kl" H 11000 6750 50  0001 C CNN
 F 3 "~" H 11000 6750 50  0001 C CNN
 	1    11000 6750

Commit message: update,
Parts:
- J14: value PCB_UART -> MAINBOARD_CONN
Changed lines of the file:
@@
 P 11350 9250
 F 0 "J14" H 11430 9242 50  0000 L CNN
-F 1 "PCB_UART" H 11430 9151 50  0000 L CNN
+F 1 "MAINBOARD_CONN" H 11430 9151 50  0000 L CNN
 F 2 "footprint-lib:s8b-ph-kl" H 11350 9250 50  0001 C CNN
 F 3 "~" H 11350 9250 50  0001 C CNN

Commit message: update,
Changed lines of the file:
@@
 Text Label 1650 6250 0    50   ~ 0
 FAN_48V_GND
-Wire Wire Line
-	2400 6350 2350 6350
 Text Label 1550 6350 0    50   ~ 0
 FAN_48V
-Wire Wire Line
-	1550 6350 2350 6350
 $Comp
 L power:GND #PWR03
 U 1 1 5BCC7684
-P 2350 6450
-F 0 "#PWR03" H 2350 6200 50  0001 C CNN
-F 1 "GND" H 2355 6277 50  0000 C CNN
-F 2 "" H 2350 6450 50  0001 C CNN
-F 3 "" H 2350 6450 50  0001 C CNN
-	1    2350 6450
-	1    0    0    -1
-$EndComp
-Wire Wire Line
-	2350 6350 2350 6450
-Wire Wire Line
-	2400 6250 1650 6250
+P 2300 6050
+F 0 "#PWR03" H 2300 5800 50  0001 C CNN
+F 1 "GND" H 2305 5877 50  0000 C CNN
+F 2 "" H 2300 6050 50  0001 C CNN
+F 3 "" H 2300 6050 50  0001 C CNN
+	1    2300 6050
+	-1   0    0    1
+$EndComp
+Wire Wire Line
+	2400 6250 2300 6250
 $Sheet
 S 6200 8400 1500 850
@@
 Text Label 3350 6550 0    50   ~ 0
 FAN_PWM_OUTPUT
-Connection ~ 2350 6350
 Text Notes 3450 6800 0    50   ~ 0
 follows PC fan ordering
@@
 	1    0    0    -1
 $EndComp
+Wire Wire Line
+	1550 6350 2400 6350
+Wire Wire Line
+	2300 6050 2300 6250
+Connection ~ 2300 6250
+Wire Wire Line
+	2300 6250 1650 6250
 $EndSCHEMATC

Commit message: basic rout complete,
Changed lines of the file:
@@
 L Connector_Generic:Conn_01x02 J4
 U 1 1 5BCB931B
-P 11000 8000
-F 0 "J4" H 11080 7992 50  0000 L CNN
-F 1 "SSR_OUTPUT" H 11080 7901 50  0000 L CNN
-F 2 "footprint-lib:s2b-ph-kl" H 11000 8000 50  0001 C CNN
-F 3 "~" H 11000 8000 50  0001 C CNN
-	1    11000 8000
-	1    0    0    -1
+P 11000 8100
+F 0 "J4" H 11080 8092 50  0000 L CNN
+F 1 "SSR_OUTPUT" H 11080 8001 50  0000 L CNN
+F 2 "footprint-lib:s2b-ph-kl" H 11000 8100 50  0001 C CNN
+F 3 "~" H 11000 8100 50  0001 C CNN
+	1    11000 8100
+	1    0    0    1
 $EndComp
 $Sheet

Commit message: remove jumper,
Parts:
- removed JP2: SCL_EN, Jumper:SolderJumper-2_P1.3mm_Open_TrianglePad1.0x1.5mm, symbol Device:Jumper_NO_Small
- removed JP3: SDA_EN, Jumper:SolderJumper-2_P1.3mm_Open_TrianglePad1.0x1.5mm, symbol Device:Jumper_NO_Small
- removed JP4: TX_EN, Jumper:SolderJumper-2_P1.3mm_Open_TrianglePad1.0x1.5mm, symbol Device:Jumper_NO_Small
- removed JP5: RX_EN, Jumper:SolderJumper-2_P1.3mm_Open_TrianglePad1.0x1.5mm, symbol Device:Jumper_NO_Small
- R5, R6: value R472,0603 -> R472,0603,NC
Connections:
- wire segments 88 -> 84
Changed lines of the file:
@@
 P 3750 2850
 F 0 "R5" H 3809 2896 50  0000 L CNN
-F 1 "R472,0603" H 3809 2805 50  0000 L CNN
+F 1 "R472,0603,NC" H 3809 2805 50  0000 L CNN
 F 2 "Resistor_SMD:R_0603_1608Metric_Pad1.05x0.95mm_HandSolder" H 3750 2850 50  0001 C CNN
 F 3 "~" H 3750 2850 50  0001 C CNN
@@
 P 3950 2850
 F 0 "R6" H 4009 2896 50  0000 L CNN
-F 1 "R472,0603" H 4009 2805 50  0000 L CNN
+F 1 "R472,0603,NC" H 4009 2805 50  0000 L CNN
 F 2 "Resistor_SMD:R_0603_1608Metric_Pad1.05x0.95mm_HandSolder" H 3950 2850 50  0001 C CNN
 F 3 "~" H 3950 2850 50  0001 C CNN
@@
 Wire Wire Line
 	5050 3300 5550 3300
-Connection ~ 3750 3200
 Text Label 9050 7850 2    50   ~ 0
 SSR_CH2_OUTPUT1
@@
 TO MAIN LANDING BOARD
 Wire Wire Line
-	3950 3300 4250 3300
-Wire Wire Line
 	3500 3300 3950 3300
-Connection ~ 3950 3300
 Wire Wire Line
 	3950 2700 3950 2750
@@
 	3950 2950 3950 3300
 Wire Wire Line
-	3700 3700 4250 3700
-Wire Wire Line
-	3750 3200 4250 3200
-Wire Wire Line
-	3700 3600 4250 3600
-Wire Wire Line
 	5050 3700 5050 3300
 Wire Wire Line
-	4450 3700 5050 3700
-Wire Wire Line
-	4950 3600 4450 3600
-Wire Wire Line
-	4450 3200 4950 3200
-Wire Wire Line
 	5550 3200 4950 3200
-Connection ~ 4950 3200
 Wire Wire Line
 	4950 3200 4950 3600
-Connection ~ 5050 3300
-Wire Wire Line
-	4450 3300 5050 3300
-$Comp
-L Device:Jumper_NO_Small JP4
-U 1 1 5BE405D0
-P 4350 3600
-F 0 "JP4" H 4350 3785 50  0000 C CNN
-F 1 "TX_EN" H 4350 3694 50  0000 C CNN
-F 2 "Jumper:SolderJumper-2_P1.3mm_Open_TrianglePad1.0x1.5mm" H 4350 3600 50  0001 C CNN
-F 3 "~" H 4350 3600 50  0001 C CNN
-	1    4350 3600
-	1    0    0    -1
-$EndComp
-$Comp
-L Device:Jumper_NO_Small JP5
-U 1 1 5BE40594
-P 4350 3700
-F 0 "JP5" H 4350 3885 50  0000 C CNN
-F 1 "RX_EN" H 4350 3794 50  0000 C CNN
-F 2 "Jumper:SolderJumper-2_P1.3mm_Open_TrianglePad1.0x1.5mm" H 4350 3700 50  0001 C CNN
-F 3 "~" H 4350 3700 50  0001 C CNN
-	1    4350 3700
-	1    0    0    -1
-$EndComp
-$Comp
-L Device:Jumper_NO_Small JP3
-U 1 1 5BDDED1D
-P 4350 3300
-F 0 "JP3" H 4350 3485 50  0000 C CNN
-F 1 "SDA_EN" H 4350 3394 50  0000 C CNN
-F 2 "Jumper:SolderJumper-2_P1.3mm_Open_TrianglePad1.0x1.5mm" H 4350 3300 50  0001 C CNN
-F 3 "~" H 4350 3300 50  0001 C CNN
-	1    4350 3300
-	1    0    0    -1
-$EndComp
-$Comp
-L Device:Jumper_NO_Small JP2
-U 1 1 5BDDECBA
-P 4350 3200
-F 0 "JP2" H 4350 3385 50  0000 C CNN
-F 1 "SCL_EN" H 4350 3294 50  0000 C CNN
-F 2 "Jumper:SolderJumper-2_P1.3mm_Open_TrianglePad1.0x1.5mm" H 4350 3200 50  0001 C CNN
-F 3 "~" H 4350 3200 50  0001 C CNN
-	1    4350 3200
-	1    0    0    -1
-$EndComp
 Wire Wire Line
 	1550 6350 2400 6350
@@
 Wire Wire Line
 	2300 6250 1650 6250
+Connection ~ 5050 3300
+Connection ~ 4950 3200
+Connection ~ 3750 3200
+Connection ~ 3950 3300
+Wire Wire Line
+	3750 3200 4950 3200
+Wire Wire Line
+	3950 3300 5050 3300
+Wire Wire Line
+	3700 3600 4950 3600
+Wire Wire Line
+	3700 3700 5050 3700
 $EndSCHEMATC

Commit message: update,
Connections:
- net labels added: PCB1_ALARM_COM
- wire segments 84 -> 87
Changed lines of the file:
@@
 	1    0    0    -1
 $EndComp
-Text Label 10400 9250 0    50   ~ 0
+Text Label 10400 9350 0    50   ~ 0
 IONAIR_TX
 Wire Wire Line
+	10400 9350 11150 9350
+Wire Wire Line
 	10400 9250 11150 9250
-Wire Wire Line
-	10400 9150 11150 9150
 $Comp
 L power:GND #PWR0119
 U 1 1 5BDC7281
-P 11000 9450
-F 0 "#PWR0119" H 11000 9200 50  0001 C CNN
-F 1 "GND" H 11005 9277 50  0000 C CNN
-F 2 "" H 11000 9450 50  0001 C CNN
-F 3 "" H 11000 9450 50  0001 C CNN
-	1    11000 9450
-	-1   0    0    -1
+P 11000 8850
+F 0 "#PWR0119" H 11000 8600 50  0001 C CNN
+F 1 "GND" H 11005 8677 50  0000 C CNN
+F 2 "" H 11000 8850 50  0001 C CNN
+F 3 "" H 11000 8850 50  0001 C CNN
+	1    11000 8850
+	-1   0    0    1
 $EndComp
 Wire Wire Line
-	11000 9450 11000 9350
+	11000 8850 11000 8950
 Wire Wire Line
-	11000 9350 11150 9350
-Text Label 10400 9150 0    50   ~ 0
+	11000 8950 11150 8950
+Text Label 10400 9250 0    50   ~ 0
 IONAIR_RX
-Text Label 10350 8950 0    50   ~ 0
+Text Label 10350 9050 0    50   ~ 0
 SSR-25-DA_P
-Text Label 10350 9050 0    50   ~ 0
+Text Label 10350 9150 0    50   ~ 0
 SSR-25-DA_N
 Wire Wire Line
+	11150 9150 10350 9150
+Wire Wire Line
 	11150 9050 10350 9050
-Wire Wire Line
-	11150 8950 10350 8950
 Wire Notes Line
 	9350 5000 9350 11100
@@
 Wire Wire Line
 	3700 3700 5050 3700
+$Comp
+L power:+5V #PWR0134
+U 1 1 5BF85C96
+P 11000 9750
+F 0 "#PWR0134" H 11000 9600 50  0001 C CNN
+F 1 "+5V" H 11015 9923 50  0000 C CNN
+F 2 "" H 11000 9750 50  0001 C CNN
+F 3 "" H 11000 9750 50  0001 C CNN
+	1    11000 9750
+	-1   0    0    1
+$EndComp
+Wire Wire Line
+	11000 9750 11000 9650
+Wire Wire Line
+	11000 9650 11150 9650
+Text Label 10400 9450 0    50   ~ 0
+PCB1_ALARM_COM
+Wire Wire Line
+	10400 9450 11150 9450
+Text GLabel 10400 9450 0    50   Input ~ 0
+PCB1_ALARM_COM
 $EndSCHEMATC
