File: pcb/_autosave-stm32_bottom_board_respin.kicad_pcb (KiCad board)
At the start: 2 copper layers, 100 x 70 mm, 90 parts, among them J1 48V_SRC, J10 FCC_B2B, J11 SSR2_CTRL, J12 POWER, J13 PMS7003S_CONN, J14 PCB_UART, J15 SWD_CONN, J2 WS2812_CTRL, J3 FAN_CTRL, J4 SSR_OUTPUT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

Commit message: update existing footprint to smaller one,
Parts:
- J1, J11, J4, J5: footprint w_conn_mkds:mkds_1,5-2 -> footprint-lib:s2b-ph-kl
- J14: footprint w_conn_mkds:mkds_1,5-3 -> footprint-lib:s8b-ph-kl
- J2, J9: footprint w_conn_mkds:mkds_1,5-3 -> footprint-lib:s3b-ph-kl
- J3: footprint w_conn_mkds:mkds_1,5-4 -> footprint-lib:s4b-ph-kl
- JP2: value Jumper_NO_Small -> SCL_EN
- JP3: value Jumper_NO_Small -> SDA_EN
- JP4: value Jumper_NO_Small -> TX_EN
- JP5: value Jumper_NO_Small -> RX_EN
- moved J14 116.0 mm to (65.4, 107.5)
Connections:
- J15 pad 1: (no net) -> /STM32_CORE/RST
- J15 pad 5: (no net) -> /STM32_CORE/SWIM
- J6 pad 1: (no net) -> Net-(J6-Pad1)
- J7 pad 10: (no net) -> Net-(J7-Pad10)
- J7 pad 11: (no net) -> Net-(J7-Pad11)
- J7 pad 12: (no net) -> Net-(J7-Pad12)
- J8 pad 3: (no net) -> Net-(J8-Pad3)
- R26 pad 1: (no net) -> 3V3
- U5 pad 10: (no net) -> /rs232_level_switch/TTL-TX2
- U5 pad 7: (no net) -> /rs232_level_switch/RS232-TX2
- U5 pad 8: (no net) -> /rs232_level_switch/RS232-RX2
- U5 pad 9: (no net) -> /rs232_level_switch/TTL-RX2
