File: pcb/_autosave-stm32_bottom_board_respin.kicad_pcb (KiCad board)
At the start: 2 copper layers, 100 x 70 mm, 93 parts, among them J1 48V_SRC, J10 FCC_B2B, J11 SSR2_CTRL, J12 POWER, J13 PMS7003S_CONN, J14 MAINBOARD_CONN, J2 WS2812_CTRL, J3 FAN_CTRL, J4 SSR_OUTPUT, J5 PURFUME_CTRL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

Commit message: update,
Routing:
- net GND: track 407.4 -> 418.2 mm, vias 5 -> 4
- net +5V: track 333.7 -> 342.3 mm
- net /IONAIR_RX: track 27.2 -> 29.9 mm
- net /IONAIR_TX: track 32.0 -> 29.5 mm
Changed lines of the file:
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@@
     (thickness 1.6)
     (drawings 20)
-    (tracks 980)
+    (tracks 972)
     (zones 0)
     (modules 93)
@@
     (solder_mask_min_width 0.25)
     (aux_axis_origin 10 10)
-    (visible_elements FFFFFFFF)
+    (visible_elements FFF9F91F)
     (pcbplotparams
       (layerselection 0x010fc_ffffffff)
@@
   (segment (start 50.76184 77.5) (end 54.5 77.5) (width 1) (layer F.Cu) (net 1) (status 20))
   (segment (start 48.6 75.4) (end 50.34849 77.14849) (width 1) (layer F.Cu) (net 1))
-  (segment (start 48.426628 84.88663) (end 48.426628 88.573372) (width 1) (layer F.Cu) (net 1))
-  (segment (start 48.426628 88.573372) (end 48 89) (width 1) (layer F.Cu) (net 1))
-  (via (at 47.8 96.2) (size 2.5) (drill 1) (layers F.Cu B.Cu) (net 1))
-  (segment (start 48 89) (end 48 96) (width 1) (layer F.Cu) (net 1))
-  (segment (start 48 96) (end 47.8 96.2) (width 1) (layer F.Cu) (net 1))
-  (segment (start 47.8 96.2) (end 49 95) (width 1) (layer B.Cu) (net 1))
-  (segment (start 54.241018 95) (end 56.341018 97.1) (width 1) (layer B.Cu) (net 1))
-  (segment (start 49 95) (end 54.241018 95) (width 1) (layer B.Cu) (net 1))
-  (segment (start 59.45001 94.04897) (end 59.99898 93.5) (width 1) (layer B.Cu) (net 1) (status 30))
-  (segment (start 58.600613 95.45001) (end 59.45001 94.600613) (width 1) (layer B.Cu) (net 1) (status 20))
-  (segment (start 58.04897 95.45001) (end 58.600613 95.45001) (width 1) (layer B.Cu) (net 1))
-  (segment (start 56.39898 97.1) (end 58.04897 95.45001) (width 1) (layer B.Cu) (net 1))
-  (segment (start 59.45001 94.600613) (end 59.45001 94.04897) (width 1) (layer B.Cu) (net 1) (status 30))
-  (segment (start 56.341018 97.1) (end 56.39898 97.1) (width 1) (layer B.Cu) (net 1))
   (segment (start 69.101 88.025) (end 61.475 88.025) (width 1) (layer F.Cu) (net 1) (status 10))
   (segment (start 59.99898 89.50102) (end 59.99898 93.5) (width 1) (layer F.Cu) (net 1) (status 20))
@@
   (segment (start 53.100001 82.523999) (end 53.100001 83.676001) (width 1) (layer B.Cu) (net 1))
   (segment (start 53.100001 83.676001) (end 52.476001 84.300001) (width 1) (layer B.Cu) (net 1))
-  (segment (start 52.476001 84.300001) (end 44.700001 84.300001) (width 1) (layer B.Cu) (net 1))
   (segment (start 41.6755 80.9) (end 44.252 78.3235) (width 1) (layer F.Cu) (net 1) (status 20))
   (segment (start 41.3 80.9) (end 41.6755 80.9) (width 1) (layer F.Cu) (net 1))
@@
   (segment (start 100.9702 44.4) (end 100.39696 44.97324) (width 1) (layer F.Cu) (net 1))
   (segment (start 105.7 44.4) (end 100.9702 44.4) (width 1) (layer F.Cu) (net 1))
+  (segment (start 51.49088 84.300001) (end 44.700001 84.300001) (width 1) (layer B.Cu) (net 1))
+  (segment (start 51.49088 84.300001) (end 51.49088 97.13976) (width 1) (layer B.Cu) (net 1))
+  (segment (start 52.476001 84.300001) (end 51.49088 84.300001) (width 1) (layer B.Cu) (net 1))
+  (segment (start 51.49088 97.13976) (end 52.49164 98.14052) (width 1) (layer B.Cu) (net 1))
+  (segment (start 52.49164 98.14052) (end 70.5358 98.14052) (width 1) (layer B.Cu) (net 1))
+  (segment (start 72.50152 96.1748) (end 72.50152 93.5) (width 1) (layer B.Cu) (net 1))
+  (segment (start 70.5358 98.14052) (end 72.50152 96.1748) (width 1) (layer B.Cu) (net 1))
   (segment (start 92.875 74.55) (end 91.4 76.025) (width 0.3) (layer F.Cu) (net 2) (status 20))
   (segment (start 98.4 74.55) (end 92.875 74.55) (width 0.3) (layer F.Cu) (net 2) (status 10))
@@
   (via (at 78.8 89.3) (size 1) (drill 0.4) (layers F.Cu B.Cu) (net 4))
   (segment (start 78.25 86.9) (end 78.8 87.45) (width 0.5) (layer B.Cu) (net 4))
-  (segment (start 78.8 87.45) (end 78.8 89.3) (width 0.5) (layer B.Cu) (net 4))
   (segment (start 79.975 89.3) (end 80.5 88.775) (width 0.5) (layer F.Cu) (net 4) (status 20))
   (segment (start 78.8 89.3) (end 79.975 89.3) (width 0.5) (layer F.Cu) (net 4))
@@
   (segment (start 72.7 30.7) (end 76.96056 34.96056) (width 0.5) (layer B.Cu) (net 4))
   (segment (start 76.96056 34.96056) (end 77.208 35.208) (width 0.5) (layer B.Cu) (net 4))
+  (segment (start 78.8 88.70696) (end 87.38616 88.70696) (width 0.5) (layer B.Cu) (net 4))
+  (segment (start 78.8 88.70696) (end 78.8 89.3) (width 0.5) (layer B.Cu) (net 4))
+  (segment (start 78.8 87.45) (end 78.8 88.70696) (width 0.5) (layer B.Cu) (net 4))
   (segment (start 81.1188 74.4614) (end 81.8414 73.7388) (width 0.3) (layer F.Cu) (net 5) (status 30))
   (segment (start 79.1744 74.4614) (end 81.1188 74.4614) (width 0.3) (layer F.Cu) (net 5) (status 30))
@@
   (segment (start 40.385 89.64) (end 40 90.025) (width 0.3) (layer F.Cu) (net 43) (status 30))
   (segment (start 44.85 89.64) (end 40.385 89.64) (width 0.3) (layer F.Cu) (net 43) (status 30))
-  (segment (start 56.00102 94) (end 60.40102 98.4) (width 0.3) (layer F.Cu) (net 48) (status 10))
-  (segment (start 56.00102 93.5) (end 56.00102 94) (width 0.3) (layer F.Cu) (net 48) (status 30))
-  (segment (start 64.10102 98.4) (end 68.50102 94) (width 0.3) (layer F.Cu) (net 48) (status 20))
-  (segment (start 68.50102 94) (end 68.50102 93.5) (width 0.3) (layer F.Cu) (net 48) (status 30))
-  (segment (start 60.40102 98.4) (end 64.10102 98.4) (width 0.3) (layer F.Cu) (net 48))
   (segment (start 51.15 87.09) (end 55.79 87.09) (width 0.3) (layer F.Cu) (net 49) (status 10))
   (segment (start 58 89.3) (end 58 93.5) (width 0.3) (layer F.Cu) (net 49) (status 20))
   (segment (start 55.79 87.09) (end 58 89.3) (width 0.3) (layer F.Cu) (net 49))
-  (segment (start 58 94) (end 60.7 96.7) (width 0.3) (layer F.Cu) (net 49) (status 10))
-  (segment (start 58 93.5) (end 58 94) (width 0.3) (layer F.Cu) (net 49) (status 30))
-  (segment (start 60.7 96.7) (end 61.4 96.7) (width 0.3) (layer F.Cu) (net 49))
-  (segment (start 61.4 96.7) (end 62.7 95.4) (width 0.3) (layer F.Cu) (net 49))
-  (segment (start 66.6 90.3) (end 67.8 90.3) (width 0.3) (layer F.Cu) (net 49))
-  (segment (start 66.4 90.5) (end 66.6 90.3) (width 0.3) (layer F.Cu) (net 49))
-  (segment (start 64.870518 90.5) (end 66.4 90.5) (width 0.3) (layer F.Cu) (net 49))
-  (segment (start 62.7 95.4) (end 62.7 92.670518) (width 0.3) (layer F.Cu) (net 49))
-  (segment (start 62.7 92.670518) (end 64.870518 90.5) (width 0.3) (layer F.Cu) (net 49))
-  (segment (start 70.5 93) (end 67.8 90.3) (width 0.3) (layer F.Cu) (net 49) (status 10))
-  (segment (start 70.5 93.5) (end 70.5 93) (width 0.3) (layer F.Cu) (net 49) (status 30))
   (segment (start 44.85 87.09) (end 42.59 87.09) (width 0.3) (layer F.Cu) (net 50) (status 10))
   (segment (start 41.225 85.725) (end 40 85.725) (width 0.3) (layer F.Cu) (net 50) (status 20))
@@
   (segment (start 56.46928 89.29624) (end 56.46928 90.86506) (width 0.3) (layer F.Cu) (net 48))
   (segment (start 56.00102 93.5) (end 56.00102 91.33332) (width 0.3) (layer F.Cu) (net 48))
+  (segment (start 56.00102 91.93874) (end 56.00102 93.5) (width 0.3) (layer B.Cu) (net 48))
+  (segment (start 56.79948 91.14028) (end 56.00102 91.93874) (width 0.3) (layer B.Cu) (net 48))
+  (segment (start 68.50102 93.5) (end 68.50102 94.78542) (width 0.3) (layer B.Cu) (net 48))
+  (segment (start 68.50102 94.78542) (end 67.056 96.23044) (width 0.3) (layer B.Cu) (net 48))
+  (segment (start 67.056 96.23044) (end 63.754 96.23044) (width 0.3) (layer B.Cu) (net 48))
+  (segment (start 63.754 96.23044) (end 61.44768 93.92412) (width 0.3) (layer B.Cu) (net 48))
+  (segment (start 61.44768 91.57208) (end 61.01588 91.14028) (width 0.3) (layer B.Cu) (net 48))
+  (segment (start 61.44768 93.92412) (end 61.44768 91.57208) (width 0.3) (layer B.Cu) (net 48))
+  (segment (start 61.01588 91.14028) (end 56.79948 91.14028) (width 0.3) (layer B.Cu) (net 48))
+  (segment (start 58 93.5) (end 58 94.91128) (width 0.3) (layer B.Cu) (net 49))
+  (segment (start 58 94.91128) (end 60.01512 96.9264) (width 0.3) (layer B.Cu) (net 49))
+  (segment (start 60.01512 96.9264) (end 69.40804 96.9264) (width 0.3) (layer B.Cu) (net 49))
+  (segment (start 70.5 95.83444) (end 70.5 93.5) (width 0.3) (layer B.Cu) (net 49))
+  (segment (start 69.40804 96.9264) (end 70.5 95.83444) (width 0.3) (layer B.Cu) (net 49))
   (segment (start 60.85 77.5) (end 60.85 78.9262) (width 0.3) (layer B.Cu) (net 54))
   (segment (start 60.85 78.9262) (end 58.07964 81.69656) (width 0.3) (layer B.Cu) (net 54))
