File: pcb/PMS5003S_interface.sch (KiCad schematic (older format))
At the start: 1 part, among them J13 Conn_01x03

Commit message: update,
Parts:
- added R? (x2): R103,0603, symbol taobao-r:R103,0603
- J13: symbol Connector_Generic:Conn_01x03 -> Connector_Generic:Conn_01x10
Connections:
- net labels added: +3V3, +5V, 3V3, PMS7003S_RESET_5, PMS7003S_RXD_7, PMS7003S_SET_10, PMS7003S_TXD_9
- net labels removed: PMS5003S_RX, PMS5003S_TX
- wire segments 4 -> 20
Other:
- note added: "PMS7003S interfacing"

Commit message: updat,
Parts:
- J13: value Conn_01x03 -> PMS7003S_CONN
Changed lines of the file:
@@
 P 3250 3750
 F 0 "J13" H 3330 3792 50  0000 L CNN
-F 1 "Conn_01x03" H 3330 3701 50  0000 L CNN
+F 1 "PMS7003S_CONN" H 3330 3701 50  0000 L CNN
 F 2 "footprint-lib:mpt_0,5%2f3-2,54" H 3250 3750 50  0001 C CNN
 F 3 "~" H 3250 3750 50  0001 C CNN

Commit message: update,
Connections:
- no-connect marks 0 -> 2
Changed lines of the file:
@@
 Wire Wire Line
 	3450 3950 4400 3950
+NoConn ~ 3450 3850
+NoConn ~ 3450 4050
 $EndSCHEMATC

Commit message: update SWD_CONN pinout,
Parts:
- added C?: CP100uf,10V, symbol taobao-cp:CP100uf,10V
Connections:
- wire segments 20 -> 22
Changed lines of the file:
@@
 NoConn ~ 3450 3850
 NoConn ~ 3450 4050
+$Comp
+L power:+5V #PWR?
+U 1 1 5C00525B
+P 2950 2450
+F 0 "#PWR?" H 2950 2300 50  0001 C CNN
+F 1 "+5V" H 2965 2623 50  0000 C CNN
+F 2 "" H 2950 2450 50  0001 C CNN
+F 3 "" H 2950 2450 50  0001 C CNN
+	1    2950 2450
+	1    0    0    -1
+$EndComp
+$Comp
+L power:GND #PWR?
+U 1 1 5C005262
+P 2950 3050
+F 0 "#PWR?" H 2950 2800 50  0001 C CNN
+F 1 "GND" H 2955 2877 50  0000 C CNN
+F 2 "" H 2950 3050 50  0001 C CNN
+F 3 "" H 2950 3050 50  0001 C CNN
+	1    2950 3050
+	1    0    0    -1
+$EndComp
+$Comp
+L taobao-cp:CP100uf,10V C?
+U 1 1 5C005569
+P 2950 2700
+F 0 "C?" H 3038 2746 50  0000 L CNN
+F 1 "CP100uf,10V" H 3038 2655 50  0000 L CNN
+F 2 "" H 2950 2700 50  0001 C CNN
+F 3 "~" H 2950 2700 50  0001 C CNN
+	1    2950 2700
+	1    0    0    -1
+$EndComp
+Wire Wire Line
+	2950 2450 2950 2600
+Wire Wire Line
+	2950 2800 2950 3050
 $EndSCHEMATC

Commit message: update,
Parts:
- gave numbers to parts that had none: 3
Changed lines of the file:
@@
 PMS7003S interfacing
 $Comp
-L power:+3V3 #PWR?
+L power:+3V3 #PWR0127
 U 1 1 5BDB40F7
 P 3550 4550
-F 0 "#PWR?" H 3550 4400 50  0001 C CNN
+F 0 "#PWR0127" H 3550 4400 50  0001 C CNN
 F 1 "+3V3" H 3565 4723 50  0000 C CNN
 F 2 "" H 3550 4550 50  0001 C CNN
@@
 $EndComp
 $Comp
-L taobao-r:R103,0603 R?
+L taobao-r:R103,0603 R25
 U 1 1 5BDB422A
 P 4000 4500
-F 0 "R?" H 3941 4454 50  0000 R CNN
+F 0 "R25" H 3941 4454 50  0000 R CNN
 F 1 "R103,0603" H 3941 4545 50  0000 R CNN
 F 2 "" H 4000 4500 50  0001 C CNN
@@
 	3450 4150 4400 4150
 $Comp
-L power:+5V #PWR?
+L power:+5V #PWR0128
 U 1 1 5BDB473F
 P 3850 3100
-F 0 "#PWR?" H 3850 2950 50  0001 C CNN
+F 0 "#PWR0128" H 3850 2950 50  0001 C CNN
 F 1 "+5V" H 3865 3273 50  0000 C CNN
 F 2 "" H 3850 3100 50  0001 C CNN
@@
 	3850 3350 3450 3350
 $Comp
-L power:GND #PWR?
+L power:GND #PWR0129
 U 1 1 5BDB4D5C
 P 4050 3200
-F 0 "#PWR?" H 4050 2950 50  0001 C CNN
+F 0 "#PWR0129" H 4050 2950 50  0001 C CNN
 F 1 "GND" H 4055 3027 50  0000 C CNN
 F 2 "" H 4050 3200 50  0001 C CNN
@@
 Connection ~ 4050 3550
 $Comp
-L tinkerforge:3V3 #PWR?
+L tinkerforge:3V3 #PWR0130
 U 1 1 5BDB511D
 P 4200 3300
-F 0 "#PWR?" H 4200 3150 50  0001 C CNN
+F 0 "#PWR0130" H 4200 3150 50  0001 C CNN
 F 1 "3V3" H 4215 3473 50  0000 C CNN
 F 2 "" H 4200 3300 50  0000 C CNN
@@
 $EndComp
 $Comp
-L taobao-r:R103,0603 R?
+L taobao-r:R103,0603 R26
 U 1 1 5BDB526A
 P 4200 3550
-F 0 "R?" H 4259 3596 50  0000 L CNN
+F 0 "R26" H 4259 3596 50  0000 L CNN
 F 1 "R103,0603" H 4259 3505 50  0000 L CNN
 F 2 "" H 4200 3550 50  0001 C CNN
@@
 NoConn ~ 3450 4050
 $Comp
-L power:+5V #PWR?
+L power:+5V #PWR0131
 U 1 1 5C00525B
 P 2950 2450
-F 0 "#PWR?" H 2950 2300 50  0001 C CNN
+F 0 "#PWR0131" H 2950 2300 50  0001 C CNN
 F 1 "+5V" H 2965 2623 50  0000 C CNN
 F 2 "" H 2950 2450 50  0001 C CNN
@@
 $EndComp
 $Comp
-L power:GND #PWR?
+L power:GND #PWR0132
 U 1 1 5C005262
 P 2950 3050
-F 0 "#PWR?" H 2950 2800 50  0001 C CNN
+F 0 "#PWR0132" H 2950 2800 50  0001 C CNN
 F 1 "GND" H 2955 2877 50  0000 C CNN
 F 2 "" H 2950 3050 50  0001 C CNN
@@
 $EndComp
 $Comp
-L taobao-cp:CP100uf,10V C?
+L taobao-cp:CP100uf,10V C21
 U 1 1 5C005569
 P 2950 2700
-F 0 "C?" H 3038 2746 50  0000 L CNN
+F 0 "C21" H 3038 2746 50  0000 L CNN
 F 1 "CP100uf,10V" H 3038 2655 50  0000 L CNN
 F 2 "" H 2950 2700 50  0001 C CNN

Commit message: assign footprint,
Parts:
- C21: footprint (none) -> Capacitor_SMD:CP_Elec_6.3x5.2
- R25, R26: footprint (none) -> Resistor_SMD:R_0603_1608Metric_Pad1.05x0.95mm_HandSolder
Changed lines of the file:
@@
 F 0 "R25" H 3941 4454 50  0000 R CNN
 F 1 "R103,0603" H 3941 4545 50  0000 R CNN
-F 2 "" H 4000 4500 50  0001 C CNN
+F 2 "Resistor_SMD:R_0603_1608Metric_Pad1.05x0.95mm_HandSolder" H 4000 4500 50  0001 C CNN
 F 3 "~" H 4000 4500 50  0001 C CNN
 	1    4000 4500
@@
 F 0 "R26" H 4259 3596 50  0000 L CNN
 F 1 "R103,0603" H 4259 3505 50  0000 L CNN
-F 2 "" H 4200 3550 50  0001 C CNN
+F 2 "Resistor_SMD:R_0603_1608Metric_Pad1.05x0.95mm_HandSolder" H 4200 3550 50  0001 C CNN
 F 3 "~" H 4200 3550 50  0001 C CNN
 	1    4200 3550
@@
 F 0 "C21" H 3038 2746 50  0000 L CNN
 F 1 "CP100uf,10V" H 3038 2655 50  0000 L CNN
-F 2 "" H 2950 2700 50  0001 C CNN
+F 2 "Capacitor_SMD:CP_Elec_6.3x5.2" H 2950 2700 50  0001 C CNN
 F 3 "~" H 2950 2700 50  0001 C CNN
 	1    2950 2700

Commit message: init commit,
Parts:
- J13: footprint footprint-lib:mpt_0,5%2f3-2,54 -> footprint-lib:s8b-ph-kl; symbol Connector_Generic:Conn_01x10 -> Connector_Generic:Conn_01x08
Connections:
- net labels removed: +3V3
- wire segments 22 -> 23
- no-connect marks 2 -> 0
Changed lines of the file:
@@
 $EndDescr
 $Comp
-L Connector_Generic:Conn_01x10 J13
+L Connector_Generic:Conn_01x08 J13
 U 1 1 5BDCE1BA
-P 3250 3750
-F 0 "J13" H 3330 3792 50  0000 L CNN
-F 1 "PMS7003S_CONN" H 3330 3701 50  0000 L CNN
-F 2 "footprint-lib:mpt_0,5%2f3-2,54" H 3250 3750 50  0001 C CNN
-F 3 "~" H 3250 3750 50  0001 C CNN
-	1    3250 3750
+P 3250 3650
+F 0 "J13" H 3330 3692 50  0000 L CNN
+F 1 "PMS7003S_CONN" H 3330 3601 50  0000 L CNN
+F 2 "footprint-lib:s8b-ph-kl" H 3250 3650 50  0001 C CNN
+F 3 "~" H 3250 3650 50  0001 C CNN
+	1    3250 3650
 	-1   0    0    -1
 $EndComp
@@
 PMS7003S interfacing
 $Comp
-L power:+3V3 #PWR0127
-U 1 1 5BDB40F7
-P 3550 4550
-F 0 "#PWR0127" H 3550 4400 50  0001 C CNN
-F 1 "+3V3" H 3565 4723 50  0000 C CNN
-F 2 "" H 3550 4550 50  0001 C CNN
-F 3 "" H 3550 4550 50  0001 C CNN
-	1    3550 4550
-	1    0    0    -1
-$EndComp
-$Comp
 L taobao-r:R103,0603 R25
 U 1 1 5BDB422A
-P 4000 4500
-F 0 "R25" H 3941 4454 50  0000 R CNN
-F 1 "R103,0603" H 3941 4545 50  0000 R CNN
-F 2 "Resistor_SMD:R_0603_1608Metric_Pad1.05x0.95mm_HandSolder" H 4000 4500 50  0001 C CNN
-F 3 "~" H 4000 4500 50  0001 C CNN
-	1    4000 4500
+P 4000 4200
+F 0 "R25" H 3941 4154 50  0000 R CNN
+F 1 "R103,0603" H 3941 4245 50  0000 R CNN
+F 2 "Resistor_SMD:R_0603_1608Metric_Pad1.05x0.95mm_HandSolder" H 4000 4200 50  0001 C CNN
+F 3 "~" H 4000 4200 50  0001 C CNN
+	1    4000 4200
 	-1   0    0    1
 $EndComp
 Wire Wire Line
-	3550 4550 3550 4700
-Wire Wire Line
-	4000 4600 4000 4700
-Wire Wire Line
-	3550 4700 4000 4700
-Wire Wire Line
-	3450 4250 4000 4250
-Wire Wire Line
-	4000 4250 4000 4400
+	4000 4300 4000 4400
+Wire Wire Line
+	3450 3950 4000 3950
+Wire Wire Line
+	4000 3950 4000 4100
+Text HLabel 4400 3550 2    50   Input ~ 0
+PMS7003S_RESET_5
 Text HLabel 4400 3750 2    50   Input ~ 0
-PMS7003S_RESET_5
+PMS7003S_RXD_7
+Text HLabel 4400 3850 2    50   Input ~ 0
+PMS7003S_TXD_9
 Text HLabel 4400 3950 2    50   Input ~ 0
-PMS7003S_RXD_7
-Text HLabel 4400 4150 2    50   Input ~ 0
-PMS7003S_TXD_9
-Text HLabel 4400 4250 2    50   Input ~ 0
 PMS7003S_SET_10
 Wire Wire Line
-	4400 4250 4000 4250
-Connection ~ 4000 4250
-Wire Wire Line
-	3450 4150 4400 4150
+	4400 3950 4000 3950
+Connection ~ 4000 3950
+Wire Wire Line
+	3450 3850 4400 3850
 $Comp
 L power:+5V #PWR0128
@@
 	3850 3100 3850 3350
 Wire Wire Line
-	3450 3450 3850 3450
-Wire Wire Line
-	3850 3450 3850 3350
-Connection ~ 3850 3350
-Wire Wire Line
 	3850 3350 3450 3350
 $Comp
 L power:GND #PWR0129
 U 1 1 5BDB4D5C
-P 4050 3200
-F 0 "#PWR0129" H 4050 2950 50  0001 C CNN
-F 1 "GND" H 4055 3027 50  0000 C CNN
-F 2 "" H 4050 3200 50  0001 C CNN
-F 3 "" H 4050 3200 50  0001 C CNN
-	1    4050 3200
+P 4050 3100
+F 0 "#PWR0129" H 4050 2850 50  0001 C CNN
+F 1 "GND" H 4055 2927 50  0000 C CNN
+F 2 "" H 4050 3100 50  0001 C CNN
+F 3 "" H 4050 3100 50  0001 C CNN
+	1    4050 3100
 	-1   0    0    1
 $EndComp
 Wire Wire Line
-	3450 3550 4050 3550
-Wire Wire Line
-	4050 3550 4050 3200
-Wire Wire Line
-	3450 3650 4050 3650
-Wire Wire Line
-	4050 3650 4050 3550
-Connection ~ 4050 3550
+	3450 3450 3600 3450
+Wire Wire Line
+	4050 3450 4050 3100
 $Comp
 L tinkerforge:3V3 #PWR0130
 U 1 1 5BDB511D
-P 4200 3300
-F 0 "#PWR0130" H 4200 3150 50  0001 C CNN
-F 1 "3V3" H 4215 3473 50  0000 C CNN
-F 2 "" H 4200 3300 50  0000 C CNN
-F 3 "" H 4200 3300 50  0000 C CNN
-	1    4200 3300
+P 4200 3100
+F 0 "#PWR0130" H 4200 2950 50  0001 C CNN
+F 1 "3V3" H 4215 3273 50  0000 C CNN
+F 2 "" H 4200 3100 50  0000 C CNN
+F 3 "" H 4200 3100 50  0000 C CNN
+	1    4200 3100
 	1    0    0    -1
 $EndComp
@@
 L taobao-r:R103,0603 R26
 U 1 1 5BDB526A
-P 4200 3550
-F 0 "R26" H 4259 3596 50  0000 L CNN
-F 1 "R103,0603" H 4259 3505 50  0000 L CNN
-F 2 "Resistor_SMD:R_0603_1608Metric_Pad1.05x0.95mm_HandSolder" H 4200 3550 50  0001 C CNN
-F 3 "~" H 4200 3550 50  0001 C CNN
-	1    4200 3550
+P 4200 3350
+F 0 "R26" H 4259 3396 50  0000 L CNN
+F 1 "R103,0603" H 4259 3305 50  0000 L CNN
+F 2 "Resistor_SMD:R_0603_1608Metric_Pad1.05x0.95mm_HandSolder" H 4200 3350 50  0001 C CNN
+F 3 "~" H 4200 3350 50  0001 C CNN
+	1    4200 3350
 	1    0    0    -1
 $EndComp
 Wire Wire Line
-	3450 3750 4200 3750
-Wire Wire Line
-	4200 3750 4200 3650
-Wire Wire Line
-	4200 3300 4200 3450
-Wire Wire Line
-	4200 3750 4400 3750
-Connection ~ 4200 3750
-Wire Wire Line
-	3450 3950 4400 3950
-NoConn ~ 3450 3850
-NoConn ~ 3450 4050
+	3450 3550 3800 3550
+Wire Wire Line
+	4200 3550 4200 3450
+Wire Wire Line
+	4200 3100 4200 3250
+Wire Wire Line
+	4200 3550 4400 3550
+Connection ~ 4200 3550
+Wire Wire Line
+	3450 3750 4400 3750
 $Comp
 L power:+5V #PWR0131
 U 1 1 5C00525B
-P 2950 2450
-F 0 "#PWR0131" H 2950 2300 50  0001 C CNN
-F 1 "+5V" H 2965 2623 50  0000 C CNN
-F 2 "" H 2950 2450 50  0001 C CNN
-F 3 "" H 2950 2450 50  0001 C CNN
-	1    2950 2450
+P 2250 2250
+F 0 "#PWR0131" H 2250 2100 50  0001 C CNN
+F 1 "+5V" H 2265 2423 50  0000 C CNN
+F 2 "" H 2250 2250 50  0001 C CNN
+F 3 "" H 2250 2250 50  0001 C CNN
+	1    2250 2250
 	1    0    0    -1
 $EndComp
@@
 L power:GND #PWR0132
 U 1 1 5C005262
-P 2950 3050
-F 0 "#PWR0132" H 2950 2800 50  0001 C CNN
-F 1 "GND" H 2955 2877 50  0000 C CNN
-F 2 "" H 2950 3050 50  0001 C CNN
-F 3 "" H 2950 3050 50  0001 C CNN
-	1    2950 3050
+P 2250 2850
+F 0 "#PWR0132" H 2250 2600 50  0001 C CNN
+F 1 "GND" H 2255 2677 50  0000 C CNN
+F 2 "" H 2250 2850 50  0001 C CNN
+F 3 "" H 2250 2850 50  0001 C CNN
+	1    2250 2850
 	1    0    0    -1
 $EndComp
@@
 L taobao-cp:CP100uf,10V C21
 U 1 1 5C005569
-P 2950 2700
-F 0 "C21" H 3038 2746 50  0000 L CNN
-F 1 "CP100uf,10V" H 3038 2655 50  0000 L CNN
-F 2 "Capacitor_SMD:CP_Elec_6.3x5.2" H 2950 2700 50  0001 C CNN
-F 3 "~" H 2950 2700 50  0001 C CNN
-	1    2950 2700
+P 2250 2500
+F 0 "C21" H 2338 2546 50  0000 L CNN
+F 1 "CP100uf,10V" H 2338 2455 50  0000 L CNN
+F 2 "Capacitor_SMD:CP_Elec_6.3x5.2" H 2250 2500 50  0001 C CNN
+F 3 "~" H 2250 2500 50  0001 C CNN
+	1    2250 2500
 	1    0    0    -1
 $EndComp
 Wire Wire Line
-	2950 2450 2950 2600
-Wire Wire Line
-	2950 2800 2950 3050
+	2250 2250 2250 2400
+Wire Wire Line
+	2250 2600 2250 2850
+Text HLabel 4400 3650 2    50   Input ~ 0
+PMS7003S_RXD_7
+Wire Wire Line
+	3450 3650 4400 3650
+Wire Wire Line
+	3800 3550 3800 4400
+Connection ~ 3800 3550
+Wire Wire Line
+	3800 3550 4200 3550
+Wire Wire Line
+	3800 4400 4000 4400
+Wire Wire Line
+	3600 3450 3600 4050
+Wire Wire Line
+	3600 4050 3450 4050
+Connection ~ 3600 3450
+Wire Wire Line
+	3600 3450 4050 3450
 $EndSCHEMATC

Commit message: update,
Connections:
- wire segments 23 -> 22
Changed lines of the file:
@@
 F 3 "~" H 4000 4200 50  0001 C CNN
 	1    4000 4200
-	-1   0    0    1
+	-1   0    0    -1
 $EndComp
 Wire Wire Line
 	4000 4300 4000 4400
-Wire Wire Line
-	3450 3950 4000 3950
-Wire Wire Line
-	4000 3950 4000 4100
 Text HLabel 4400 3550 2    50   Input ~ 0
 PMS7003S_RESET_5
+Text HLabel 4400 3650 2    50   Input ~ 0
+PMS7003S_RXD_7
 Text HLabel 4400 3750 2    50   Input ~ 0
-PMS7003S_RXD_7
+PMS7003S_TXD_9
 Text HLabel 4400 3850 2    50   Input ~ 0
-PMS7003S_TXD_9
-Text HLabel 4400 3950 2    50   Input ~ 0
 PMS7003S_SET_10
 Wire Wire Line
-	4400 3950 4000 3950
-Connection ~ 4000 3950
-Wire Wire Line
-	3450 3850 4400 3850
+	3450 3750 4400 3750
 $Comp
 L power:+5V #PWR0128
@@
 Connection ~ 4200 3550
 Wire Wire Line
-	3450 3750 4400 3750
+	3450 3650 4400 3650
 $Comp
 L power:+5V #PWR0131
@@
 Wire Wire Line
 	2250 2600 2250 2850
-Text HLabel 4400 3650 2    50   Input ~ 0
-PMS7003S_RXD_7
-Wire Wire Line
-	3450 3650 4400 3650
 Wire Wire Line
 	3800 3550 3800 4400
@@
 Wire Wire Line
 	3600 3450 4050 3450
+Wire Wire Line
+	3450 3850 4000 3850
+Wire Wire Line
+	4400 3850 4000 3850
+Connection ~ 4000 3850
+Wire Wire Line
+	4000 3850 4000 4100
 $EndSCHEMATC
