File: pcb/PMS5003S_interface.sch (KiCad schematic (older format))
At the start: 4 parts, among them J13 PMS7003S_CONN

Commit message: fix power symbol,
Connections:
- net labels added: +3V3
- net labels removed: 3V3
Changed lines of the file:
@@
 	4050 3450 4050 3100
-$Comp
-L tinkerforge:3V3 #PWR0130
-U 1 1 5BDB511D
-P 4200 3100
-F 0 "#PWR0130" H 4200 2950 50  0001 C CNN
-F 1 "3V3" H 4215 3273 50  0000 C CNN
-F 2 "" H 4200 3100 50  0000 C CNN
-F 3 "" H 4200 3100 50  0000 C CNN
-	1    4200 3100
-	1    0    0    -1
-$EndComp
 $Comp
 L taobao-r:R103,0603 R26
@@
 Wire Wire Line
 	4000 3850 4000 4100
+$Comp
+L power:+3V3 #PWR?
+U 1 1 5BDC6BC2
+P 4200 3100
+F 0 "#PWR?" H 4200 2950 50  0001 C CNN
+F 1 "+3V3" H 4250 3300 50  0000 C CNN
+F 2 "" H 4200 3100 50  0001 C CNN
+F 3 "" H 4200 3100 50  0001 C CNN
+	1    4200 3100
+	1    0    0    -1
+$EndComp
 $EndSCHEMATC

Commit message: update,
Connections:
- wire segments 22 -> 21
Changed lines of the file:
@@
 $EndComp
-Wire Wire Line
-	3450 3550 3800 3550
 Wire Wire Line
 	4200 3550 4200 3450
@@
 	2250 2600 2250 2850
 Wire Wire Line
-	3800 3550 3800 4400
-Connection ~ 3800 3550
-Wire Wire Line
-	3800 3550 4200 3550
-Wire Wire Line
-	3800 4400 4000 4400
-Wire Wire Line
 	3600 3450 3600 4050
 Wire Wire Line
@@
 	1    0    0    -1
 $EndComp
+Wire Wire Line
+	3450 3550 4200 3550
+$Comp
+L power:+3V3 #PWR0133
+U 1 1 5BEE893F
+P 3700 4300
+F 0 "#PWR0133" H 3700 4150 50  0001 C CNN
+F 1 "+3V3" H 3750 4500 50  0000 C CNN
+F 2 "" H 3700 4300 50  0001 C CNN
+F 3 "" H 3700 4300 50  0001 C CNN
+	1    3700 4300
+	1    0    0    -1
+$EndComp
+Wire Wire Line
+	3700 4300 3700 4400
+Wire Wire Line
+	3700 4400 4000 4400
 $EndSCHEMATC

Commit message: update,
Parts:
- renumbered C21 to C?, J13 to J?, R25 to R?, R26 to R?
Changed lines of the file:
@@
 EESchema Schematic File Version 4
+LIBS:backplane-cache
 LIBS:stm32_bottom_board_respin-cache
 EELAYER 26 0
@@
 $Descr A4 11693 8268
 encoding utf-8
-Sheet 8 8
+Sheet 9 9
 Title ""
 Date ""
@@
 $EndDescr
 $Comp
-L Connector_Generic:Conn_01x08 J13
+L Connector_Generic:Conn_01x08 J?
 U 1 1 5BDCE1BA
 P 3250 3650
-F 0 "J13" H 3330 3692 50  0000 L CNN
+F 0 "J?" H 3330 3692 50  0000 L CNN
 F 1 "PMS7003S_CONN" H 3330 3601 50  0000 L CNN
 F 2 "footprint-lib:s8b-ph-kl" H 3250 3650 50  0001 C CNN
@@
 PMS7003S interfacing
 $Comp
-L taobao-r:R103,0603 R25
+L taobao-r:R103,0603 R?
 U 1 1 5BDB422A
 P 4000 4200
-F 0 "R25" H 3941 4154 50  0000 R CNN
+F 0 "R?" H 3941 4154 50  0000 R CNN
 F 1 "R103,0603" H 3941 4245 50  0000 R CNN
 F 2 "Resistor_SMD:R_0603_1608Metric_Pad1.05x0.95mm_HandSolder" H 4000 4200 50  0001 C CNN
@@
 	3450 3750 4400 3750
 $Comp
-L power:+5V #PWR0128
+L power:+5V #PWR?
 U 1 1 5BDB473F
 P 3850 3100
-F 0 "#PWR0128" H 3850 2950 50  0001 C CNN
+F 0 "#PWR?" H 3850 2950 50  0001 C CNN
 F 1 "+5V" H 3865 3273 50  0000 C CNN
 F 2 "" H 3850 3100 50  0001 C CNN
@@
 	3850 3350 3450 3350
 $Comp
-L power:GND #PWR0129
+L power:GND #PWR?
 U 1 1 5BDB4D5C
 P 4050 3100
-F 0 "#PWR0129" H 4050 2850 50  0001 C CNN
+F 0 "#PWR?" H 4050 2850 50  0001 C CNN
 F 1 "GND" H 4055 2927 50  0000 C CNN
 F 2 "" H 4050 3100 50  0001 C CNN
@@
 	4050 3450 4050 3100
 $Comp
-L taobao-r:R103,0603 R26
+L taobao-r:R103,0603 R?
 U 1 1 5BDB526A
 P 4200 3350
-F 0 "R26" H 4259 3396 50  0000 L CNN
+F 0 "R?" H 4259 3396 50  0000 L CNN
 F 1 "R103,0603" H 4259 3305 50  0000 L CNN
 F 2 "Resistor_SMD:R_0603_1608Metric_Pad1.05x0.95mm_HandSolder" H 4200 3350 50  0001 C CNN
@@
 	3450 3650 4400 3650
 $Comp
-L power:+5V #PWR0131
+L power:+5V #PWR?
 U 1 1 5C00525B
 P 2250 2250
-F 0 "#PWR0131" H 2250 2100 50  0001 C CNN
+F 0 "#PWR?" H 2250 2100 50  0001 C CNN
 F 1 "+5V" H 2265 2423 50  0000 C CNN
 F 2 "" H 2250 2250 50  0001 C CNN
@@
 $EndComp
 $Comp
-L power:GND #PWR0132
+L power:GND #PWR?
 U 1 1 5C005262
 P 2250 2850
-F 0 "#PWR0132" H 2250 2600 50  0001 C CNN
+F 0 "#PWR?" H 2250 2600 50  0001 C CNN
 F 1 "GND" H 2255 2677 50  0000 C CNN
 F 2 "" H 2250 2850 50  0001 C CNN
@@
 $EndComp
 $Comp
-L taobao-cp:CP100uf,10V C21
+L taobao-cp:CP100uf,10V C?
 U 1 1 5C005569
 P 2250 2500
-F 0 "C21" H 2338 2546 50  0000 L CNN
+F 0 "C?" H 2338 2546 50  0000 L CNN
 F 1 "CP100uf,10V" H 2338 2455 50  0000 L CNN
 F 2 "Capacitor_SMD:CP_Elec_6.3x5.2" H 2250 2500 50  0001 C CNN
@@
 	4000 3850 4000 4100
 $Comp
-L power:+3V3 #PWR0127
+L power:+3V3 #PWR?
 U 1 1 5BDC6BC2
 P 4200 3100
-F 0 "#PWR0127" H 4200 2950 50  0001 C CNN
+F 0 "#PWR?" H 4200 2950 50  0001 C CNN
 F 1 "+3V3" H 4250 3300 50  0000 C CNN
 F 2 "" H 4200 3100 50  0001 C CNN
@@
 	3450 3550 4200 3550
 $Comp
-L power:+3V3 #PWR0133
+L power:+3V3 #PWR?
 U 1 1 5BEE893F
 P 3700 4300
-F 0 "#PWR0133" H 3700 4150 50  0001 C CNN
+F 0 "#PWR?" H 3700 4150 50  0001 C CNN
 F 1 "+3V3" H 3750 4500 50  0000 C CNN
 F 2 "" H 3700 4300 50  0001 C CNN
