File: pcb/STM32_CORE.sch (KiCad schematic (older format))
At the start: 34 parts, among them J12 POWER, J6 Conn_01x14, J7 Conn_01x12, J8 Conn_01x15, SW1 SW_Push, U3 STM32F103C8T6, U4 AMS1117-3.3, Y1 O8M, Y2 O_EPSON_32.768K

Commit message: update,
Parts:
- gave numbers to parts that had none: 1
Changed lines of the file:
@@
 	1250 1900 1250 2150
 $Comp
-L power:GND #PWR?
+L power:GND #PWR0125
 U 1 1 5BEEEFFB
 P 1250 1200
-F 0 "#PWR?" H 1250 950 50  0001 C CNN
+F 0 "#PWR0125" H 1250 950 50  0001 C CNN
 F 1 "GND" H 1255 1027 50  0000 C CNN
 F 2 "" H 1250 1200 50  0001 C CNN
@@
 	1250 1400 1250 1200
 $Comp
-L power:+3V3 #PWR?
+L power:+3V3 #PWR0126
 U 1 1 5BF1D935
 P 1450 1150
-F 0 "#PWR?" H 1450 1000 50  0001 C CNN
+F 0 "#PWR0126" H 1450 1000 50  0001 C CNN
 F 1 "+3V3" H 1500 1350 50  0000 C CNN
 F 2 "" H 1450 1150 50  0001 C CNN
@@
 	1350 1400 1350 950
 $Comp
-L Connector_Generic:Conn_02x04_Odd_Even J?
+L Connector_Generic:Conn_02x04_Odd_Even J15
 U 1 1 5BFAD103
 P 1250 1600
-F 0 "J?" V 1254 1312 50  0000 R CNN
+F 0 "J15" V 1254 1312 50  0000 R CNN
 F 1 "SWD_CONN" V 1345 1312 50  0000 R CNN
 F 2 "" H 1250 1600 50  0001 C CNN

Commit message: assign footprint,
Parts:
- J15: footprint (none) -> Connector_PinSocket_2.54mm:PinSocket_2x04_P2.54mm_Vertical
- R10, R11, R12, R13, R9: footprint Resistor_SMD:R_0805_2012Metric_Pad1.15x1.40mm_HandSolder -> Resistor_SMD:R_0603_1608Metric_Pad1.05x0.95mm_HandSolder
Changed lines of the file:
@@
 F 0 "R11" H 14259 5346 50  0000 L CNN
 F 1 "R511" H 14259 5255 50  0000 L CNN
-F 2 "Resistor_SMD:R_0805_2012Metric_Pad1.15x1.40mm_HandSolder" H 14200 5300 50  0001 C CNN
+F 2 "Resistor_SMD:R_0603_1608Metric_Pad1.05x0.95mm_HandSolder" H 14200 5300 50  0001 C CNN
 F 3 "~" H 14200 5300 50  0001 C CNN
 	1    14200 5300
@@
 F 0 "R13" H 14909 5346 50  0000 L CNN
 F 1 "R511" H 14909 5255 50  0000 L CNN
-F 2 "Resistor_SMD:R_0805_2012Metric_Pad1.15x1.40mm_HandSolder" H 14850 5300 50  0001 C CNN
+F 2 "Resistor_SMD:R_0603_1608Metric_Pad1.05x0.95mm_HandSolder" H 14850 5300 50  0001 C CNN
 F 3 "~" H 14850 5300 50  0001 C CNN
 	1    14850 5300
@@
 F 0 "R12" H 14559 2446 50  0000 L CNN
 F 1 "R103" H 14559 2355 50  0000 L CNN
-F 2 "Resistor_SMD:R_0805_2012Metric_Pad1.15x1.40mm_HandSolder" H 14500 2400 50  0001 C CNN
+F 2 "Resistor_SMD:R_0603_1608Metric_Pad1.05x0.95mm_HandSolder" H 14500 2400 50  0001 C CNN
 F 3 "~" H 14500 2400 50  0001 C CNN
 	1    14500 2400
@@
 F 0 "R9" V 11304 1800 50  0000 C CNN
 F 1 "R104" V 11395 1800 50  0000 C CNN
-F 2 "Resistor_SMD:R_0805_2012Metric_Pad1.15x1.40mm_HandSolder" H 11500 1800 50  0001 C CNN
+F 2 "Resistor_SMD:R_0603_1608Metric_Pad1.05x0.95mm_HandSolder" H 11500 1800 50  0001 C CNN
 F 3 "~" H 11500 1800 50  0001 C CNN
 	1    11500 1800
@@
 F 0 "R10" V 12954 1800 50  0000 C CNN
 F 1 "R104" V 13045 1800 50  0000 C CNN
-F 2 "Resistor_SMD:R_0805_2012Metric_Pad1.15x1.40mm_HandSolder" H 13150 1800 50  0001 C CNN
+F 2 "Resistor_SMD:R_0603_1608Metric_Pad1.05x0.95mm_HandSolder" H 13150 1800 50  0001 C CNN
 F 3 "~" H 13150 1800 50  0001 C CNN
 	1    13150 1800
@@
 F 0 "J15" V 1254 1312 50  0000 R CNN
 F 1 "SWD_CONN" V 1345 1312 50  0000 R CNN
-F 2 "" H 1250 1600 50  0001 C CNN
+F 2 "Connector_PinSocket_2.54mm:PinSocket_2x04_P2.54mm_Vertical" H 1250 1600 50  0001 C CNN
 F 3 "~" H 1250 1600 50  0001 C CNN
 	1    1250 1600

Commit message: update,
Parts:
- J12: footprint w_conn_mkds:mkds_1,5-3 -> footprint-lib:s3b-ph-kl
Changed lines of the file:
@@
 F 0 "J12" H 1520 5325 50  0000 C CNN
 F 1 "POWER" H 1520 5416 50  0000 C CNN
-F 2 "w_conn_mkds:mkds_1,5-3" H 1600 5650 50  0001 C CNN
+F 2 "footprint-lib:s3b-ph-kl" H 1600 5650 50  0001 C CNN
 F 3 "~" H 1600 5650 50  0001 C CNN
 	1    1600 5650

Commit message: update,
Parts:
- removed JP1: Jumper_NO_Small, Jumper:SolderJumper-2_P1.3mm_Open_TrianglePad1.0x1.5mm, symbol Device:Jumper_NO_Small
Connections:
- wire segments 201 -> 200
Changed lines of the file:
@@
 Wire Wire Line
 	6100 1100 6100 1250
-$Comp
-L Device:Jumper_NO_Small JP1
-U 1 1 5BE05EFF
-P 2250 4350
-F 0 "JP1" H 2250 4535 50  0000 C CNN
-F 1 "Jumper_NO_Small" H 2250 4444 50  0000 C CNN
-F 2 "Jumper:SolderJumper-2_P1.3mm_Open_TrianglePad1.0x1.5mm" H 2250 4350 50  0001 C CNN
-F 3 "~" H 2250 4350 50  0001 C CNN
-	1    2250 4350
-	1    0    0    1
-$EndComp
-Wire Wire Line
-	1950 4350 2150 4350
-Wire Wire Line
-	2350 4350 2500 4350
 Text Label 2250 4150 2    50   ~ 0
 PB9
@@
 Text Notes 1350 6300 0    50   ~ 0
 update to incidate the +3V3 is not necessary
+Wire Wire Line
+	1950 4350 2500 4350
 $EndSCHEMATC

Commit message: fix power symbol,
Changed lines of the file:
@@
 	2350 5650 1800 5650
-$Comp
-L tinkerforge:+5V #PWR0114
-U 1 1 5BD3EFE4
-P 14200 4750
-F 0 "#PWR0114" H 14200 4600 50  0001 C CNN
-F 1 "+5V" H 14215 4923 50  0000 C CNN
-F 2 "" H 14200 4750 50  0000 C CNN
-F 3 "" H 14200 4750 50  0000 C CNN
-	1    14200 4750
-	1    0    0    -1
-$EndComp
 $Comp
 L taobao-osc:O_EPSON_32.768K Y2
@@
 Wire Wire Line
 	1950 4350 2500 4350
+$Comp
+L power:+5V #PWR?
+U 1 1 5BDC3128
+P 14200 4750
+F 0 "#PWR?" H 14200 4600 50  0001 C CNN
+F 1 "+5V" H 14250 4950 50  0000 C CNN
+F 2 "" H 14200 4750 50  0001 C CNN
+F 3 "" H 14200 4750 50  0001 C CNN
+	1    14200 4750
+	1    0    0    -1
+$EndComp
 $EndSCHEMATC

Commit message: update,
Parts:
- removed J15: SWD_CONN, Connector_PinSocket_2.54mm:PinSocket_2x04_P2.54mm_Vertical, symbol Connector_Generic:Conn_02x04_Odd_Even
- added U7: waveshare-swd-pinsocket, footprint-lib.pretty:waveshare-swd-pinsocket, symbol taobao-components:waveshare-swd-pinsocket
Changed lines of the file:
@@
 L power:GND #PWR0109
 U 1 1 5BD06547
-P 1250 2150
-F 0 "#PWR0109" H 1250 1900 50  0001 C CNN
-F 1 "GND" H 1255 1977 50  0000 C CNN
-F 2 "" H 1250 2150 50  0001 C CNN
-F 3 "" H 1250 2150 50  0001 C CNN
-	1    1250 2150
-	-1   0    0    -1
-$EndComp
-Text Label 1150 2550 1    50   ~ 0
+P 1050 950
+F 0 "#PWR0109" H 1050 700 50  0001 C CNN
+F 1 "GND" H 1055 777 50  0000 C CNN
+F 2 "" H 1050 950 50  0001 C CNN
+F 3 "" H 1050 950 50  0001 C CNN
+	1    1050 950
+	0    1    -1   0
+$EndComp
+Text Label 650  850  0    50   ~ 0
 SWIO
-Text Label 1350 2550 1    50   ~ 0
+Text Label 650  1050 0    50   ~ 0
 SWCLK
 Wire Wire Line
-	1350 1900 1350 2550
-Wire Wire Line
-	1150 1900 1150 2550
+	1300 1050 650  1050
+Wire Wire Line
+	1300 850  650  850
 $Comp
 L power:+3V3 #PWR0110
 U 1 1 5BD06554
-P 1450 2150
-F 0 "#PWR0110" H 1450 2000 50  0001 C CNN
-F 1 "+3V3" H 1500 2350 50  0000 C CNN
-F 2 "" H 1450 2150 50  0001 C CNN
-F 3 "" H 1450 2150 50  0001 C CNN
-	1    1450 2150
-	-1   0    0    1
+P 1050 1150
+F 0 "#PWR0110" H 1050 1000 50  0001 C CNN
+F 1 "+3V3" H 1100 1350 50  0000 C CNN
+F 2 "" H 1050 1150 50  0001 C CNN
+F 3 "" H 1050 1150 50  0001 C CNN
+	1    1050 1150
+	0    -1   -1   0
 $EndComp
 $Comp
@@
 STM32_FAN_RPM
 Wire Wire Line
-	1450 1900 1450 2150
-Wire Wire Line
-	1250 1900 1250 2150
+	1300 1150 1050 1150
+Wire Wire Line
+	1300 950  1050 950
 $Comp
 L power:GND #PWR0125
 U 1 1 5BEEEFFB
-P 1250 1200
-F 0 "#PWR0125" H 1250 950 50  0001 C CNN
-F 1 "GND" H 1255 1027 50  0000 C CNN
-F 2 "" H 1250 1200 50  0001 C CNN
-F 3 "" H 1250 1200 50  0001 C CNN
-	1    1250 1200
-	1    0    0    1
-$EndComp
-Wire Wire Line
-	1250 1400 1250 1200
+P 2500 950
+F 0 "#PWR0125" H 2500 700 50  0001 C CNN
+F 1 "GND" H 2505 777 50  0000 C CNN
+F 2 "" H 2500 950 50  0001 C CNN
+F 3 "" H 2500 950 50  0001 C CNN
+	1    2500 950
+	0    -1   1    0
+$EndComp
+Wire Wire Line
+	2300 950  2500 950
 $Comp
 L power:+3V3 #PWR0126
 U 1 1 5BF1D935
-P 1450 1150
-F 0 "#PWR0126" H 1450 1000 50  0001 C CNN
-F 1 "+3V3" H 1500 1350 50  0000 C CNN
-F 2 "" H 1450 1150 50  0001 C CNN
-F 3 "" H 1450 1150 50  0001 C CNN
-	1    1450 1150
-	1    0    0    -1
-$EndComp
-Wire Wire Line
-	1450 1400 1450 1150
-Text Label 1150 950  3    50   ~ 0
+P 2550 1150
+F 0 "#PWR0126" H 2550 1000 50  0001 C CNN
+F 1 "+3V3" H 2600 1350 50  0000 C CNN
+F 2 "" H 2550 1150 50  0001 C CNN
+F 3 "" H 2550 1150 50  0001 C CNN
+	1    2550 1150
+	0    1    1    0
+$EndComp
+Wire Wire Line
+	2300 1150 2550 1150
+Text Label 2750 850  2    50   ~ 0
 RST
 Wire Wire Line
-	1150 1400 1150 950
-Text Label 1350 950  3    50   ~ 0
+	2300 850  2750 850
+Text Label 2750 1050 2    50   ~ 0
 SWIM
 Wire Wire Line
-	1350 1400 1350 950
-$Comp
-L Connector_Generic:Conn_02x04_Odd_Even J15
-U 1 1 5BFAD103
-P 1250 1600
-F 0 "J15" V 1254 1312 50  0000 R CNN
-F 1 "SWD_CONN" V 1345 1312 50  0000 R CNN
-F 2 "Connector_PinSocket_2.54mm:PinSocket_2x04_P2.54mm_Vertical" H 1250 1600 50  0001 C CNN
-F 3 "~" H 1250 1600 50  0001 C CNN
-	1    1250 1600
-	0    -1   1    0
-$EndComp
+	2300 1050 2750 1050
 Text Notes 10950 5300 2    50   ~ 0
 to stablize power from power supply ->
@@
 	1950 4350 2500 4350
 $Comp
-L power:+5V #PWR?
+L power:+5V #PWR0114
 U 1 1 5BDC3128
 P 14200 4750
-F 0 "#PWR?" H 14200 4600 50  0001 C CNN
+F 0 "#PWR0114" H 14200 4600 50  0001 C CNN
 F 1 "+5V" H 14250 4950 50  0000 C CNN
 F 2 "" H 14200 4750 50  0001 C CNN
@@
 	1    0    0    -1
 $EndComp
+$Comp
+L taobao-components:waveshare-swd-pinsocket U7
+U 1 1 5BDC76BE
+P 1800 1000
+F 0 "U7" H 1800 1450 50  0000 C CNN
+F 1 "waveshare-swd-pinsocket" H 1800 1350 50  0000 C CNN
+F 2 "footprint-lib.pretty:waveshare-swd-pinsocket" H 1750 750 50  0001 C CNN
+F 3 "" H 1750 750 50  0001 C CNN
+	1    1800 1000
+	1    0    0    -1
+$EndComp

Commit message: basic rout complete,
Changed lines of the file:
@@
 $EndComp
 Wire Wire Line
-	2500 4350 2500 4500
+	2500 3050 2500 2900
 $Comp
 L power:GND #PWR018
@@
 L power:+5V #PWR021
 U 1 1 5BCACB86
-P 2500 4500
-F 0 "#PWR021" H 2500 4350 50  0001 C CNN
-F 1 "+5V" H 2500 4700 50  0000 C CNN
-F 2 "" H 2500 4500 50  0001 C CNN
-F 3 "" H 2500 4500 50  0001 C CNN
-	1    2500 4500
-	1    0    0    1
+P 2500 2900
+F 0 "#PWR021" H 2500 2750 50  0001 C CNN
+F 1 "+5V" H 2500 3100 50  0000 C CNN
+F 2 "" H 2500 2900 50  0001 C CNN
+F 3 "" H 2500 2900 50  0001 C CNN
+	1    2500 2900
+	1    0    0    -1
 $EndComp
 $Comp
@@
 update to incidate the +3V3 is not necessary
 Wire Wire Line
-	1950 4350 2500 4350
+	1950 3050 2500 3050
 $Comp
 L power:+5V #PWR0114

Commit message: update,
Parts:
- added D9: LED_GREEN, LED_SMD:LED_0603_1608Metric_Pad1.05x0.95mm_HandSolder, symbol taobao-components:LED_GREEN
- added R27: R102,0603, Resistor_SMD:R_0603_1608Metric_Pad1.05x0.95mm_HandSolder, symbol taobao-r:R102,0603
Connections:
- wire segments 200 -> 203
Changed lines of the file:
@@
 Wire Wire Line
 	6100 2100 6100 2000
+Text GLabel 10000 3050 2    50   Input ~ 0
+STM32_PMS7003S_RESET
 Text GLabel 10000 2950 2    50   Input ~ 0
-STM32_PMS7003S_RESET
-Text GLabel 10000 3050 2    50   Input ~ 0
 STM32_PMS7003S_SET
 Text GLabel 8350 1250 1    50   Input ~ 0
@@
 	1    0    0    -1
 $EndComp
+$Comp
+L power:GND #PWR0130
+U 1 1 5BE8F4B2
+P 5500 3450
+F 0 "#PWR0130" H 5500 3200 50  0001 C CNN
+F 1 "GND" H 5505 3277 50  0000 C CNN
+F 2 "" H 5500 3450 50  0001 C CNN
+F 3 "" H 5500 3450 50  0001 C CNN
+	1    5500 3450
+	1    0    0    -1
+$EndComp
+Text Label 5500 2500 3    50   ~ 0
+PC13
+$Comp
+L taobao-r:R102,0603 R27
+U 1 1 5BEA8193
+P 5500 2900
+F 0 "R27" H 5600 2950 50  0000 L CNN
+F 1 "R102,0603" H 5600 2900 50  0000 L CNN
+F 2 "Resistor_SMD:R_0603_1608Metric_Pad1.05x0.95mm_HandSolder" H 5500 2900 50  0001 C CNN
+F 3 "~" H 5500 2900 50  0001 C CNN
+	1    5500 2900
+	1    0    0    -1
+$EndComp
+$Comp
+L taobao-components:LED_GREEN D9
+U 1 1 5BEA8346
+P 5500 3150
+F 0 "D9" V 5550 3050 50  0000 R CNN
+F 1 "LED_GREEN" V 5500 3050 50  0000 R CNN
+F 2 "LED_SMD:LED_0603_1608Metric_Pad1.05x0.95mm_HandSolder" V 5500 3150 50  0001 C CNN
+F 3 "" V 5500 3150 50  0001 C CNN
+	1    5500 3150
+	0    -1   -1   0
+$EndComp
+Wire Wire Line
+	5500 2500 5500 2800
+Wire Wire Line
+	5500 3000 5500 3050
+Wire Wire Line
+	5500 3250 5500 3450
 $EndSCHEMATC
