File: pcb/FAN_PWM_DRIVER.sch (KiCad schematic (older format))
At the start: 3 parts, among them Q2 SS9013_J3

Commit message: update,
Parts:
- added D?: 1N4148, symbol taobao-d:1N4148
- added R?: R103, symbol taobao-r:R103
Connections:
- net labels added: FAN_RPM, STM32_FAN_RPM
- wire segments 9 -> 14
Changed lines of the file:
@@
 	1    0    0    -1
 $EndComp
+Text HLabel 1750 3900 0    50   Input ~ 0
+STM32_FAN_RPM
+$Comp
+L power:VDD #PWR?
+U 1 1 5BDC0579
+P 2350 3350
+F 0 "#PWR?" H 2350 3200 50  0001 C CNN
+F 1 "VDD" H 2367 3523 50  0000 C CNN
+F 2 "" H 2350 3350 50  0001 C CNN
+F 3 "" H 2350 3350 50  0001 C CNN
+	1    2350 3350
+	1    0    0    -1
+$EndComp
+$Comp
+L taobao-r:R103 R?
+U 1 1 5BDC0610
+P 2350 3600
+F 0 "R?" H 2409 3646 50  0000 L CNN
+F 1 "R103" H 2409 3555 50  0000 L CNN
+F 2 "" H 2350 3600 50  0001 C CNN
+F 3 "~" H 2350 3600 50  0001 C CNN
+	1    2350 3600
+	1    0    0    -1
+$EndComp
+$Comp
+L taobao-d:1N4148 D?
+U 1 1 5BDC3BB5
+P 2550 3900
+F 0 "D?" H 2550 3695 50  0000 C CNN
+F 1 "1N4148" H 2550 3786 50  0000 C CNN
+F 2 "" V 2550 3900 50  0001 C CNN
+F 3 "~" V 2550 3900 50  0001 C CNN
+	1    2550 3900
+	-1   0    0    1
+$EndComp
+Wire Wire Line
+	2350 3350 2350 3500
+Wire Wire Line
+	1750 3900 2350 3900
+Wire Wire Line
+	2350 3900 2350 3700
+Wire Wire Line
+	2350 3900 2450 3900
+Connection ~ 2350 3900
+Text HLabel 3750 3900 2    50   Input ~ 0
+FAN_RPM
+Wire Wire Line
+	2650 3900 3750 3900
 $EndSCHEMATC

Commit message: update,
Connections:
- net labels removed: FAN_PWM_GND, FAN_PWM_OUTPUT_GND
- wire segments 14 -> 12
Changed lines of the file:
@@
 	1    0    0    -1
 $EndComp
-Wire Wire Line
-	2850 2400 2850 2550
 Text Label 3650 1850 2    50   ~ 0
 FAN_PWM_OUTPUT
@@
 Wire Wire Line
 	2850 1850 2850 2000
-Text Label 3750 2550 2    50   ~ 0
-FAN_PWM_OUTPUT_GND
-Wire Wire Line
-	3750 2550 2850 2550
-Connection ~ 2850 2550
-Wire Wire Line
-	2850 2550 2850 2700
 Text HLabel 3750 1850 2    50   Input ~ 0
 FAN_PWM_OUTPUT
-Text HLabel 3750 2550 2    50   Input ~ 0
-FAN_PWM_GND
 $Comp
 L power:VDD #PWR015
@@
 Wire Wire Line
 	2650 3900 3750 3900
+Wire Wire Line
+	2850 2400 2850 2700
 $EndSCHEMATC

Commit message: update,
Parts:
- gave numbers to parts that had none: 2
Changed lines of the file:
@@
 STM32_FAN_RPM
 $Comp
-L power:VDD #PWR?
+L power:VDD #PWR0124
 U 1 1 5BDC0579
 P 2350 3350
-F 0 "#PWR?" H 2350 3200 50  0001 C CNN
+F 0 "#PWR0124" H 2350 3200 50  0001 C CNN
 F 1 "VDD" H 2367 3523 50  0000 C CNN
 F 2 "" H 2350 3350 50  0001 C CNN
@@
 $EndComp
 $Comp
-L taobao-r:R103 R?
+L taobao-r:R103 R24
 U 1 1 5BDC0610
 P 2350 3600
-F 0 "R?" H 2409 3646 50  0000 L CNN
+F 0 "R24" H 2409 3646 50  0000 L CNN
 F 1 "R103" H 2409 3555 50  0000 L CNN
 F 2 "" H 2350 3600 50  0001 C CNN
@@
 $EndComp
 $Comp
-L taobao-d:1N4148 D?
+L taobao-d:1N4148 D8
 U 1 1 5BDC3BB5
 P 2550 3900
-F 0 "D?" H 2550 3695 50  0000 C CNN
+F 0 "D8" H 2550 3695 50  0000 C CNN
 F 1 "1N4148" H 2550 3786 50  0000 C CNN
 F 2 "" V 2550 3900 50  0001 C CNN

Commit message: assign footprint,
Parts:
- D8: footprint (none) -> Diode_SMD:D_SOD-323_HandSoldering
- R24: footprint (none) -> Resistor_SMD:R_0603_1608Metric_Pad1.05x0.95mm_HandSolder
- R7, R8: footprint Resistor_SMD:R_0805_2012Metric_Pad1.15x1.40mm_HandSolder -> Resistor_SMD:R_0603_1608Metric_Pad1.05x0.95mm_HandSolder
Changed lines of the file:
@@
 F 0 "R7" V 1954 2200 50  0000 C CNN
 F 1 "R471" V 2045 2200 50  0000 C CNN
-F 2 "Resistor_SMD:R_0805_2012Metric_Pad1.15x1.40mm_HandSolder" H 2150 2200 50  0001 C CNN
+F 2 "Resistor_SMD:R_0603_1608Metric_Pad1.05x0.95mm_HandSolder" H 2150 2200 50  0001 C CNN
 F 3 "~" H 2150 2200 50  0001 C CNN
 	1    2150 2200
@@
 F 0 "R8" H 2909 1646 50  0000 L CNN
 F 1 "R331" H 2909 1555 50  0000 L CNN
-F 2 "Resistor_SMD:R_0805_2012Metric_Pad1.15x1.40mm_HandSolder" H 2850 1600 50  0001 C CNN
+F 2 "Resistor_SMD:R_0603_1608Metric_Pad1.05x0.95mm_HandSolder" H 2850 1600 50  0001 C CNN
 F 3 "~" H 2850 1600 50  0001 C CNN
 	1    2850 1600
@@
 F 0 "R24" H 2409 3646 50  0000 L CNN
 F 1 "R103" H 2409 3555 50  0000 L CNN
-F 2 "" H 2350 3600 50  0001 C CNN
+F 2 "Resistor_SMD:R_0603_1608Metric_Pad1.05x0.95mm_HandSolder" H 2350 3600 50  0001 C CNN
 F 3 "~" H 2350 3600 50  0001 C CNN
 	1    2350 3600
@@
 F 0 "D8" H 2550 3695 50  0000 C CNN
 F 1 "1N4148" H 2550 3786 50  0000 C CNN
-F 2 "" V 2550 3900 50  0001 C CNN
+F 2 "Diode_SMD:D_SOD-323_HandSoldering" V 2550 3900 50  0001 C CNN
 F 3 "~" V 2550 3900 50  0001 C CNN
 	1    2550 3900

Commit message: update,
Parts:
- renumbered D8 to D?, Q2 to Q?, R7 to R?, R8 to R?, R24 to R?
Changed lines of the file:
@@
 EESchema Schematic File Version 4
+LIBS:backplane-cache
 LIBS:stm32_bottom_board_respin-cache
 EELAYER 26 0
@@
 $Descr A4 11693 8268
 encoding utf-8
-Sheet 4 8
+Sheet 4 9
 Title ""
 Date ""
@@
 $EndDescr
 $Comp
-L taobao-r:R471 R7
+L taobao-r:R471 R?
 U 1 1 5BCBA355
 P 2150 2200
-F 0 "R7" V 1954 2200 50  0000 C CNN
+F 0 "R?" V 1954 2200 50  0000 C CNN
 F 1 "R471" V 2045 2200 50  0000 C CNN
 F 2 "Resistor_SMD:R_0603_1608Metric_Pad1.05x0.95mm_HandSolder" H 2150 2200 50  0001 C CNN
@@
 $EndComp
 $Comp
-L taobao-r:R331 R8
+L taobao-r:R331 R?
 U 1 1 5BCBA411
 P 2850 1600
-F 0 "R8" H 2909 1646 50  0000 L CNN
+F 0 "R?" H 2909 1646 50  0000 L CNN
 F 1 "R331" H 2909 1555 50  0000 L CNN
 F 2 "Resistor_SMD:R_0603_1608Metric_Pad1.05x0.95mm_HandSolder" H 2850 1600 50  0001 C CNN
@@
 	2850 1700 2850 1850
 $Comp
-L power:GND #PWR016
+L power:GND #PWR?
 U 1 1 5BCBA643
 P 2850 2700
-F 0 "#PWR016" H 2850 2450 50  0001 C CNN
+F 0 "#PWR?" H 2850 2450 50  0001 C CNN
 F 1 "GND" H 2855 2527 50  0000 C CNN
 F 2 "" H 2850 2700 50  0001 C CNN
@@
 FAN_PWM_OUTPUT
 $Comp
-L power:VDD #PWR015
+L power:VDD #PWR?
 U 1 1 5BCBA5C6
 P 2850 1300
-F 0 "#PWR015" H 2850 1150 50  0001 C CNN
+F 0 "#PWR?" H 2850 1150 50  0001 C CNN
 F 1 "VDD" H 2867 1473 50  0000 C CNN
 F 2 "" H 2850 1300 50  0001 C CNN
@@
 $EndComp
 $Comp
-L taobao-transistor:SS9013_J3 Q2
+L taobao-transistor:SS9013_J3 Q?
 U 1 1 5BCBC4D0
 P 2750 2200
-AR Path="/5BCBC4D0" Ref="Q2"  Part="1"
-AR Path="/5BCBA20B/5BCBC4D0" Ref="Q2"  Part="1"
-F 0 "Q2" H 2950 2250 50  0000 L CNN
+AR Path="/5BCBC4D0" Ref="Q?"  Part="1"
+AR Path="/5BCBA20B/5BCBC4D0" Ref="Q?"  Part="1"
+F 0 "Q?" H 2950 2250 50  0000 L CNN
 F 1 "SS9013_J3" H 2950 2200 50  0000 L CNN
 F 2 "Package_TO_SOT_SMD:SOT-23_Handsoldering" H 2950 2125 50  0001 L CIN
@@
 STM32_FAN_RPM
 $Comp
-L power:VDD #PWR0124
+L power:VDD #PWR?
 U 1 1 5BDC0579
 P 2350 3350
-F 0 "#PWR0124" H 2350 3200 50  0001 C CNN
+F 0 "#PWR?" H 2350 3200 50  0001 C CNN
 F 1 "VDD" H 2367 3523 50  0000 C CNN
 F 2 "" H 2350 3350 50  0001 C CNN
@@
 $EndComp
 $Comp
-L taobao-r:R103 R24
+L taobao-r:R103 R?
 U 1 1 5BDC0610
 P 2350 3600
-F 0 "R24" H 2409 3646 50  0000 L CNN
+F 0 "R?" H 2409 3646 50  0000 L CNN
 F 1 "R103" H 2409 3555 50  0000 L CNN
 F 2 "Resistor_SMD:R_0603_1608Metric_Pad1.05x0.95mm_HandSolder" H 2350 3600 50  0001 C CNN
@@
 $EndComp
 $Comp
-L taobao-d:1N4148 D8
+L taobao-d:1N4148 D?
 U 1 1 5BDC3BB5
 P 2550 3900
-F 0 "D8" H 2550 3695 50  0000 C CNN
+F 0 "D?" H 2550 3695 50  0000 C CNN
 F 1 "1N4148" H 2550 3786 50  0000 C CNN
 F 2 "Diode_SMD:D_SOD-323_HandSoldering" V 2550 3900 50  0001 C CNN
