File: pcb/SSR_DRIVER.sch (KiCad schematic (older format))
At the start: 7 parts, among them Q1 2N3904(1AM), U2 OMRON-G3MB-202P

Commit message: update adding SSR2 on pcb and ioc,
Parts:
- added D?: LED_BLUE, LED_SMD:LED_0805_2012Metric_Pad1.15x1.40mm_HandSolder, symbol taobao-components:LED_RED
- added Q?: 2N3904(1AM), Package_TO_SOT_SMD:SOT-23_Handsoldering, symbol taobao-transistor:2N3904(1AM)
- added R? (x2): R331, Resistor_SMD:R_0805_2012Metric_Pad1.15x1.40mm_HandSolder, symbol taobao-r:R331
- added R?: R103, Resistor_SMD:R_0805_2012Metric_Pad1.15x1.40mm_HandSolder, symbol taobao-r:R103
- added R?: R151, Resistor_SMD:R_0805_2012Metric_Pad1.15x1.40mm_HandSolder, symbol taobao-r:R151
- added U?: OMRON-G3MB-202P, footprint-lib:OMRON-G3MB-202P, symbol Relay_SolidState:S102S01
Connections:
- net GND: now also Q?.2 (E), R?.2
- net VDD: now also D?.2 (A), R?.1
- net STM32_SSR_OUTPUT renamed STM32_SSR1_OUTPUT
- new net: Q?.1 (B), R?.1, R?.1
- new net: D?.1 (K), R?.1
- new net: Q?.3 (C), R?.2, U?.4
- new net: R?.2, U?.3
- new net SSR_CH2_OUTPUT1: U?.2
- new net SSR_CH2_OUTPUT2: U?.1
- new net STM32_SSR2_OUTPUT: R?.2
Changed lines of the file:
@@
 U 1 1 5BCB4B6E
 P 4500 3000
+AR Path="/5BCB4A39/5BCB4B6E" Ref="R1"  Part="1"
+AR Path="/5BE41138/5BCB4B6E" Ref="R?"  Part="1"
 F 0 "R1" V 4304 3000 50  0000 C CNN
 F 1 "R331" V 4395 3000 50  0000 C CNN
@@
 $EndComp
 Text HLabel 4000 3000 0    50   Input ~ 0
-STM32_SSR_OUTPUT
+STM32_SSR1_OUTPUT
 $Comp
 L taobao-r:R103 R2
 U 1 1 5BCB4C36
 P 4750 3400
+AR Path="/5BCB4A39/5BCB4C36" Ref="R2"  Part="1"
+AR Path="/5BE41138/5BCB4C36" Ref="R?"  Part="1"
 F 0 "R2" H 4809 3446 50  0000 L CNN
 F 1 "R103" H 4809 3355 50  0000 L CNN
@@
 U 1 1 5BCB4D36
 P 4950 3850
+AR Path="/5BCB4A39/5BCB4D36" Ref="#PWR011"  Part="1"
+AR Path="/5BE41138/5BCB4D36" Ref="#PWR?"  Part="1"
 F 0 "#PWR011" H 4950 3600 50  0001 C CNN
 F 1 "GND" H 4955 3677 50  0000 C CNN
@@
 U 1 1 5BCB4F0A
 P 4800 2200
+AR Path="/5BCB4A39/5BCB4F0A" Ref="D1"  Part="1"
+AR Path="/5BE41138/5BCB4F0A" Ref="D?"  Part="1"
 F 0 "D1" V 4846 2132 50  0000 R CNN
 F 1 "LED_BLUE" V 4755 2132 50  0000 R CNN
@@
 U 1 1 5BCB4FB1
 P 4800 2500
+AR Path="/5BCB4A39/5BCB4FB1" Ref="R3"  Part="1"
+AR Path="/5BE41138/5BCB4FB1" Ref="R?"  Part="1"
 F 0 "R3" H 4859 2546 50  0000 L CNN
 F 1 "R331" H 4859 2455 50  0000 L CNN
@@
 U 1 1 5BCB51DC
 P 5350 2300
+AR Path="/5BCB4A39/5BCB51DC" Ref="R4"  Part="1"
+AR Path="/5BE41138/5BCB51DC" Ref="R?"  Part="1"
 F 0 "R4" H 5409 2346 50  0000 L CNN
 F 1 "R151" H 5409 2255 50  0000 L CNN
@@
 U 1 1 5BCB53B0
 P 6150 2400
+AR Path="/5BCB4A39/5BCB53B0" Ref="U2"  Part="1"
+AR Path="/5BE41138/5BCB53B0" Ref="U?"  Part="1"
 F 0 "U2" H 6150 2083 50  0000 C CNN
 F 1 "OMRON-G3MB-202P" H 6150 2174 50  0000 C CNN
@@
 U 1 1 5BCBF013
 P 5050 1900
+AR Path="/5BCB4A39/5BCBF013" Ref="#PWR012"  Part="1"
+AR Path="/5BE41138/5BCBF013" Ref="#PWR?"  Part="1"
 F 0 "#PWR012" H 5050 1750 50  0001 C CNN
 F 1 "VDD" H 5067 2073 50  0000 C CNN
@@
 AR Path="/5BCBBF31" Ref="Q1"  Part="1"
 AR Path="/5BCB4A39/5BCBBF31" Ref="Q1"  Part="1"
+AR Path="/5BE41138/5BCBBF31" Ref="Q?"  Part="1"
 F 0 "Q1" H 5300 3050 50  0000 L CNN
 F 1 "2N3904(1AM)" H 5300 3000 50  0000 L CNN
@@
 	1    0    0    -1
 $EndComp
+$Comp
+L taobao-r:R331 R?
+U 1 1 5BE460BB
+P 4400 5550
+AR Path="/5BCB4A39/5BE460BB" Ref="R?"  Part="1"
+AR Path="/5BE41138/5BE460BB" Ref="R?"  Part="1"
+F 0 "R?" V 4204 5550 50  0000 C CNN
+F 1 "R331" V 4295 5550 50  0000 C CNN
+F 2 "Resistor_SMD:R_0805_2012Metric_Pad1.15x1.40mm_HandSolder" H 4400 5550 50  0001 C CNN
+F 3 "~" H 4400 5550 50  0001 C CNN
+	1    4400 5550
+	0    1    1    0
+$EndComp
+Text HLabel 3900 5550 0    50   Input ~ 0
+STM32_SSR2_OUTPUT
+$Comp
+L taobao-r:R103 R?
+U 1 1 5BE460C2
+P 4650 5950
+AR Path="/5BCB4A39/5BE460C2" Ref="R?"  Part="1"
+AR Path="/5BE41138/5BE460C2" Ref="R?"  Part="1"
+F 0 "R?" H 4709 5996 50  0000 L CNN
+F 1 "R103" H 4709 5905 50  0000 L CNN
+F 2 "Resistor_SMD:R_0805_2012Metric_Pad1.15x1.40mm_HandSolder" H 4650 5950 50  0001 C CNN
+F 3 "~" H 4650 5950 50  0001 C CNN
+	1    4650 5950
+	1    0    0    -1
+$EndComp
+Wire Wire Line
+	3900 5550 4300 5550
+Wire Wire Line
+	4500 5550 4650 5550
+Wire Wire Line
+	4650 5550 4650 5850
+Wire Wire Line
+	4800 5550 4650 5550
+Connection ~ 4650 5550
+Wire Wire Line
+	4650 6050 4650 6200
+Wire Wire Line
+	4650 6200 4850 6200
+Wire Wire Line
+	5100 6200 5100 5750
+$Comp
+L power:GND #PWR?
+U 1 1 5BE460D0
+P 4850 6400
+AR Path="/5BCB4A39/5BE460D0" Ref="#PWR?"  Part="1"
+AR Path="/5BE41138/5BE460D0" Ref="#PWR?"  Part="1"
+F 0 "#PWR?" H 4850 6150 50  0001 C CNN
+F 1 "GND" H 4855 6227 50  0000 C CNN
+F 2 "" H 4850 6400 50  0001 C CNN
+F 3 "" H 4850 6400 50  0001 C CNN
+	1    4850 6400
+	1    0    0    -1
+$EndComp
+Wire Wire Line
+	4850 6400 4850 6200
+Connection ~ 4850 6200
+Wire Wire Line
+	4850 6200 5100 6200
+$Comp
+L taobao-components:LED_RED D?
+U 1 1 5BE460D9
+P 4700 4750
+AR Path="/5BCB4A39/5BE460D9" Ref="D?"  Part="1"
+AR Path="/5BE41138/5BE460D9" Ref="D?"  Part="1"
+F 0 "D?" V 4746 4682 50  0000 R CNN
+F 1 "LED_BLUE" V 4655 4682 50  0000 R CNN
+F 2 "LED_SMD:LED_0805_2012Metric_Pad1.15x1.40mm_HandSolder" V 4700 4750 50  0001 C CNN
+F 3 "~" V 4700 4750 50  0001 C CNN
+	1    4700 4750
+	0    -1   -1   0
+$EndComp
+$Comp
+L taobao-r:R331 R?
+U 1 1 5BE460DF
+P 4700 5050
+AR Path="/5BCB4A39/5BE460DF" Ref="R?"  Part="1"
+AR Path="/5BE41138/5BE460DF" Ref="R?"  Part="1"
+F 0 "R?" H 4759 5096 50  0000 L CNN
+F 1 "R331" H 4759 5005 50  0000 L CNN
+F 2 "Resistor_SMD:R_0805_2012Metric_Pad1.15x1.40mm_HandSolder" H 4700 5050 50  0001 C CNN
+F 3 "~" H 4700 5050 50  0001 C CNN
+	1    4700 5050
+	1    0    0    -1
+$EndComp
+Wire Wire Line
+	4700 5150 4700 5250
+Wire Wire Line
+	4700 5250 5100 5250
+Wire Wire Line
+	5100 5250 5100 5350
+Wire Wire Line
+	4700 4550 4700 4650
+Wire Wire Line
+	4700 4850 4700 4950
+$Comp
+L taobao-r:R151 R?
+U 1 1 5BE460EA
+P 5250 4850
+AR Path="/5BCB4A39/5BE460EA" Ref="R?"  Part="1"
+AR Path="/5BE41138/5BE460EA" Ref="R?"  Part="1"
+F 0 "R?" H 5309 4896 50  0000 L CNN
+F 1 "R151" H 5309 4805 50  0000 L CNN
+F 2 "Resistor_SMD:R_0805_2012Metric_Pad1.15x1.40mm_HandSolder" H 5250 4850 50  0001 C CNN
+F 3 "~" H 5250 4850 50  0001 C CNN
+	1    5250 4850
+	1    0    0    -1
+$EndComp
+Wire Wire Line
+	5250 4550 5250 4750
+$Comp
+L Relay_SolidState:S102S01 U?
+U 1 1 5BE460F1
+P 6050 4950
+AR Path="/5BCB4A39/5BE460F1" Ref="U?"  Part="1"
+AR Path="/5BE41138/5BE460F1" Ref="U?"  Part="1"
+F 0 "U?" H 6050 4633 50  0000 C CNN
+F 1 "OMRON-G3MB-202P" H 6050 4724 50  0000 C CNN
+F 2 "footprint-lib:OMRON-G3MB-202P" H 5850 4750 50  0001 L CIN
+F 3 "http://www.sharp-world.com/products/device/lineup/data/pdf/datasheet/s102s01_e.pdf" H 6015 4950 50  0001 L CNN
+	1    6050 4950
+	1    0    0    1
+$EndComp
+Wire Wire Line
+	5250 4950 5250 5050
+Wire Wire Line
+	5250 5050 5750 5050
+Wire Wire Line
+	5100 5250 5600 5250
+Wire Wire Line
+	5600 5250 5600 4850
+Wire Wire Line
+	5600 4850 5750 4850
+Connection ~ 5100 5250
+Text Label 7350 4850 2    50   ~ 0
+SSR_CH2_OUTPUT1
+Text Label 7350 5050 2    50   ~ 0
+SSR_CH2_OUTPUT2
+Text HLabel 7600 4850 2    50   Input ~ 0
+SSR_CH2_OUTPUT1
+Text HLabel 7600 5050 2    50   Input ~ 0
+SSR_CH2_OUTPUT2
+Wire Wire Line
+	6350 4850 7600 4850
+Wire Wire Line
+	6350 5050 7600 5050
+$Comp
+L power:VDD #PWR?
+U 1 1 5BE46103
+P 4950 4450
+AR Path="/5BCB4A39/5BE46103" Ref="#PWR?"  Part="1"
+AR Path="/5BE41138/5BE46103" Ref="#PWR?"  Part="1"
+F 0 "#PWR?" H 4950 4300 50  0001 C CNN
+F 1 "VDD" H 4967 4623 50  0000 C CNN
+F 2 "" H 4950 4450 50  0001 C CNN
+F 3 "" H 4950 4450 50  0001 C CNN
+	1    4950 4450
+	1    0    0    -1
+$EndComp
+Wire Wire Line
+	4950 4450 4950 4550
+Wire Wire Line
+	4950 4550 4700 4550
+Wire Wire Line
+	4950 4550 5250 4550
+Connection ~ 4950 4550
+$Comp
+L taobao-transistor:2N3904(1AM) Q?
+U 1 1 5BE4610D
+P 5000 5550
+AR Path="/5BE4610D" Ref="Q?"  Part="1"
+AR Path="/5BCB4A39/5BE4610D" Ref="Q?"  Part="1"
+AR Path="/5BE41138/5BE4610D" Ref="Q?"  Part="1"
+F 0 "Q?" H 5200 5600 50  0000 L CNN
+F 1 "2N3904(1AM)" H 5200 5550 50  0000 L CNN
+F 2 "Package_TO_SOT_SMD:SOT-23_Handsoldering" H 5200 5475 50  0001 L CIN
+F 3 "" H 5000 5550 50  0001 L CNN
+	1    5000 5550
+	1    0    0    -1
+$EndComp

Commit message: update,
Other:
- moved on the sheet: D?, Q?, R?, U?
Changed lines of the file:
@@
 L taobao-r:R331 R?
 U 1 1 5BE460BB
-P 4400 5550
+P 4500 5550
 AR Path="/5BCB4A39/5BE460BB" Ref="R?"  Part="1"
 AR Path="/5BE41138/5BE460BB" Ref="R?"  Part="1"
-F 0 "R?" V 4204 5550 50  0000 C CNN
-F 1 "R331" V 4295 5550 50  0000 C CNN
-F 2 "Resistor_SMD:R_0805_2012Metric_Pad1.15x1.40mm_HandSolder" H 4400 5550 50  0001 C CNN
-F 3 "~" H 4400 5550 50  0001 C CNN
-	1    4400 5550
+F 0 "R?" V 4304 5550 50  0000 C CNN
+F 1 "R331" V 4395 5550 50  0000 C CNN
+F 2 "Resistor_SMD:R_0805_2012Metric_Pad1.15x1.40mm_HandSolder" H 4500 5550 50  0001 C CNN
+F 3 "~" H 4500 5550 50  0001 C CNN
+	1    4500 5550
 	0    1    1    0
 $EndComp
-Text HLabel 3900 5550 0    50   Input ~ 0
+Text HLabel 4000 5550 0    50   Input ~ 0
 STM32_SSR2_OUTPUT
 $Comp
 L taobao-r:R103 R?
 U 1 1 5BE460C2
-P 4650 5950
+P 4750 5950
 AR Path="/5BCB4A39/5BE460C2" Ref="R?"  Part="1"
 AR Path="/5BE41138/5BE460C2" Ref="R?"  Part="1"
-F 0 "R?" H 4709 5996 50  0000 L CNN
-F 1 "R103" H 4709 5905 50  0000 L CNN
-F 2 "Resistor_SMD:R_0805_2012Metric_Pad1.15x1.40mm_HandSolder" H 4650 5950 50  0001 C CNN
-F 3 "~" H 4650 5950 50  0001 C CNN
-	1    4650 5950
+F 0 "R?" H 4809 5996 50  0000 L CNN
+F 1 "R103" H 4809 5905 50  0000 L CNN
+F 2 "Resistor_SMD:R_0805_2012Metric_Pad1.15x1.40mm_HandSolder" H 4750 5950 50  0001 C CNN
+F 3 "~" H 4750 5950 50  0001 C CNN
+	1    4750 5950
 	1    0    0    -1
 $EndComp
 Wire Wire Line
-	3900 5550 4300 5550
+	4000 5550 4400 5550
 Wire Wire Line
-	4500 5550 4650 5550
+	4600 5550 4750 5550
 Wire Wire Line
-	4650 5550 4650 5850
+	4750 5550 4750 5850
 Wire Wire Line
-	4800 5550 4650 5550
-Connection ~ 4650 5550
+	4900 5550 4750 5550
+Connection ~ 4750 5550
 Wire Wire Line
-	4650 6050 4650 6200
+	4750 6050 4750 6200
 Wire Wire Line
-	4650 6200 4850 6200
+	4750 6200 4950 6200
 Wire Wire Line
-	5100 6200 5100 5750
+	5200 6200 5200 5750
 $Comp
 L power:GND #PWR?
 U 1 1 5BE460D0
-P 4850 6400
+P 4950 6400
 AR Path="/5BCB4A39/5BE460D0" Ref="#PWR?"  Part="1"
 AR Path="/5BE41138/5BE460D0" Ref="#PWR?"  Part="1"
-F 0 "#PWR?" H 4850 6150 50  0001 C CNN
-F 1 "GND" H 4855 6227 50  0000 C CNN
-F 2 "" H 4850 6400 50  0001 C CNN
-F 3 "" H 4850 6400 50  0001 C CNN
-	1    4850 6400
+F 0 "#PWR?" H 4950 6150 50  0001 C CNN
+F 1 "GND" H 4955 6227 50  0000 C CNN
+F 2 "" H 4950 6400 50  0001 C CNN
+F 3 "" H 4950 6400 50  0001 C CNN
+	1    4950 6400
 	1    0    0    -1
 $EndComp
 Wire Wire Line
-	4850 6400 4850 6200
-Connection ~ 4850 6200
+	4950 6400 4950 6200
+Connection ~ 4950 6200
 Wire Wire Line
-	4850 6200 5100 6200
+	4950 6200 5200 6200
 $Comp
 L taobao-components:LED_RED D?
 U 1 1 5BE460D9
-P 4700 4750
+P 4800 4750
 AR Path="/5BCB4A39/5BE460D9" Ref="D?"  Part="1"
 AR Path="/5BE41138/5BE460D9" Ref="D?"  Part="1"
-F 0 "D?" V 4746 4682 50  0000 R CNN
-F 1 "LED_BLUE" V 4655 4682 50  0000 R CNN
-F 2 "LED_SMD:LED_0805_2012Metric_Pad1.15x1.40mm_HandSolder" V 4700 4750 50  0001 C CNN
-F 3 "~" V 4700 4750 50  0001 C CNN
-	1    4700 4750
+F 0 "D?" V 4846 4682 50  0000 R CNN
+F 1 "LED_BLUE" V 4755 4682 50  0000 R CNN
+F 2 "LED_SMD:LED_0805_2012Metric_Pad1.15x1.40mm_HandSolder" V 4800 4750 50  0001 C CNN
+F 3 "~" V 4800 4750 50  0001 C CNN
+	1    4800 4750
 	0    -1   -1   0
 $EndComp
@@
 L taobao-r:R331 R?
 U 1 1 5BE460DF
-P 4700 5050
+P 4800 5050
 AR Path="/5BCB4A39/5BE460DF" Ref="R?"  Part="1"
 AR Path="/5BE41138/5BE460DF" Ref="R?"  Part="1"
-F 0 "R?" H 4759 5096 50  0000 L CNN
-F 1 "R331" H 4759 5005 50  0000 L CNN
-F 2 "Resistor_SMD:R_0805_2012Metric_Pad1.15x1.40mm_HandSolder" H 4700 5050 50  0001 C CNN
-F 3 "~" H 4700 5050 50  0001 C CNN
-	1    4700 5050
+F 0 "R?" H 4859 5096 50  0000 L CNN
+F 1 "R331" H 4859 5005 50  0000 L CNN
+F 2 "Resistor_SMD:R_0805_2012Metric_Pad1.15x1.40mm_HandSolder" H 4800 5050 50  0001 C CNN
+F 3 "~" H 4800 5050 50  0001 C CNN
+	1    4800 5050
 	1    0    0    -1
 $EndComp
 Wire Wire Line
-	4700 5150 4700 5250
+	4800 5150 4800 5250
 Wire Wire Line
-	4700 5250 5100 5250
+	4800 5250 5200 5250
 Wire Wire Line
-	5100 5250 5100 5350
+	5200 5250 5200 5350
 Wire Wire Line
-	4700 4550 4700 4650
+	4800 4550 4800 4650
 Wire Wire Line
-	4700 4850 4700 4950
+	4800 4850 4800 4950
 $Comp
 L taobao-r:R151 R?
 U 1 1 5BE460EA
-P 5250 4850
+P 5350 4850
 AR Path="/5BCB4A39/5BE460EA" Ref="R?"  Part="1"
 AR Path="/5BE41138/5BE460EA" Ref="R?"  Part="1"
-F 0 "R?" H 5309 4896 50  0000 L CNN
-F 1 "R151" H 5309 4805 50  0000 L CNN
-F 2 "Resistor_SMD:R_0805_2012Metric_Pad1.15x1.40mm_HandSolder" H 5250 4850 50  0001 C CNN
-F 3 "~" H 5250 4850 50  0001 C CNN
-	1    5250 4850
+F 0 "R?" H 5409 4896 50  0000 L CNN
+F 1 "R151" H 5409 4805 50  0000 L CNN
+F 2 "Resistor_SMD:R_0805_2012Metric_Pad1.15x1.40mm_HandSolder" H 5350 4850 50  0001 C CNN
+F 3 "~" H 5350 4850 50  0001 C CNN
+	1    5350 4850
 	1    0    0    -1
 $EndComp
 Wire Wire Line
-	5250 4550 5250 4750
+	5350 4550 5350 4750
 $Comp
 L Relay_SolidState:S102S01 U?
 U 1 1 5BE460F1
-P 6050 4950
+P 6150 4950
 AR Path="/5BCB4A39/5BE460F1" Ref="U?"  Part="1"
 AR Path="/5BE41138/5BE460F1" Ref="U?"  Part="1"
-F 0 "U?" H 6050 4633 50  0000 C CNN
-F 1 "OMRON-G3MB-202P" H 6050 4724 50  0000 C CNN
-F 2 "footprint-lib:OMRON-G3MB-202P" H 5850 4750 50  0001 L CIN
-F 3 "http://www.sharp-world.com/products/device/lineup/data/pdf/datasheet/s102s01_e.pdf" H 6015 4950 50  0001 L CNN
-	1    6050 4950
+F 0 "U?" H 6150 4633 50  0000 C CNN
+F 1 "OMRON-G3MB-202P" H 6150 4724 50  0000 C CNN
+F 2 "footprint-lib:OMRON-G3MB-202P" H 5950 4750 50  0001 L CIN
+F 3 "http://www.sharp-world.com/products/device/lineup/data/pdf/datasheet/s102s01_e.pdf" H 6115 4950 50  0001 L CNN
+	1    6150 4950
 	1    0    0    1
 $EndComp
 Wire Wire Line
-	5250 4950 5250 5050
+	5350 4950 5350 5050
 Wire Wire Line
-	5250 5050 5750 5050
+	5350 5050 5850 5050
 Wire Wire Line
-	5100 5250 5600 5250
+	5200 5250 5700 5250
 Wire Wire Line
-	5600 5250 5600 4850
+	5700 5250 5700 4850
 Wire Wire Line
-	5600 4850 5750 4850
-Connection ~ 5100 5250
-Text Label 7350 4850 2    50   ~ 0
+	5700 4850 5850 4850
+Connection ~ 5200 5250
+Text Label 7450 4850 2    50   ~ 0
 SSR_CH2_OUTPUT1
-Text Label 7350 5050 2    50   ~ 0
+Text Label 7450 5050 2    50   ~ 0
 SSR_CH2_OUTPUT2
-Text HLabel 7600 4850 2    50   Input ~ 0
+Text HLabel 7700 4850 2    50   Input ~ 0
 SSR_CH2_OUTPUT1
-Text HLabel 7600 5050 2    50   Input ~ 0
+Text HLabel 7700 5050 2    50   Input ~ 0
 SSR_CH2_OUTPUT2
 Wire Wire Line
-	6350 4850 7600 4850
+	6450 4850 7700 4850
 Wire Wire Line
-	6350 5050 7600 5050
+	6450 5050 7700 5050
 $Comp
 L power:VDD #PWR?
 U 1 1 5BE46103
-P 4950 4450
+P 5050 4450
 AR Path="/5BCB4A39/5BE46103" Ref="#PWR?"  Part="1"
 AR Path="/5BE41138/5BE46103" Ref="#PWR?"  Part="1"
-F 0 "#PWR?" H 4950 4300 50  0001 C CNN
-F 1 "VDD" H 4967 4623 50  0000 C CNN
-F 2 "" H 4950 4450 50  0001 C CNN
-F 3 "" H 4950 4450 50  0001 C CNN
-	1    4950 4450
+F 0 "#PWR?" H 5050 4300 50  0001 C CNN
+F 1 "VDD" H 5067 4623 50  0000 C CNN
+F 2 "" H 5050 4450 50  0001 C CNN
+F 3 "" H 5050 4450 50  0001 C CNN
+	1    5050 4450
 	1    0    0    -1
 $EndComp
 Wire Wire Line
-	4950 4450 4950 4550
+	5050 4450 5050 4550
 Wire Wire Line
-	4950 4550 4700 4550
+	5050 4550 4800 4550
 Wire Wire Line
-	4950 4550 5250 4550
-Connection ~ 4950 4550
+	5050 4550 5350 4550
+Connection ~ 5050 4550
 $Comp
 L taobao-transistor:2N3904(1AM) Q?
 U 1 1 5BE4610D
-P 5000 5550
+P 5100 5550
 AR Path="/5BE4610D" Ref="Q?"  Part="1"
 AR Path="/5BCB4A39/5BE4610D" Ref="Q?"  Part="1"
 AR Path="/5BE41138/5BE4610D" Ref="Q?"  Part="1"
-F 0 "Q?" H 5200 5600 50  0000 L CNN
-F 1 "2N3904(1AM)" H 5200 5550 50  0000 L CNN
-F 2 "Package_TO_SOT_SMD:SOT-23_Handsoldering" H 5200 5475 50  0001 L CIN
-F 3 "" H 5000 5550 50  0001 L CNN
-	1    5000 5550
+F 0 "Q?" H 5300 5600 50  0000 L CNN
+F 1 "2N3904(1AM)" H 5300 5550 50  0000 L CNN
+F 2 "Package_TO_SOT_SMD:SOT-23_Handsoldering" H 5300 5475 50  0001 L CIN
+F 3 "" H 5100 5550 50  0001 L CNN
+	1    5100 5550
 	1    0    0    -1
 $EndComp

Commit message: update,
Parts:
- gave numbers to parts that had none: 7
Changed lines of the file:
@@
 $EndComp
 $Comp
-L taobao-r:R331 R?
+L taobao-r:R331 R16
 U 1 1 5BE460BB
 P 4500 5550
-AR Path="/5BCB4A39/5BE460BB" Ref="R?"  Part="1"
+AR Path="/5BCB4A39/5BE460BB" Ref="R16"  Part="1"
 AR Path="/5BE41138/5BE460BB" Ref="R?"  Part="1"
-F 0 "R?" V 4304 5550 50  0000 C CNN
+F 0 "R16" V 4304 5550 50  0000 C CNN
 F 1 "R331" V 4395 5550 50  0000 C CNN
 F 2 "Resistor_SMD:R_0805_2012Metric_Pad1.15x1.40mm_HandSolder" H 4500 5550 50  0001 C CNN
@@
 STM32_SSR2_OUTPUT
 $Comp
-L taobao-r:R103 R?
+L taobao-r:R103 R17
 U 1 1 5BE460C2
 P 4750 5950
-AR Path="/5BCB4A39/5BE460C2" Ref="R?"  Part="1"
+AR Path="/5BCB4A39/5BE460C2" Ref="R17"  Part="1"
 AR Path="/5BE41138/5BE460C2" Ref="R?"  Part="1"
-F 0 "R?" H 4809 5996 50  0000 L CNN
+F 0 "R17" H 4809 5996 50  0000 L CNN
 F 1 "R103" H 4809 5905 50  0000 L CNN
 F 2 "Resistor_SMD:R_0805_2012Metric_Pad1.15x1.40mm_HandSolder" H 4750 5950 50  0001 C CNN
@@
 	5200 6200 5200 5750
 $Comp
-L power:GND #PWR?
+L power:GND #PWR0120
 U 1 1 5BE460D0
 P 4950 6400
-AR Path="/5BCB4A39/5BE460D0" Ref="#PWR?"  Part="1"
+AR Path="/5BCB4A39/5BE460D0" Ref="#PWR0120"  Part="1"
 AR Path="/5BE41138/5BE460D0" Ref="#PWR?"  Part="1"
-F 0 "#PWR?" H 4950 6150 50  0001 C CNN
+F 0 "#PWR0120" H 4950 6150 50  0001 C CNN
 F 1 "GND" H 4955 6227 50  0000 C CNN
 F 2 "" H 4950 6400 50  0001 C CNN
@@
 	4950 6200 5200 6200
 $Comp
-L taobao-components:LED_RED D?
+L taobao-components:LED_RED D6
 U 1 1 5BE460D9
 P 4800 4750
-AR Path="/5BCB4A39/5BE460D9" Ref="D?"  Part="1"
+AR Path="/5BCB4A39/5BE460D9" Ref="D6"  Part="1"
 AR Path="/5BE41138/5BE460D9" Ref="D?"  Part="1"
-F 0 "D?" V 4846 4682 50  0000 R CNN
+F 0 "D6" V 4846 4682 50  0000 R CNN
 F 1 "LED_BLUE" V 4755 4682 50  0000 R CNN
 F 2 "LED_SMD:LED_0805_2012Metric_Pad1.15x1.40mm_HandSolder" V 4800 4750 50  0001 C CNN
@@
 $EndComp
 $Comp
-L taobao-r:R331 R?
+L taobao-r:R331 R18
 U 1 1 5BE460DF
 P 4800 5050
-AR Path="/5BCB4A39/5BE460DF" Ref="R?"  Part="1"
+AR Path="/5BCB4A39/5BE460DF" Ref="R18"  Part="1"
 AR Path="/5BE41138/5BE460DF" Ref="R?"  Part="1"
-F 0 "R?" H 4859 5096 50  0000 L CNN
+F 0 "R18" H 4859 5096 50  0000 L CNN
 F 1 "R331" H 4859 5005 50  0000 L CNN
 F 2 "Resistor_SMD:R_0805_2012Metric_Pad1.15x1.40mm_HandSolder" H 4800 5050 50  0001 C CNN
@@
 	4800 4850 4800 4950
 $Comp
-L taobao-r:R151 R?
+L taobao-r:R151 R19
 U 1 1 5BE460EA
 P 5350 4850
-AR Path="/5BCB4A39/5BE460EA" Ref="R?"  Part="1"
+AR Path="/5BCB4A39/5BE460EA" Ref="R19"  Part="1"
 AR Path="/5BE41138/5BE460EA" Ref="R?"  Part="1"
-F 0 "R?" H 5409 4896 50  0000 L CNN
+F 0 "R19" H 5409 4896 50  0000 L CNN
 F 1 "R151" H 5409 4805 50  0000 L CNN
 F 2 "Resistor_SMD:R_0805_2012Metric_Pad1.15x1.40mm_HandSolder" H 5350 4850 50  0001 C CNN
@@
 	5350 4550 5350 4750
 $Comp
-L Relay_SolidState:S102S01 U?
+L Relay_SolidState:S102S01 U6
 U 1 1 5BE460F1
 P 6150 4950
-AR Path="/5BCB4A39/5BE460F1" Ref="U?"  Part="1"
+AR Path="/5BCB4A39/5BE460F1" Ref="U6"  Part="1"
 AR Path="/5BE41138/5BE460F1" Ref="U?"  Part="1"
-F 0 "U?" H 6150 4633 50  0000 C CNN
+F 0 "U6" H 6150 4633 50  0000 C CNN
 F 1 "OMRON-G3MB-202P" H 6150 4724 50  0000 C CNN
 F 2 "footprint-lib:OMRON-G3MB-202P" H 5950 4750 50  0001 L CIN
@@
 	6450 5050 7700 5050
 $Comp
-L power:VDD #PWR?
+L power:VDD #PWR0121
 U 1 1 5BE46103
 P 5050 4450
-AR Path="/5BCB4A39/5BE46103" Ref="#PWR?"  Part="1"
+AR Path="/5BCB4A39/5BE46103" Ref="#PWR0121"  Part="1"
 AR Path="/5BE41138/5BE46103" Ref="#PWR?"  Part="1"
-F 0 "#PWR?" H 5050 4300 50  0001 C CNN
+F 0 "#PWR0121" H 5050 4300 50  0001 C CNN
 F 1 "VDD" H 5067 4623 50  0000 C CNN
 F 2 "" H 5050 4450 50  0001 C CNN
@@
 P 5100 5550
 AR Path="/5BE4610D" Ref="Q?"  Part="1"
-AR Path="/5BCB4A39/5BE4610D" Ref="Q?"  Part="1"
+AR Path="/5BCB4A39/5BE4610D" Ref="Q3"  Part="1"
 AR Path="/5BE41138/5BE4610D" Ref="Q?"  Part="1"
-F 0 "Q?" H 5300 5600 50  0000 L CNN
+F 0 "Q3" H 5300 5600 50  0000 L CNN
 F 1 "2N3904(1AM)" H 5300 5550 50  0000 L CNN
 F 2 "Package_TO_SOT_SMD:SOT-23_Handsoldering" H 5300 5475 50  0001 L CIN

Commit message: assign footprint,
Parts:
- R1, R16, R17, R18, R19, R2, R3, R4: footprint Resistor_SMD:R_0805_2012Metric_Pad1.15x1.40mm_HandSolder -> Resistor_SMD:R_0603_1608Metric_Pad1.05x0.95mm_HandSolder
Changed lines of the file:
@@
 F 0 "R1" V 4304 3000 50  0000 C CNN
 F 1 "R331" V 4395 3000 50  0000 C CNN
-F 2 "Resistor_SMD:R_0805_2012Metric_Pad1.15x1.40mm_HandSolder" H 4500 3000 50  0001 C CNN
+F 2 "Resistor_SMD:R_0603_1608Metric_Pad1.05x0.95mm_HandSolder" H 4500 3000 50  0001 C CNN
 F 3 "~" H 4500 3000 50  0001 C CNN
 	1    4500 3000
@@
 F 0 "R2" H 4809 3446 50  0000 L CNN
 F 1 "R103" H 4809 3355 50  0000 L CNN
-F 2 "Resistor_SMD:R_0805_2012Metric_Pad1.15x1.40mm_HandSolder" H 4750 3400 50  0001 C CNN
+F 2 "Resistor_SMD:R_0603_1608Metric_Pad1.05x0.95mm_HandSolder" H 4750 3400 50  0001 C CNN
 F 3 "~" H 4750 3400 50  0001 C CNN
 	1    4750 3400
@@
 F 0 "R3" H 4859 2546 50  0000 L CNN
 F 1 "R331" H 4859 2455 50  0000 L CNN
-F 2 "Resistor_SMD:R_0805_2012Metric_Pad1.15x1.40mm_HandSolder" H 4800 2500 50  0001 C CNN
+F 2 "Resistor_SMD:R_0603_1608Metric_Pad1.05x0.95mm_HandSolder" H 4800 2500 50  0001 C CNN
 F 3 "~" H 4800 2500 50  0001 C CNN
 	1    4800 2500
@@
 F 0 "R4" H 5409 2346 50  0000 L CNN
 F 1 "R151" H 5409 2255 50  0000 L CNN
-F 2 "Resistor_SMD:R_0805_2012Metric_Pad1.15x1.40mm_HandSolder" H 5350 2300 50  0001 C CNN
+F 2 "Resistor_SMD:R_0603_1608Metric_Pad1.05x0.95mm_HandSolder" H 5350 2300 50  0001 C CNN
 F 3 "~" H 5350 2300 50  0001 C CNN
 	1    5350 2300
@@
 F 0 "R16" V 4304 5550 50  0000 C CNN
 F 1 "R331" V 4395 5550 50  0000 C CNN
-F 2 "Resistor_SMD:R_0805_2012Metric_Pad1.15x1.40mm_HandSolder" H 4500 5550 50  0001 C CNN
+F 2 "Resistor_SMD:R_0603_1608Metric_Pad1.05x0.95mm_HandSolder" H 4500 5550 50  0001 C CNN
 F 3 "~" H 4500 5550 50  0001 C CNN
 	1    4500 5550
@@
 F 0 "R17" H 4809 5996 50  0000 L CNN
 F 1 "R103" H 4809 5905 50  0000 L CNN
-F 2 "Resistor_SMD:R_0805_2012Metric_Pad1.15x1.40mm_HandSolder" H 4750 5950 50  0001 C CNN
+F 2 "Resistor_SMD:R_0603_1608Metric_Pad1.05x0.95mm_HandSolder" H 4750 5950 50  0001 C CNN
 F 3 "~" H 4750 5950 50  0001 C CNN
 	1    4750 5950
@@
 F 0 "R18" H 4859 5096 50  0000 L CNN
 F 1 "R331" H 4859 5005 50  0000 L CNN
-F 2 "Resistor_SMD:R_0805_2012Metric_Pad1.15x1.40mm_HandSolder" H 4800 5050 50  0001 C CNN
+F 2 "Resistor_SMD:R_0603_1608Metric_Pad1.05x0.95mm_HandSolder" H 4800 5050 50  0001 C CNN
 F 3 "~" H 4800 5050 50  0001 C CNN
 	1    4800 5050
@@
 F 0 "R19" H 5409 4896 50  0000 L CNN
 F 1 "R151" H 5409 4805 50  0000 L CNN
-F 2 "Resistor_SMD:R_0805_2012Metric_Pad1.15x1.40mm_HandSolder" H 5350 4850 50  0001 C CNN
+F 2 "Resistor_SMD:R_0603_1608Metric_Pad1.05x0.95mm_HandSolder" H 5350 4850 50  0001 C CNN
 F 3 "~" H 5350 4850 50  0001 C CNN
 	1    5350 4850
