File: pcb/SSR_DRIVER.sch (KiCad schematic (older format))
At the start: 14 parts, among them Q1 2N3904(1AM), Q3 2N3904(1AM), U2 OMRON-G3MB-202P, U6 OMRON-G3MB-202P

Commit message: update,
Parts:
- U2: footprint footprint-lib:OMRON-G3MB-202P -> footprint-lib.pretty:OMRON-G3MB-202P
Changed lines of the file:
@@
 F 0 "U2" H 6150 2083 50  0000 C CNN
 F 1 "OMRON-G3MB-202P" H 6150 2174 50  0000 C CNN
-F 2 "footprint-lib:OMRON-G3MB-202P" H 5950 2200 50  0001 L CIN
+F 2 "footprint-lib.pretty:OMRON-G3MB-202P" H 5950 2200 50  0001 L CIN
 F 3 "http://www.sharp-world.com/products/device/lineup/data/pdf/datasheet/s102s01_e.pdf" H 6115 2400 50  0001 L CNN
 	1    6150 2400

Commit message: update,
Parts:
- renumbered D1 to D?, D6 to D?, Q1 to Q?, Q3 to Q?, R1 to R?, R2 to R?, R3 to R?, R4 to R?, R16 to R?, R17 to R?, R18 to R?, R19 to R?, U2 to U?, U6 to U?
Changed lines of the file:
@@
 EESchema Schematic File Version 4
+LIBS:backplane-cache
 LIBS:stm32_bottom_board_respin-cache
 EELAYER 26 0
@@
 $Descr A4 11693 8268
 encoding utf-8
-Sheet 2 8
+Sheet 2 9
 Title ""
 Date ""
@@
 $EndDescr
 $Comp
-L taobao-r:R331 R1
+L taobao-r:R331 R?
 U 1 1 5BCB4B6E
 P 4500 3000
-AR Path="/5BCB4A39/5BCB4B6E" Ref="R1"  Part="1"
+AR Path="/5BCB4A39/5BCB4B6E" Ref="R?"  Part="1"
 AR Path="/5BE41138/5BCB4B6E" Ref="R?"  Part="1"
-F 0 "R1" V 4304 3000 50  0000 C CNN
+F 0 "R?" V 4304 3000 50  0000 C CNN
 F 1 "R331" V 4395 3000 50  0000 C CNN
 F 2 "Resistor_SMD:R_0603_1608Metric_Pad1.05x0.95mm_HandSolder" H 4500 3000 50  0001 C CNN
@@
 STM32_SSR1_OUTPUT
 $Comp
-L taobao-r:R103 R2
+L taobao-r:R103 R?
 U 1 1 5BCB4C36
 P 4750 3400
-AR Path="/5BCB4A39/5BCB4C36" Ref="R2"  Part="1"
+AR Path="/5BCB4A39/5BCB4C36" Ref="R?"  Part="1"
 AR Path="/5BE41138/5BCB4C36" Ref="R?"  Part="1"
-F 0 "R2" H 4809 3446 50  0000 L CNN
+F 0 "R?" H 4809 3446 50  0000 L CNN
 F 1 "R103" H 4809 3355 50  0000 L CNN
 F 2 "Resistor_SMD:R_0603_1608Metric_Pad1.05x0.95mm_HandSolder" H 4750 3400 50  0001 C CNN
@@
 	5200 3650 5200 3200
 $Comp
-L power:GND #PWR011
+L power:GND #PWR?
 U 1 1 5BCB4D36
 P 4950 3850
-AR Path="/5BCB4A39/5BCB4D36" Ref="#PWR011"  Part="1"
+AR Path="/5BCB4A39/5BCB4D36" Ref="#PWR?"  Part="1"
 AR Path="/5BE41138/5BCB4D36" Ref="#PWR?"  Part="1"
-F 0 "#PWR011" H 4950 3600 50  0001 C CNN
+F 0 "#PWR?" H 4950 3600 50  0001 C CNN
 F 1 "GND" H 4955 3677 50  0000 C CNN
 F 2 "" H 4950 3850 50  0001 C CNN
@@
 	4950 3650 5200 3650
 $Comp
-L taobao-components:LED_RED D1
+L taobao-components:LED_RED D?
 U 1 1 5BCB4F0A
 P 4800 2200
-AR Path="/5BCB4A39/5BCB4F0A" Ref="D1"  Part="1"
+AR Path="/5BCB4A39/5BCB4F0A" Ref="D?"  Part="1"
 AR Path="/5BE41138/5BCB4F0A" Ref="D?"  Part="1"
-F 0 "D1" V 4846 2132 50  0000 R CNN
+F 0 "D?" V 4846 2132 50  0000 R CNN
 F 1 "LED_BLUE" V 4755 2132 50  0000 R CNN
 F 2 "LED_SMD:LED_0805_2012Metric_Pad1.15x1.40mm_HandSolder" V 4800 2200 50  0001 C CNN
@@
 $EndComp
 $Comp
-L taobao-r:R331 R3
+L taobao-r:R331 R?
 U 1 1 5BCB4FB1
 P 4800 2500
-AR Path="/5BCB4A39/5BCB4FB1" Ref="R3"  Part="1"
+AR Path="/5BCB4A39/5BCB4FB1" Ref="R?"  Part="1"
 AR Path="/5BE41138/5BCB4FB1" Ref="R?"  Part="1"
-F 0 "R3" H 4859 2546 50  0000 L CNN
+F 0 "R?" H 4859 2546 50  0000 L CNN
 F 1 "R331" H 4859 2455 50  0000 L CNN
 F 2 "Resistor_SMD:R_0603_1608Metric_Pad1.05x0.95mm_HandSolder" H 4800 2500 50  0001 C CNN
@@
 	4800 2300 4800 2400
 $Comp
-L taobao-r:R151 R4
+L taobao-r:R151 R?
 U 1 1 5BCB51DC
 P 5350 2300
-AR Path="/5BCB4A39/5BCB51DC" Ref="R4"  Part="1"
+AR Path="/5BCB4A39/5BCB51DC" Ref="R?"  Part="1"
 AR Path="/5BE41138/5BCB51DC" Ref="R?"  Part="1"
-F 0 "R4" H 5409 2346 50  0000 L CNN
+F 0 "R?" H 5409 2346 50  0000 L CNN
 F 1 "R151" H 5409 2255 50  0000 L CNN
 F 2 "Resistor_SMD:R_0603_1608Metric_Pad1.05x0.95mm_HandSolder" H 5350 2300 50  0001 C CNN
@@
 	5350 2000 5350 2200
 $Comp
-L Relay_SolidState:S102S01 U2
+L Relay_SolidState:S102S01 U?
 U 1 1 5BCB53B0
 P 6150 2400
-AR Path="/5BCB4A39/5BCB53B0" Ref="U2"  Part="1"
+AR Path="/5BCB4A39/5BCB53B0" Ref="U?"  Part="1"
 AR Path="/5BE41138/5BCB53B0" Ref="U?"  Part="1"
-F 0 "U2" H 6150 2083 50  0000 C CNN
+F 0 "U?" H 6150 2083 50  0000 C CNN
 F 1 "OMRON-G3MB-202P" H 6150 2174 50  0000 C CNN
 F 2 "footprint-lib.pretty:OMRON-G3MB-202P" H 5950 2200 50  0001 L CIN
@@
 	6450 2500 7700 2500
 $Comp
-L power:VDD #PWR012
+L power:VDD #PWR?
 U 1 1 5BCBF013
 P 5050 1900
-AR Path="/5BCB4A39/5BCBF013" Ref="#PWR012"  Part="1"
+AR Path="/5BCB4A39/5BCBF013" Ref="#PWR?"  Part="1"
 AR Path="/5BE41138/5BCBF013" Ref="#PWR?"  Part="1"
-F 0 "#PWR012" H 5050 1750 50  0001 C CNN
+F 0 "#PWR?" H 5050 1750 50  0001 C CNN
 F 1 "VDD" H 5067 2073 50  0000 C CNN
 F 2 "" H 5050 1900 50  0001 C CNN
@@
 Connection ~ 5050 2000
 $Comp
-L taobao-transistor:2N3904(1AM) Q1
+L taobao-transistor:2N3904(1AM) Q?
 U 1 1 5BCBBF31
 P 5100 3000
-AR Path="/5BCBBF31" Ref="Q1"  Part="1"
-AR Path="/5BCB4A39/5BCBBF31" Ref="Q1"  Part="1"
+AR Path="/5BCBBF31" Ref="Q?"  Part="1"
+AR Path="/5BCB4A39/5BCBBF31" Ref="Q?"  Part="1"
 AR Path="/5BE41138/5BCBBF31" Ref="Q?"  Part="1"
-F 0 "Q1" H 5300 3050 50  0000 L CNN
+F 0 "Q?" H 5300 3050 50  0000 L CNN
 F 1 "2N3904(1AM)" H 5300 3000 50  0000 L CNN
 F 2 "Package_TO_SOT_SMD:SOT-23_Handsoldering" H 5300 2925 50  0001 L CIN
@@
 $EndComp
 $Comp
-L taobao-r:R331 R16
+L taobao-r:R331 R?
 U 1 1 5BE460BB
 P 4500 5550
-AR Path="/5BCB4A39/5BE460BB" Ref="R16"  Part="1"
+AR Path="/5BCB4A39/5BE460BB" Ref="R?"  Part="1"
 AR Path="/5BE41138/5BE460BB" Ref="R?"  Part="1"
-F 0 "R16" V 4304 5550 50  0000 C CNN
+F 0 "R?" V 4304 5550 50  0000 C CNN
 F 1 "R331" V 4395 5550 50  0000 C CNN
 F 2 "Resistor_SMD:R_0603_1608Metric_Pad1.05x0.95mm_HandSolder" H 4500 5550 50  0001 C CNN
@@
 STM32_SSR2_OUTPUT
 $Comp
-L taobao-r:R103 R17
+L taobao-r:R103 R?
 U 1 1 5BE460C2
 P 4750 5950
-AR Path="/5BCB4A39/5BE460C2" Ref="R17"  Part="1"
+AR Path="/5BCB4A39/5BE460C2" Ref="R?"  Part="1"
 AR Path="/5BE41138/5BE460C2" Ref="R?"  Part="1"
-F 0 "R17" H 4809 5996 50  0000 L CNN
+F 0 "R?" H 4809 5996 50  0000 L CNN
 F 1 "R103" H 4809 5905 50  0000 L CNN
 F 2 "Resistor_SMD:R_0603_1608Metric_Pad1.05x0.95mm_HandSolder" H 4750 5950 50  0001 C CNN
@@
 	5200 6200 5200 5750
 $Comp
-L power:GND #PWR0120
+L power:GND #PWR?
 U 1 1 5BE460D0
 P 4950 6400
-AR Path="/5BCB4A39/5BE460D0" Ref="#PWR0120"  Part="1"
+AR Path="/5BCB4A39/5BE460D0" Ref="#PWR?"  Part="1"
 AR Path="/5BE41138/5BE460D0" Ref="#PWR?"  Part="1"
-F 0 "#PWR0120" H 4950 6150 50  0001 C CNN
+F 0 "#PWR?" H 4950 6150 50  0001 C CNN
 F 1 "GND" H 4955 6227 50  0000 C CNN
 F 2 "" H 4950 6400 50  0001 C CNN
@@
 	4950 6200 5200 6200
 $Comp
-L taobao-components:LED_RED D6
+L taobao-components:LED_RED D?
 U 1 1 5BE460D9
 P 4800 4750
-AR Path="/5BCB4A39/5BE460D9" Ref="D6"  Part="1"
+AR Path="/5BCB4A39/5BE460D9" Ref="D?"  Part="1"
 AR Path="/5BE41138/5BE460D9" Ref="D?"  Part="1"
-F 0 "D6" V 4846 4682 50  0000 R CNN
+F 0 "D?" V 4846 4682 50  0000 R CNN
 F 1 "LED_BLUE" V 4755 4682 50  0000 R CNN
 F 2 "LED_SMD:LED_0805_2012Metric_Pad1.15x1.40mm_HandSolder" V 4800 4750 50  0001 C CNN
@@
 $EndComp
 $Comp
-L taobao-r:R331 R18
+L taobao-r:R331 R?
 U 1 1 5BE460DF
 P 4800 5050
-AR Path="/5BCB4A39/5BE460DF" Ref="R18"  Part="1"
+AR Path="/5BCB4A39/5BE460DF" Ref="R?"  Part="1"
 AR Path="/5BE41138/5BE460DF" Ref="R?"  Part="1"
-F 0 "R18" H 4859 5096 50  0000 L CNN
+F 0 "R?" H 4859 5096 50  0000 L CNN
 F 1 "R331" H 4859 5005 50  0000 L CNN
 F 2 "Resistor_SMD:R_0603_1608Metric_Pad1.05x0.95mm_HandSolder" H 4800 5050 50  0001 C CNN
@@
 	4800 4850 4800 4950
 $Comp
-L taobao-r:R151 R19
+L taobao-r:R151 R?
 U 1 1 5BE460EA
 P 5350 4850
-AR Path="/5BCB4A39/5BE460EA" Ref="R19"  Part="1"
+AR Path="/5BCB4A39/5BE460EA" Ref="R?"  Part="1"
 AR Path="/5BE41138/5BE460EA" Ref="R?"  Part="1"
-F 0 "R19" H 5409 4896 50  0000 L CNN
+F 0 "R?" H 5409 4896 50  0000 L CNN
 F 1 "R151" H 5409 4805 50  0000 L CNN
 F 2 "Resistor_SMD:R_0603_1608Metric_Pad1.05x0.95mm_HandSolder" H 5350 4850 50  0001 C CNN
@@
 	5350 4550 5350 4750
 $Comp
-L Relay_SolidState:S102S01 U6
+L Relay_SolidState:S102S01 U?
 U 1 1 5BE460F1
 P 6150 4950
-AR Path="/5BCB4A39/5BE460F1" Ref="U6"  Part="1"
+AR Path="/5BCB4A39/5BE460F1" Ref="U?"  Part="1"
 AR Path="/5BE41138/5BE460F1" Ref="U?"  Part="1"
-F 0 "U6" H 6150 4633 50  0000 C CNN
+F 0 "U?" H 6150 4633 50  0000 C CNN
 F 1 "OMRON-G3MB-202P" H 6150 4724 50  0000 C CNN
 F 2 "footprint-lib:OMRON-G3MB-202P" H 5950 4750 50  0001 L CIN
@@
 	6450 5050 7700 5050
 $Comp
-L power:VDD #PWR0121
+L power:VDD #PWR?
 U 1 1 5BE46103
 P 5050 4450
-AR Path="/5BCB4A39/5BE46103" Ref="#PWR0121"  Part="1"
+AR Path="/5BCB4A39/5BE46103" Ref="#PWR?"  Part="1"
 AR Path="/5BE41138/5BE46103" Ref="#PWR?"  Part="1"
-F 0 "#PWR0121" H 5050 4300 50  0001 C CNN
+F 0 "#PWR?" H 5050 4300 50  0001 C CNN
 F 1 "VDD" H 5067 4623 50  0000 C CNN
 F 2 "" H 5050 4450 50  0001 C CNN
@@
 P 5100 5550
 AR Path="/5BE4610D" Ref="Q?"  Part="1"
-AR Path="/5BCB4A39/5BE4610D" Ref="Q3"  Part="1"
+AR Path="/5BCB4A39/5BE4610D" Ref="Q?"  Part="1"
 AR Path="/5BE41138/5BE4610D" Ref="Q?"  Part="1"
-F 0 "Q3" H 5300 5600 50  0000 L CNN
+F 0 "Q?" H 5300 5600 50  0000 L CNN
 F 1 "2N3904(1AM)" H 5300 5550 50  0000 L CNN
 F 2 "Package_TO_SOT_SMD:SOT-23_Handsoldering" H 5300 5475 50  0001 L CIN
