File: pcb/WS2812_PWM_DRIVER.sch (KiCad schematic (older format))
At the start: 1 part, among them U1 74AHCT1G125

Commit message: update,
Parts:
- renumbered U1 to U?
Changed lines of the file:
@@
 EESchema Schematic File Version 4
+LIBS:backplane-cache
 LIBS:stm32_bottom_board_respin-cache
 EELAYER 26 0
@@
 $Descr A4 11693 8268
 encoding utf-8
-Sheet 6 8
+Sheet 6 9
 Title ""
 Date ""
@@
 $EndDescr
 $Comp
-L taobao-components:74AHCT1G125 U1
+L taobao-components:74AHCT1G125 U?
 U 1 1 5BCB46C2
 P 5400 3200
-AR Path="/5BCB46C2" Ref="U1"  Part="1"
-AR Path="/5BCB4060/5BCB46C2" Ref="U1"  Part="1"
-F 0 "U1" H 5375 3026 50  0000 C CNN
+AR Path="/5BCB46C2" Ref="U?"  Part="1"
+AR Path="/5BCB4060/5BCB46C2" Ref="U?"  Part="1"
+F 0 "U?" H 5375 3026 50  0000 C CNN
 F 1 "74AHCT1G125" H 5375 2935 50  0000 C CNN
 F 2 "Package_TO_SOT_SMD:SOT-23-5_HandSoldering" H 5400 3200 50  0001 C CNN
@@
 	4500 3200 5100 3200
 $Comp
-L power:VDD #PWR010
+L power:VDD #PWR?
 U 1 1 5BCB476F
 P 5550 2750
-F 0 "#PWR010" H 5550 2600 50  0001 C CNN
+F 0 "#PWR?" H 5550 2600 50  0001 C CNN
 F 1 "VDD" H 5567 2923 50  0000 C CNN
 F 2 "" H 5550 2750 50  0001 C CNN
@@
 $EndComp
 $Comp
-L power:GND #PWR08
+L power:GND #PWR?
 U 1 1 5BCB47D3
 P 5250 2750
-F 0 "#PWR08" H 5250 2500 50  0001 C CNN
+F 0 "#PWR?" H 5250 2500 50  0001 C CNN
 F 1 "GND" H 5255 2577 50  0000 C CNN
 F 2 "" H 5250 2750 50  0001 C CNN
@@
 	5450 2850 5450 3150
 $Comp
-L power:GND #PWR09
+L power:GND #PWR?
 U 1 1 5BCB4815
 P 5450 3700
-F 0 "#PWR09" H 5450 3450 50  0001 C CNN
+F 0 "#PWR?" H 5450 3450 50  0001 C CNN
 F 1 "GND" H 5455 3527 50  0000 C CNN
 F 2 "" H 5450 3700 50  0001 C CNN
