File: pcb/rs232_level_switch.sch (KiCad schematic (older format))
At the start: 6 parts, among them U5 SP3232EEN

Commit message: update,
Parts:
- added D4, D5: LED_GREEN, LED_SMD:LED_0805_2012Metric_Pad1.15x1.40mm_HandSolder, symbol taobao-components:LED_GREEN
- added R14, R15: R102, Resistor_SMD:R_0805_2012Metric_Pad1.15x1.40mm_HandSolder, symbol taobao-r:R511
Connections:
- net TTL-RX1: now also D5.1 (K)
- net TTL-TX1: now also D4.1 (K)
- net VDD: now also R14.1, R15.1
- new net: D4.2 (A), R14.2
- new net: D5.2 (A), R15.2
Changed lines of the file:
@@
 Wire Wire Line
 	5700 4550 5700 4700
-Wire Wire Line
-	4500 3900 5100 3900
-Wire Wire Line
-	4500 4100 5100 4100
-Text HLabel 4500 3900 0    50   Input ~ 0
+Text HLabel 3350 3900 0    50   Input ~ 0
 TTL-TX1
-Text HLabel 4500 4000 0    50   Input ~ 0
+Text HLabel 3350 4000 0    50   Input ~ 0
 TTL-TX2
-Text HLabel 4500 4100 0    50   Input ~ 0
+Text HLabel 3350 4100 0    50   Input ~ 0
 TTL-RX1
-Text HLabel 4500 4200 0    50   Input ~ 0
+Text HLabel 3350 4200 0    50   Input ~ 0
 TTL-RX2
-Wire Wire Line
-	4500 4000 5100 4000
-Wire Wire Line
-	5100 4200 4500 4200
 Wire Wire Line
 	6300 3900 6800 3900
@@
 	1    0    0    -1
 $EndComp
+$Comp
+L taobao-r:R511 R14
+U 1 1 5BD94646
+P 3700 3250
+F 0 "R14" H 3642 3296 50  0000 R CNN
+F 1 "R102" H 3642 3205 50  0000 R CNN
+F 2 "Resistor_SMD:R_0805_2012Metric_Pad1.15x1.40mm_HandSolder" H 3700 3250 50  0001 C CNN
+F 3 "~" H 3700 3250 50  0001 C CNN
+	1    3700 3250
+	1    0    0    -1
+$EndComp
+$Comp
+L taobao-components:LED_GREEN D4
+U 1 1 5BD94746
+P 3700 3600
+F 0 "D4" V 3746 3697 50  0000 L CNN
+F 1 "LED_GREEN" V 3655 3697 50  0000 L CNN
+F 2 "LED_SMD:LED_0805_2012Metric_Pad1.15x1.40mm_HandSolder" V 3700 3600 50  0001 C CNN
+F 3 "" V 3700 3600 50  0001 C CNN
+	1    3700 3600
+	0    -1   -1   0
+$EndComp
+Wire Wire Line
+	5100 3900 3700 3900
+Wire Wire Line
+	5100 4000 3350 4000
+Wire Wire Line
+	5100 4100 3900 4100
+Wire Wire Line
+	5100 4200 3350 4200
+$Comp
+L taobao-r:R511 R15
+U 1 1 5BD95DFC
+P 3900 3250
+F 0 "R15" H 3959 3296 50  0000 L CNN
+F 1 "R102" H 3959 3205 50  0000 L CNN
+F 2 "Resistor_SMD:R_0805_2012Metric_Pad1.15x1.40mm_HandSolder" H 3900 3250 50  0001 C CNN
+F 3 "~" H 3900 3250 50  0001 C CNN
+	1    3900 3250
+	1    0    0    -1
+$EndComp
+$Comp
+L taobao-components:LED_GREEN D5
+U 1 1 5BD95E02
+P 3900 3600
+F 0 "D5" V 3946 3532 50  0000 R CNN
+F 1 "LED_GREEN" V 3855 3532 50  0000 R CNN
+F 2 "LED_SMD:LED_0805_2012Metric_Pad1.15x1.40mm_HandSolder" V 3900 3600 50  0001 C CNN
+F 3 "" V 3900 3600 50  0001 C CNN
+	1    3900 3600
+	0    -1   -1   0
+$EndComp
+$Comp
+L power:VDD #PWR0108
+U 1 1 5BD961A3
+P 3800 3050
+F 0 "#PWR0108" H 3800 2900 50  0001 C CNN
+F 1 "VDD" H 3817 3223 50  0000 C CNN
+F 2 "" H 3800 3050 50  0001 C CNN
+F 3 "" H 3800 3050 50  0001 C CNN
+	1    3800 3050
+	1    0    0    -1
+$EndComp
+Wire Wire Line
+	3800 3050 3800 3100
+Wire Wire Line
+	3800 3100 3700 3100
+Wire Wire Line
+	3700 3100 3700 3150
+Wire Wire Line
+	3800 3100 3900 3100
+Wire Wire Line
+	3900 3100 3900 3150
+Connection ~ 3800 3100
+Wire Wire Line
+	3700 3350 3700 3500
+Wire Wire Line
+	3900 3350 3900 3500
+Wire Wire Line
+	3700 3700 3700 3900
+Connection ~ 3700 3900
+Wire Wire Line
+	3700 3900 3350 3900
+Wire Wire Line
+	3900 3700 3900 4100
+Connection ~ 3900 4100
+Wire Wire Line
+	3900 4100 3350 4100
 $EndSCHEMATC

Commit message: assign footprint,
Parts:
- R14, R15: footprint Resistor_SMD:R_0805_2012Metric_Pad1.15x1.40mm_HandSolder -> Resistor_SMD:R_0603_1608Metric_Pad1.05x0.95mm_HandSolder
Changed lines of the file:
@@
 F 0 "R14" H 3642 3296 50  0000 R CNN
 F 1 "R102" H 3642 3205 50  0000 R CNN
-F 2 "Resistor_SMD:R_0805_2012Metric_Pad1.15x1.40mm_HandSolder" H 3700 3250 50  0001 C CNN
+F 2 "Resistor_SMD:R_0603_1608Metric_Pad1.05x0.95mm_HandSolder" H 3700 3250 50  0001 C CNN
 F 3 "~" H 3700 3250 50  0001 C CNN
 	1    3700 3250
@@
 F 0 "R15" H 3959 3296 50  0000 L CNN
 F 1 "R102" H 3959 3205 50  0000 L CNN
-F 2 "Resistor_SMD:R_0805_2012Metric_Pad1.15x1.40mm_HandSolder" H 3900 3250 50  0001 C CNN
+F 2 "Resistor_SMD:R_0603_1608Metric_Pad1.05x0.95mm_HandSolder" H 3900 3250 50  0001 C CNN
 F 3 "~" H 3900 3250 50  0001 C CNN
 	1    3900 3250

Commit message: update,
Parts:
- renumbered C15 to C?, C16 to C?, C17 to C?, C18 to C?, C19 to C?, D4 to D?, D5 to D?, R14 to R?, R15 to R?, U5 to U?
Changed lines of the file:
@@
 EESchema Schematic File Version 4
+LIBS:backplane-cache
 LIBS:stm32_bottom_board_respin-cache
 EELAYER 26 0
@@
 $Descr A4 11693 8268
 encoding utf-8
-Sheet 7 8
+Sheet 7 9
 Title ""
 Date ""
@@
 $EndDescr
 $Comp
-L taobao-c:C104 C15
+L taobao-c:C104 C?
 U 1 1 5BCE722E
 P 4900 3150
-F 0 "C15" H 4992 3196 50  0000 L CNN
+F 0 "C?" H 4992 3196 50  0000 L CNN
 F 1 "C104" H 4992 3105 50  0000 L CNN
 F 2 "Capacitor_SMD:C_0805_2012Metric_Pad1.15x1.40mm_HandSolder" H 4900 3150 50  0001 C CNN
@@
 	4900 3300 5100 3300
 $Comp
-L taobao-c:C104 C16
+L taobao-c:C104 C?
 U 1 1 5BCE7274
 P 4900 3600
-F 0 "C16" H 4992 3646 50  0000 L CNN
+F 0 "C?" H 4992 3646 50  0000 L CNN
 F 1 "C104" H 4992 3555 50  0000 L CNN
 F 2 "Capacitor_SMD:C_0805_2012Metric_Pad1.15x1.40mm_HandSolder" H 4900 3600 50  0001 C CNN
@@
 	4900 3750 4900 3700
 $Comp
-L taobao-c:C104 C17
+L taobao-c:C104 C?
 U 1 1 5BCE86C7
 P 6050 2350
-F 0 "C17" V 5821 2350 50  0000 C CNN
+F 0 "C?" V 5821 2350 50  0000 C CNN
 F 1 "C104" V 5912 2350 50  0000 C CNN
 F 2 "Capacitor_SMD:C_0805_2012Metric_Pad1.15x1.40mm_HandSolder" H 6050 2350 50  0001 C CNN
@@
 $EndComp
 $Comp
-L power:VDD #PWR0102
+L power:VDD #PWR?
 U 1 1 5BCE8CF9
 P 5700 1850
-F 0 "#PWR0102" H 5700 1700 50  0001 C CNN
+F 0 "#PWR?" H 5700 1700 50  0001 C CNN
 F 1 "VDD" H 5717 2023 50  0000 C CNN
 F 2 "" H 5700 1850 50  0001 C CNN
@@
 	5700 2350 5700 2700
 $Comp
-L taobao-c:C104 C18
+L taobao-c:C104 C?
 U 1 1 5BCE8DB1
 P 6700 3050
-F 0 "C18" V 6471 3050 50  0000 C CNN
+F 0 "C?" V 6471 3050 50  0000 C CNN
 F 1 "C104" V 6562 3050 50  0000 C CNN
 F 2 "Capacitor_SMD:C_0805_2012Metric_Pad1.15x1.40mm_HandSolder" H 6700 3050 50  0001 C CNN
@@
 $EndComp
 $Comp
-L taobao-c:C104 C19
+L taobao-c:C104 C?
 U 1 1 5BCE8DF5
 P 6700 3450
-F 0 "C19" V 6471 3450 50  0000 C CNN
+F 0 "C?" V 6471 3450 50  0000 C CNN
 F 1 "C104" V 6562 3450 50  0000 C CNN
 F 2 "Capacitor_SMD:C_0805_2012Metric_Pad1.15x1.40mm_HandSolder" H 6700 3450 50  0001 C CNN
@@
 Connection ~ 6950 3050
 $Comp
-L power:GND #PWR0103
+L power:GND #PWR?
 U 1 1 5BCE9117
 P 6950 3600
-F 0 "#PWR0103" H 6950 3350 50  0001 C CNN
+F 0 "#PWR?" H 6950 3350 50  0001 C CNN
 F 1 "GND" H 6955 3427 50  0000 C CNN
 F 2 "" H 6950 3600 50  0001 C CNN
@@
 Connection ~ 6950 3450
 $Comp
-L power:GND #PWR0104
+L power:GND #PWR?
 U 1 1 5BCE9791
 P 5700 4700
-F 0 "#PWR0104" H 5700 4450 50  0001 C CNN
+F 0 "#PWR?" H 5700 4450 50  0001 C CNN
 F 1 "GND" H 5705 4527 50  0000 C CNN
 F 2 "" H 5700 4700 50  0001 C CNN
@@
 RS232-RX2
 $Comp
-L taobao-components:SP3232EEN U5
+L taobao-components:SP3232EEN U?
 U 1 1 5BCEE512
 P 5700 3500
-F 0 "U5" H 5700 4478 50  0000 C CNN
+F 0 "U?" H 5700 4478 50  0000 C CNN
 F 1 "SP3232EEN" H 5700 4387 50  0000 C CNN
 F 2 "footprint-lib:SOP-16_4.4x10.4mm_Pitch1.27mm" H 5700 3000 50  0001 C CNN
@@
 $EndComp
 $Comp
-L taobao-r:R511 R14
+L taobao-r:R511 R?
 U 1 1 5BD94646
 P 3700 3250
-F 0 "R14" H 3642 3296 50  0000 R CNN
+F 0 "R?" H 3642 3296 50  0000 R CNN
 F 1 "R102" H 3642 3205 50  0000 R CNN
 F 2 "Resistor_SMD:R_0603_1608Metric_Pad1.05x0.95mm_HandSolder" H 3700 3250 50  0001 C CNN
@@
 $EndComp
 $Comp
-L taobao-components:LED_GREEN D4
+L taobao-components:LED_GREEN D?
 U 1 1 5BD94746
 P 3700 3600
-F 0 "D4" V 3746 3697 50  0000 L CNN
+F 0 "D?" V 3746 3697 50  0000 L CNN
 F 1 "LED_GREEN" V 3655 3697 50  0000 L CNN
 F 2 "LED_SMD:LED_0805_2012Metric_Pad1.15x1.40mm_HandSolder" V 3700 3600 50  0001 C CNN
@@
 	5100 4200 3350 4200
 $Comp
-L taobao-r:R511 R15
+L taobao-r:R511 R?
 U 1 1 5BD95DFC
 P 3900 3250
-F 0 "R15" H 3959 3296 50  0000 L CNN
+F 0 "R?" H 3959 3296 50  0000 L CNN
 F 1 "R102" H 3959 3205 50  0000 L CNN
 F 2 "Resistor_SMD:R_0603_1608Metric_Pad1.05x0.95mm_HandSolder" H 3900 3250 50  0001 C CNN
@@
 $EndComp
 $Comp
-L taobao-components:LED_GREEN D5
+L taobao-components:LED_GREEN D?
 U 1 1 5BD95E02
 P 3900 3600
-F 0 "D5" V 3946 3532 50  0000 R CNN
+F 0 "D?" V 3946 3532 50  0000 R CNN
 F 1 "LED_GREEN" V 3855 3532 50  0000 R CNN
 F 2 "LED_SMD:LED_0805_2012Metric_Pad1.15x1.40mm_HandSolder" V 3900 3600 50  0001 C CNN
@@
 $EndComp
 $Comp
-L power:VDD #PWR0108
+L power:VDD #PWR?
 U 1 1 5BD961A3
 P 3800 3050
-F 0 "#PWR0108" H 3800 2900 50  0001 C CNN
+F 0 "#PWR?" H 3800 2900 50  0001 C CNN
 F 1 "VDD" H 3817 3223 50  0000 C CNN
 F 2 "" H 3800 3050 50  0001 C CNN
