File: backplane/_autosave-backplane.kicad_pcb (KiCad board)
At the start: 2 copper layers, 200 x 300 mm, 14 parts, among them J1 Conn_PCB1, J10 Conn_SSR_INPUT, J12 Conn_SSR_PCB2, J13 Conn_01x05, J15 Screw_Terminal_AQ_2, J16 Screw_Terminal_AQ_1, J17 Screw_Terminal_O3_1, J18 Conn_TO_ION_AIR, J2 Conn_PCB2, J23 PCB1_COMM_CONNECTOR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

Commit message: update,
Parts:
- J15: footprint backplate:Pin_Header_Straight_1x04_Pitch2.54mm -> footprint-lib:mpt_0,5%2f4-2,54
- J16, J17: footprint backplate:PhoenixContact_MCV_1,5_4-G-3.5_1x04_P3.50mm_Vertical_handsolder -> footprint-lib:mpt_0,5%2f4-2,54

Commit message: update J17,
Parts:
- J15: footprint footprint-lib:mpt_0,5%2f4-2,54 -> backplate:Pin_Header_Straight_1x04_Pitch2.54mm
- J16: footprint footprint-lib:mpt_0,5%2f4-2,54 -> backplate:PhoenixContact_MCV_1,5_4-G-3.5_1x04_P3.50mm_Vertical_handsolder
- moved J17 4.57 mm to (11.5, 167.1)
Connections:
- J17 pad 1: /O3_1_GND -> /O3_1_SHIELD
- J17 pad 2: /O3_1_24V -> /O3_1_SENSOR
- J17 pad 3: /O3_1_SENSOR -> /O3_1_24V
- J17 pad 4: /O3_1_SHIELD -> /O3_1_GND
