File: backplane/backplane.kicad_pcb (KiCad board)
At the start: 2 copper layers, 200 x 300 mm, 14 parts, among them J1 Conn_PCB1, J10 Conn_SSR_INPUT, J12 Conn_SSR_PCB2, J13 Conn_01x05, J15 Screw_Terminal_AQ_2, J16 Screw_Terminal_AQ_1, J17 Screw_Terminal_O3_1, J18 Conn_TO_ION_AIR, J2 Conn_PCB2, J23 PCB1_COMM_CONNECTOR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

Commit message: update,
Parts:
- J13: footprint backplate:PhoenixContact_MCV_1,5_8-G-3.5_1x05_P3.50mm_Vertical_handsolder -> footprint-lib:mpt_0,5%2f5-2,54
- J16, J17: footprint backplate:PhoenixContact_MCV_1,5_4-G-3.5_1x04_P3.50mm_Vertical_handsolder -> footprint-lib:mpt_0,5%2f4-2,54
- moved J17 4.57 mm to (11.5, 167.1)
Connections:
- J13 pad 1: /flow_sensor_shield -> /flow_sensor_GND
- J13 pad 2: /flow_sensor_%RH -> /flow_sensor_24V
- J13 pad 4: /flow_sensor_24V -> /flow_sensor_%RH
- J13 pad 5: /flow_sensor_GND -> /flow_sensor_shield
- J16 pad 1: /AQ1_GND -> /AQ1_SHIELD
- J16 pad 2: /AQ1_5V -> /AQ1_SENSOR
- J16 pad 3: /AQ1_SENSOR -> /AQ1_5V
- J16 pad 4: /AQ1_SHIELD -> /AQ1_GND
- J17 pad 1: /O3_1_GND -> /O3_1_SHIELD
- J17 pad 2: /O3_1_24V -> /O3_1_SENSOR
- J17 pad 3: /O3_1_SENSOR -> /O3_1_24V
- J17 pad 4: /O3_1_SHIELD -> /O3_1_GND

Commit message: update,
Parts:
- J13: value Conn_01x05 -> FLOW_SENSOR
- J15: value Screw_Terminal_AQ_2 -> AQ2_SENSOR; footprint backplate:Pin_Header_Straight_1x04_Pitch2.54mm -> footprint-lib:mpt_0,5%2f4-2,54; moved to F.Cu
- J16: value Screw_Terminal_AQ_1 -> AQ1_SENSOR
- J17: value Screw_Terminal_O3_1 -> O3_SENSOR
- J3: value Conn_SSR_INPUT -> SSR_CONTROL
- J4: value Conn_01x08 -> TO_CONTROL_BOARD
- moved J15 132.4 mm to (11.5, 189.1), turned to 270 degrees
- moved J17 12.0 mm to (11.5, 155.1)
- moved J16 10.5 mm to (11.7, 173.1)
- moved J13 0.21 mm to (11.5, 202.4)
Connections:
- J15 pad 1: /AQ2_SHIELD -> /AQ2_GND
- J15 pad 2: /AQ2_SENSOR -> /AQ2_5V
- J15 pad 3: /AQ2_5V -> /AQ2_SENSOR
- J15 pad 4: /AQ2_GND -> /AQ2_SHIELD
Routing:
- net GND: track 408.8 -> 684.6 mm
- net /AQ2_SHIELD: track 31.1 -> 175.4 mm
- net /AQ2_SENSOR: track 32.5 -> 171.6 mm
- net /AQ2_5V: track 32.0 -> 165.6 mm
- net /AQ2_GND: track 31.1 -> 159.4 mm
- net /flow_sensor_%RH: track 214.0 -> 236.4 mm
- net /SSR-24-DA_P: track 38.9 -> 52.4 mm
- net /PCB1_232_RX: track 38.6 -> 48.6 mm
- net /SSR-24-DA_N: track 30.6 -> 40.1 mm
- net /O3_1_SHIELD: track 233.0 -> 239.0 mm
- net /AQ1_SENSOR: track 225.3 -> 219.5 mm
- net /O3_1_SENSOR: track 245.9 -> 251.5 mm
- net /O3_1_24V: track 240.8 -> 246.0 mm
- net /O3_1_GND: track 252.1 -> 256.9 mm
- net /AQ1_GND: track 231.6 -> 226.9 mm
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Other:
- net class 1 mil: clearance 0.5 -> 0.2
- net class 2 mil: clearance 1 -> 0.2
- board text removed: "220V SUPPLY"
- board text removed: "AQ1"
- board text removed: "AQ2"
- board text removed: "O3 SENSOR"
- board text removed: "SSR_CONTROL"

Commit message: update,
Parts:
- added RLY***: relay_SSR-xxDA, w_relay:relay_SSR-xxDA, F.Cu at (40.1, 180.3)
- moved J3 70.7 mm to (40.1, 124.1)
Routing:
- net GND: track 684.6 -> 363.8 mm
- net +5V: track 280.8 -> 323.7 mm
- net /SSR-24-DA_N: track 40.1 -> 74.5 mm
- net /SSR-24-DA_P: track 52.4 -> 78.7 mm
- net /flow_sensor_%RH: track 236.4 -> 249.6 mm
- net /AQ2_5V: track 165.6 -> 178.1 mm
- net /flow_sensor_24V: track 253.7 -> 264.6 mm
- net /flow_sensor_GND: track 213.2 -> 222.5 mm
- net /To_J1_P11: track 201.9 -> 194.0 mm
- net /flow_sensor_FLOW: track 214.4 -> 222.2 mm
- net /AQ2_GND: track 159.4 -> 166.5 mm
- net /To_J1_P3: track 200.2 -> 194.0 mm
- net /To_J1_P6: track 215.7 -> 221.1 mm
- net /To_J1_P5: track 195.1 -> 190.4 mm
- net /To_J1_P10: track 197.5 -> 202.2 mm
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
Commit message: update board mounting hole,
Parts:
- removed RLY***: relay_SSR-xxDA, w_relay:relay_SSR-xxDA
- added H1: PCB2, MountingHole:MountingHole_3.2mm_M3_DIN965, F.Cu at (80.7, 124.8)
- added H2: PCB2, MountingHole:MountingHole_3.2mm_M3_DIN965, F.Cu at (189.2, 107.0)
- added H3: PCB2, MountingHole:MountingHole_3.2mm_M3_DIN965, F.Cu at (197.7, 150.8)
- added H4: PCB2, MountingHole:MountingHole_3.2mm_M3_DIN965, F.Cu at (106.2, 107.0)
- added H5: PCB1, MountingHole:MountingHole_3.2mm_M3_DIN965, F.Cu at (196.7, 206.2)
- added H6: PCB1, MountingHole:MountingHole_3.2mm_M3_DIN965, F.Cu at (189.2, 7.00)
- added H7: PCB1, MountingHole:MountingHole_3.2mm_M3_DIN965, F.Cu at (120.2, 259.8)
- added H8: PCB1, MountingHole:MountingHole_3.2mm_M3_DIN965, F.Cu at (106.2, 7.00)
- added H9: PCB1, MountingHole:MountingHole_3.2mm_M3_DIN965, F.Cu at (184.2, 259.8)
Other:
- outline, holes or cut-outs redrawn

Commit message: update,
Parts:
- added H10: PCB1, MountingHole:MountingHole_3.2mm_M3_DIN965, F.Cu at (28.0, 145.0)
- added H11: PCB1, MountingHole:MountingHole_3.2mm_M3_DIN965, F.Cu at (188.0, 145.0)
- added H12: PCB1, MountingHole:MountingHole_3.2mm_M3_DIN965, F.Cu at (28.0, 15.0)
- added H13: PCB1, MountingHole:MountingHole_3.2mm_M3_DIN965, F.Cu at (28.0, 275.0)
- added H14: PCB1, MountingHole:MountingHole_3.2mm_M3_DIN965, F.Cu at (188.0, 15.0)
- added H15: PCB1, MountingHole:MountingHole_3.2mm_M3_DIN965, F.Cu at (188.0, 275.0)
Other:
- outline, holes or cut-outs redrawn
Changed lines of the file:
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@@
   (general
     (thickness 1.6)
-    (drawings 27)
+    (drawings 20)
     (tracks 457)
     (zones 0)
-    (modules 23)
+    (modules 29)
     (nets 45)
   )
@@
     (add_net /PWR_SOURCE_SSR_L_1)
     (add_net /SSR_PCB2_L_2)
+  )
+  (module MountingHole:MountingHole_3.2mm_M3_DIN965 locked (layer F.Cu)
+    (at 187.999998 275)
+    (descr "Mounting Hole 3.2mm, no annular, M3, DIN965")
+    (tags "mounting hole 3.2mm no annular m3 din965")
+    (attr virtual)
+    (fp_text reference H15 (at 0 -3.8) (layer F.SilkS)
+      (effects (font (size 1 1) (thickness 0.15)))
+    )
+    (fp_text value PCB1 (at 0 3.8) (layer F.Fab)
+      (effects (font (size 1 1) (thickness 0.15)))
+    )
+    (fp_circle (center 0 0) (end 3.05 0) (layer F.CrtYd) (width 0.05))
+    (fp_circle (center 0 0) (end 2.8 0) (layer Cmts.User) (width 0.15))
+    (fp_text user %R (at 0.3 0) (layer F.Fab)
+      (effects (font (size 1 1) (thickness 0.15)))
+    )
+    (pad 1 np_thru_hole circle (at 0 0) (size 3.2 3.2) (drill 3.2) (layers *.Cu *.Mask))
+  )
+  (module MountingHole:MountingHole_3.2mm_M3_DIN965 locked (layer F.Cu)
+    (at 187.999998 15)
+    (descr "Mounting Hole 3.2mm, no annular, M3, DIN965")
+    (tags "mounting hole 3.2mm no annular m3 din965")
+    (attr virtual)
+    (fp_text reference H14 (at 0 -3.8) (layer F.SilkS)
+      (effects (font (size 1 1) (thickness 0.15)))
+    )
+    (fp_text value PCB1 (at 0 3.8) (layer F.Fab)
+      (effects (font (size 1 1) (thickness 0.15)))
+    )
+    (fp_text user %R (at 0.3 0) (layer F.Fab)
+      (effects (font (size 1 1) (thickness 0.15)))
+    )
+    (fp_circle (center 0 0) (end 2.8 0) (layer Cmts.User) (width 0.15))
+    (fp_circle (center 0 0) (end 3.05 0) (layer F.CrtYd) (width 0.05))
+    (pad 1 np_thru_hole circle (at 0 0) (size 3.2 3.2) (drill 3.2) (layers *.Cu *.Mask))
+  )
+  (module MountingHole:MountingHole_3.2mm_M3_DIN965 locked (layer F.Cu)
+    (at 27.983998 275)
+    (descr "Mounting Hole 3.2mm, no annular, M3, DIN965")
+    (tags "mounting hole 3.2mm no annular m3 din965")
+    (attr virtual)
+    (fp_text reference H13 (at 0 -3.8) (layer F.SilkS)
+      (effects (font (size 1 1) (thickness 0.15)))
+    )
+    (fp_text value PCB1 (at 0 3.8) (layer F.Fab)
+      (effects (font (size 1 1) (thickness 0.15)))
+    )
+    (fp_circle (center 0 0) (end 3.05 0) (layer F.CrtYd) (width 0.05))
+    (fp_circle (center 0 0) (end 2.8 0) (layer Cmts.User) (width 0.15))
+    (fp_text user %R (at 0.3 0) (layer F.Fab)
+      (effects (font (size 1 1) (thickness 0.15)))
+    )
+    (pad 1 np_thru_hole circle (at 0 0) (size 3.2 3.2) (drill 3.2) (layers *.Cu *.Mask))
+  )
+  (module MountingHole:MountingHole_3.2mm_M3_DIN965 locked (layer F.Cu)
+    (at 27.999998 15)
+    (descr "Mounting Hole 3.2mm, no annular, M3, DIN965")
+    (tags "mounting hole 3.2mm no annular m3 din965")
+    (attr virtual)
+    (fp_text reference H12 (at 0 -3.8) (layer F.SilkS)
+      (effects (font (size 1 1) (thickness 0.15)))
+    )
+    (fp_text value PCB1 (at 0 3.8) (layer F.Fab)
+      (effects (font (size 1 1) (thickness 0.15)))
+    )
+    (fp_text user %R (at 0.3 0) (layer F.Fab)
+      (effects (font (size 1 1) (thickness 0.15)))
+    )
+    (fp_circle (center 0 0) (end 2.8 0) (layer Cmts.User) (width 0.15))
+    (fp_circle (center 0 0) (end 3.05 0) (layer F.CrtYd) (width 0.05))
+    (pad 1 np_thru_hole circle (at 0 0) (size 3.2 3.2) (drill 3.2) (layers *.Cu *.Mask))
+  )
+  (module MountingHole:MountingHole_3.2mm_M3_DIN965 locked (layer F.Cu)
+    (at 187.999998 145)
+    (descr "Mounting Hole 3.2mm, no annular, M3, DIN965")
+    (tags "mounting hole 3.2mm no annular m3 din965")
+    (attr virtual)
+    (fp_text reference H11 (at 0 -3.8) (layer F.SilkS)
+      (effects (font (size 1 1) (thickness 0.15)))
+    )
+    (fp_text value PCB1 (at 0 3.8) (layer F.Fab)
+      (effects (font (size 1 1) (thickness 0.15)))
+    )
+    (fp_circle (center 0 0) (end 3.05 0) (layer F.CrtYd) (width 0.05))
+    (fp_circle (center 0 0) (end 2.8 0) (layer Cmts.User) (width 0.15))
+    (fp_text user %R (at 0.3 0) (layer F.Fab)
+      (effects (font (size 1 1) (thickness 0.15)))
+    )
+    (pad 1 np_thru_hole circle (at 0 0) (size 3.2 3.2) (drill 3.2) (layers *.Cu *.Mask))
+  )
+  (module MountingHole:MountingHole_3.2mm_M3_DIN965 locked (layer F.Cu)
+    (at 27.999998 145)
+    (descr "Mounting Hole 3.2mm, no annular, M3, DIN965")
+    (tags "mounting hole 3.2mm no annular m3 din965")
+    (attr virtual)
+    (fp_text reference H10 (at 0 -3.8) (layer F.SilkS)
+      (effects (font (size 1 1) (thickness 0.15)))
+    )
+    (fp_text value PCB1 (at 0 3.8) (layer F.Fab)
+      (effects (font (size 1 1) (thickness 0.15)))
+    )
+    (fp_text user %R (at 0.3 0) (layer F.Fab)
+      (effects (font (size 1 1) (thickness 0.15)))
+    )
+    (fp_circle (center 0 0) (end 2.8 0) (layer Cmts.User) (width 0.15))
+    (fp_circle (center 0 0) (end 3.05 0) (layer F.CrtYd) (width 0.05))
+    (pad 1 np_thru_hole circle (at 0 0) (size 3.2 3.2) (drill 3.2) (layers *.Cu *.Mask))
   )
   (module MountingHole:MountingHole_3.2mm_M3_DIN965 locked (layer F.Cu)
@@
   (gr_circle (center 101 202) (end 102.5 202) (layer Edge.Cuts) (width 1))
   (gr_circle (center 101 199) (end 114 199) (layer Edge.Cuts) (width 1))
-  (gr_circle (center 27.999998 15) (end 26.999998 15) (layer Edge.Cuts) (width 1))
-  (gr_circle (center 187.999998 15) (end 186.999998 15) (layer Edge.Cuts) (width 1))
-  (gr_circle (center 187.999998 145) (end 186.999998 145) (layer Edge.Cuts) (width 1))
-  (gr_circle (center 27.999998 145) (end 26.999998 145) (layer Edge.Cuts) (width 1))
-  (gr_circle (center 27.983998 275) (end 26.983998 275) (layer Edge.Cuts) (width 1))
-  (gr_circle (center 187.999998 275) (end 186.999998 275) (layer Edge.Cuts) (width 1))
-  (gr_line (start 207.930998 223.25) (end 207.930998 243.25) (angle 90) (layer Dwgs.User) (width 0.2))
-  (gr_line (start 197.930998 243.25) (end 207.930998 243.25) (angle 90) (layer Dwgs.User) (width 0.2))
-  (gr_line (start 197.930998 223.25) (end 197.930998 243.25) (angle 90) (layer Dwgs.User) (width 0.2))
-  (gr_line (start 207.930998 223.25) (end 197.930998 223.25) (angle 90) (layer Dwgs.User) (width 0.2))
-  (gr_text "220V \nTO PCB2" (at 17.78 288.29) (layer F.SilkS)
+  (gr_line (start 189.931 248.25) (end 199.931 248.25) (angle 90) (layer Dwgs.User) (width 0.2))
+  (gr_line (start 189.931 228.25) (end 189.931 248.25) (angle 90) (layer Dwgs.User) (width 0.2))
+  (gr_line (start 199.931 228.25) (end 189.931 228.25) (angle 90) (layer Dwgs.User) (width 0.2))
+  (gr_text "220V \nTO PCB2" (at 31.636 287.8) (layer F.SilkS)
     (effects (font (size 3 3) (thickness 0.5)) (justify right))
   )
-  (gr_circle (center 187.999998 145) (end 190.999998 145) (layer Edge.Cuts) (width 1))
-  (gr_circle (center 27.999998 145) (end 30.999998 145) (layer Edge.Cuts) (width 1))
-  (gr_circle (center 187.999998 15) (end 193.999998 15) (layer Edge.Cuts) (width 1))
-  (gr_circle (center 27.999998 15) (end 33.999998 15) (layer Edge.Cuts) (width 1))
-  (gr_circle (center 187.999998 275) (end 193.999998 275) (layer Edge.Cuts) (width 1))
-  (gr_circle (center 27.999998 275) (end 33.999998 275) (layer Edge.Cuts) (width 1))
-  (gr_line (start 7.999998 295) (end 207.999998 295) (angle 90) (layer Dwgs.User) (width 1))
-  (gr_line (start 207.999998 -5) (end 207.999998 295) (angle 90) (layer Dwgs.User) (width 1))
-  (gr_line (start 7.999998 -5) (end 207.999998 -5) (angle 90) (layer Dwgs.User) (width 1))
-  (gr_line (start 7.999998 -5) (end 7.999998 295) (angle 90) (layer Dwgs.User) (width 1))
+  (gr_circle (center 187.999998 145) (end 190.999998 145) (layer Dwgs.User) (width 1))
+  (gr_circle (center 27.999998 145) (end 30.999998 145) (layer Dwgs.User) (width 1))
+  (gr_circle (center 187.999998 15) (end 193.999998 15) (layer Dwgs.User) (width 1))
+  (gr_circle (center 27.999998 15) (end 33.999998 15) (layer Dwgs.User) (width 1))
+  (gr_circle (center 187.999998 275) (end 193.999998 275) (layer Dwgs.User) (width 1))
+  (gr_circle (center 27.999998 275) (end 33.999998 275) (layer Dwgs.User) (width 1))
+  (gr_line (start 0 300) (end 200 300) (angle 90) (layer Dwgs.User) (width 1))
+  (gr_line (start 200 0) (end 200 300) (angle 90) (layer Dwgs.User) (width 1))
+  (gr_line (start 0 0) (end 200 0) (angle 90) (layer Dwgs.User) (width 1))
+  (gr_line (start 0 0) (end 0 300) (angle 90) (layer Dwgs.User) (width 1))
   (segment (start 89.1 94.9) (end 89.1 99.114) (width 1) (layer B.Cu) (net 1) (status 10))
   (segment (start 164.709648 240.24) (end 177.999998 240.24) (width 1) (layer B.Cu) (net 1) (status 20))
@@
     (polygon
       (pts
-        (xy 0.254 235.084269) (xy 75.692 234.830269) (xy 75.692 296.672) (xy 0 296.926) (xy 0.254 296.926)
+        (xy 0.254 235.084269) (xy 75.692 234.830269) (xy 75.692 299.003) (xy 0 299.257) (xy 0.254 296.926)
       )
     )

Commit message: update,
Parts:
- added H16: HEATSINK_SCREW, MountingHole:MountingHole_3.2mm_M3_DIN965, F.Cu at (101.0, 202.0)
Other:
- outline, holes or cut-outs redrawn
Changed lines of the file:
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@@
   (general
     (thickness 1.6)
-    (drawings 20)
+    (drawings 19)
     (tracks 457)
     (zones 0)
-    (modules 29)
+    (modules 30)
     (nets 45)
   )
@@
     (38 B.Mask user)
     (39 F.Mask user)
-    (40 Dwgs.User user hide)
+    (40 Dwgs.User user)
     (41 Cmts.User user)
     (42 Eco1.User user)
@@
     (add_net /PWR_SOURCE_SSR_L_1)
     (add_net /SSR_PCB2_L_2)
+  )
+  (module MountingHole:MountingHole_3.2mm_M3_DIN965 locked (layer F.Cu)
+    (at 101 202)
+    (descr "Mounting Hole 3.2mm, no annular, M3, DIN965")
+    (tags "mounting hole 3.2mm no annular m3 din965")
+    (attr virtual)
+    (fp_text reference H16 (at 0 -3.8) (layer F.SilkS)
+      (effects (font (size 1 1) (thickness 0.15)))
+    )
+    (fp_text value HEATSINK_SCREW (at 0 3.8) (layer F.Fab)
+      (effects (font (size 1 1) (thickness 0.15)))
+    )
+    (fp_text user %R (at 0.3 0) (layer F.Fab)
+      (effects (font (size 1 1) (thickness 0.15)))
+    )
+    (fp_circle (center 0 0) (end 2.8 0) (layer Cmts.User) (width 0.15))
+    (fp_circle (center 0 0) (end 3.05 0) (layer F.CrtYd) (width 0.05))
+    (pad 1 np_thru_hole circle (at 0 0) (size 3.2 3.2) (drill 3.2) (layers *.Cu *.Mask))
   )
   (module MountingHole:MountingHole_3.2mm_M3_DIN965 locked (layer F.Cu)
@@
   (gr_line (start 200 0) (end 200 300) (layer Edge.Cuts) (width 1))
   (gr_line (start 0 0) (end 200 0) (layer Edge.Cuts) (width 1))
-  (gr_circle (center 101 202) (end 102.5 202) (layer Edge.Cuts) (width 1))
-  (gr_circle (center 101 199) (end 114 199) (layer Edge.Cuts) (width 1))
+  (gr_circle (center 101 199) (end 114 199) (layer Dwgs.User) (width 1))
   (gr_line (start 189.931 248.25) (end 199.931 248.25) (angle 90) (layer Dwgs.User) (width 0.2))
   (gr_line (start 189.931 228.25) (end 189.931 248.25) (angle 90) (layer Dwgs.User) (width 0.2))
@@
     (effects (font (size 3 3) (thickness 0.5)) (justify right))
   )
-  (gr_circle (center 187.999998 145) (end 190.999998 145) (layer Dwgs.User) (width 1))
-  (gr_circle (center 27.999998 145) (end 30.999998 145) (layer Dwgs.User) (width 1))
+  (gr_circle (center 187.999998 145) (end 193.999998 145) (layer Dwgs.User) (width 1))
+  (gr_circle (center 27.999998 145) (end 33.999998 145) (layer Dwgs.User) (width 1))
   (gr_circle (center 187.999998 15) (end 193.999998 15) (layer Dwgs.User) (width 1))
   (gr_circle (center 27.999998 15) (end 33.999998 15) (layer Dwgs.User) (width 1))

Commit message: update,
Parts:
- added G***: LOGO, w_logo:Logo_silk_high_voltage_10x8.5mm, F.Cu at (68.7, 240.8)
Routing:
- net +5V: track 323.7 -> 277.0 mm, vias 0 -> 2
- net GND: track 363.8 -> 334.2 mm
- net /PCB1_ALARM_COM: track 277.5 -> 264.4 mm
- net /SSR-24-DA_P: track 78.7 -> 75.4 mm
- net /SSR-24-DA_N: track 74.5 -> 71.5 mm
- net /PCB1_232_TX: track 44.0 -> 43.3 mm
Other:
- net class 0.5 mil: clearance 0.1 -> 1
- net class 1 mil: clearance 0.2 -> 1
- net class 2 mil: clearance 0.2 -> 1
- net class Default: clearance 0.3 -> 1
- rule trace_clearance: 0.3 -> 1

Commit message: update,
Parts:
- moved J4 5.52 mm to (12.0, 74.1)
Routing:
- net GND: track 334.2 -> 288.5 mm
- net /flow_sensor_24V: track 264.6 -> 284.3 mm
- net /flow_sensor_%RH: track 249.6 -> 232.5 mm
- net /PCB1_232_RX: track 49.1 -> 34.4 mm
- net /O3_1_GND: track 256.9 -> 246.5 mm
- net /flow_sensor_GND: track 222.5 -> 213.7 mm
- net /To_J1_P4: track 228.5 -> 236.0 mm
- net /To_J1_P2: track 235.2 -> 242.1 mm
- net /PCB1_ALARM_COM: track 264.4 -> 257.6 mm
- net +5V: track 277.0 -> 271.1 mm
- net /To_J1_P14: track 167.8 -> 173.6 mm
- net /To_J1_P8: track 227.9 -> 233.0 mm
- net /To_J1_P10: track 202.2 -> 206.1 mm
- net /To_J1_P6: track 221.1 -> 224.9 mm
- net /To_J1_P11: track 194.0 -> 190.3 mm
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Other:
- net class 0.5 mil removed
- net class Default: trace_width 0.2 -> 1
- rule trace_min: 0.2 -> 0.3
