File: backplane/backplane.kicad_pcb (KiCad board)
At the start: 2 copper layers, 200 x 300 mm, 117 parts, among them J1 Conn_PCB1, J10 Conn_SSR_INPUT, J11 FAN, J12 Conn_SSR_PCB2, J13 FLOW, J14 FCC_B2B, J15 AQ2, J16 AQ1, J17 O3, J18 Conn_TO_ION_AIR, J2 Conn_PCB2, J22 POWER, J23 PCB1_COMM_CONNECTOR, J24 Conn_01x14, J25 PCB1_ALARM, J26 Conn_01x12, J27 Conn_01x15, J28 PMS7003S_CONN, J3 SSR_CONTROL, J4 TO_CONTROL_BOARD, J5 Conn_SSR_POWER_SOURCE, J6 48V_SRC, J7 WS2812, J8 PURFUME, J9 SSR2, Q1 2N3904(1AM), Q2 2N3904(1AM), Q3 2N3904(1AM), Q4 SS9013_J3, SW1 SW_Push, U1 OMRON-G3MB-202P, U2 OMRON-G3MB-202P, U3 waveshare-swd-pinsocket, U4 STM32F103C8T6, U5 AMS1117-3.3, U6 74AHCT1G125, U7 SP3232EEN, Y1 O8M, Y2 O_EPSON_32.768K

Commit message: update,
Parts:
- moved Q3 29.6 mm to (62.2, 95.9)
- moved D3 29.6 mm to (58.0, 90.3)
- moved R12 29.6 mm to (62.2, 100.4)
- moved R13 29.6 mm to (61.8, 90.3)
- moved R14 29.6 mm to (57.1, 93.3)
- moved R11 29.6 mm to (57.9, 96.5)
- moved C21 25.0 mm to (14.7, 89.1)
- moved J28 25.0 mm to (6.46, 80.1)
- moved R26 25.0 mm to (13.0, 83.1)
- moved R27 25.0 mm to (11.4, 75.2)
- moved D1 18.0 mm to (43.2, 107.3)
- moved J8 18.0 mm to (6.28, 110.0)
- moved J9 18.0 mm to (6.28, 96.9)
- moved Q1 18.0 mm to (42.1, 111.5)
- moved R3 18.0 mm to (48.3, 112.5)
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Routing:
- net SSR-25-DA_P: track 60.5 -> 95.0 mm
- net SSR-25-DA_N: track 71.6 -> 97.2 mm, vias 0 -> 2
- net GND: track 854.4 -> 878.9 mm, vias 14 -> 13
- net Net-(Q2-Pad3): track 25.8 -> 46.1 mm
- net STM32_SSR1_OUTPUT: track 65.3 -> 84.6 mm
- net STM32_SSR2_OUTPUT: track 45.8 -> 64.3 mm, vias 1 -> 2
- net STM32_PMS7003S_SET: track 137.4 -> 119.8 mm
- net /stm32_board/STM32_CORE/RESET: track 73.8 -> 57.1 mm, vias 3 -> 2
- net /stm32_board/WS2812_PWM_TERMINAL: track 22.8 -> 10.7 mm
- net +3V3: track 315.7 -> 305.9 mm
- net STM32_PMS7003S_TXD: track 95.8 -> 86.2 mm
- net /stm32_board/STM32_CORE/OSCOUT: track 34.6 -> 41.1 mm
- net Net-(Q1-Pad1): track 10.7 -> 6.72 mm, vias 2 -> 0
- net STM32_PMS7003S_RESET: track 127.2 -> 123.2 mm
- net /stm32_board/STM32_CORE/PC15: track 29.6 -> 32.7 mm
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
Commit message: update,
Parts:
- moved J17 3.00 mm to (11.5, 158.1)
Routing:
- net /O3_1_SHIELD: track 246.1 -> 248.2 mm
- net /O3_1_SENSOR: track 258.2 -> 260.1 mm
- net /O3_1_GND: track 253.3 -> 254.5 mm
- net /O3_1_24V: track 252.4 -> 253.6 mm
Changed lines of the file:
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@@
     (thickness 1.6)
     (drawings 22)
-    (tracks 1584)
+    (tracks 1590)
     (zones 0)
     (modules 117)
@@
   )
   (module footprint-lib:mpt_0,5%2f4-2,54 locked (layer F.Cu)
-    (at 11.476 155.13 270)
+    (at 11.476 158.13 270)
     (descr "4-way 2.54mm pitch terminal block, Phoenix MPT series")
     (clearance 0.3)
@@
   (segment (start 138.938 226.773132) (end 150.456 238.291132) (width 1) (layer B.Cu) (net 26))
   (segment (start 151.685998 268.779998) (end 151.685998 273.498) (width 1) (layer B.Cu) (net 26) (status 20))
-  (via (at 42.856 148.06) (size 3) (drill 0.4) (layers F.Cu B.Cu) (net 26))
-  (segment (start 53.736 158.94) (end 42.856 148.06) (width 1) (layer B.Cu) (net 26))
-  (segment (start 86.120674 158.94) (end 53.736 158.94) (width 1) (layer B.Cu) (net 26))
-  (segment (start 39.596 151.32) (end 11.476 151.32) (width 1) (layer F.Cu) (net 26) (status 20))
-  (segment (start 42.856 148.06) (end 39.596 151.32) (width 1) (layer F.Cu) (net 26))
+  (via (at 42.856 146.97) (size 3) (drill 0.4) (layers F.Cu B.Cu) (net 26))
   (segment (start 137.069285 200.406) (end 137.069285 194.473285) (width 1) (layer B.Cu) (net 27))
   (segment (start 137.069285 200.406) (end 137.069285 194.31) (width 1) (layer B.Cu) (net 27))
@@
   (segment (start 138.76731 223.774) (end 137.668 222.67469) (width 1) (layer B.Cu) (net 27))
   (segment (start 140.716 225.72269) (end 138.76731 223.774) (width 1) (layer B.Cu) (net 27))
-  (segment (start 137.069285 204.216) (end 137.069285 192.890167) (width 1) (layer B.Cu) (net 27))
-  (segment (start 137.069285 192.890167) (end 112.999139 168.820021) (width 1) (layer B.Cu) (net 27))
-  (segment (start 112.999139 168.820021) (end 98.829136 168.82002) (width 1) (layer B.Cu) (net 27))
-  (segment (start 98.829136 168.82002) (end 86.409116 156.4) (width 1) (layer B.Cu) (net 27))
   (segment (start 152.456011 237.462701) (end 140.716 225.72269) (width 1) (layer B.Cu) (net 27))
   (segment (start 156.765998 273.498) (end 156.765998 268.779998) (width 1) (layer B.Cu) (net 27) (status 10))
   (segment (start 156.765998 268.779998) (end 152.456011 264.470011) (width 1) (layer B.Cu) (net 27))
   (segment (start 152.456011 264.470011) (end 152.456011 237.462701) (width 1) (layer B.Cu) (net 27))
-  (via (at 48.226 147.67) (size 3) (drill 0.4) (layers F.Cu B.Cu) (net 27))
-  (segment (start 56.956 156.4) (end 48.226 147.67) (width 1) (layer B.Cu) (net 27))
-  (segment (start 86.409116 156.4) (end 56.956 156.4) (width 1) (layer B.Cu) (net 27))
-  (segment (start 42.036 153.86) (end 11.476 153.86) (width 1) (layer F.Cu) (net 27) (status 20))
-  (segment (start 48.226 147.67) (end 42.036 153.86) (width 1) (layer F.Cu) (net 27))
+  (segment (start 54.826 158.94) (end 42.856 146.97) (width 1) (layer B.Cu) (net 26))
+  (segment (start 74.24 158.94) (end 54.826 158.94) (width 1) (layer B.Cu) (net 26))
+  (segment (start 86.120674 158.94) (end 74.24 158.94) (width 1) (layer B.Cu) (net 26))
+  (segment (start 35.506 154.32) (end 42.856 146.97) (width 1) (layer F.Cu) (net 26))
+  (segment (start 11.476 154.32) (end 35.506 154.32) (width 1) (layer F.Cu) (net 26))
+  (segment (start 98.829136 168.82002) (end 86.409116 156.4) (width 1) (layer B.Cu) (net 27))
+  (segment (start 57.774786 156.4) (end 49.744494 148.369708) (width 1) (layer B.Cu) (net 27))
+  (segment (start 112.999139 168.820021) (end 98.829136 168.82002) (width 1) (layer B.Cu) (net 27))
+  (segment (start 137.069285 192.890167) (end 112.999139 168.820021) (width 1) (layer B.Cu) (net 27))
+  (segment (start 137.069285 204.216) (end 137.069285 192.890167) (width 1) (layer B.Cu) (net 27))
+  (segment (start 46.744496 148.369708) (end 48.244495 146.869709) (width 1) (layer F.Cu) (net 27))
+  (segment (start 86.409116 156.4) (end 57.774786 156.4) (width 1) (layer B.Cu) (net 27))
+  (segment (start 49.744494 148.369708) (end 48.244495 146.869709) (width 1) (layer B.Cu) (net 27))
+  (via (at 48.244495 146.869709) (size 3) (drill 0.4) (layers F.Cu B.Cu) (net 27))
+  (segment (start 38.254204 156.86) (end 46.744496 148.369708) (width 1) (layer F.Cu) (net 27))
+  (segment (start 11.476 156.86) (end 38.254204 156.86) (width 1) (layer F.Cu) (net 27))
   (segment (start 139.210142 201.168) (end 139.210142 192.278) (width 1) (layer B.Cu) (net 28))
   (segment (start 141.693885 223.52) (end 139.954 221.780115) (width 1) (layer B.Cu) (net 28))
   (segment (start 139.210142 201.168) (end 139.210142 221.036257) (width 1) (layer B.Cu) (net 28))
   (segment (start 139.210142 221.036257) (end 141.693885 223.52) (width 1) (layer B.Cu) (net 28))
-  (segment (start 139.210142 192.202584) (end 138.92845 191.92089) (width 1) (layer B.Cu) (net 28))
-  (segment (start 138.92845 191.92089) (end 113.827571 166.820011) (width 1) (layer B.Cu) (net 28))
-  (segment (start 99.657568 166.82001) (end 86.697558 153.86) (width 1) (layer B.Cu) (net 28))
-  (segment (start 139.210142 201.168) (end 139.210142 192.202584) (width 1) (layer B.Cu) (net 28))
-  (segment (start 113.827571 166.820011) (end 99.657568 166.82001) (width 1) (layer B.Cu) (net 28))
   (segment (start 161.845998 273.498) (end 161.845998 268.779998) (width 1) (layer B.Cu) (net 28) (status 10))
   (segment (start 154.456022 261.390022) (end 154.456022 236.282137) (width 1) (layer B.Cu) (net 28))
   (segment (start 161.845998 268.779998) (end 154.456022 261.390022) (width 1) (layer B.Cu) (net 28))
   (segment (start 154.456022 236.282137) (end 141.693885 223.52) (width 1) (layer B.Cu) (net 28))
-  (segment (start 60.486 153.86) (end 53.596 146.97) (width 1) (layer B.Cu) (net 28))
   (via (at 53.596 146.97) (size 3) (drill 0.4) (layers F.Cu B.Cu) (net 28))
-  (segment (start 86.697558 153.86) (end 60.486 153.86) (width 1) (layer B.Cu) (net 28))
-  (segment (start 44.166 156.4) (end 11.476 156.4) (width 1) (layer F.Cu) (net 28) (status 20))
-  (segment (start 53.596 146.97) (end 44.166 156.4) (width 1) (layer F.Cu) (net 28))
   (segment (start 166.925998 268.779998) (end 156.464 258.318) (width 1) (layer B.Cu) (net 29) (status 40000))
   (segment (start 166.925998 273.498) (end 166.925998 268.779998) (width 1) (layer B.Cu) (net 29) (status 40010))
@@
   (segment (start 143.002 221.575411) (end 142.24 220.813411) (width 1) (layer B.Cu) (net 29) (status 40000))
   (segment (start 156.464 235.037411) (end 143.002 221.575411) (width 1) (layer B.Cu) (net 29) (status 40000))
-  (segment (start 141.350999 206.248) (end 141.350999 191.514999) (width 1) (layer B.Cu) (net 29) (status 40000))
   (segment (start 141.350999 206.248) (end 141.350999 199.898) (width 1) (layer B.Cu) (net 29) (status 40000))
+  (via (at 59.036 146.97) (size 3) (drill 0.4) (layers F.Cu B.Cu) (net 29))
+  (segment (start 60.486 153.86) (end 53.596 146.97) (width 1) (layer B.Cu) (net 28))
+  (segment (start 139.210142 201.168) (end 139.210142 192.202584) (width 1) (layer B.Cu) (net 28))
+  (segment (start 139.210142 192.202584) (end 138.92845 191.92089) (width 1) (layer B.Cu) (net 28))
+  (segment (start 138.92845 191.92089) (end 113.827571 166.820011) (width 1) (layer B.Cu) (net 28))
+  (segment (start 113.827571 166.820011) (end 99.657568 166.82001) (width 1) (layer B.Cu) (net 28))
+  (segment (start 99.657568 166.82001) (end 86.697558 153.86) (width 1) (layer B.Cu) (net 28))
+  (segment (start 86.697558 153.86) (end 60.486 153.86) (width 1) (layer B.Cu) (net 28))
+  (segment (start 41.166 159.4) (end 53.596 146.97) (width 1) (layer F.Cu) (net 28))
+  (segment (start 11.476 159.4) (end 41.166 159.4) (width 1) (layer F.Cu) (net 28))
+  (segment (start 63.386 151.32) (end 59.036 146.97) (width 1) (layer B.Cu) (net 29))
   (segment (start 100.486 164.82) (end 86.986 151.32) (width 1) (layer B.Cu) (net 29))
+  (segment (start 86.986 151.32) (end 63.386 151.32) (width 1) (layer B.Cu) (net 29))
   (segment (start 114.656 164.82) (end 100.486 164.82) (width 1) (layer B.Cu) (net 29))
   (segment (start 141.350999 191.514999) (end 114.656 164.82) (width 1) (layer B.Cu) (net 29))
-  (via (at 59.036 146.97) (size 3) (drill 0.4) (layers F.Cu B.Cu) (net 29))
-  (segment (start 86.986 151.32) (end 63.386 151.32) (width 1) (layer B.Cu) (net 29))
-  (segment (start 63.386 151.32) (end 59.036 146.97) (width 1) (layer B.Cu) (net 29))
-  (segment (start 47.066 158.94) (end 11.476 158.94) (width 1) (layer F.Cu) (net 29) (status 20))
-  (segment (start 59.036 146.97) (end 47.066 158.94) (width 1) (layer F.Cu) (net 29))
+  (segment (start 141.350999 206.248) (end 141.350999 191.514999) (width 1) (layer B.Cu) (net 29))
+  (segment (start 57.536001 148.469999) (end 59.036 146.97) (width 1) (layer F.Cu) (net 29))
+  (segment (start 45.355989 160.650011) (end 57.536001 148.469999) (width 1) (layer F.Cu) (net 29))
+  (segment (start 24.139989 160.650011) (end 45.355989 160.650011) (width 1) (layer F.Cu) (net 29))
+  (segment (start 11.476 161.94) (end 22.85 161.94) (width 1) (layer F.Cu) (net 29))
+  (segment (start 22.85 161.94) (end 24.139989 160.650011) (width 1) (layer F.Cu) (net 29))
   (segment (start 111.76 244.214) (end 111.76 270.764) (width 1) (layer B.Cu) (net 30) (status 40000))
   (segment (start 111.76 270.764) (end 119.38 278.384) (width 1) (layer B.Cu) (net 30) (status 40000))

Commit message: update,
Parts:
- moved C7 2.00 mm to (33.4, 8.56)
Routing:
- net GND: track 878.9 -> 856.0 mm, vias 13 -> 12
- net SSR-25-DA_P: track 95.0 -> 82.9 mm
- net /stm32_board/FAN_RPM: track 57.8 -> 68.2 mm, vias 1 -> 0
- net STM32_PMS7003S_RESET: track 123.2 -> 113.6 mm
- net STM32_WS2812_OUTPUT: track 89.6 -> 83.4 mm
- net Net-(R10-Pad2): track 18.8 -> 14.1 mm
- net STM32_SSR2_OUTPUT: track 64.3 -> 68.7 mm
- net /stm32_board/STM32_CORE/SWIO: track 62.2 -> 65.6 mm
- net STM32_SSR-25-DA_OUTPUT: track 86.6 -> 90.0 mm
- net B2B_UART_TX: track 41.5 -> 44.2 mm
- net /stm32_board/STM32_CORE/RESET: track 57.1 -> 59.6 mm
- net SSR-25-DA_N: track 97.2 -> 95.4 mm
- net IONAIR-TTL-TX: track 57.2 -> 58.9 mm
- net IONAIR_RX: track 137.4 -> 135.9 mm
- net +3V3: track 305.9 -> 304.5 mm
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
Commit message: update,
Routing:
- net +3V3: track 304.5 -> 290.0 mm
- net SSR-25-DA_N: track 95.4 -> 87.2 mm
- net STM32_PMS7003S_RESET: track 113.6 -> 117.8 mm
- net GND: track 856.0 -> 858.9 mm
- net STM32_PMS7003S_SET: track 119.8 -> 117.7 mm
- net IONAIR_TX: track 145.8 -> 144.1 mm
- net +5V: track 701.6 -> 699.9 mm, vias 17 -> 15
- net IONAIR_RX: track 135.9 -> 134.2 mm
- net STM32_PMS7003S_TXD: track 86.2 -> 84.7 mm
- net STM32_PMS7003S_RXD: track 92.7 -> 91.4 mm
- net IONAIR-TTL-RX: track 53.1 -> 54.4 mm
- net STM32_SSR2_OUTPUT: track 68.7 -> 69.8 mm
- net /stm32_board/WS2812_PWM_TERMINAL: track 10.7 -> 11.5 mm
- net STM32_SSR-25-DA_OUTPUT: track 90.0 -> 90.6 mm

Commit message: update,
Parts:
- moved D2 45.8 mm to (6.28, 102.4), turned to 270 degrees
- moved R8 40.7 mm to (11.3, 102.4), turned to 270 degrees
- moved D1 37.8 mm to (6.28, 115.5), turned to 270 degrees
- moved R7 28.8 mm to (11.3, 115.5), turned to 270 degrees
- moved D6 1.96 mm to (16.2, 26.7)
- moved R21 1.57 mm to (16.0, 30.3)
- moved R23 0.36 mm to (9.92, 30.3)
Routing:
- net Net-(Q1-Pad3): track 13.3 -> 34.4 mm, vias 0 -> 1
- net Net-(Q2-Pad3): track 46.0 -> 64.2 mm
- net +5V: track 699.9 -> 714.3 mm, vias 15 -> 18
- net Net-(D1-Pad1): track 2.44 -> 5.06 mm
- net Net-(D2-Pad1): track 3.00 -> 5.06 mm
- net Net-(D7-Pad1): track 4.94 -> 3.64 mm
- net /stm32_board/SSR_CH2_OUTPUT1: track 18.0 -> 17.4 mm

Commit message: update,
Routing:
- net +5V: track 714.3 -> 703.1 mm, vias 18 -> 16

Commit message: update,
Routing:
- net +5V: track 703.1 -> 703.4 mm, vias 16 -> 17
Changed lines of the file:
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@@
     (thickness 1.6)
     (drawings 22)
-    (tracks 1520)
+    (tracks 1523)
     (zones 0)
     (modules 117)
@@
   (segment (start 12.416 134.13024) (end 6.283501 134.13024) (width 0.75) (layer B.Cu) (net 37) (status 20))
   (segment (start 12.416 134.13024) (end 8.476 134.13024) (width 0.75) (layer B.Cu) (net 37))
-  (segment (start 20.14576 134.13024) (end 6.283501 134.13024) (width 0.75) (layer F.Cu) (net 37) (status 20))
-  (segment (start 22.696 131.58) (end 20.14576 134.13024) (width 0.75) (layer F.Cu) (net 37))
   (segment (start 56.238472 91.047499) (end 56.988472 90.297499) (width 0.75) (layer F.Cu) (net 37) (status 20))
   (segment (start 56.238472 93.2975) (end 56.238472 91.047499) (width 0.75) (layer F.Cu) (net 37) (status 10))
@@
   (via (at 56.01 127.9) (size 1) (drill 0.4) (layers F.Cu B.Cu) (net 37))
   (segment (start 53.09 130.82) (end 56.01 127.9) (width 0.75) (layer B.Cu) (net 37))
-  (segment (start 22.696 130.82) (end 53.09 130.82) (width 0.75) (layer B.Cu) (net 37))
   (segment (start 55.334102 127.224102) (end 56.01 127.9) (width 0.75) (layer F.Cu) (net 37))
   (segment (start 53.440442 127.224102) (end 55.334102 127.224102) (width 0.75) (layer F.Cu) (net 37) (status 10))
@@
   (segment (start 26.9 104.827106) (end 26.9 104.12) (width 0.75) (layer F.Cu) (net 37))
   (segment (start 26.9 116.19) (end 26.9 104.827106) (width 0.75) (layer F.Cu) (net 37))
-  (segment (start 22.696 121.3) (end 22.696 120.394) (width 0.75) (layer F.Cu) (net 37))
   (segment (start 23.96 119.13) (end 26.9 116.19) (width 0.75) (layer F.Cu) (net 37))
-  (segment (start 22.696 120.394) (end 23.96 119.13) (width 0.75) (layer F.Cu) (net 37))
   (segment (start 22.88 120.21) (end 23.96 119.13) (width 0.75) (layer F.Cu) (net 37))
-  (segment (start 22.696 121.3) (end 22.696 131.58) (width 0.75) (layer F.Cu) (net 37))
+  (segment (start 20.14576 134.13024) (end 6.283501 134.13024) (width 0.75) (layer F.Cu) (net 37))
+  (segment (start 22.696 131.58) (end 20.14576 134.13024) (width 0.75) (layer F.Cu) (net 37))
+  (segment (start 23.96 119.13) (end 22.696 120.394) (width 0.75) (layer F.Cu) (net 37))
+  (via (at 22.696 130.03) (size 1) (drill 0.4) (layers F.Cu B.Cu) (net 37))
+  (segment (start 25.64 130.82) (end 53.09 130.82) (width 0.75) (layer B.Cu) (net 37))
+  (segment (start 25.64 130.82) (end 23.486 130.82) (width 0.75) (layer B.Cu) (net 37))
+  (segment (start 22.696 120.394) (end 22.696 130.03) (width 0.75) (layer F.Cu) (net 37))
+  (segment (start 22.696 130.03) (end 22.696 131.58) (width 0.75) (layer F.Cu) (net 37))
+  (segment (start 23.486 130.82) (end 22.696 130.03) (width 0.75) (layer B.Cu) (net 37))
   (segment (start 33.9737 46.01223) (end 35.5485 47.58703) (width 0.5) (layer F.Cu) (net 40) (status 20))
   (segment (start 32.3485 46.01223) (end 33.9737 46.01223) (width 0.5) (layer F.Cu) (net 40) (status 10))
@@
   (segment (start 45.7485 29.56223) (end 46.2735 29.03723) (width 0.5) (layer F.Cu) (net 121) (status 20))
   (segment (start 45.7485 31.43723) (end 45.7485 29.56223) (width 0.5) (layer F.Cu) (net 121) (status 10))
-  (segment (start 11.133501 101.39542) (end 11.283501 101.54542) (width 0.5) (layer F.Cu) (net 122) (status 1000030))
-  (segment (start 6.283501 101.39542) (end 11.133501 101.39542) (width 0.5) (layer F.Cu) (net 122) (status 1000030))
+  (segment (start 11.133501 101.39542) (end 11.283501 101.54542) (width 0.5) (layer F.Cu) (net 122) (status 30))
+  (segment (start 6.283501 101.39542) (end 11.133501 101.39542) (width 0.5) (layer F.Cu) (net 122) (status 30))
   (segment (start 11.133501 114.51542) (end 11.283501 114.66542) (width 0.5) (layer F.Cu) (net 123) (status 30))
   (segment (start 6.283501 114.51542) (end 11.133501 114.51542) (width 0.5) (layer F.Cu) (net 123) (status 30))

Commit message: update,
Parts:
- moved R14 38.3 mm to (27.3, 117.4)
- moved D3 36.9 mm to (45.5, 125.1)
- moved R13 36.1 mm to (45.7, 122.5), turned to 180 degrees
Routing:
- net Net-(Q2-Pad3): track 64.2 -> 41.1 mm
- net +5V: track 703.4 -> 683.3 mm, vias 17 -> 16
- net SSR-25-DA_P: track 82.9 -> 98.4 mm
- net GND: track 859.3 -> 851.8 mm
- net SSR-25-DA_N: track 87.2 -> 94.2 mm
- net Net-(Q1-Pad3): track 34.4 -> 39.5 mm
- net /stm32_board/STM32_CORE/OSCOUT: track 41.1 -> 39.5 mm
- net IONAIR-TTL-TX: track 58.9 -> 60.2 mm
- net STM32_PCB1_ALARM_COM: track 102.7 -> 103.7 mm
- net /stm32_board/STM32_CORE/RESET: track 59.6 -> 58.6 mm
- net IONAIR-TTL-RX: track 54.4 -> 53.7 mm
- net /stm32_board/STM32_CORE/PA0: track 18.8 -> 19.5 mm
- net Net-(D3-Pad1): track 1.90 -> 2.51 mm
- net /stm32_board/STM32_CORE/PA1: track 17.8 -> 18.4 mm
