File: backplane/PMS5003S_interface.sch (KiCad schematic (older format))
At the start: 4 parts, among them J28 PMS7003S_CONN

Commit message: backport footprint from pcb,
Parts:
- J28: footprint footprint-lib:s8b-ph-kl -> Connector_JST:JST_XH_S08B-XH-A_1x08_P2.50mm_Horizontal
Changed lines of the file:
@@
 F 0 "J28" H 3330 3692 50  0000 L CNN
 F 1 "PMS7003S_CONN" H 3330 3601 50  0000 L CNN
-F 2 "footprint-lib:s8b-ph-kl" H 3250 3650 50  0001 C CNN
+F 2 "Connector_JST:JST_XH_S08B-XH-A_1x08_P2.50mm_Horizontal" H 3250 3650 50  0001 C CNN
 F 3 "~" H 3250 3650 50  0001 C CNN
 	1    3250 3650
