File: backplane/backplane.sch (KiCad schematic (older format))
At the start: 23 parts, among them J1 Conn_PCB1, J10 Conn_SSR_INPUT, J12 Conn_SSR_PCB2, J13 FLOW_SENSOR, J15 AQ2_SENSOR, J16 AQ1_SENSOR, J17 O3_SENSOR, J18 Conn_TO_ION_AIR, J2 Conn_PCB2, J23 PCB1_COMM_CONNECTOR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

Commit message: update,
Parts:
- added H? (x6): PCB1, MountingHole:MountingHole_3.2mm_M3_DIN965, symbol Mechanical:MountingHole
- gave numbers to parts that had none: 9
Changed lines of the file:
@@
 	6550 2200 7850 2200
 $Comp
-L Mechanical:MountingHole H?
+L Mechanical:MountingHole H1
 U 1 1 5BE6E1EE
 P 7750 4950
-F 0 "H?" H 7850 4996 50  0000 L CNN
+F 0 "H1" H 7850 4996 50  0000 L CNN
 F 1 "PCB2" H 7850 4905 50  0000 L CNN
 F 2 "MountingHole:MountingHole_3.2mm_M3_DIN965" H 7750 4950 50  0001 C CNN
@@
 $EndComp
 $Comp
-L Mechanical:MountingHole H?
+L Mechanical:MountingHole H2
 U 1 1 5BE6E3BE
 P 7750 5150
-F 0 "H?" H 7850 5196 50  0000 L CNN
+F 0 "H2" H 7850 5196 50  0000 L CNN
 F 1 "PCB2" H 7850 5105 50  0000 L CNN
 F 2 "MountingHole:MountingHole_3.2mm_M3_DIN965" H 7750 5150 50  0001 C CNN
@@
 $EndComp
 $Comp
-L Mechanical:MountingHole H?
+L Mechanical:MountingHole H3
 U 1 1 5BE6E3F6
 P 7750 5350
-F 0 "H?" H 7850 5396 50  0000 L CNN
+F 0 "H3" H 7850 5396 50  0000 L CNN
 F 1 "PCB2" H 7850 5305 50  0000 L CNN
 F 2 "MountingHole:MountingHole_3.2mm_M3_DIN965" H 7750 5350 50  0001 C CNN
@@
 $EndComp
 $Comp
-L Mechanical:MountingHole H?
+L Mechanical:MountingHole H4
 U 1 1 5BE6E42C
 P 7750 5550
-F 0 "H?" H 7850 5596 50  0000 L CNN
+F 0 "H4" H 7850 5596 50  0000 L CNN
 F 1 "PCB2" H 7850 5505 50  0000 L CNN
 F 2 "MountingHole:MountingHole_3.2mm_M3_DIN965" H 7750 5550 50  0001 C CNN
@@
 $EndComp
 $Comp
-L Mechanical:MountingHole H?
+L Mechanical:MountingHole H5
 U 1 1 5BE6E69F
 P 8500 4950
-F 0 "H?" H 8600 4996 50  0000 L CNN
+F 0 "H5" H 8600 4996 50  0000 L CNN
 F 1 "PCB1" H 8600 4905 50  0000 L CNN
 F 2 "MountingHole:MountingHole_3.2mm_M3_DIN965" H 8500 4950 50  0001 C CNN
@@
 $EndComp
 $Comp
-L Mechanical:MountingHole H?
+L Mechanical:MountingHole H6
 U 1 1 5BE74A69
 P 8500 5150
-F 0 "H?" H 8600 5196 50  0000 L CNN
+F 0 "H6" H 8600 5196 50  0000 L CNN
 F 1 "PCB1" H 8600 5105 50  0000 L CNN
 F 2 "MountingHole:MountingHole_3.2mm_M3_DIN965" H 8500 5150 50  0001 C CNN
@@
 $EndComp
 $Comp
-L Mechanical:MountingHole H?
+L Mechanical:MountingHole H7
 U 1 1 5BE77C40
 P 8500 5350
-F 0 "H?" H 8600 5396 50  0000 L CNN
+F 0 "H7" H 8600 5396 50  0000 L CNN
 F 1 "PCB1" H 8600 5305 50  0000 L CNN
 F 2 "MountingHole:MountingHole_3.2mm_M3_DIN965" H 8500 5350 50  0001 C CNN
@@
 $EndComp
 $Comp
-L Mechanical:MountingHole H?
+L Mechanical:MountingHole H8
 U 1 1 5BE77C46
 P 8500 5550
-F 0 "H?" H 8600 5596 50  0000 L CNN
+F 0 "H8" H 8600 5596 50  0000 L CNN
 F 1 "PCB1" H 8600 5505 50  0000 L CNN
 F 2 "MountingHole:MountingHole_3.2mm_M3_DIN965" H 8500 5550 50  0001 C CNN
@@
 $EndComp
 $Comp
-L Mechanical:MountingHole H?
+L Mechanical:MountingHole H9
 U 1 1 5BE7ADFF
 P 8500 5750
-F 0 "H?" H 8600 5796 50  0000 L CNN
+F 0 "H9" H 8600 5796 50  0000 L CNN
 F 1 "PCB1" H 8600 5705 50  0000 L CNN
 F 2 "MountingHole:MountingHole_3.2mm_M3_DIN965" H 8500 5750 50  0001 C CNN
@@
 	1    0    0    -1
 $EndComp
+$Comp
+L Mechanical:MountingHole H?
+U 1 1 5BE7E2A8
+P 9550 4950
+F 0 "H?" H 9650 4996 50  0000 L CNN
+F 1 "PCB1" H 9650 4905 50  0000 L CNN
+F 2 "MountingHole:MountingHole_3.2mm_M3_DIN965" H 9550 4950 50  0001 C CNN
+F 3 "~" H 9550 4950 50  0001 C CNN
+	1    9550 4950
+	1    0    0    -1
+$EndComp
+$Comp
+L Mechanical:MountingHole H?
+U 1 1 5BE7E2AE
+P 9550 5150
+F 0 "H?" H 9650 5196 50  0000 L CNN
+F 1 "PCB1" H 9650 5105 50  0000 L CNN
+F 2 "MountingHole:MountingHole_3.2mm_M3_DIN965" H 9550 5150 50  0001 C CNN
+F 3 "~" H 9550 5150 50  0001 C CNN
+	1    9550 5150
+	1    0    0    -1
+$EndComp
+$Comp
+L Mechanical:MountingHole H?
+U 1 1 5BE7E2B4
+P 9550 5350
+F 0 "H?" H 9650 5396 50  0000 L CNN
+F 1 "PCB1" H 9650 5305 50  0000 L CNN
+F 2 "MountingHole:MountingHole_3.2mm_M3_DIN965" H 9550 5350 50  0001 C CNN
+F 3 "~" H 9550 5350 50  0001 C CNN
+	1    9550 5350
+	1    0    0    -1
+$EndComp
+$Comp
+L Mechanical:MountingHole H?
+U 1 1 5BE7E2BA
+P 9550 5550
+F 0 "H?" H 9650 5596 50  0000 L CNN
+F 1 "PCB1" H 9650 5505 50  0000 L CNN
+F 2 "MountingHole:MountingHole_3.2mm_M3_DIN965" H 9550 5550 50  0001 C CNN
+F 3 "~" H 9550 5550 50  0001 C CNN
+	1    9550 5550
+	1    0    0    -1
+$EndComp
+$Comp
+L Mechanical:MountingHole H?
+U 1 1 5BE7E2C0
+P 9550 5750
+F 0 "H?" H 9650 5796 50  0000 L CNN
+F 1 "PCB1" H 9650 5705 50  0000 L CNN
+F 2 "MountingHole:MountingHole_3.2mm_M3_DIN965" H 9550 5750 50  0001 C CNN
+F 3 "~" H 9550 5750 50  0001 C CNN
+	1    9550 5750
+	1    0    0    -1
+$EndComp
+$Comp
+L Mechanical:MountingHole H?
+U 1 1 5BE81489
+P 9550 5950
+F 0 "H?" H 9650 5996 50  0000 L CNN
+F 1 "PCB1" H 9650 5905 50  0000 L CNN
+F 2 "MountingHole:MountingHole_3.2mm_M3_DIN965" H 9550 5950 50  0001 C CNN
+F 3 "~" H 9550 5950 50  0001 C CNN
+	1    9550 5950
+	1    0    0    -1
+$EndComp

Commit message: update,
Parts:
- added H?: HEATSINK_SCREW, MountingHole:MountingHole_3.2mm_M3_DIN965, symbol Mechanical:MountingHole
- gave numbers to parts that had none: 6
Changed lines of the file:
@@
 $EndComp
 $Comp
-L Mechanical:MountingHole H?
+L Mechanical:MountingHole H10
 U 1 1 5BE7E2A8
 P 9550 4950
-F 0 "H?" H 9650 4996 50  0000 L CNN
+F 0 "H10" H 9650 4996 50  0000 L CNN
 F 1 "PCB1" H 9650 4905 50  0000 L CNN
 F 2 "MountingHole:MountingHole_3.2mm_M3_DIN965" H 9550 4950 50  0001 C CNN
@@
 $EndComp
 $Comp
-L Mechanical:MountingHole H?
+L Mechanical:MountingHole H11
 U 1 1 5BE7E2AE
 P 9550 5150
-F 0 "H?" H 9650 5196 50  0000 L CNN
+F 0 "H11" H 9650 5196 50  0000 L CNN
 F 1 "PCB1" H 9650 5105 50  0000 L CNN
 F 2 "MountingHole:MountingHole_3.2mm_M3_DIN965" H 9550 5150 50  0001 C CNN
@@
 $EndComp
 $Comp
-L Mechanical:MountingHole H?
+L Mechanical:MountingHole H12
 U 1 1 5BE7E2B4
 P 9550 5350
-F 0 "H?" H 9650 5396 50  0000 L CNN
+F 0 "H12" H 9650 5396 50  0000 L CNN
 F 1 "PCB1" H 9650 5305 50  0000 L CNN
 F 2 "MountingHole:MountingHole_3.2mm_M3_DIN965" H 9550 5350 50  0001 C CNN
@@
 $EndComp
 $Comp
-L Mechanical:MountingHole H?
+L Mechanical:MountingHole H13
 U 1 1 5BE7E2BA
 P 9550 5550
-F 0 "H?" H 9650 5596 50  0000 L CNN
+F 0 "H13" H 9650 5596 50  0000 L CNN
 F 1 "PCB1" H 9650 5505 50  0000 L CNN
 F 2 "MountingHole:MountingHole_3.2mm_M3_DIN965" H 9550 5550 50  0001 C CNN
@@
 $EndComp
 $Comp
-L Mechanical:MountingHole H?
+L Mechanical:MountingHole H14
 U 1 1 5BE7E2C0
 P 9550 5750
-F 0 "H?" H 9650 5796 50  0000 L CNN
+F 0 "H14" H 9650 5796 50  0000 L CNN
 F 1 "PCB1" H 9650 5705 50  0000 L CNN
 F 2 "MountingHole:MountingHole_3.2mm_M3_DIN965" H 9550 5750 50  0001 C CNN
@@
 $EndComp
 $Comp
-L Mechanical:MountingHole H?
+L Mechanical:MountingHole H15
 U 1 1 5BE81489
 P 9550 5950
-F 0 "H?" H 9650 5996 50  0000 L CNN
+F 0 "H15" H 9650 5996 50  0000 L CNN
 F 1 "PCB1" H 9650 5905 50  0000 L CNN
 F 2 "MountingHole:MountingHole_3.2mm_M3_DIN965" H 9550 5950 50  0001 C CNN
@@
 	1    0    0    -1
 $EndComp
+$Comp
+L Mechanical:MountingHole H?
+U 1 1 5BE84A69
+P 10300 4950
+F 0 "H?" H 10400 4996 50  0000 L CNN
+F 1 "HEATSINK_SCREW" H 10400 4905 50  0000 L CNN
+F 2 "MountingHole:MountingHole_3.2mm_M3_DIN965" H 10300 4950 50  0001 C CNN
+F 3 "~" H 10300 4950 50  0001 C CNN
+	1    10300 4950
+	1    0    0    -1
+$EndComp

Commit message: update,
Parts:
- H10, H11, H12, H13, H14, H15: value PCB1 -> MAINBOARD
- gave numbers to parts that had none: 1
Changed lines of the file:
@@
 L Mechanical:MountingHole H10
 U 1 1 5BE7E2A8
-P 9550 4950
-F 0 "H10" H 9650 4996 50  0000 L CNN
-F 1 "PCB1" H 9650 4905 50  0000 L CNN
-F 2 "MountingHole:MountingHole_3.2mm_M3_DIN965" H 9550 4950 50  0001 C CNN
-F 3 "~" H 9550 4950 50  0001 C CNN
-	1    9550 4950
+P 9100 4950
+F 0 "H10" H 9200 4996 50  0000 L CNN
+F 1 "MAINBOARD" H 9200 4905 50  0000 L CNN
+F 2 "MountingHole:MountingHole_3.2mm_M3_DIN965" H 9100 4950 50  0001 C CNN
+F 3 "~" H 9100 4950 50  0001 C CNN
+	1    9100 4950
 	1    0    0    -1
 $EndComp
@@
 L Mechanical:MountingHole H11
 U 1 1 5BE7E2AE
-P 9550 5150
-F 0 "H11" H 9650 5196 50  0000 L CNN
-F 1 "PCB1" H 9650 5105 50  0000 L CNN
-F 2 "MountingHole:MountingHole_3.2mm_M3_DIN965" H 9550 5150 50  0001 C CNN
-F 3 "~" H 9550 5150 50  0001 C CNN
-	1    9550 5150
+P 9100 5150
+F 0 "H11" H 9200 5196 50  0000 L CNN
+F 1 "MAINBOARD" H 9200 5105 50  0000 L CNN
+F 2 "MountingHole:MountingHole_3.2mm_M3_DIN965" H 9100 5150 50  0001 C CNN
+F 3 "~" H 9100 5150 50  0001 C CNN
+	1    9100 5150
 	1    0    0    -1
 $EndComp
@@
 L Mechanical:MountingHole H12
 U 1 1 5BE7E2B4
-P 9550 5350
-F 0 "H12" H 9650 5396 50  0000 L CNN
-F 1 "PCB1" H 9650 5305 50  0000 L CNN
-F 2 "MountingHole:MountingHole_3.2mm_M3_DIN965" H 9550 5350 50  0001 C CNN
-F 3 "~" H 9550 5350 50  0001 C CNN
-	1    9550 5350
+P 9100 5350
+F 0 "H12" H 9200 5396 50  0000 L CNN
+F 1 "MAINBOARD" H 9200 5305 50  0000 L CNN
+F 2 "MountingHole:MountingHole_3.2mm_M3_DIN965" H 9100 5350 50  0001 C CNN
+F 3 "~" H 9100 5350 50  0001 C CNN
+	1    9100 5350
 	1    0    0    -1
 $EndComp
@@
 L Mechanical:MountingHole H13
 U 1 1 5BE7E2BA
-P 9550 5550
-F 0 "H13" H 9650 5596 50  0000 L CNN
-F 1 "PCB1" H 9650 5505 50  0000 L CNN
-F 2 "MountingHole:MountingHole_3.2mm_M3_DIN965" H 9550 5550 50  0001 C CNN
-F 3 "~" H 9550 5550 50  0001 C CNN
-	1    9550 5550
+P 9100 5550
+F 0 "H13" H 9200 5596 50  0000 L CNN
+F 1 "MAINBOARD" H 9200 5505 50  0000 L CNN
+F 2 "MountingHole:MountingHole_3.2mm_M3_DIN965" H 9100 5550 50  0001 C CNN
+F 3 "~" H 9100 5550 50  0001 C CNN
+	1    9100 5550
 	1    0    0    -1
 $EndComp
@@
 L Mechanical:MountingHole H14
 U 1 1 5BE7E2C0
-P 9550 5750
-F 0 "H14" H 9650 5796 50  0000 L CNN
-F 1 "PCB1" H 9650 5705 50  0000 L CNN
-F 2 "MountingHole:MountingHole_3.2mm_M3_DIN965" H 9550 5750 50  0001 C CNN
-F 3 "~" H 9550 5750 50  0001 C CNN
-	1    9550 5750
+P 9100 5750
+F 0 "H14" H 9200 5796 50  0000 L CNN
+F 1 "MAINBOARD" H 9200 5705 50  0000 L CNN
+F 2 "MountingHole:MountingHole_3.2mm_M3_DIN965" H 9100 5750 50  0001 C CNN
+F 3 "~" H 9100 5750 50  0001 C CNN
+	1    9100 5750
 	1    0    0    -1
 $EndComp
@@
 L Mechanical:MountingHole H15
 U 1 1 5BE81489
-P 9550 5950
-F 0 "H15" H 9650 5996 50  0000 L CNN
-F 1 "PCB1" H 9650 5905 50  0000 L CNN
-F 2 "MountingHole:MountingHole_3.2mm_M3_DIN965" H 9550 5950 50  0001 C CNN
-F 3 "~" H 9550 5950 50  0001 C CNN
-	1    9550 5950
+P 9100 5950
+F 0 "H15" H 9200 5996 50  0000 L CNN
+F 1 "MAINBOARD" H 9200 5905 50  0000 L CNN
+F 2 "MountingHole:MountingHole_3.2mm_M3_DIN965" H 9100 5950 50  0001 C CNN
+F 3 "~" H 9100 5950 50  0001 C CNN
+	1    9100 5950
 	1    0    0    -1
 $EndComp
 $Comp
-L Mechanical:MountingHole H?
+L Mechanical:MountingHole H16
 U 1 1 5BE84A69
-P 10300 4950
-F 0 "H?" H 10400 4996 50  0000 L CNN
-F 1 "HEATSINK_SCREW" H 10400 4905 50  0000 L CNN
-F 2 "MountingHole:MountingHole_3.2mm_M3_DIN965" H 10300 4950 50  0001 C CNN
-F 3 "~" H 10300 4950 50  0001 C CNN
-	1    10300 4950
+P 9700 4950
+F 0 "H16" H 9800 4996 50  0000 L CNN
+F 1 "HEATSINK_SCREW" H 9800 4905 50  0000 L CNN
+F 2 "MountingHole:MountingHole_3.2mm_M3_DIN965" H 9700 4950 50  0001 C CNN
+F 3 "~" H 9700 4950 50  0001 C CNN
+	1    9700 4950
 	1    0    0    -1
 $EndComp

Commit message: update,
Parts:
- H1, H3: value PCB2 -> PCB1
- H6, H8: value PCB1 -> PCB2
- J13: value FLOW_SENSOR -> FLOW; footprint footprint-lib:mpt_0,5%2f5-2,54 -> footprint-lib:flow_mpt_0,5%2f5-2,54
- J15: value AQ2_SENSOR -> AQ2; footprint footprint-lib:mpt_0,5%2f4-2,54 -> footprint-lib:AQ_mpt_0,5%2f4-2,54
- J16: value AQ1_SENSOR -> AQ1; footprint footprint-lib:mpt_0,5%2f4-2,54 -> footprint-lib:AQ_mpt_0,5%2f4-2,54
- J17: value O3_SENSOR -> O3
Changed lines of the file:
@@
 Text Label 2550 5650 2    60   ~ 0
 AQ2_SENSOR
+Text Label 2550 6550 2    60   ~ 0
+AQ1_GND
 Text Label 2550 6250 2    60   ~ 0
-AQ1_GND
-Text Label 2550 6550 2    60   ~ 0
 AQ1_SHIELD
-Text Label 2550 6450 2    60   ~ 0
+Text Label 2550 6350 2    60   ~ 0
 AQ1_SENSOR
 Wire Wire Line
-	1850 6450 2550 6450
+	1850 6350 2550 6350
+Wire Wire Line
+	1850 6250 2550 6250
 Wire Wire Line
 	1850 6550 2550 6550
-Wire Wire Line
-	1850 6250 2550 6250
 $Comp
 L bluepill:Screw_Terminal_01x04 J15
@@
 P 1650 5750
 F 0 "J15" H 1650 5950 50  0000 C CNN
-F 1 "AQ2_SENSOR" H 1650 5450 50  0000 C CNN
-F 2 "footprint-lib:mpt_0,5%2f4-2,54" H 1650 5750 50  0001 C CNN
+F 1 "AQ2" H 1650 5450 50  0000 C CNN
+F 2 "footprint-lib:AQ_mpt_0,5%2f4-2,54" H 1650 5750 50  0001 C CNN
 F 3 "" H 1650 5750 50  0001 C CNN
 	1    1650 5750
@@
 P 1650 6450
 F 0 "J16" H 1650 6650 50  0000 C CNN
-F 1 "AQ1_SENSOR" H 1650 6150 50  0000 C CNN
-F 2 "footprint-lib:mpt_0,5%2f4-2,54" H 1650 6450 50  0001 C CNN
+F 1 "AQ1" H 1650 6150 50  0000 C CNN
+F 2 "footprint-lib:AQ_mpt_0,5%2f4-2,54" H 1650 6450 50  0001 C CNN
 F 3 "" H 1650 6450 50  0001 C CNN
 	1    1650 6450
 	-1   0    0    1
 $EndComp
-Text Label 2550 6350 2    60   ~ 0
+Text Label 2550 6450 2    60   ~ 0
 AQ1_5V
 Wire Wire Line
-	2550 6350 1850 6350
+	2550 6450 1850 6450
+Text Label 2550 7300 2    60   ~ 0
+O3_1_GND
 Text Label 2550 7000 2    60   ~ 0
-O3_1_GND
-Text Label 2550 7300 2    60   ~ 0
 O3_1_SHIELD
-Text Label 2550 7200 2    60   ~ 0
+Text Label 2550 7100 2    60   ~ 0
 O3_1_SENSOR
 Wire Wire Line
-	1850 7200 2550 7200
+	1850 7100 2550 7100
+Wire Wire Line
+	1850 7000 2550 7000
 Wire Wire Line
 	1850 7300 2550 7300
-Wire Wire Line
-	1850 7000 2550 7000
 $Comp
 L bluepill:Screw_Terminal_01x04 J17
@@
 P 1650 7200
 F 0 "J17" H 1650 7400 50  0000 C CNN
-F 1 "O3_SENSOR" H 1650 6900 50  0000 C CNN
+F 1 "O3" H 1650 6900 50  0000 C CNN
 F 2 "footprint-lib:mpt_0,5%2f4-2,54" H 1650 7200 50  0001 C CNN
 F 3 "" H 1650 7200 50  0001 C CNN
@@
 	-1   0    0    1
 $EndComp
-Text Label 2550 7100 2    60   ~ 0
+Text Label 2550 7200 2    60   ~ 0
 O3_1_24V
 Wire Wire Line
-	2550 7100 1850 7100
+	2550 7200 1850 7200
 $Comp
 L bluepill:Conn_01x18 J18
@@
 P 4100 1250
 F 0 "J13" H 4020 1667 50  0000 C CNN
-F 1 "FLOW_SENSOR" H 4020 1576 50  0000 C CNN
-F 2 "footprint-lib:mpt_0,5%2f5-2,54" H 4100 1250 50  0001 C CNN
+F 1 "FLOW" H 4020 1576 50  0000 C CNN
+F 2 "footprint-lib:flow_mpt_0,5%2f5-2,54" H 4100 1250 50  0001 C CNN
 F 3 "~" H 4100 1250 50  0001 C CNN
 	1    4100 1250
@@
 P 7750 4950
 F 0 "H1" H 7850 4996 50  0000 L CNN
-F 1 "PCB2" H 7850 4905 50  0000 L CNN
+F 1 "PCB1" H 7850 4905 50  0000 L CNN
 F 2 "MountingHole:MountingHole_3.2mm_M3_DIN965" H 7750 4950 50  0001 C CNN
 F 3 "~" H 7750 4950 50  0001 C CNN
@@
 P 7750 5350
 F 0 "H3" H 7850 5396 50  0000 L CNN
-F 1 "PCB2" H 7850 5305 50  0000 L CNN
+F 1 "PCB1" H 7850 5305 50  0000 L CNN
 F 2 "MountingHole:MountingHole_3.2mm_M3_DIN965" H 7750 5350 50  0001 C CNN
 F 3 "~" H 7750 5350 50  0001 C CNN
@@
 P 8500 5150
 F 0 "H6" H 8600 5196 50  0000 L CNN
-F 1 "PCB1" H 8600 5105 50  0000 L CNN
+F 1 "PCB2" H 8600 5105 50  0000 L CNN
 F 2 "MountingHole:MountingHole_3.2mm_M3_DIN965" H 8500 5150 50  0001 C CNN
 F 3 "~" H 8500 5150 50  0001 C CNN
@@
 P 8500 5550
 F 0 "H8" H 8600 5596 50  0000 L CNN
-F 1 "PCB1" H 8600 5505 50  0000 L CNN
+F 1 "PCB2" H 8600 5505 50  0000 L CNN
 F 2 "MountingHole:MountingHole_3.2mm_M3_DIN965" H 8500 5550 50  0001 C CNN
 F 3 "~" H 8500 5550 50  0001 C CNN

Commit message: update,
Connections:
- net labels added: IONAIR_RX, IONAIR_TX, SSR-25-DA_N, SSR-25-DA_P
- net labels removed: SSR-24-DA_N, SSR-24-DA_P
Changed lines of the file:
@@
 $Descr A4 11693 8268
 encoding utf-8
-Sheet 1 1
+Sheet 1 9
 Title ""
 Date ""
@@
 $EndComp
 Text Label 9000 3000 0    60   ~ 0
-SSR-24-DA_P
+SSR-25-DA_P
 Text Label 9000 3100 0    60   ~ 0
-SSR-24-DA_N
+SSR-25-DA_N
 Text Label 9000 3200 0    60   ~ 0
 PCB1_232_RX
@@
 $EndComp
 Wire Wire Line
-	9000 3000 10000 3000
-Wire Wire Line
-	9000 3100 10000 3100
-Wire Wire Line
-	9000 3200 10000 3200
-Wire Wire Line
-	9000 3300 10000 3300
+	8450 3000 10000 3000
+Wire Wire Line
+	8450 3100 10000 3100
 Wire Wire Line
 	10000 2900 9350 2900
@@
 	9350 2900 9350 2750
 Text Label 7550 2900 2    60   ~ 0
-SSR-24-DA_P
+SSR-25-DA_P
 Text Label 7550 3000 2    60   ~ 0
-SSR-24-DA_N
+SSR-25-DA_N
 Wire Wire Line
 	7550 2900 6550 2900
@@
 	1    0    0    -1
 $EndComp
+$Sheet
+S 6500 6600 1550 900
+U 5BEEE39B
+F0 "stm32_board" 60
+F1 "stm32_board.sch" 60
+$EndSheet
+Text Label 8450 3300 0    50   ~ 0
+IONAIR_TX
+Text Label 8450 3200 0    50   ~ 0
+IONAIR_RX
+Text GLabel 9000 3400 0    50   Input ~ 0
+PCB1_ALARM_COM
+Wire Wire Line
+	8450 3300 10000 3300
+Wire Wire Line
+	8450 3200 10000 3200
+Text GLabel 8450 3200 0    60   Input ~ 0
+IONAIR_RX
+Text GLabel 8450 3300 0    60   Input ~ 0
+IONAIR_TX
+Text GLabel 8450 3000 0    60   Input ~ 0
+SSR-25-DA_P
+Text GLabel 8450 3100 0    60   Input ~ 0
+SSR-25-DA_N
 $EndSCHEMATC

Commit message: update,
Changed lines of the file:
@@
 $Descr A4 11693 8268
 encoding utf-8
-Sheet 1 9
+Sheet 1 10
 Title ""
 Date ""
@@
 Text GLabel 8450 3100 0    60   Input ~ 0
 SSR-25-DA_N
+Text GLabel 6550 2100 0    60   Input ~ 0
+IONAIR_RX
+Text GLabel 6550 2200 0    60   Input ~ 0
+IONAIR_TX
 $EndSCHEMATC

Commit message: align mounting hole,
Parts:
- added H? (x4): STM32_MOUNT, MountingHole:MountingHole_3.7mm, symbol Mechanical:MountingHole
- H1, H16, H2, H3, H4, H5, H6, H7, H8, H9: footprint MountingHole:MountingHole_3.2mm_M3_DIN965 -> MountingHole:MountingHole_3.7mm
Changed lines of the file:
@@
 F 0 "H1" H 7850 4996 50  0000 L CNN
 F 1 "PCB1" H 7850 4905 50  0000 L CNN
-F 2 "MountingHole:MountingHole_3.2mm_M3_DIN965" H 7750 4950 50  0001 C CNN
+F 2 "MountingHole:MountingHole_3.7mm" H 7750 4950 50  0001 C CNN
 F 3 "~" H 7750 4950 50  0001 C CNN
 	1    7750 4950
@@
 F 0 "H2" H 7850 5196 50  0000 L CNN
 F 1 "PCB2" H 7850 5105 50  0000 L CNN
-F 2 "MountingHole:MountingHole_3.2mm_M3_DIN965" H 7750 5150 50  0001 C CNN
+F 2 "MountingHole:MountingHole_3.7mm" H 7750 5150 50  0001 C CNN
 F 3 "~" H 7750 5150 50  0001 C CNN
 	1    7750 5150
@@
 F 0 "H3" H 7850 5396 50  0000 L CNN
 F 1 "PCB1" H 7850 5305 50  0000 L CNN
-F 2 "MountingHole:MountingHole_3.2mm_M3_DIN965" H 7750 5350 50  0001 C CNN
+F 2 "MountingHole:MountingHole_3.7mm" H 7750 5350 50  0001 C CNN
 F 3 "~" H 7750 5350 50  0001 C CNN
 	1    7750 5350
@@
 F 0 "H4" H 7850 5596 50  0000 L CNN
 F 1 "PCB2" H 7850 5505 50  0000 L CNN
-F 2 "MountingHole:MountingHole_3.2mm_M3_DIN965" H 7750 5550 50  0001 C CNN
+F 2 "MountingHole:MountingHole_3.7mm" H 7750 5550 50  0001 C CNN
 F 3 "~" H 7750 5550 50  0001 C CNN
 	1    7750 5550
@@
 F 0 "H5" H 8600 4996 50  0000 L CNN
 F 1 "PCB1" H 8600 4905 50  0000 L CNN
-F 2 "MountingHole:MountingHole_3.2mm_M3_DIN965" H 8500 4950 50  0001 C CNN
+F 2 "MountingHole:MountingHole_3.7mm" H 8500 4950 50  0001 C CNN
 F 3 "~" H 8500 4950 50  0001 C CNN
 	1    8500 4950
@@
 F 0 "H6" H 8600 5196 50  0000 L CNN
 F 1 "PCB2" H 8600 5105 50  0000 L CNN
-F 2 "MountingHole:MountingHole_3.2mm_M3_DIN965" H 8500 5150 50  0001 C CNN
+F 2 "MountingHole:MountingHole_3.7mm" H 8500 5150 50  0001 C CNN
 F 3 "~" H 8500 5150 50  0001 C CNN
 	1    8500 5150
@@
 F 0 "H7" H 8600 5396 50  0000 L CNN
 F 1 "PCB1" H 8600 5305 50  0000 L CNN
-F 2 "MountingHole:MountingHole_3.2mm_M3_DIN965" H 8500 5350 50  0001 C CNN
+F 2 "MountingHole:MountingHole_3.7mm" H 8500 5350 50  0001 C CNN
 F 3 "~" H 8500 5350 50  0001 C CNN
 	1    8500 5350
@@
 F 0 "H8" H 8600 5596 50  0000 L CNN
 F 1 "PCB2" H 8600 5505 50  0000 L CNN
-F 2 "MountingHole:MountingHole_3.2mm_M3_DIN965" H 8500 5550 50  0001 C CNN
+F 2 "MountingHole:MountingHole_3.7mm" H 8500 5550 50  0001 C CNN
 F 3 "~" H 8500 5550 50  0001 C CNN
 	1    8500 5550
@@
 F 0 "H9" H 8600 5796 50  0000 L CNN
 F 1 "PCB1" H 8600 5705 50  0000 L CNN
-F 2 "MountingHole:MountingHole_3.2mm_M3_DIN965" H 8500 5750 50  0001 C CNN
+F 2 "MountingHole:MountingHole_3.7mm" H 8500 5750 50  0001 C CNN
 F 3 "~" H 8500 5750 50  0001 C CNN
 	1    8500 5750
@@
 F 0 "H16" H 9800 4996 50  0000 L CNN
 F 1 "HEATSINK_SCREW" H 9800 4905 50  0000 L CNN
-F 2 "MountingHole:MountingHole_3.2mm_M3_DIN965" H 9700 4950 50  0001 C CNN
+F 2 "MountingHole:MountingHole_3.7mm" H 9700 4950 50  0001 C CNN
 F 3 "~" H 9700 4950 50  0001 C CNN
 	1    9700 4950
@@
 Text GLabel 6550 2200 0    60   Input ~ 0
 IONAIR_TX
+$Comp
+L Mechanical:MountingHole H?
+U 1 1 5BF6BD7A
+P 6650 4950
+F 0 "H?" H 6750 4996 50  0000 L CNN
+F 1 "STM32_MOUNT" H 6750 4905 50  0000 L CNN
+F 2 "MountingHole:MountingHole_3.7mm" H 6650 4950 50  0001 C CNN
+F 3 "~" H 6650 4950 50  0001 C CNN
+	1    6650 4950
+	1    0    0    -1
+$EndComp
+$Comp
+L Mechanical:MountingHole H?
+U 1 1 5BF6BD80
+P 6650 5150
+F 0 "H?" H 6750 5196 50  0000 L CNN
+F 1 "STM32_MOUNT" H 6750 5105 50  0000 L CNN
+F 2 "MountingHole:MountingHole_3.7mm" H 6650 5150 50  0001 C CNN
+F 3 "~" H 6650 5150 50  0001 C CNN
+	1    6650 5150
+	1    0    0    -1
+$EndComp
+$Comp
+L Mechanical:MountingHole H?
+U 1 1 5BF6BD86
+P 6650 5350
+F 0 "H?" H 6750 5396 50  0000 L CNN
+F 1 "STM32_MOUNT" H 6750 5305 50  0000 L CNN
+F 2 "MountingHole:MountingHole_3.7mm" H 6650 5350 50  0001 C CNN
+F 3 "~" H 6650 5350 50  0001 C CNN
+	1    6650 5350
+	1    0    0    -1
+$EndComp
+$Comp
+L Mechanical:MountingHole H?
+U 1 1 5BF6BD8C
+P 6650 5550
+F 0 "H?" H 6750 5596 50  0000 L CNN
+F 1 "STM32_MOUNT" H 6750 5505 50  0000 L CNN
+F 2 "MountingHole:MountingHole_3.7mm" H 6650 5550 50  0001 C CNN
+F 3 "~" H 6650 5550 50  0001 C CNN
+	1    6650 5550
+	1    0    0    -1
+$EndComp
 $EndSCHEMATC
