File: backplane/backplane.sch (KiCad schematic (older format))
At the start: 34 parts, among them J1 Conn_PCB1, J10 Conn_SSR_INPUT, J12 Conn_SSR_PCB2, J13 FLOW, J15 AQ2, J16 AQ1, J17 O3, J18 Conn_TO_ION_AIR, J2 Conn_PCB2, J23 PCB1_COMM_CONNECTOR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

Commit message: backport footprint from pcb,
Parts:
- H1, H16, H2, H3, H4, H5, H6, H7, H8, H9: footprint MountingHole:MountingHole_3.7mm -> MountingHole:MountingHole_5.3mm_M5_DIN965
- J4: footprint footprint-lib:s8b-ph-kl -> Connector_JST:JST_XH_S08B-XH-A_1x08_P2.50mm_Horizontal
Changed lines of the file:
@@
 F 0 "J4" H 10280 3192 50  0000 L CNN
 F 1 "TO_CONTROL_BOARD" H 10280 3101 50  0000 L CNN
-F 2 "footprint-lib:s8b-ph-kl" H 10200 3200 50  0001 C CNN
+F 2 "Connector_JST:JST_XH_S08B-XH-A_1x08_P2.50mm_Horizontal" H 10200 3200 50  0001 C CNN
 F 3 "~" H 10200 3200 50  0001 C CNN
 	1    10200 3200
@@
 F 0 "H1" H 7850 4996 50  0000 L CNN
 F 1 "PCB1" H 7850 4905 50  0000 L CNN
-F 2 "MountingHole:MountingHole_3.7mm" H 7750 4950 50  0001 C CNN
+F 2 "MountingHole:MountingHole_5.3mm_M5_DIN965" H 7750 4950 50  0001 C CNN
 F 3 "~" H 7750 4950 50  0001 C CNN
 	1    7750 4950
@@
 F 0 "H2" H 7850 5196 50  0000 L CNN
 F 1 "PCB2" H 7850 5105 50  0000 L CNN
-F 2 "MountingHole:MountingHole_3.7mm" H 7750 5150 50  0001 C CNN
+F 2 "MountingHole:MountingHole_5.3mm_M5_DIN965" H 7750 5150 50  0001 C CNN
 F 3 "~" H 7750 5150 50  0001 C CNN
 	1    7750 5150
@@
 F 0 "H3" H 7850 5396 50  0000 L CNN
 F 1 "PCB1" H 7850 5305 50  0000 L CNN
-F 2 "MountingHole:MountingHole_3.7mm" H 7750 5350 50  0001 C CNN
+F 2 "MountingHole:MountingHole_5.3mm_M5_DIN965" H 7750 5350 50  0001 C CNN
 F 3 "~" H 7750 5350 50  0001 C CNN
 	1    7750 5350
@@
 F 0 "H4" H 7850 5596 50  0000 L CNN
 F 1 "PCB2" H 7850 5505 50  0000 L CNN
-F 2 "MountingHole:MountingHole_3.7mm" H 7750 5550 50  0001 C CNN
+F 2 "MountingHole:MountingHole_5.3mm_M5_DIN965" H 7750 5550 50  0001 C CNN
 F 3 "~" H 7750 5550 50  0001 C CNN
 	1    7750 5550
@@
 F 0 "H5" H 8600 4996 50  0000 L CNN
 F 1 "PCB1" H 8600 4905 50  0000 L CNN
-F 2 "MountingHole:MountingHole_3.7mm" H 8500 4950 50  0001 C CNN
+F 2 "MountingHole:MountingHole_5.3mm_M5_DIN965" H 8500 4950 50  0001 C CNN
 F 3 "~" H 8500 4950 50  0001 C CNN
 	1    8500 4950
@@
 F 0 "H6" H 8600 5196 50  0000 L CNN
 F 1 "PCB2" H 8600 5105 50  0000 L CNN
-F 2 "MountingHole:MountingHole_3.7mm" H 8500 5150 50  0001 C CNN
+F 2 "MountingHole:MountingHole_5.3mm_M5_DIN965" H 8500 5150 50  0001 C CNN
 F 3 "~" H 8500 5150 50  0001 C CNN
 	1    8500 5150
@@
 F 0 "H7" H 8600 5396 50  0000 L CNN
 F 1 "PCB1" H 8600 5305 50  0000 L CNN
-F 2 "MountingHole:MountingHole_3.7mm" H 8500 5350 50  0001 C CNN
+F 2 "MountingHole:MountingHole_5.3mm_M5_DIN965" H 8500 5350 50  0001 C CNN
 F 3 "~" H 8500 5350 50  0001 C CNN
 	1    8500 5350
@@
 F 0 "H8" H 8600 5596 50  0000 L CNN
 F 1 "PCB2" H 8600 5505 50  0000 L CNN
-F 2 "MountingHole:MountingHole_3.7mm" H 8500 5550 50  0001 C CNN
+F 2 "MountingHole:MountingHole_5.3mm_M5_DIN965" H 8500 5550 50  0001 C CNN
 F 3 "~" H 8500 5550 50  0001 C CNN
 	1    8500 5550
@@
 F 0 "H9" H 8600 5796 50  0000 L CNN
 F 1 "PCB1" H 8600 5705 50  0000 L CNN
-F 2 "MountingHole:MountingHole_3.7mm" H 8500 5750 50  0001 C CNN
+F 2 "MountingHole:MountingHole_5.3mm_M5_DIN965" H 8500 5750 50  0001 C CNN
 F 3 "~" H 8500 5750 50  0001 C CNN
 	1    8500 5750
@@
 F 0 "H16" H 9800 4996 50  0000 L CNN
 F 1 "HEATSINK_SCREW" H 9800 4905 50  0000 L CNN
-F 2 "MountingHole:MountingHole_3.7mm" H 9700 4950 50  0001 C CNN
+F 2 "MountingHole:MountingHole_5.3mm_M5_DIN965" H 9700 4950 50  0001 C CNN
 F 3 "~" H 9700 4950 50  0001 C CNN
 	1    9700 4950
