File: backplane/backplane.sch (KiCad schematic (older format))
At the start: 34 parts, among them J1 Conn_PCB1, J10 Conn_SSR_INPUT, J12 Conn_SSR_PCB2, J13 FLOW, J15 AQ2, J16 AQ1, J17 O3, J18 Conn_TO_ION_AIR, J2 Conn_PCB2, J23 PCB1_COMM_CONNECTOR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

Commit message: update,
Parts:
- gave numbers to parts that had none: 4
Changed lines of the file:
@@
 IONAIR_TX
 $Comp
-L Mechanical:MountingHole H?
+L Mechanical:MountingHole H17
 U 1 1 5BF6BD7A
 P 6650 4950
-F 0 "H?" H 6750 4996 50  0000 L CNN
+F 0 "H17" H 6750 4996 50  0000 L CNN
 F 1 "STM32_MOUNT" H 6750 4905 50  0000 L CNN
 F 2 "MountingHole:MountingHole_3.7mm" H 6650 4950 50  0001 C CNN
@@
 $EndComp
 $Comp
-L Mechanical:MountingHole H?
+L Mechanical:MountingHole H18
 U 1 1 5BF6BD80
 P 6650 5150
-F 0 "H?" H 6750 5196 50  0000 L CNN
+F 0 "H18" H 6750 5196 50  0000 L CNN
 F 1 "STM32_MOUNT" H 6750 5105 50  0000 L CNN
 F 2 "MountingHole:MountingHole_3.7mm" H 6650 5150 50  0001 C CNN
@@
 $EndComp
 $Comp
-L Mechanical:MountingHole H?
+L Mechanical:MountingHole H19
 U 1 1 5BF6BD86
 P 6650 5350
-F 0 "H?" H 6750 5396 50  0000 L CNN
+F 0 "H19" H 6750 5396 50  0000 L CNN
 F 1 "STM32_MOUNT" H 6750 5305 50  0000 L CNN
 F 2 "MountingHole:MountingHole_3.7mm" H 6650 5350 50  0001 C CNN
@@
 $EndComp
 $Comp
-L Mechanical:MountingHole H?
+L Mechanical:MountingHole H20
 U 1 1 5BF6BD8C
 P 6650 5550
-F 0 "H?" H 6750 5596 50  0000 L CNN
+F 0 "H20" H 6750 5596 50  0000 L CNN
 F 1 "STM32_MOUNT" H 6750 5505 50  0000 L CNN
 F 2 "MountingHole:MountingHole_3.7mm" H 6650 5550 50  0001 C CNN
@@
 	1    0    0    -1
 $EndComp
+Text GLabel 3700 3650 2    60   Input ~ 0
+PWR_SOURCE_SSR_L_1
+Text GLabel 3700 3750 2    60   Input ~ 0
+SSR_PCB2_L_2
 $EndSCHEMATC

Commit message: update,
Connections:
- net labels added: RELAY_N, RELAY_P
Changed lines of the file:
@@
 Text GLabel 8450 3300 0    60   Input ~ 0
 IONAIR_TX
-Text GLabel 8450 3000 0    60   Input ~ 0
-SSR-25-DA_P
-Text GLabel 8450 3100 0    60   Input ~ 0
-SSR-25-DA_N
 Text GLabel 6550 2100 0    60   Input ~ 0
 IONAIR_RX
@@
 Text GLabel 3700 3750 2    60   Input ~ 0
 SSR_PCB2_L_2
+Text GLabel 8450 3000 0    60   Input ~ 0
+RELAY_P
+Text GLabel 8450 3100 0    60   Input ~ 0
+RELAY_N
 $EndSCHEMATC

Commit message: update,
Changed lines of the file:
@@
 	6400 1300 8100 1300
 Wire Wire Line
-	6550 2100 7850 2100
+	6550 2200 7850 2200
 Wire Wire Line
 	6550 2000 7500 2000
 Text Label 6550 2000 0    60   ~ 0
 PCB1_UART_COM
+Text Label 6550 2200 0    60   ~ 0
+PCB1_232_RX
 Text Label 6550 2100 0    60   ~ 0
-PCB1_232_RX
-Text Label 6550 2200 0    60   ~ 0
 PCB1_232_TX
 $Comp
@@
 L bluepill:Conn_01x02 J3
 U 1 1 5BEF34ED
-P 6350 2900
-F 0 "J3" H 6350 3000 50  0000 C CNN
-F 1 "SSR_CONTROL" H 6350 2700 50  0000 C CNN
-F 2 "footprint-lib:mpt_0,5%2f2-2,54" H 6350 2900 50  0001 C CNN
-F 3 "" H 6350 2900 50  0001 C CNN
-	1    6350 2900
-	-1   0    0    -1
+P 6350 3000
+F 0 "J3" H 6350 3100 50  0000 C CNN
+F 1 "SSR_CONTROL" H 6350 2800 50  0000 C CNN
+F 2 "footprint-lib:mpt_0,5%2f2-2,54" H 6350 3000 50  0001 C CNN
+F 3 "" H 6350 3000 50  0001 C CNN
+	1    6350 3000
+	-1   0    0    1
 $EndComp
 Text Label 9000 3000 0    60   ~ 0
@@
 	7500 2000 7850 2000
 Wire Wire Line
-	6550 2200 7850 2200
+	6550 2100 7850 2100
 $Comp
 L Mechanical:MountingHole H1
@@
 Text GLabel 8450 3300 0    60   Input ~ 0
 IONAIR_TX
+Text GLabel 6550 2200 0    60   Input ~ 0
+IONAIR_RX
 Text GLabel 6550 2100 0    60   Input ~ 0
-IONAIR_RX
-Text GLabel 6550 2200 0    60   Input ~ 0
 IONAIR_TX
 $Comp

Commit message: update,
Other:
- note added: "1: IONAIR GND\n2: IONAIR RX PIN\n3: IONAIR TX PIN"
Changed lines of the file:
@@
 Text GLabel 8450 3100 0    60   Input ~ 0
 RELAY_N
+Text Notes 8200 2200 0    60   ~ 0
+1: IONAIR GND\n2: IONAIR RX PIN\n3: IONAIR TX PIN
 $EndSCHEMATC
