File: backplane/SSR-25-DA_DRIVER.sch (KiCad schematic (older format))
At the start: 6 parts, among them Q3 2N3904(1AM)

Commit message: update,
Parts:
- added D11: SD_M7, Diode_SMD:D_SOD-123, symbol taobao-sd:SD_M7
- added K1: SLA-05VDC-SL-C, footprint-lib:SLA-05VDC-SL-C, symbol taobao-relay:SLA-05VDC-SL-C
Connections:
- net labels added: POWER_CONTROL_COM, POWER_CONTROL_NO
- net labels removed: SSR-25-DA_N, SSR-25-DA_P
- wire segments 21 -> 31
Changed lines of the file:
@@
 	6250 3250 6250 3350
-Wire Wire Line
-	5850 2550 5850 2650
 Wire Wire Line
 	5850 2850 5850 2950
@@
 L taobao-r:R151 R?
 U 1 1 5BDCB69D
-P 6400 2850
+P 6400 2000
 AR Path="/5BCB4A39/5BDCB69D" Ref="R?"  Part="1"
 AR Path="/5BE41138/5BDCB69D" Ref="R?"  Part="1"
 AR Path="/5BCB679F/5BDCB69D" Ref="R?"  Part="1"
 AR Path="/5BEEE39B/5BCB679F/5BDCB69D" Ref="R14"  Part="1"
-F 0 "R14" H 6459 2896 50  0000 L CNN
-F 1 "R151" H 6459 2805 50  0000 L CNN
-F 2 "Resistor_SMD:R_0603_1608Metric_Pad1.05x0.95mm_HandSolder" H 6400 2850 50  0001 C CNN
-F 3 "~" H 6400 2850 50  0001 C CNN
-	1    6400 2850
+F 0 "R14" H 6459 2046 50  0000 L CNN
+F 1 "R151" H 6459 1955 50  0000 L CNN
+F 2 "Resistor_SMD:R_0603_1608Metric_Pad1.05x0.95mm_HandSolder" H 6400 2000 50  0001 C CNN
+F 3 "~" H 6400 2000 50  0001 C CNN
+	1    6400 2000
 	1    0    0    -1
 $EndComp
 Wire Wire Line
-	6400 2550 6400 2750
+	6400 1700 6400 1900
 Wire Wire Line
-	6400 2950 6400 3050
+	6400 2100 6400 2200
 Wire Wire Line
-	6400 3050 6900 3050
+	6400 2200 6500 2200
 Connection ~ 6250 3250
 $Comp
 L power:VDD #PWR?
 U 1 1 5BDCB6B8
-P 6100 2450
+P 6100 1600
 AR Path="/5BCB4A39/5BDCB6B8" Ref="#PWR?"  Part="1"
 AR Path="/5BE41138/5BDCB6B8" Ref="#PWR?"  Part="1"
 AR Path="/5BCB679F/5BDCB6B8" Ref="#PWR?"  Part="1"
 AR Path="/5BEEE39B/5BCB679F/5BDCB6B8" Ref="#PWR0125"  Part="1"
-F 0 "#PWR0125" H 6100 2300 50  0001 C CNN
-F 1 "VDD" H 6117 2623 50  0000 C CNN
-F 2 "" H 6100 2450 50  0001 C CNN
-F 3 "" H 6100 2450 50  0001 C CNN
-	1    6100 2450
+F 0 "#PWR0125" H 6100 1450 50  0001 C CNN
+F 1 "VDD" H 6117 1773 50  0000 C CNN
+F 2 "" H 6100 1600 50  0001 C CNN
+F 3 "" H 6100 1600 50  0001 C CNN
+	1    6100 1600
 	1    0    0    -1
 $EndComp
 Wire Wire Line
-	6100 2450 6100 2550
+	6100 1600 6100 1700
 Wire Wire Line
-	6100 2550 5850 2550
+	6100 1700 5850 1700
 Wire Wire Line
-	6100 2550 6400 2550
-Connection ~ 6100 2550
+	6100 1700 6400 1700
+Connection ~ 6100 1700
 $Comp
 L taobao-transistor:2N3904(1AM) Q?
@@
 	1    0    0    -1
 $EndComp
-Text HLabel 6900 3250 2    50   Input ~ 0
-SSR-25-DA_N
-Text HLabel 6900 3050 2    50   Input ~ 0
-SSR-25-DA_P
+Text HLabel 7650 3250 2    50   Input ~ 0
+POWER_CONTROL_COM
+Text HLabel 7650 2200 2    50   Input ~ 0
+POWER_CONTROL_NO
 Wire Wire Line
-	6250 3250 6900 3250
+	6250 3250 6500 3250
+$Comp
+L taobao-relay:SLA-05VDC-SL-C K1
+U 1 1 5BFF6769
+P 7100 2700
+F 0 "K1" H 7530 2746 50  0000 L CNN
+F 1 "SLA-05VDC-SL-C" H 7530 2655 50  0000 L CNN
+F 2 "footprint-lib:SLA-05VDC-SL-C" H 7550 2650 50  0001 L CNN
+F 3 "http://www.omron.com/ecb/products/pdf/en-g5le.pdf" H 7100 2300 50  0001 C CNN
+	1    7100 2700
+	1    0    0    -1
+$EndComp
+Wire Wire Line
+	5850 1700 5850 2650
+Wire Wire Line
+	6900 2200 6900 2400
+Wire Wire Line
+	6900 3000 6900 3250
+$Comp
+L taobao-sd:SD_M7 D11
+U 1 1 5BFF70E1
+P 6500 2750
+F 0 "D11" V 6454 2818 50  0000 L CNN
+F 1 "SD_M7" V 6545 2818 50  0000 L CNN
+F 2 "Diode_SMD:D_SOD-123" V 6500 2750 50  0001 C CNN
+F 3 "~" V 6500 2750 50  0001 C CNN
+	1    6500 2750
+	0    1    1    0
+$EndComp
+Wire Wire Line
+	6500 2650 6500 2200
+Connection ~ 6500 2200
+Wire Wire Line
+	6500 2200 6900 2200
+Wire Wire Line
+	6500 2850 6500 3250
+Connection ~ 6500 3250
+Wire Wire Line
+	6500 3250 6900 3250
+Wire Wire Line
+	7300 3000 7300 3250
+Wire Wire Line
+	7300 3250 7650 3250
+Wire Wire Line
+	7650 2200 7400 2200
+Wire Wire Line
+	7400 2200 7400 2400
 $EndSCHEMATC
