File: backplane/SSR-25-DA_DRIVER.sch (KiCad schematic (older format))
At the start: 8 parts, among them K1 SLA-05VDC-SL-C, Q3 2N3904(1AM)

Commit message: update,
Connections:
- net labels added: RELAY_N, RELAY_P
- wire segments 31 -> 37
Changed lines of the file:
@@
 Connection ~ 6500 2200
 Wire Wire Line
-	6500 2200 6900 2200
+	6500 2200 6800 2200
 Wire Wire Line
 	6500 2850 6500 3250
 Connection ~ 6500 3250
 Wire Wire Line
-	6500 3250 6900 3250
+	6500 3250 6800 3250
 Wire Wire Line
 	7300 3000 7300 3250
@@
 EndData
 $EndBitmap
+Text GLabel 6900 2050 2    60   Input ~ 0
+RELAY_P
+Wire Wire Line
+	6900 2050 6800 2050
+Wire Wire Line
+	6800 2050 6800 2200
+Connection ~ 6800 2200
+Wire Wire Line
+	6800 2200 6900 2200
+Text GLabel 6900 3400 2    60   Input ~ 0
+RELAY_N
+Wire Wire Line
+	6800 3250 6800 3400
+Wire Wire Line
+	6800 3400 6900 3400
+Connection ~ 6800 3250
+Wire Wire Line
+	6800 3250 6900 3250
 $EndSCHEMATC

Commit message: update resistor for relay,
Parts:
- R14: value R151 -> R220
Changed lines of the file:
@@
 AR Path="/5BEEE39B/5BCB679F/5BDCB69D" Ref="R14"  Part="1"
 F 0 "R14" H 6459 2046 50  0000 L CNN
-F 1 "R151" H 6459 1955 50  0000 L CNN
+F 1 "R220" H 6459 1955 50  0000 L CNN
 F 2 "Resistor_SMD:R_0603_1608Metric_Pad1.05x0.95mm_HandSolder" H 6400 2000 50  0001 C CNN
 F 3 "~" H 6400 2000 50  0001 C CNN

Commit message: fix R14 for coil relay,
Parts:
- R14: value R220 -> R100
Changed lines of the file:
@@
 AR Path="/5BEEE39B/5BCB679F/5BDCB69D" Ref="R14"  Part="1"
 F 0 "R14" H 6459 2046 50  0000 L CNN
-F 1 "R220" H 6459 1955 50  0000 L CNN
+F 1 "R100" H 6459 1955 50  0000 L CNN
 F 2 "Resistor_SMD:R_0603_1608Metric_Pad1.05x0.95mm_HandSolder" H 6400 2000 50  0001 C CNN
 F 3 "~" H 6400 2000 50  0001 C CNN

Commit message: as fit resistor value to actual working value,
Parts:
- Q3: value 2N3904(1AM) -> SS9013(J3)
- R11: value R331 -> R103
- R12: value R103 -> R331
Changed lines of the file:
@@
 AR Path="/5BEEE39B/5BCB679F/5BDCB66A" Ref="R11"  Part="1"
 F 0 "R11" V 5354 3550 50  0000 C CNN
-F 1 "R331" V 5445 3550 50  0000 C CNN
+F 1 "R103" V 5445 3550 50  0000 C CNN
 F 2 "Resistor_SMD:R_0603_1608Metric_Pad1.05x0.95mm_HandSolder" H 5550 3550 50  0001 C CNN
 F 3 "~" H 5550 3550 50  0001 C CNN
@@
 AR Path="/5BEEE39B/5BCB679F/5BDCB672" Ref="R12"  Part="1"
 F 0 "R12" H 5859 3996 50  0000 L CNN
-F 1 "R103" H 5859 3905 50  0000 L CNN
+F 1 "R331" H 5859 3905 50  0000 L CNN
 F 2 "Resistor_SMD:R_0603_1608Metric_Pad1.05x0.95mm_HandSolder" H 5800 3950 50  0001 C CNN
 F 3 "~" H 5800 3950 50  0001 C CNN
@@
 AR Path="/5BEEE39B/5BCB679F/5BDCB6C2" Ref="Q3"  Part="1"
 F 0 "Q3" H 6350 3600 50  0000 L CNN
-F 1 "2N3904(1AM)" H 6350 3550 50  0000 L CNN
+F 1 "SS9013(J3)" H 6350 3550 50  0000 L CNN
 F 2 "Package_TO_SOT_SMD:SOT-23_Handsoldering" H 6350 3475 50  0001 L CIN
 F 3 "" H 6150 3550 50  0001 L CNN
