File: backplane/stm32_board.sch (KiCad schematic (older format))
At the start: 11 parts, among them J11 FAN, J14 FCC_B2B, J19 PCB_UART, J20 SSR_25, J6 48V_SRC, J7 WS2812, J8 PURFUME, J9 SSR2

Commit message: update,
Changed lines of the file:
@@
 $Descr A3 16535 11693
 encoding utf-8
-Sheet 2 9
+Sheet 2 10
 Title ""
 Date ""
@@
 Text GLabel 15800 8200 2    60   Input ~ 0
 SSR-25-DA_N
+$Sheet
+S 6200 11050 1500 850
+U 5BF2E866
+F0 "IONAIR_ALARM" 50
+F1 "IONAIR_ALARM.sch" 50
+$EndSheet
 $EndSCHEMATC

Commit message: update,
Parts:
- removed J19: PCB_UART, footprint-lib:s3b-ph-kl, symbol Connector_Generic:Conn_01x03
- removed J20: SSR_25, footprint-lib:s2b-ph-kl, symbol Connector_Generic:Conn_01x02
Connections:
- wire segments 78 -> 72
Changed lines of the file:
@@
 Wire Wire Line
 	14450 8100 15800 8100
-Text Label 10000 8000 0    50   ~ 0
-SSR-25-DA_P
-Text Label 10000 8100 0    50   ~ 0
-SSR-25-DA_N
-Wire Wire Line
-	10800 8100 10000 8100
-Wire Wire Line
-	10800 8000 10000 8000
-$Comp
-L Connector_Generic:Conn_01x02 J20
-U 1 1 5BCB931B
-P 11000 8100
-F 0 "J20" H 11080 8092 50  0000 L CNN
-F 1 "SSR_25" H 11080 8001 50  0000 L CNN
-F 2 "footprint-lib:s2b-ph-kl" H 11000 8100 50  0001 C CNN
-F 3 "~" H 11000 8100 50  0001 C CNN
-	1    11000 8100
-	1    0    0    1
-$EndComp
 $Sheet
 S 6200 6150 1500 750
@@
 Text Label 15200 6850 2    50   ~ 0
 IONAIR_RX
-$Comp
-L Connector_Generic:Conn_01x03 J19
-U 1 1 5BCF033A
-P 11000 6750
-F 0 "J19" H 11080 6742 50  0000 L CNN
-F 1 "PCB_UART" H 11080 6651 50  0000 L CNN
-F 2 "footprint-lib:s3b-ph-kl" H 11000 6750 50  0001 C CNN
-F 3 "~" H 11000 6750 50  0001 C CNN
-	1    11000 6750
-	1    0    0    -1
-$EndComp
-Text Label 10050 6750 0    50   ~ 0
-IONAIR_TX
-Wire Wire Line
-	10050 6750 10800 6750
-Wire Wire Line
-	10050 6650 10800 6650
 Wire Wire Line
 	3500 3200 3750 3200
@@
 Wire Wire Line
 	6000 8750 6200 8750
-$Comp
-L power:GND #PWR0111
-U 1 1 5BD58CE7
-P 10650 6950
-F 0 "#PWR0111" H 10650 6700 50  0001 C CNN
-F 1 "GND" H 10655 6777 50  0000 C CNN
-F 2 "" H 10650 6950 50  0001 C CNN
-F 3 "" H 10650 6950 50  0001 C CNN
-	1    10650 6950
-	-1   0    0    -1
-$EndComp
-Wire Wire Line
-	10650 6950 10650 6850
-Wire Wire Line
-	10650 6850 10800 6850
 Text GLabel 12750 6750 0    50   Input ~ 0
 IONAIR-TTL-TX
-Text Label 10050 6650 0    50   ~ 0
-IONAIR_RX
 $Comp
 L power:+5V #PWR0112

Commit message: backport footprint from pcb,
Parts:
- J11: footprint footprint-lib:s4b-ph-kl -> Connector_JST:JST_XH_S04B-XH-A_1x04_P2.50mm_Horizontal
- J6, J8, J9: footprint footprint-lib:s2b-ph-kl -> Connector_JST:JST_XH_S02B-XH-A_1x02_P2.50mm_Horizontal
- J7: footprint footprint-lib:s3b-ph-kl -> Connector_JST:JST_XH_S03B-XH-A_1x03_P2.50mm_Horizontal
Changed lines of the file:
@@
 F 0 "J7" H 3330 8942 50  0000 L CNN
 F 1 "WS2812" H 3330 8851 50  0000 L CNN
-F 2 "footprint-lib:s3b-ph-kl" H 3250 8900 50  0001 C CNN
+F 2 "Connector_JST:JST_XH_S03B-XH-A_1x03_P2.50mm_Horizontal" H 3250 8900 50  0001 C CNN
 F 3 "~" H 3250 8900 50  0001 C CNN
 	1    3250 8900
@@
 F 0 "J8" H 4280 7292 50  0000 L CNN
 F 1 "PURFUME" H 4280 7201 50  0000 L CNN
-F 2 "footprint-lib:s2b-ph-kl" H 4200 7300 50  0001 C CNN
+F 2 "Connector_JST:JST_XH_S02B-XH-A_1x02_P2.50mm_Horizontal" H 4200 7300 50  0001 C CNN
 F 3 "~" H 4200 7300 50  0001 C CNN
 	1    4200 7300
@@
 F 0 "J11" H 4430 6342 50  0000 L CNN
 F 1 "FAN" H 4430 6251 50  0000 L CNN
-F 2 "footprint-lib:s4b-ph-kl" H 4350 6350 50  0001 C CNN
+F 2 "Connector_JST:JST_XH_S04B-XH-A_1x04_P2.50mm_Horizontal" H 4350 6350 50  0001 C CNN
 F 3 "~" H 4350 6350 50  0001 C CNN
 	1    4350 6350
@@
 F 0 "J6" H 2680 6242 50  0000 L CNN
 F 1 "48V_SRC" H 2680 6151 50  0000 L CNN
-F 2 "footprint-lib:s2b-ph-kl" H 2600 6250 50  0001 C CNN
+F 2 "Connector_JST:JST_XH_S02B-XH-A_1x02_P2.50mm_Horizontal" H 2600 6250 50  0001 C CNN
 F 3 "~" H 2600 6250 50  0001 C CNN
 	1    2600 6250
@@
 F 0 "J9" H 4280 7642 50  0000 L CNN
 F 1 "SSR2" H 4280 7551 50  0000 L CNN
-F 2 "footprint-lib:s2b-ph-kl" H 4200 7650 50  0001 C CNN
+F 2 "Connector_JST:JST_XH_S02B-XH-A_1x02_P2.50mm_Horizontal" H 4200 7650 50  0001 C CNN
 F 3 "~" H 4200 7650 50  0001 C CNN
 	1    4200 7650

Commit message: update,
Connections:
- net labels added: PWR_SOURCE_SSR_L_1, SSR_PCB2_L_2
- net labels removed: SSR-25-DA_N, SSR-25-DA_P
Changed lines of the file:
@@
 F1 "SSR-25-DA_DRIVER.sch" 50
 F2 "STM32_SSR-25-DA_OUTPUT" I L 12950 7850 50
-F3 "SSR-25-DA_P" I R 14450 8100 50
-F4 "SSR-25-DA_N" I R 14450 8200 50
-$EndSheet
-Text Label 15800 8100 2    50   ~ 0
-SSR-25-DA_P
-Text Label 15800 8200 2    50   ~ 0
-SSR-25-DA_N
+F3 "POWER_CONTROL_COM" I R 14450 8200 60
+F4 "POWER_CONTROL_NO" I R 14450 8100 60
+$EndSheet
 Wire Wire Line
 	14450 8200 15800 8200
@@
 Text GLabel 15200 6750 2    60   Input ~ 0
 IONAIR_TX
-Text GLabel 15800 8100 2    60   Input ~ 0
-SSR-25-DA_P
-Text GLabel 15800 8200 2    60   Input ~ 0
-SSR-25-DA_N
 $Sheet
 S 6200 11050 1500 850
@@
 F1 "IONAIR_ALARM.sch" 50
 $EndSheet
+Text GLabel 15800 8100 2    60   Input ~ 0
+PWR_SOURCE_SSR_L_1
+Text GLabel 15800 8200 2    60   Input ~ 0
+SSR_PCB2_L_2
 $EndSCHEMATC

Commit message: update,
Connections:
- wire segments 72 -> 73
Changed lines of the file:
@@
 $EndComp
 Wire Wire Line
-	5550 2800 5000 2800
+	5550 2800 5450 2800
 Wire Wire Line
 	5000 2800 5000 2750
 Wire Wire Line
-	5150 2650 5150 2700
-Wire Wire Line
-	5150 2700 5550 2700
+	5150 3450 5150 3400
+Wire Wire Line
+	5150 3400 5550 3400
 Text GLabel 3500 3300 0    50   Input ~ 0
 I2C_SDA
@@
 L power:+5V #PWR0112
 U 1 1 5BCE34B6
-P 5150 2650
-F 0 "#PWR0112" H 5150 2500 50  0001 C CNN
-F 1 "+5V" H 5200 2850 50  0000 C CNN
-F 2 "" H 5150 2650 50  0001 C CNN
-F 3 "" H 5150 2650 50  0001 C CNN
-	1    5150 2650
-	1    0    0    -1
+P 5150 3450
+F 0 "#PWR0112" H 5150 3300 50  0001 C CNN
+F 1 "+5V" H 5200 3650 50  0000 C CNN
+F 2 "" H 5150 3450 50  0001 C CNN
+F 3 "" H 5150 3450 50  0001 C CNN
+	1    5150 3450
+	1    0    0    1
 $EndComp
 $Comp
@@
 Text Notes 3450 6800 0    50   ~ 0
 follows PC fan ordering
-$Comp
-L power:GND #PWR0114
-U 1 1 5BE0459B
-P 5400 3600
-F 0 "#PWR0114" H 5400 3350 50  0001 C CNN
-F 1 "GND" H 5405 3427 50  0000 C CNN
-F 2 "" H 5400 3600 50  0001 C CNN
-F 3 "" H 5400 3600 50  0001 C CNN
-	1    5400 3600
-	1    0    0    -1
-$EndComp
-Wire Wire Line
-	5400 3600 5400 3400
-Wire Wire Line
-	5400 3400 5550 3400
 $Comp
 L power:+3V3 #PWR0115
@@
 Text GLabel 15800 8200 2    60   Input ~ 0
 SSR_PCB2_L_2
+Wire Wire Line
+	5550 2700 5450 2700
+Wire Wire Line
+	5450 2700 5450 2800
+Connection ~ 5450 2800
+Wire Wire Line
+	5450 2800 5000 2800
 $EndSCHEMATC

Commit message: update,
Connections:
- net labels added: EXT_TRIGGER
- wire segments 73 -> 71
Changed lines of the file:
@@
 L power:GND #PWR0110
 U 1 1 5BD0F41D
-P 5000 2750
-F 0 "#PWR0110" H 5000 2500 50  0001 C CNN
-F 1 "GND" H 5005 2577 50  0000 C CNN
-F 2 "" H 5000 2750 50  0001 C CNN
-F 3 "" H 5000 2750 50  0001 C CNN
-	1    5000 2750
+P 5000 2650
+F 0 "#PWR0110" H 5000 2400 50  0001 C CNN
+F 1 "GND" H 5005 2477 50  0000 C CNN
+F 2 "" H 5000 2650 50  0001 C CNN
+F 3 "" H 5000 2650 50  0001 C CNN
+	1    5000 2650
 	-1   0    0    1
 $EndComp
 Wire Wire Line
-	5550 2800 5450 2800
-Wire Wire Line
-	5000 2800 5000 2750
+	5000 2700 5000 2650
 Wire Wire Line
 	5150 3450 5150 3400
@@
 SSR_PCB2_L_2
 Wire Wire Line
-	5550 2700 5450 2700
-Wire Wire Line
-	5450 2700 5450 2800
-Connection ~ 5450 2800
-Wire Wire Line
-	5450 2800 5000 2800
+	5000 2700 5550 2700
+Text GLabel 4800 2800 0    50   Input ~ 0
+EXT_TRIGGER
+Wire Wire Line
+	4800 2800 5550 2800
 $EndSCHEMATC

Commit message: update,
Parts:
- J11: footprint Connector_JST:JST_XH_S04B-XH-A_1x04_P2.50mm_Horizontal -> Connector_JST:JST_XH_S04B-XH-A-1_1x04_P2.50mm_Horizontal
- J6: footprint Connector_JST:JST_XH_S02B-XH-A_1x02_P2.50mm_Horizontal -> Connector_JST:JST_XH_S02B-XH-A-1_1x02_P2.50mm_Horizontal
- J7: footprint Connector_JST:JST_XH_S03B-XH-A_1x03_P2.50mm_Horizontal -> Connector_JST:JST_XH_S03B-XH-A-1_1x03_P2.50mm_Horizontal
Changed lines of the file:
@@
 F 0 "J7" H 3330 8942 50  0000 L CNN
 F 1 "WS2812" H 3330 8851 50  0000 L CNN
-F 2 "Connector_JST:JST_XH_S03B-XH-A_1x03_P2.50mm_Horizontal" H 3250 8900 50  0001 C CNN
+F 2 "Connector_JST:JST_XH_S03B-XH-A-1_1x03_P2.50mm_Horizontal" H 3250 8900 50  0001 C CNN
 F 3 "~" H 3250 8900 50  0001 C CNN
 	1    3250 8900
@@
 F 0 "J11" H 4430 6342 50  0000 L CNN
 F 1 "FAN" H 4430 6251 50  0000 L CNN
-F 2 "Connector_JST:JST_XH_S04B-XH-A_1x04_P2.50mm_Horizontal" H 4350 6350 50  0001 C CNN
+F 2 "Connector_JST:JST_XH_S04B-XH-A-1_1x04_P2.50mm_Horizontal" H 4350 6350 50  0001 C CNN
 F 3 "~" H 4350 6350 50  0001 C CNN
 	1    4350 6350
@@
 F 0 "J6" H 2680 6242 50  0000 L CNN
 F 1 "48V_SRC" H 2680 6151 50  0000 L CNN
-F 2 "Connector_JST:JST_XH_S02B-XH-A_1x02_P2.50mm_Horizontal" H 2600 6250 50  0001 C CNN
+F 2 "Connector_JST:JST_XH_S02B-XH-A-1_1x02_P2.50mm_Horizontal" H 2600 6250 50  0001 C CNN
 F 3 "~" H 2600 6250 50  0001 C CNN
 	1    2600 6250

Commit message: add optional LED power supply from main 5V,
Parts:
- added JP?: Jumper_NO_Small, Jumper:SolderJumper-2_P1.3mm_Open_TrianglePad1.0x1.5mm, symbol Device:Jumper_NO_Small
Connections:
- wire segments 71 -> 75
Changed lines of the file:
@@
 L taobao-components:VWS2812 #PWR0106
 U 1 1 5BCB629E
-P 4200 8650
-F 0 "#PWR0106" H 4200 8500 50  0001 C CNN
-F 1 "VWS2812" H 4217 8823 50  0000 C CNN
-F 2 "" H 4200 8650 50  0001 C CNN
-F 3 "" H 4200 8650 50  0001 C CNN
-	1    4200 8650
+P 4500 8650
+F 0 "#PWR0106" H 4500 8500 50  0001 C CNN
+F 1 "VWS2812" H 4517 8823 50  0000 C CNN
+F 2 "" H 4500 8650 50  0001 C CNN
+F 3 "" H 4500 8650 50  0001 C CNN
+	1    4500 8650
 	1    0    0    -1
 $EndComp
@@
 	1    0    0    -1
 $EndComp
-Wire Wire Line
-	4200 8650 4200 8750
 Wire Wire Line
 	4200 8950 4200 9100
@@
 Wire Wire Line
 	4800 2800 5550 2800
+$Comp
+L power:+5V #PWR?
+U 1 1 5C0C4F7B
+P 4200 8350
+F 0 "#PWR?" H 4200 8200 50  0001 C CNN
+F 1 "+5V" H 4215 8523 50  0000 C CNN
+F 2 "" H 4200 8350 50  0001 C CNN
+F 3 "" H 4200 8350 50  0001 C CNN
+	1    4200 8350
+	1    0    0    -1
+$EndComp
+Wire Wire Line
+	4500 8650 4500 8700
+Wire Wire Line
+	4500 8700 4200 8700
+Wire Wire Line
+	4200 8700 4200 8750
+$Comp
+L Device:Jumper_NO_Small JP?
+U 1 1 5C0C8C74
+P 4200 8500
+F 0 "JP?" V 4154 8548 50  0000 L CNN
+F 1 "Jumper_NO_Small" V 4245 8548 50  0000 L CNN
+F 2 "Jumper:SolderJumper-2_P1.3mm_Open_TrianglePad1.0x1.5mm" H 4200 8500 50  0001 C CNN
+F 3 "~" H 4200 8500 50  0001 C CNN
+	1    4200 8500
+	0    1    1    0
+$EndComp
+Wire Wire Line
+	4200 8350 4200 8400
+Wire Wire Line
+	4200 8600 4200 8700
+Connection ~ 4200 8700
 $EndSCHEMATC
