File: backplane/stm32_board.sch (KiCad schematic (older format))
At the start: 10 parts, among them J11 FAN, J14 FCC_B2B, J6 48V_SRC, J7 WS2812, J8 PURFUME, J9 SSR2

Commit message: fix R14 for coil relay,
Parts:
- gave numbers to parts that had none: 1
Changed lines of the file:
@@
 	4800 2800 5550 2800
 $Comp
-L power:+5V #PWR?
+L power:+5V #PWR0111
 U 1 1 5C0C4F7B
 P 4200 8350
-F 0 "#PWR?" H 4200 8200 50  0001 C CNN
+F 0 "#PWR0111" H 4200 8200 50  0001 C CNN
 F 1 "+5V" H 4215 8523 50  0000 C CNN
 F 2 "" H 4200 8350 50  0001 C CNN
@@
 	4200 8700 4200 8750
 $Comp
-L Device:Jumper_NO_Small JP?
+L Device:Jumper_NO_Small JP1
 U 1 1 5C0C8C74
 P 4200 8500
-F 0 "JP?" V 4154 8548 50  0000 L CNN
+F 0 "JP1" V 4154 8548 50  0000 L CNN
 F 1 "Jumper_NO_Small" V 4245 8548 50  0000 L CNN
 F 2 "Jumper:SolderJumper-2_P1.3mm_Open_TrianglePad1.0x1.5mm" H 4200 8500 50  0001 C CNN
