File: backplane/STM32_CORE.sch (KiCad schematic (older format))
At the start: 35 parts, among them J22 POWER, J24 Conn_01x14, J26 Conn_01x12, J27 Conn_01x15, SW1 SW_Push, U3 waveshare-swd-pinsocket, U4 STM32F103C8T6, U5 AMS1117-3.3, Y1 O8M, Y2 O_EPSON_32.768K

Commit message: update,
Connections:
- net labels added: STM32_PCB1_ALARM_COM
- net labels removed: PCB1_ALARM_COM
Changed lines of the file:
@@
 $Descr A3 16535 11693
 encoding utf-8
-Sheet 6 9
+Sheet 6 10
 Title ""
 Date ""
@@
 Wire Wire Line
 	5500 3250 5500 3450
-Text GLabel 8100 4750 3    50   Input ~ 0
-PCB1_ALARM_COM
+Text GLabel 8100 4750 3    60   Input ~ 0
+STM32_PCB1_ALARM_COM
 $EndSCHEMATC

Commit message: backport footprint from pcb,
Parts:
- J22: footprint footprint-lib:s3b-ph-kl -> Connector_JST:JST_XH_S03B-XH-A_1x03_P2.50mm_Horizontal
Changed lines of the file:
@@
 F 0 "J22" H 1520 5325 50  0000 C CNN
 F 1 "POWER" H 1520 5416 50  0000 C CNN
-F 2 "footprint-lib:s3b-ph-kl" H 1600 5650 50  0001 C CNN
+F 2 "Connector_JST:JST_XH_S03B-XH-A_1x03_P2.50mm_Horizontal" H 1600 5650 50  0001 C CNN
 F 3 "~" H 1600 5650 50  0001 C CNN
 	1    1600 5650

Commit message: update,
Connections:
- net labels added: EXT_TRIGGER
Changed lines of the file:
@@
 Text GLabel 8100 4750 3    60   Input ~ 0
 STM32_PCB1_ALARM_COM
+Text GLabel 10000 3250 2    60   Input ~ 0
+EXT_TRIGGER
 $EndSCHEMATC

Commit message: update,
Parts:
- Y1: footprint w_crystal:hc-49_smd -> footprint-lib:hc-49_smd
- renumbered BOOT1 to BOOT0, BOOT2 to BOOT1
Changed lines of the file:
@@
 F 0 "Y1" V 14654 6788 50  0000 L CNN
 F 1 "O8M" V 14745 6788 50  0000 L CNN
-F 2 "w_crystal:hc-49_smd" H 14700 6700 50  0001 C CNN
+F 2 "footprint-lib:hc-49_smd" H 14700 6700 50  0001 C CNN
 F 3 "~" H 14700 6700 50  0001 C CNN
 	1    14700 6700
@@
 	14500 3100 14500 3350
 $Comp
-L Jumper:SolderJumper_3_Open BOOT1
+L Jumper:SolderJumper_3_Open BOOT0
 U 1 1 5BCF8FA5
 P 11900 1800
-F 0 "BOOT1" V 11854 1868 50  0000 L CNN
+F 0 "BOOT0" V 11854 1868 50  0000 L CNN
 F 1 "JUMPER" V 11945 1868 50  0000 L CNN
 F 2 "Jumper:SolderJumper-3_P2.0mm_Open_TrianglePad1.0x1.5mm" H 11900 1800 50  0001 C CNN
@@
 $EndComp
 $Comp
-L Jumper:SolderJumper_3_Open BOOT2
+L Jumper:SolderJumper_3_Open BOOT1
 U 1 1 5BCF9021
 P 12750 1800
-F 0 "BOOT2" V 12704 1868 50  0000 L CNN
+F 0 "BOOT1" V 12704 1868 50  0000 L CNN
 F 1 "JUMPER" V 12795 1868 50  0000 L CNN
 F 2 "Jumper:SolderJumper-3_P2.0mm_Open_TrianglePad1.0x1.5mm" H 12750 1800 50  0001 C CNN

Commit message: update,
Parts:
- J22: footprint Connector_JST:JST_XH_S03B-XH-A_1x03_P2.50mm_Horizontal -> Connector_JST:JST_XH_S03B-XH-A-1_1x03_P2.50mm_Horizontal
Changed lines of the file:
@@
 F 0 "J22" H 1520 5325 50  0000 C CNN
 F 1 "POWER" H 1520 5416 50  0000 C CNN
-F 2 "Connector_JST:JST_XH_S03B-XH-A_1x03_P2.50mm_Horizontal" H 1600 5650 50  0001 C CNN
+F 2 "Connector_JST:JST_XH_S03B-XH-A-1_1x03_P2.50mm_Horizontal" H 1600 5650 50  0001 C CNN
 F 3 "~" H 1600 5650 50  0001 C CNN
 	1    1600 5650

Commit message: as fit resistor value to actual working value,
Parts:
- Y1: symbol taobao-osc:O8M -> backplane-rescue:O8M-taobao-osc
- Y2: symbol taobao-osc:O_EPSON_32.768K -> backplane-rescue:O_EPSON_32.768K-taobao-osc
Changed lines of the file:
@@
 $EndComp
 $Comp
-L taobao-osc:O8M Y1
+L backplane-rescue:O8M-taobao-osc Y1
 U 1 1 5BCC6C8D
 P 14700 6700
+AR Path="/5BCC6C8D" Ref="Y1"  Part="1"
+AR Path="/5BEEE39B/5BCB6FA2/5BCC6C8D" Ref="Y1"  Part="1"
 F 0 "Y1" V 14654 6788 50  0000 L CNN
 F 1 "O8M" V 14745 6788 50  0000 L CNN
@@
 	2350 5650 1800 5650
 $Comp
-L taobao-osc:O_EPSON_32.768K Y2
+L backplane-rescue:O_EPSON_32.768K-taobao-osc Y2
 U 1 1 5BD58864
 P 14700 7500
